Commit message: Added Transmission and used robot_state_publisher

File: robot/description/urdf/side_wheels.urdf.xacro (robot description, xacro)
@@ -1,5 +1,4 @@
 <?xml version="1.0"?>
 <robot name="side_wheels" xmlns:xacro="http://ros.org/wiki/xacro">
-    <!-- TODO: include Transmission later for use with motors -->
     <!-- Constants -->
     <xacro:property name="wheel_vertical_offset" value="-0.61759696"/>
@@ -19,4 +18,14 @@
             izx="0.00" izy="-1.15" izz="0.87"
             />
+    </xacro:macro>
+    <!-- Motor Transmissions -->
+    <xacro:macro name="Transmission" params="joint">
+        <transmission name="trans_${joint}">
+            <type>transmission_interface/SimpleTransmission</type>
+            <joint name="${joint}">
+                <hardwareInterface>EffortJointInterface</hardwareInterface>
+            </joint>
+            <actuator name="${joint}_motor"/>
+        </transmission>
     </xacro:macro>
     <!-- left wheel -->
@@ -45,4 +54,5 @@
         <axis xyz="0 1 0"/>
     </joint>
+    <xacro:Transmission joint="left_wheel_joint"/>
     <!-- right wheel -->
     <link name="right_wheel_link">
@@ -70,3 +80,4 @@
         <axis xyz="0 1 0"/>
     </joint>
+    <xacro:Transmission joint="right_wheel_joint"/>
 </robot>
