Commit message: added Lidar plugin

File: robot/description/urdf/base_laser.urdf.xacro (robot description, xacro)
@@ -19,5 +19,5 @@
          <origin xyz="0 0 0" rpy="0 0 0"/>
          <geometry>
-           <mesh filename="package://description//rdf.meshes/hokuyo.dae"/>
+           <mesh filename="package://description//urdf/meshes/hokuyo.dae"/>
          </geometry>
       </collision>

Commit message: changed 'hokuyo' name to 'laser' for consistency

File: robot/description/urdf/base_laser.urdf.xacro (robot description, xacro)
@@ -7,6 +7,6 @@
    <link name="base_laser">
         <inertial>
-            <mass value="${hokuyo_mass}"/>
-            <xacro:box_inertia mass="${hokuyo_mass}" length="${hokuyo_length}" width="${hokuyo_width}" height="${hokuyo_height}"/>
+            <mass value="${laser_mass}"/>
+            <xacro:box_inertia mass="${laser_mass}" length="${laser_length}" width="${laser_width}" height="${laser_height}"/>
         </inertial>
       <visual>

Commit message: Added tf_prefix to all links

File: robot/description/urdf/base_laser.urdf.xacro (robot description, xacro)
@@ -5,5 +5,5 @@
    <xacro:include filename="$(find description)/urdf/inertias.xacro"/>
    <!-- LIDAR link -->
-   <link name="base_laser">
+   <link name="${tf_prefix}/base_laser">
         <inertial>
             <mass value="${laser_mass}"/>

File: robot/description/urdf/caffeine.gazebo.xacro (robot description, xacro)
@@ -8,6 +8,6 @@
             <robotNamespace>${robotNamespace}</robotNamespace>
             <updateRate>${diff_drive_update_rate}</updateRate>
-            <leftJoint>${wheel_left_joint}</leftJoint>
-            <rightJoint>${wheel_right_joint}</rightJoint>
+	    <leftJoint>${tf_prefix}/${wheel_left_joint}</leftJoint>
+	    <rightJoint>${tf_prefix}/${wheel_right_joint}</rightJoint>
             <wheelSeparation>${wheels_separation}</wheelSeparation>
             <wheelDiameter>${wheel_diameter}</wheelDiameter>
@@ -34,5 +34,5 @@
     </gazebo>
     <!-- LIDAR -->
-   <gazebo reference="base_laser">
+    <gazebo reference="${tf_prefix}/base_laser">
       <sensor type="ray" name="gpu_hokuyo_sensor">
          <pose>0 0 0 0 0 0</pose>
@@ -65,5 +65,5 @@
             <robotNamespace>${robotNamespace}</robotNamespace>
             <topicName>${laser_topicName}</topicName>
-            <frameName>${laser_frameName}</frameName>
+	    <frameName>${tf_prefix}/${laser_frameName}</frameName>
          </plugin>
       </sensor>

File: robot/description/urdf/caffeine.urdf.xacro (robot description, xacro)
@@ -1,40 +1,33 @@
 <?xml version="1.0"?>
 <robot name="caffeine" xmlns:xacro="http://ros.org/wiki/xacro">
-    <xacro:arg name="tf_prefix" default="caffeine"/>
     <!-- Includes -->
     <xacro:include filename="$(find description)/urdf/constants.xacro"/>
     <xacro:include filename="$(find description)/urdf/caffeine.gazebo.xacro"/>
     <!-- base_link: origin of the robot; located in the middle, on the top of the base plate -->
-    <link name="$(arg tf_prefix)/base_link"/>
+    <link name="${tf_prefix}/base_link"/>
     <!-- chassis_link: geometric center of the robot; used as the parent in which all other links connect to -->
-    <xacro:include filename="$(find description)/urdf/chassis_link.urdf.xacro">
-        <xacro:arg name="tf_prefix" value="$(arg tf_prefix)"/>
-    </xacro:include>
-    <joint name="$(arg tf_prefix)/chassis_link_joint" type="fixed">
-        <parent link="$(arg tf_prefix)/base_link"/>
-        <child link="$(arg tf_prefix)/chassis_link"/>
+    <xacro:include filename="$(find description)/urdf/chassis_link.urdf.xacro"/>
+    <joint name="${tf_prefix}/chassis_link_joint" type="fixed">
+	<parent link="${tf_prefix}/base_link"/>
+	<child link="${tf_prefix}/chassis_link"/>
         <origin rpy="0 0 0" xyz="0 0 ${chassis_to_base_link_dist}"/>
     </joint>
     <!-- stand_link: origin for anything on the stand; located in the middle, on the top of the stand plate -->
-    <xacro:include filename="$(find description)/urdf/stand_link.urdf.xacro">
-        <xacro:arg name="tf_prefix" value="$(arg tf_prefix)"/>
-    </xacro:include>
-    <joint name="$(arg tf_prefix)/stand_link_joint" type="fixed">
-        <parent link="$(arg tf_prefix)/chassis_link"/>
-        <child link="$(arg tf_prefix)/stand_link"/>
+    <xacro:include filename="$(find description)/urdf/stand_link.urdf.xacro"/>
+    <joint name="${tf_prefix}/stand_link_joint" type="fixed">
+	<parent link="${tf_prefix}/chassis_link"/>
+	<child link="${tf_prefix}/stand_link"/>
         <origin rpy="0 0 0" xyz="0 0 ${chassis_to_stand_link_dist}"/>
     </joint>
     <!-- wheels: associated to wheels that can be moved by a motor -->
-    <xacro:include filename="$(find description)/urdf/side_wheels.urdf.xacro">
-        <xacro:arg name="tf_prefix" value="$(arg tf_prefix)"/>
-    </xacro:include>
+    <xacro:include filename="$(find description)/urdf/side_wheels.urdf.xacro"/>
     <!-- wheels: front and back casters -->
     <xacro:include filename="$(find description)/urdf/casters.urdf.xacro"/>
-    <!-- base_laser: LIDAR at front of Caffeine -->
-    <xacro:include filename="$(find description)/urdf/base_laser.urdf.xacro"/>
-    <joint name="base_laser_joint" type="fixed">
-        <parent link="base_link"/>
-        <child link="base_laser"/>
-        <origin xyz="${laser_x_dist} 0 ${laser_z_dist}" rpy="0 0 0"/>
+   <!-- base_laser: LIDAR at front of Caffeine -->
+   <xacro:include filename="$(find description)/urdf/base_laser.urdf.xacro"/>
+   <joint name="${tf_prefix}/base_laser_joint" type="fixed">
+      <parent link="${tf_prefix}/base_link"/>
+      <child link="${tf_prefix}/base_laser"/>
+      <origin xyz="${laser_x_dist} 0 ${laser_z_dist}" rpy="0 0 0"/>
    </joint>
 </robot>

File: robot/description/urdf/casters.urdf.xacro (robot description, xacro)
@@ -1,10 +1,9 @@
 <?xml version="1.0"?>
 <robot name="caster_wheels" xmlns:xacro="http://ros.org/wiki/xacro">
-    <xacro:arg name="tf_prefix" default="caffeine"/>
     <!-- Includes -->
     <xacro:include filename="$(find description)/urdf/constants.xacro"/>
     <xacro:include filename="$(find description)/urdf/inertias.xacro"/>
     <!-- Front caster definition -->
-    <link name="$(arg tf_prefix)/front_caster_link">
+    <link name="${tf_prefix}/front_caster_link">
         <visual>
             <origin rpy="0 0 0" xyz="0 0 0"/>
@@ -25,12 +24,12 @@
     </link>
     <!-- NOTE: using a fixed joint prevents Caffeine spawning tipped over -->
-    <joint name="$(arg tf_prefix)/front_caster_link_joint" type="fixed">
+    <joint name="${tf_prefix}/front_caster_link_joint" type="fixed">
         <!-- <axis xyz="0 0 1"/> -->
-        <parent link="$(arg tf_prefix)/chassis_link"/>
-        <child link="$(arg tf_prefix)/front_caster_link"/>
+	<parent link="${tf_prefix}/chassis_link"/>
+	<child link="${tf_prefix}/front_caster_link"/>
         <origin rpy="0 0 0" xyz="${casters_separation / 2.0} 0 ${caster_vertical_offset}"/>
     </joint>
     <!-- Back caster definition -->
-    <link name="$(arg tf_prefix)/back_caster_link">
+    <link name="${tf_prefix}/back_caster_link">
         <visual>
             <origin rpy="0 0 0" xyz="0 0 0"/>
@@ -51,12 +50,12 @@
     </link>
     <!-- NOTE: using a fixed joint prevents Caffeine spawning tipped over -->
-    <joint name="$(arg tf_prefix)/back_caster_link_joint" type="fixed">
+    <joint name="${tf_prefix}/back_caster_link_joint" type="fixed">
         <!-- <axis xyz="0 0 1"/> -->
-        <parent link="$(arg tf_prefix)/chassis_link"/>
-        <child link="$(arg tf_prefix)/back_caster_link"/>
+	<parent link="${tf_prefix}/chassis_link"/>
+	<child link="${tf_prefix}/back_caster_link"/>
         <origin rpy="0 0 0" xyz="-${casters_separation / 2.0} 0 ${caster_vertical_offset}"/>
     </joint>
     <!-- Front caster wheel definition -->
-    <link name="$(arg tf_prefix)/front_caster_wheel">
+    <link name="${tf_prefix}/front_caster_wheel">
         <visual>
             <origin rpy="0 0 0" xyz="0 0 0"/>
@@ -76,12 +75,12 @@
         </inertial>
     </link>
-    <joint name="$(arg tf_prefix)/front_caster_wheel_joint" type="continuous">
-        <parent link="$(arg tf_prefix)/front_caster_link"/>
-        <child link="$(arg tf_prefix)/front_caster_wheel"/>
+    <joint name="${tf_prefix}/front_caster_wheel_joint" type="continuous">
+	<parent link="${tf_prefix}/front_caster_link"/>
+	<child link="${tf_prefix}/front_caster_wheel"/>
         <origin rpy="0 0 0" xyz="${caster_link_to_wheel_dist_x} 0 ${caster_link_to_wheel_dist_z}"/>
         <axis xyz="0 1 0"/>
     </joint>
     <!-- Back caster wheel definition -->
-    <link name="$(arg tf_prefix)/back_caster_wheel">
+    <link name="${tf_prefix}/back_caster_wheel">
         <visual>
             <origin rpy="0 0 0" xyz="0 0 0"/>
@@ -101,7 +100,7 @@
         </inertial>
     </link>
-    <joint name="$(arg tf_prefix)/back_caster_wheel_joint" type="continuous">
-        <parent link="$(arg tf_prefix)/back_caster_link"/>
-        <child link="$(arg tf_prefix)/back_caster_wheel"/>
+    <joint name="${tf_prefix}/back_caster_wheel_joint" type="continuous">
+	<parent link="${tf_prefix}/back_caster_link"/>
+	<child link="${tf_prefix}/back_caster_wheel"/>
         <origin rpy="0 0 0" xyz="-${caster_link_to_wheel_dist_x} 0 ${caster_link_to_wheel_dist_z}"/>
         <axis xyz="0 1 0"/>

File: robot/description/urdf/chassis_link.urdf.xacro (robot description, xacro)
@@ -1,10 +1,9 @@
 <?xml version="1.0"?>
 <robot name="chassis" xmlns:xacro="http://ros.org/wiki/xacro">
-    <xacro:arg name="tf_prefix" default="caffeine"/>
     <!-- Includes -->
     <xacro:include filename="$(find description)/urdf/constants.xacro"/>
     <xacro:include filename="$(find description)/urdf/inertias.xacro"/>
     <!-- Chassis link definition; chassis link is associated with the centroid of the bounding box of the robot and the chassis_link.dae file-->
-    <link name="$(arg tf_prefix)/chassis_link">
+    <link name="${tf_prefix}/chassis_link">
         <visual>
             <origin rpy="0 0 0" xyz="0 0 0"/>

File: robot/description/urdf/constants.xacro (robot description, xacro)
@@ -3,4 +3,5 @@
     <!-- Caffeine -->
     <xacro:property name="robotNamespace" value="caffeine"/>
+    <xacro:property name="tf_prefix" value="caffeine"/>
     <!-- Drivebase -->
    <xacro:property name="base_length" value="1.268"/>

File: robot/description/urdf/side_wheels.urdf.xacro (robot description, xacro)
@@ -1,5 +1,4 @@
 <?xml version="1.0"?>
 <robot name="side_wheels" xmlns:xacro="http://ros.org/wiki/xacro">
-    <xacro:arg name="tf_prefix" default="caffeine"/>
     <!-- Includes -->
     <xacro:include filename="$(find description)/urdf/constants.xacro"/>
@@ -16,5 +15,5 @@
     </xacro:macro>
     <!-- left wheel -->
-    <link name="$(arg tf_prefix)/left_wheel_link">
+    <link name="${tf_prefix}/left_wheel_link">
         <visual>
             <origin rpy="0 0 0" xyz="0 0 0"/>
@@ -34,13 +33,13 @@
         </inertial>
     </link>
-    <joint name="$(arg tf_prefix)/left_wheel_joint" type="continuous">
-        <parent link="$(arg tf_prefix)/chassis_link"/>
-        <child link="$(arg tf_prefix)/left_wheel_link"/>
+    <joint name="${tf_prefix}/left_wheel_joint" type="continuous">
+	<parent link="${tf_prefix}/chassis_link"/>
+	<child link="${tf_prefix}/left_wheel_link"/>
         <origin xyz= "0 ${wheels_separation / 2.0} ${wheel_vertical_offset}"/>
         <axis xyz="0 1 0"/>
     </joint>
-    <xacro:Transmission joint="$(arg tf_prefix)/left_wheel_joint"/>
+    <xacro:Transmission joint="${tf_prefix}/left_wheel_joint"/>
     <!-- right wheel -->
-    <link name="$(arg tf_prefix)/right_wheel_link">
+    <link name="${tf_prefix}/right_wheel_link">
         <visual>
             <origin rpy="0 0 0" xyz="0 0 0"/>
@@ -60,10 +59,10 @@
         </inertial>
     </link>
-    <joint name="$(arg tf_prefix)/right_wheel_joint" type="continuous">
-        <parent link="$(arg tf_prefix)/chassis_link"/>
-        <child link="$(arg tf_prefix)/right_wheel_link"/>
+    <joint name="${tf_prefix}/right_wheel_joint" type="continuous">
+	<parent link="${tf_prefix}/chassis_link"/>
+	<child link="${tf_prefix}/right_wheel_link"/>
         <origin xyz= "0 -${wheels_separation / 2.0} ${wheel_vertical_offset}"/>
         <axis xyz="0 1 0"/>
     </joint>
-    <xacro:Transmission joint="$(arg tf_prefix)/right_wheel_joint"/>
+    <xacro:Transmission joint="${tf_prefix}/right_wheel_joint"/>
 </robot>

File: robot/description/urdf/stand_link.urdf.xacro (robot description, xacro)
@@ -1,5 +1,4 @@
 <?xml version="1.0"?>
 <robot name="stand_link" xmlns:xacro="http://ros.org/wiki/xacro">
-    <xacro:arg name="tf_prefix" default="caffeine"/>
     <!-- Includes -->
     <xacro:include filename="$(find description)/urdf/constants.xacro"/>
@@ -7,5 +6,5 @@
     <!-- Stand link; this is a dummy link that is used to make camera placement and other sensors on the stand more convenient -->
     <!-- Stand link definition. Note: purposely left blank -->
-    <link name="$(arg tf_prefix)/stand_link">
+    <link name="${tf_prefix}/stand_link">
     </link>
 </robot>
