Commit message: Added caster_links

File: robot/description/urdf/caffeine.urdf.xacro (robot description, xacro)
@@ -24,3 +24,16 @@
         <origin rpy="0 0 0" xyz="0 0 ${chassis_to_stand_link_dist}"/>
     </joint>
+    <xacro:include filename="$(find description)/urdf/casters.urdf.xacro"/>
+    <joint name="front_caster_link_joint" type="continuous">
+        <axis xyz="0 0 1"/>
+        <parent link="chassis_link"/>
+        <child link="front_caster_link"/>
+        <origin rpy="0 0 0" xyz="${chassis_to_front_caster_link_dist_x} 0 ${chassis_to_caster_link_dist_z}"/>
+    </joint>
+    <joint name="base_caster_link_joint" type="continuous">
+        <axis xyz="0 0 1"/>
+        <parent link="chassis_link"/>
+        <child link="back_caster_link"/>
+        <origin rpy="0 0 0" xyz="${chassis_to_back_caster_link_dist_x} 0 ${chassis_to_caster_link_dist_z}"/>
+    </joint>
 </robot>

File: robot/description/urdf/caffeine_constants.xacro (robot description, xacro)
@@ -4,3 +4,7 @@
     <xacro:property name="chassis_to_base_link_dist" value="0.501747"/>
     <xacro:property name="chassis_to_stand_link_dist" value="0.713459"/>
+    <xacro:property name="chassis_to_front_caster_link_dist_x" value="0.55951056"/>
+    <xacro:property name="chassis_to_back_caster_link_dist_x" value="-0.55951056"/>
+    <!-- Applicable to both casters -->
+    <xacro:property name="chassis_to_caster_link_dist_z" value="-0.619167561"/>
 </robot>

File: robot/description/urdf/chassis_link.urdf.xacro (robot description, xacro)
@@ -2,5 +2,5 @@
 <robot name="chassis" xmlns:xacro="http://ros.org/wiki/xacro">
     <!-- Constants for chassis_link -->
-    <xacro:property name="chassis_link_mass" value="30.0"/>
+    <xacro:property name="chassis_link_mass" value="33.9"/>
     <xacro:macro name="chassis_link_inertia">
         <inertia

Commit message: Added left and right wheels

File: robot/description/urdf/caffeine.urdf.xacro (robot description, xacro)
@@ -24,3 +24,5 @@
         <origin rpy="0 0 0" xyz="0 0 ${chassis_to_stand_link_dist}"/>
     </joint>
+    <!-- wheels: associated to wheels that can be moved by a motor -->
+    <xacro:include filename="$(find description)/urdf/side_wheels.urdf.xacro"/>
 </robot>

File: robot/description/urdf/side_wheels.urdf.xacro (robot description, xacro)
@@ -2,4 +2,71 @@
 <robot name="side_wheels" xmlns:xacro="http://ros.org/wiki/xacro">
     <!-- TODO: include Transmission later for use with motors -->
-    <!-- TODO: populate this file with definitions and constants for left, right wheels -->
+    <!-- Constants -->
+    <xacro:property name="wheel_vertical_offset" value="-0.61759696"/>
+    <xacro:property name="wheels_separation" value="0.875"/>
+    <xacro:property name="wheel_mass" value="4.45"/>
+    <xacro:macro name="left_wheel_inertia">
+        <inertia
+            ixx="2.43" ixy="0.00" ixz="0.00"
+            iyx="0.00" iyy="1.60" iyz="1.15"
+            izx="0.00" izy="1.15" izz="0.87"
+            />
+    </xacro:macro>
+    <xacro:macro name="right_wheel_inertia">
+        <inertia
+            ixx="2.43" ixy="0.00" ixz="0.00"
+            iyx="0.00" iyy="1.60" iyz="-1.15"
+            izx="0.00" izy="-1.15" izz="0.87"
+            />
+    </xacro:macro>
+    <!-- left wheel -->
+    <link name="left_wheel_link">
+        <visual>
+            <origin rpy="0 0 0" xyz="0 0 0"/>
+            <geometry>
+                <mesh filename="package://description/urdf/meshes/left_wheel.dae"/>
+            </geometry>
+        </visual>
+        <collision>
+            <origin rpy="0 0 0" xyz="0 0 0"/>
+            <geometry>
+                <mesh filename="package://description/urdf/meshes/left_wheel.dae"/>
+            </geometry>
+        </collision>
+        <inertial>
+            <mass value="${wheel_mass}"/>
+            <xacro:left_wheel_inertia/>
+        </inertial>
+    </link>
+    <joint name="left_wheel_joint" type="continuous">
+        <parent link="chassis_link"/>
+        <child link="left_wheel_link"/>
+        <origin xyz= "0 ${wheels_separation / 2.0} ${wheel_vertical_offset}"/>
+        <axis xyz="0 1 0"/>
+    </joint>
+    <!-- right wheel -->
+    <link name="right_wheel_link">
+        <visual>
+            <origin rpy="0 0 0" xyz="0 0 0"/>
+            <geometry>
+                <mesh filename="package://description/urdf/meshes/right_wheel.dae"/>
+            </geometry>
+        </visual>
+        <collision>
+            <origin rpy="0 0 0" xyz="0 0 0"/>
+            <geometry>
+                <mesh filename="package://description/urdf/meshes/right_wheel.dae"/>
+            </geometry>
+        </collision>
+        <inertial>
+            <mass value="${wheel_mass}"/>
+            <xacro:right_wheel_inertia/>
+        </inertial>
+    </link>
+    <joint name="right_wheel_joint" type="continuous">
+        <parent link="chassis_link"/>
+        <child link="right_wheel_link"/>
+        <origin xyz= "0 -${wheels_separation / 2.0} ${wheel_vertical_offset}"/>
+        <axis xyz="0 1 0"/>
+    </joint>
 </robot>

Commit message: Moved caster joint definitions to caster_link.urdf.xacro

File: robot/description/urdf/caffeine.urdf.xacro (robot description, xacro)
@@ -28,15 +28,3 @@
     <!-- wheels: front and back casters -->
     <xacro:include filename="$(find description)/urdf/casters.urdf.xacro"/>
-    <joint name="front_caster_link_joint" type="continuous">
-        <axis xyz="0 0 1"/>
-        <parent link="chassis_link"/>
-        <child link="front_caster_link"/>
-        <origin rpy="0 0 0" xyz="${chassis_to_front_caster_link_dist_x} 0 ${chassis_to_caster_link_dist_z}"/>
-    </joint>
-    <joint name="base_caster_link_joint" type="continuous">
-        <axis xyz="0 0 1"/>
-        <parent link="chassis_link"/>
-        <child link="back_caster_link"/>
-        <origin rpy="0 0 0" xyz="${chassis_to_back_caster_link_dist_x} 0 ${chassis_to_caster_link_dist_z}"/>
-    </joint>
 </robot>

File: robot/description/urdf/caffeine_constants.xacro (robot description, xacro)
@@ -4,7 +4,3 @@
     <xacro:property name="chassis_to_base_link_dist" value="0.501747"/>
     <xacro:property name="chassis_to_stand_link_dist" value="0.713459"/>
-    <xacro:property name="chassis_to_front_caster_link_dist_x" value="0.55951056"/>
-    <xacro:property name="chassis_to_back_caster_link_dist_x" value="-0.55951056"/>
-    <!-- Applicable to both casters -->
-    <xacro:property name="chassis_to_caster_link_dist_z" value="-0.619167561"/>
 </robot>

File: robot/description/urdf/casters.urdf.xacro (robot description, xacro)
@@ -4,5 +4,5 @@
     <!-- Note: this file contains definitions for both the casters & the caster wheels -->
     <!-- When included, only use front_caster_link and back_caster_link (joints for the wheels are defined in this file) -->
-    <!-- Constants related to casters -->
+    <!-- Constants related to casters link definition  -->
     <!-- Note: mass can be used across both casters -->
     <xacro:property name="caster_link_mass" value="0.5"/>
@@ -21,4 +21,7 @@
         />
     </xacro:macro>
+    <!-- Constants realted to casters joint definition -->
+    <xacro:property name="casters_separation" value="1.12"/>
+    <xacro:property name="caster_vertical_offset" value="-0.619167561"/>
     <!-- Front caster link definition -->
     <link name="front_caster_link">
@@ -40,4 +43,11 @@
         </inertial>
     </link>
+    <!-- Front caster joint definition -->
+    <joint name="front_caster_link_joint" type="continuous">
+        <axis xyz="0 0 1"/>
+        <parent link="chassis_link"/>
+        <child link="front_caster_link"/>
+        <origin rpy="0 0 0" xyz="${casters_separation / 2.0} 0 ${caster_vertical_offset}"/>
+    </joint>
     <!-- Back caster link definition -->
     <link name="back_caster_link">
@@ -59,4 +69,11 @@
         </inertial>
     </link>
+    <!-- Back caster joint definition -->
+    <joint name="back_caster_link_joint" type="continuous">
+        <axis xyz="0 0 1"/>
+        <parent link="chassis_link"/>
+        <child link="back_caster_link"/>
+        <origin rpy="0 0 0" xyz="-${casters_separation / 2.0} 0 ${caster_vertical_offset}"/>
+    </joint>
     <!-- Wheel definitions and joints -->
     <!-- Constants related to caster wheel definition -->
@@ -77,7 +94,6 @@
     </xacro:macro>
     <!-- Constants related to caster wheel joint definition -->
-    <xacro:property name="front_caster_link_to_front_caster_wheel_dist_x" value="0.03621719"/>
-    <xacro:property name="back_caster_link_to_back_caster_wheel_dist_x" value="-0.03621719"/>
-    <xacro:property name="caster_link_to_caster_wheel_dist_z" value="-0.04361749"/>
+    <xacro:property name="caster_link_to_wheel_dist_x" value="0.03621719"/>
+    <xacro:property name="caster_link_to_wheel_dist_z" value="-0.04361749"/>
     <!-- Front caster wheel definition -->
     <link name="front_caster_wheel">
@@ -104,5 +120,5 @@
         <parent link="front_caster_link"/>
         <child link="front_caster_wheel"/>
-        <origin rpy="0 0 0" xyz="${front_caster_link_to_front_caster_wheel_dist_x} 0 ${caster_link_to_caster_wheel_dist_z}"/>
+        <origin rpy="0 0 0" xyz="${caster_link_to_wheel_dist_x} 0 ${caster_link_to_wheel_dist_z}"/>
     </joint>
      <!-- Back caster wheel definition -->
@@ -126,9 +142,9 @@
      </link>
     <!-- Back caster wheel joint -->
-     <joint name="back_caster_wheel_joint" type="continuous">
-         <axis xyz="0 1 0"/>
-         <parent link="back_caster_link"/>
-         <child link="back_caster_wheel"/>
-         <origin rpy="0 0 0" xyz="${back_caster_link_to_back_caster_wheel_dist_x} 0 ${caster_link_to_caster_wheel_dist_z}"/>
-     </joint>
+    <joint name="back_caster_wheel_joint" type="continuous">
+        <axis xyz="0 1 0"/>
+        <parent link="back_caster_link"/>
+        <child link="back_caster_wheel"/>
+        <origin rpy="0 0 0" xyz="-${caster_link_to_wheel_dist_x} 0 ${caster_link_to_wheel_dist_z}"/>
+    </joint>
 </robot>

Commit message: Added gazebo plugins and wheel diameter constant

File: robot/description/urdf/caffeine.urdf.xacro (robot description, xacro)
@@ -28,3 +28,5 @@
     <!-- wheels: front and back casters -->
     <xacro:include filename="$(find description)/urdf/casters.urdf.xacro"/>
+    <!-- Include gazebo file -->
+    <xacro:include filename="$(find description)/urdf/caffeine.gazebo.xacro"/>
 </robot>

File: robot/description/urdf/side_wheels.urdf.xacro (robot description, xacro)
@@ -4,4 +4,5 @@
     <xacro:property name="wheel_vertical_offset" value="-0.61759696"/>
     <xacro:property name="wheels_separation" value="0.875"/>
+    <xacro:property name="wheel_diameter" value="0.25"/> <!-- TODO: update this value -->
     <xacro:property name="wheel_mass" value="4.45"/>
     <xacro:macro name="left_wheel_inertia">

Commit message: added Lidar Plug-in

File: robot/description/urdf/caffeine.urdf.xacro (robot description, xacro)
@@ -24,3 +24,29 @@
     <!-- wheels: front and back casters -->
     <xacro:include filename="$(find description)/urdf/casters.urdf.xacro"/>
+   <!-- LIDAR link -->
+   <link name="base_laser">
+        <inertial>
+            <mass value="${hokuyo_mass}"/>
+            <xacro:box_inertia mass="${hokuyo_mass}" length="${hokuyo_length}" width="${hokuyo_width}" height="${hokuyo_height}"/>
+        </inertial>
+      <visual>
+         <origin xyz="0 0 0" rpy="0 0 0"/>
+         <geometry>
+            <mesh filename="package:///description/meshes/hokuyo.dae"/>
+         </geometry>
+      </visual>
+      <collision>
+         <origin xyz="0 0 0" rpy="0 0 0"/>
+         <geometry>
+            <mesh filename="package:///description/meshes/hokuyo.dae"/>
+         </geometry>
+      </collision>
+   </link>
+   <!-- LIDAR joint -->
+   <!-- TODO: double check xyz location-->
+   <joint name="base_laser_joint" type="fixed">
+      <parent link="base_link"/>
+      <child link="base_laser"/>
+      <origin xyz="${laser_x_dist} 0 ${laser_z_dist}" rpy="0 0 0"/>
+   </joint>
 </robot>

Commit message: Added tf_prefix to all elements of our URDF

File: robot/description/urdf/caffeine.urdf.xacro (robot description, xacro)
@@ -1,26 +1,35 @@
 <?xml version="1.0"?>
 <robot name="caffeine" xmlns:xacro="http://ros.org/wiki/xacro">
+    <xacro:arg name="tf_prefix" default="caffeine"/>
     <!-- Includes -->
     <xacro:include filename="$(find description)/urdf/constants.xacro"/>
     <xacro:include filename="$(find description)/urdf/caffeine.gazebo.xacro"/>
     <!-- base_link: origin of the robot; located in the middle, on the top of the base plate -->
-    <link name="base_link"/>
+    <link name="$(arg tf_prefix)/base_link"/>
     <!-- chassis_link: geometric center of the robot; used as the parent in which all other links connect to -->
-    <xacro:include filename="$(find description)/urdf/chassis_link.urdf.xacro"/>
-    <joint name="chassis_link_joint" type="fixed">
-        <parent link="base_link"/>
-        <child link="chassis_link"/>
+    <xacro:include filename="$(find description)/urdf/chassis_link.urdf.xacro">
+        <xacro:arg name="tf_prefix" value="$(arg tf_prefix)"/>
+    </xacro:include>
+    <joint name="$(arg tf_prefix)/chassis_link_joint" type="fixed">
+        <parent link="$(arg tf_prefix)/base_link"/>
+        <child link="$(arg tf_prefix)/chassis_link"/>
         <origin rpy="0 0 0" xyz="0 0 ${chassis_to_base_link_dist}"/>
     </joint>
     <!-- stand_link: origin for anything on the stand; located in the middle, on the top of the stand plate -->
-    <xacro:include filename="$(find description)/urdf/stand_link.urdf.xacro"/>
-    <joint name="stand_link_joint" type="fixed">
-        <parent link="chassis_link"/>
-        <child link="stand_link"/>
+    <xacro:include filename="$(find description)/urdf/stand_link.urdf.xacro">
+        <xacro:arg name="tf_prefix" value="$(arg tf_prefix)"/>
+    </xacro:include>
+    <joint name="$(arg tf_prefix)/stand_link_joint" type="fixed">
+        <parent link="$(arg tf_prefix)/chassis_link"/>
+        <child link="$(arg tf_prefix)/stand_link"/>
         <origin rpy="0 0 0" xyz="0 0 ${chassis_to_stand_link_dist}"/>
     </joint>
     <!-- wheels: associated to wheels that can be moved by a motor -->
-    <xacro:include filename="$(find description)/urdf/side_wheels.urdf.xacro"/>
+    <xacro:include filename="$(find description)/urdf/side_wheels.urdf.xacro">
+        <xacro:arg name="tf_prefix" value="$(arg tf_prefix)"/>
+    </xacro:include>
     <!-- wheels: front and back casters -->
-    <xacro:include filename="$(find description)/urdf/casters.urdf.xacro"/>
+    <xacro:include filename="$(find description)/urdf/casters.urdf.xacro">
+        <xacro:arg name="tf_prefix" value="$(arg tf_prefix)"/>
+    </xacro:include>
 </robot>

File: robot/description/urdf/casters.urdf.xacro (robot description, xacro)
@@ -1,9 +1,10 @@
 <?xml version="1.0"?>
 <robot name="caster_wheels" xmlns:xacro="http://ros.org/wiki/xacro">
+    <xacro:arg name="tf_prefix" default="caffeine"/>
     <!-- Includes -->
     <xacro:include filename="$(find description)/urdf/constants.xacro"/>
     <xacro:include filename="$(find description)/urdf/inertias.xacro"/>
     <!-- Front caster definition -->
-    <link name="front_caster_link">
+    <link name="$(arg tf_prefix)/front_caster_link">
         <visual>
             <origin rpy="0 0 0" xyz="0 0 0"/>
@@ -24,12 +25,12 @@
     </link>
     <!-- NOTE: using a fixed joint prevents Caffeine spawning tipped over -->
-    <joint name="front_caster_link_joint" type="fixed">
+    <joint name="$(arg tf_prefix)/front_caster_link_joint" type="fixed">
         <!-- <axis xyz="0 0 1"/> -->
-        <parent link="chassis_link"/>
-        <child link="front_caster_link"/>
+        <parent link="$(arg tf_prefix)/chassis_link"/>
+        <child link="$(arg tf_prefix)/front_caster_link"/>
         <origin rpy="0 0 0" xyz="${casters_separation / 2.0} 0 ${caster_vertical_offset}"/>
     </joint>
     <!-- Back caster definition -->
-    <link name="back_caster_link">
+    <link name="$(arg tf_prefix)/back_caster_link">
         <visual>
             <origin rpy="0 0 0" xyz="0 0 0"/>
@@ -50,12 +51,12 @@
     </link>
     <!-- NOTE: using a fixed joint prevents Caffeine spawning tipped over -->
-    <joint name="back_caster_link_joint" type="fixed">
+    <joint name="$(arg tf_prefix)/back_caster_link_joint" type="fixed">
         <!-- <axis xyz="0 0 1"/> -->
-        <parent link="chassis_link"/>
-        <child link="back_caster_link"/>
+        <parent link="$(arg tf_prefix)/chassis_link"/>
+        <child link="$(arg tf_prefix)/back_caster_link"/>
         <origin rpy="0 0 0" xyz="-${casters_separation / 2.0} 0 ${caster_vertical_offset}"/>
     </joint>
     <!-- Front caster wheel definition -->
-    <link name="front_caster_wheel">
+    <link name="$(arg tf_prefix)/front_caster_wheel">
         <visual>
             <origin rpy="0 0 0" xyz="0 0 0"/>
@@ -75,12 +76,12 @@
         </inertial>
     </link>
-    <joint name="front_caster_wheel_joint" type="continuous">
-        <parent link="front_caster_link"/>
-        <child link="front_caster_wheel"/>
+    <joint name="$(arg tf_prefix)/front_caster_wheel_joint" type="continuous">
+        <parent link="$(arg tf_prefix)/front_caster_link"/>
+        <child link="$(arg tf_prefix)/front_caster_wheel"/>
         <origin rpy="0 0 0" xyz="${caster_link_to_wheel_dist_x} 0 ${caster_link_to_wheel_dist_z}"/>
         <axis xyz="0 1 0"/>
     </joint>
     <!-- Back caster wheel definition -->
-    <link name="back_caster_wheel">
+    <link name="$(arg tf_prefix)/back_caster_wheel">
         <visual>
             <origin rpy="0 0 0" xyz="0 0 0"/>
@@ -100,7 +101,7 @@
         </inertial>
     </link>
-    <joint name="back_caster_wheel_joint" type="continuous">
-        <parent link="back_caster_link"/>
-        <child link="back_caster_wheel"/>
+    <joint name="$(arg tf_prefix)/back_caster_wheel_joint" type="continuous">
+        <parent link="$(arg tf_prefix)/back_caster_link"/>
+        <child link="$(arg tf_prefix)/back_caster_wheel"/>
         <origin rpy="0 0 0" xyz="-${caster_link_to_wheel_dist_x} 0 ${caster_link_to_wheel_dist_z}"/>
         <axis xyz="0 1 0"/>

File: robot/description/urdf/chassis_link.urdf.xacro (robot description, xacro)
@@ -1,9 +1,10 @@
 <?xml version="1.0"?>
 <robot name="chassis" xmlns:xacro="http://ros.org/wiki/xacro">
+    <xacro:arg name="tf_prefix" default="caffeine"/>
     <!-- Includes -->
     <xacro:include filename="$(find description)/urdf/constants.xacro"/>
     <xacro:include filename="$(find description)/urdf/inertias.xacro"/>
     <!-- Chassis link definition; chassis link is associated with the centroid of the bounding box of the robot and the chassis_link.dae file-->
-    <link name="chassis_link">
+    <link name="$(arg tf_prefix)/chassis_link">
         <visual>
             <origin rpy="0 0 0" xyz="0 0 0"/>

File: robot/description/urdf/side_wheels.urdf.xacro (robot description, xacro)
@@ -1,4 +1,5 @@
 <?xml version="1.0"?>
 <robot name="side_wheels" xmlns:xacro="http://ros.org/wiki/xacro">
+    <xacro:arg name="tf_prefix" default="caffeine"/>
     <!-- Includes -->
     <xacro:include filename="$(find description)/urdf/constants.xacro"/>
@@ -15,5 +16,5 @@
     </xacro:macro>
     <!-- left wheel -->
-    <link name="left_wheel_link">
+    <link name="$(arg tf_prefix)/left_wheel_link">
         <visual>
             <origin rpy="0 0 0" xyz="0 0 0"/>
@@ -33,13 +34,13 @@
         </inertial>
     </link>
-    <joint name="left_wheel_joint" type="continuous">
-        <parent link="chassis_link"/>
-        <child link="left_wheel_link"/>
+    <joint name="$(arg tf_prefix)/left_wheel_joint" type="continuous">
+        <parent link="$(arg tf_prefix)/chassis_link"/>
+        <child link="$(arg tf_prefix)/left_wheel_link"/>
         <origin xyz= "0 ${wheels_separation / 2.0} ${wheel_vertical_offset}"/>
         <axis xyz="0 1 0"/>
     </joint>
-    <xacro:Transmission joint="left_wheel_joint"/>
+    <xacro:Transmission joint="$(arg tf_prefix)/left_wheel_joint"/>
     <!-- right wheel -->
-    <link name="right_wheel_link">
+    <link name="$(arg tf_prefix)/right_wheel_link">
         <visual>
             <origin rpy="0 0 0" xyz="0 0 0"/>
@@ -59,10 +60,10 @@
         </inertial>
     </link>
-    <joint name="right_wheel_joint" type="continuous">
-        <parent link="chassis_link"/>
-        <child link="right_wheel_link"/>
+    <joint name="$(arg tf_prefix)/right_wheel_joint" type="continuous">
+        <parent link="$(arg tf_prefix)/chassis_link"/>
+        <child link="$(arg tf_prefix)/right_wheel_link"/>
         <origin xyz= "0 -${wheels_separation / 2.0} ${wheel_vertical_offset}"/>
         <axis xyz="0 1 0"/>
     </joint>
-    <xacro:Transmission joint="right_wheel_joint"/>
+    <xacro:Transmission joint="$(arg tf_prefix)/right_wheel_joint"/>
 </robot>

File: robot/description/urdf/stand_link.urdf.xacro (robot description, xacro)
@@ -1,4 +1,5 @@
 <?xml version="1.0"?>
 <robot name="stand_link" xmlns:xacro="http://ros.org/wiki/xacro">
+    <xacro:arg name="tf_prefix" default="caffeine"/>
     <!-- Includes -->
     <xacro:include filename="$(find description)/urdf/constants.xacro"/>
@@ -6,5 +7,5 @@
     <!-- Stand link; this is a dummy link that is used to make camera placement and other sensors on the stand more convenient -->
     <!-- Stand link definition. Note: purposely left blank -->
-    <link name="stand_link">
+    <link name="$(arg tf_prefix)/stand_link">
     </link>
 </robot>
