Commit message: Resolving spacing issues

File: robot/description/urdf/caffeine.urdf.xacro (robot description, xacro)
@@ -26,8 +26,8 @@
    <!-- base_laser: LIDAR at front of Caffeine -->
    <xacro:include filename="$(find description)/urdf/base_laser.urdf.xacro"/>
-    <joint name="${tf_prefix}/base_laser_joint" type="fixed">
+   <joint name="${tf_prefix}/base_laser_joint" type="fixed">
         <parent link="${tf_prefix}/base_link"/>
         <child link="${tf_prefix}/base_laser"/>
         <origin xyz="${laser_x_dist} 0 ${laser_z_dist}" rpy="0 0 0"/>
-    </joint>
+   </joint>
 </robot>

File: robot/description/urdf/casters.urdf.xacro (robot description, xacro)
@@ -26,6 +26,6 @@
     <joint name="${tf_prefix}/front_caster_link_joint" type="fixed">
         <!-- <axis xyz="0 0 1"/> -->
-	    <parent link="${tf_prefix}/chassis_link"/>
-	    <child link="${tf_prefix}/front_caster_link"/>
+        <parent link="${tf_prefix}/chassis_link"/>
+        <child link="${tf_prefix}/front_caster_link"/>
         <origin rpy="0 0 0" xyz="${casters_separation / 2.0} 0 ${caster_vertical_offset}"/>
     </joint>
@@ -52,6 +52,6 @@
     <joint name="${tf_prefix}/back_caster_link_joint" type="fixed">
         <!-- <axis xyz="0 0 1"/> -->
-	    <parent link="${tf_prefix}/chassis_link"/>
-	    <child link="${tf_prefix}/back_caster_link"/>
+        <parent link="${tf_prefix}/chassis_link"/>
+        <child link="${tf_prefix}/back_caster_link"/>
         <origin rpy="0 0 0" xyz="-${casters_separation / 2.0} 0 ${caster_vertical_offset}"/>
     </joint>
@@ -76,6 +76,6 @@
     </link>
     <joint name="${tf_prefix}/front_caster_wheel_joint" type="continuous">
-	    <parent link="${tf_prefix}/front_caster_link"/>
-	    <child link="${tf_prefix}/front_caster_wheel"/>
+        <parent link="${tf_prefix}/front_caster_link"/>
+        <child link="${tf_prefix}/front_caster_wheel"/>
         <origin rpy="0 0 0" xyz="${caster_link_to_wheel_dist_x} 0 ${caster_link_to_wheel_dist_z}"/>
         <axis xyz="0 1 0"/>
@@ -101,6 +101,6 @@
     </link>
     <joint name="${tf_prefix}/back_caster_wheel_joint" type="continuous">
-	    <parent link="${tf_prefix}/back_caster_link"/>
-	    <child link="${tf_prefix}/back_caster_wheel"/>
+        <parent link="${tf_prefix}/back_caster_link"/>
+        <child link="${tf_prefix}/back_caster_wheel"/>
         <origin rpy="0 0 0" xyz="-${caster_link_to_wheel_dist_x} 0 ${caster_link_to_wheel_dist_z}"/>
         <axis xyz="0 1 0"/>

File: robot/description/urdf/side_wheels.urdf.xacro (robot description, xacro)
@@ -34,6 +34,6 @@
     </link>
     <joint name="${tf_prefix}/left_wheel_joint" type="continuous">
-	    <parent link="${tf_prefix}/chassis_link"/>
-	    <child link="${tf_prefix}/left_wheel_link"/>
+        <parent link="${tf_prefix}/chassis_link"/>
+        <child link="${tf_prefix}/left_wheel_link"/>
         <origin xyz= "0 ${wheels_separation / 2.0} ${wheel_vertical_offset}"/>
         <axis xyz="0 1 0"/>
@@ -60,6 +60,6 @@
     </link>
     <joint name="${tf_prefix}/right_wheel_joint" type="continuous">
-	    <parent link="${tf_prefix}/chassis_link"/>
-    	<child link="${tf_prefix}/right_wheel_link"/>
+        <parent link="${tf_prefix}/chassis_link"/>
+        <child link="${tf_prefix}/right_wheel_link"/>
         <origin xyz= "0 -${wheels_separation / 2.0} ${wheel_vertical_offset}"/>
         <axis xyz="0 1 0"/>
