Commit message: fixing zed camera height

File: robot/description/urdf/stand_link.urdf.xacro (robot description, xacro)
@@ -27,5 +27,5 @@
     </link>
     <joint name="${tf_prefix}/zed_camera_joint" type="fixed">
-        <origin xyz="${stand_length/2 - ZED_camera_width} 0 0" rpy="0 0 0"/>
+        <origin xyz="${stand_length/2 - ZED_camera_width} 0 ${ZED_camera_height / 2.0}" rpy="0 0 0"/>
         <parent link="${tf_prefix}/stand_link"/>
         <child link="${tf_prefix}/zed_camera_link"/>

Commit message: Added pitch to camera link

File: robot/description/urdf/stand_link.urdf.xacro (robot description, xacro)
@@ -10,5 +10,5 @@
     <link name="${tf_prefix}/zed_camera_link">
         <visual>
-            <origin xyz="0 0 0" rpy="0 0 0"/>
+            <origin xyz="0 0 0" rpy="0 ${ZED_camera_pitch} 0"/>
             <geometry>
             <box size="${ZED_camera_width} ${ZED_camera_length} ${ZED_camera_height}"/>

Commit message: Added pitch to camera link joint

File: robot/description/urdf/stand_link.urdf.xacro (robot description, xacro)
@@ -10,5 +10,5 @@
     <link name="${tf_prefix}/zed_camera_link">
         <visual>
-            <origin xyz="0 0 0" rpy="0 ${ZED_camera_pitch} 0"/>
+            <origin xyz="0 0 0" rpy="0 0 0"/>
             <geometry>
             <box size="${ZED_camera_width} ${ZED_camera_length} ${ZED_camera_height}"/>
@@ -27,5 +27,5 @@
     </link>
     <joint name="${tf_prefix}/zed_camera_joint" type="fixed">
-        <origin xyz="${stand_length/2 - ZED_camera_width} 0 ${ZED_camera_height / 2.0}" rpy="0 0 0"/>
+        <origin xyz="${stand_length/2 - ZED_camera_width} 0 ${ZED_camera_height / 2.0}" rpy="0 ${ZED_camera_pitch} 0"/>
         <parent link="${tf_prefix}/stand_link"/>
         <child link="${tf_prefix}/zed_camera_link"/>
