Commit message: Moved all constants to constants.xacro

File: robot/description/urdf/caffeine.gazebo.xacro (robot description, xacro)
@@ -1,5 +1,6 @@
 <?xml version="1.0"?>
 <robot name="caffeine_sim" xmlns:xacro="http://ros.org/wiki/xacro">
-    <xacro:property name="diff_drive_update_rate" value="30.0"/>
+    <!-- Constants -->
+    <xacro:include filename="$(find description)/urdf/constants.xacro"/>
     <!-- differential drive control support -->
     <!-- TODO: update parameters once they become known -->
@@ -30,5 +31,5 @@
         <plugin name="gazebo_ros_control" filename="libgazebo_ros_control.so">
             <!-- TODO: put namespace if necessary -->
-            <robotNamespace></robotNamespace>
+            <robotNamespace>caffeine</robotNamespace>
         </plugin>
     </gazebo>

File: robot/description/urdf/caffeine.urdf.xacro (robot description, xacro)
@@ -1,9 +1,8 @@
 <?xml version="1.0"?>
 <robot name="caffeine" xmlns:xacro="http://ros.org/wiki/xacro">
-    <!-- Includes -->
-    <xacro:include filename="$(find description)/urdf/caffeine_constants.xacro"/>
+    <!-- Constants -->
+    <xacro:include filename="$(find description)/urdf/constants.xacro"/>
     <!-- Base link; dummy link. This is the base for everything else. Located at the plate centroid of the plate of the robot -->
-    <link name="base_link">
-    </link>
+    <link name="base_link"/>
     <!-- Chassis link; this link is associated with the main body of the robot. Located at centroid of bounding box around chassis+stand -->
     <!-- This link is associated with chassis_link.dae -->

File: robot/description/urdf/casters.urdf.xacro (robot description, xacro)
@@ -4,7 +4,7 @@
     <!-- Note: this file contains definitions for both the casters & the caster wheels -->
     <!-- When included, only use front_caster_link and back_caster_link (joints for the wheels are defined in this file) -->
-    <!-- Constants related to casters link definition  -->
+    <!-- Constants -->
+    <xacro:include filename="$(find description)/urdf/constants.xacro"/>
     <!-- Note: mass can be used across both casters -->
-    <xacro:property name="caster_link_mass" value="0.5"/>
     <xacro:macro name="front_caster_link_inertia">
         <inertia
@@ -21,7 +21,4 @@
         />
     </xacro:macro>
-    <!-- Constants realted to casters joint definition -->
-    <xacro:property name="casters_separation" value="1.12"/>
-    <xacro:property name="caster_vertical_offset" value="-0.619167561"/>
     <!-- Front caster link definition -->
     <link name="front_caster_link">
@@ -77,6 +74,4 @@
     </joint>
     <!-- Wheel definitions and joints -->
-    <!-- Constants related to caster wheel definition -->
-    <xacro:property name="caster_wheel_mass" value="0.7"/>
     <xacro:macro name="front_caster_wheel_inertia">
         <inertia
@@ -93,7 +88,4 @@
         />
     </xacro:macro>
-    <!-- Constants related to caster wheel joint definition -->
-    <xacro:property name="caster_link_to_wheel_dist_x" value="0.03621719"/>
-    <xacro:property name="caster_link_to_wheel_dist_z" value="-0.04361749"/>
     <!-- Front caster wheel definition -->
     <link name="front_caster_wheel">

File: robot/description/urdf/chassis_link.urdf.xacro (robot description, xacro)
@@ -1,6 +1,7 @@
 <?xml version="1.0"?>
 <robot name="chassis" xmlns:xacro="http://ros.org/wiki/xacro">
-    <!-- Constants for chassis_link -->
-    <xacro:property name="chassis_link_mass" value="33.9"/>
+    <!-- Constants -->
+    <xacro:include filename="$(find description)/urdf/constants.xacro"/>
+    <!-- Inertias -->
     <xacro:macro name="chassis_link_inertia">
         <inertia

File: robot/description/urdf/side_wheels.urdf.xacro (robot description, xacro)
@@ -2,8 +2,6 @@
 <robot name="side_wheels" xmlns:xacro="http://ros.org/wiki/xacro">
     <!-- Constants -->
-    <xacro:property name="wheel_vertical_offset" value="-0.61759696"/>
-    <xacro:property name="wheels_separation" value="0.875"/>
-    <xacro:property name="wheel_diameter" value="0.25"/> <!-- TODO: update this value -->
-    <xacro:property name="wheel_mass" value="4.45"/>
+    <xacro:include filename="$(find description)/urdf/constants.xacro"/>
+    <!-- Inertias -->
     <xacro:macro name="left_wheel_inertia">
         <inertia

File: robot/description/urdf/stand_link.urdf.xacro (robot description, xacro)
@@ -1,4 +1,6 @@
 <?xml version="1.0"?>
 <robot name="stand_link" xmlns:xacro="http://ros.org/wiki/xacro">
+    <!-- Constants -->
+    <xacro:include filename="$(find description)/urdf/constants.xacro"/>
     <!-- Stand link; this is a dummy link that is used to make camera placement and other sensors on the stand more convenient -->
     <!-- Stand link definition. Note: purposely left blank -->

Commit message: added Lidar Plug-in

File: robot/description/urdf/caffeine.gazebo.xacro (robot description, xacro)
@@ -34,3 +34,40 @@
         </plugin>
     </gazebo>
+    <!-- LIDAR plug-in -->
+    <!-- TODO: Double check the numbers-->
+   <gazebo reference="base_laser">
+      <sensor type="ray" name="gpu_hokuyo_sensor">
+         <pose>0 0 0 0 0 0</pose>
+         <visualize>${laser_visualize}</visualize>
+        <update_rate>${laser_update_rate}</update_rate>
+         <ray>
+            <scan>
+               <horizontal>
+                  <samples>${laser_horizontal_samples}</samples>
+                  <resolution>${laser_horizontal_resolution}</resolution>
+                  <min_angle>${laser_horizontal_min_angle}</min_angle>
+                  <max_angle>${laser_horizontal_max_angle}</max_angle>
+               </horizontal>
+            </scan>
+            <range>
+               <min>${laser_range_min_angle}</min>
+               <max>${laser_range_max_angle}</max>
+               <resolution>${laser_range_resolution}</resolution>
+            </range>
+            <noise>
+               <type>gaussian</type>
+               <!-- Noise based on gazebosim.org's tutorial on writing gazebo plugins w/ ROS. The comment they put will be reproduced:
+                    Noise parameters based on published spec for Hokuyo laser achieving "+-30mm" accuracy at range < 10 m. A mean of
+                    0.0m and stddev of 0.01m will put 99.7% of samples within 0.03m of the true reading. -->
+               <mean>${laser_mean}</mean>
+               <stddev>${laser_stddev}</stddev>
+            </noise>
+         </ray>
+         <plugin name="gazebo_ros_hokuyo_controller" filename="libgazebo_ros_laser.so">
+            <topicName>
+            scan</topicName>
+            <frameName>base_laser</frameName>
+         </plugin>
+      </sensor>
+   </gazebo>
 </robot>

File: robot/description/urdf/constants.xacro (robot description, xacro)
@@ -19,3 +19,21 @@
     <!-- Gazebo Motor -->
     <xacro:property name="diff_drive_update_rate" value="30.0"/>
+    <!-- Constants for hokuyo 2D LIDAR sensor -->
+    <xacro:property name="laser_visualize" value="false"/>
+    <xacro:property name="laser_update_rate" value="30"/>
+    <xacro:property name="laser_horizontal_samples" value="1080"/>
+    <xacro:property name="laser_horizontal_resolution" value="1"/>
+    <xacro:property name="laser_horizontal_min_angle" value="-2.356"/>
+    <xacro:property name="laser_horizontal_max_angle" value="2.356"/>
+    <xacro:property name="laser_range_min_angle" value="0.1"/>
+    <xacro:property name="laser_range_max_angle" value="5.6"/>
+    <xacro:property name="laser_range_resolution" value="0.01"/>
+    <xacro:property name="laser_mean" value="0.0"/>
+    <xacro:property name="laser_stddev" value="0.1"/>
+    <xacro:property name="hokuyo_length" value="0.05"/>
+    <xacro:property name="hokuyo_width" value="0.05"/>
+    <xacro:property name="hokuyo_height" value="0.07"/>
+    <xacro:property name="hokuyo_mass" value="0.16"/>
+    <xacro:property name="laser_x_dist" value="0.07"/>
+    <xacro:property name="laser_z_dist" value="0.16"/>
 </robot>

File: robot/description/urdf/inertias.xacro (robot description, xacro)
@@ -32,3 +32,13 @@
         />
     </xacro:macro>
+    <xacro:macro name="box_inertia" params="mass length width height">
+        <inertia
+            ixx="${mass * (height*height + length*length)/12.0}"
+                        ixy="0.0"
+            ixz="0.0"
+                        iyy="${mass * (width*width + length*length)/12.0}"
+                        iyz="0.0"
+            izz="${mass * (width*width + height*height)/12.0}"
+        />
+    </xacro:macro>
 </robot>

Commit message: added Lidar plugin

File: robot/description/urdf/caffeine.gazebo.xacro (robot description, xacro)
@@ -65,7 +65,6 @@
          </ray>
          <plugin name="gazebo_ros_hokuyo_controller" filename="libgazebo_ros_laser.so">
-            <topicName>
-            scan</topicName>
-            <frameName>base_laser</frameName>
+            <topicName>${laser_topicName}</topicName>
+            <frameName>${laser_frameName}</frameName>
          </plugin>
       </sensor>

File: robot/description/urdf/caffeine.urdf.xacro (robot description, xacro)
@@ -24,23 +24,4 @@
     <!-- wheels: front and back casters -->
     <xacro:include filename="$(find description)/urdf/casters.urdf.xacro"/>
-   <!-- LIDAR link -->
-   <link name="base_laser">
-        <inertial>
-            <mass value="${hokuyo_mass}"/>
-            <xacro:box_inertia mass="${hokuyo_mass}" length="${hokuyo_length}" width="${hokuyo_width}" height="${hokuyo_height}"/>
-        </inertial>
-      <visual>
-         <origin xyz="0 0 0" rpy="0 0 0"/>
-         <geometry>
-            <mesh filename="package:///description/meshes/hokuyo.dae"/>
-         </geometry>
-      </visual>
-      <collision>
-         <origin xyz="0 0 0" rpy="0 0 0"/>
-         <geometry>
-            <mesh filename="package:///description/meshes/hokuyo.dae"/>
-         </geometry>
-      </collision>
-   </link>
    <!-- LIDAR joint -->
    <!-- TODO: double check xyz location-->

File: robot/description/urdf/constants.xacro (robot description, xacro)
@@ -31,9 +31,11 @@
     <xacro:property name="laser_mean" value="0.0"/>
     <xacro:property name="laser_stddev" value="0.1"/>
+    <xacro:property name="laser_topicName" value="scan"/>
+    <xacro:property name="laser_frameName" value="base_laser"/>
     <xacro:property name="hokuyo_length" value="0.05"/>
     <xacro:property name="hokuyo_width" value="0.05"/>
     <xacro:property name="hokuyo_height" value="0.07"/>
     <xacro:property name="hokuyo_mass" value="0.16"/>
-    <xacro:property name="laser_x_dist" value="0.07"/>
-    <xacro:property name="laser_z_dist" value="0.16"/>
+    <xacro:property name="laser_x_dist" value="0.3"/>
+    <xacro:property name="laser_z_dist" value="0.0"/>
 </robot>

Commit message: added Lidar plugin

File: robot/description/urdf/caffeine.gazebo.xacro (robot description, xacro)
@@ -51,15 +51,15 @@
             </scan>
             <range>
-               <min>${laser_range_min_angle}</min>
-               <max>${laser_range_max_angle}</max>
+               <min>${laser_range_min}</min>
+               <max>${laser_range_max}</max>
                <resolution>${laser_range_resolution}</resolution>
             </range>
             <noise>
-               <type>gaussian</type>
+               <type>${laser_noise_type}</type>
                <!-- Noise based on gazebosim.org's tutorial on writing gazebo plugins w/ ROS. The comment they put will be reproduced:
                     Noise parameters based on published spec for Hokuyo laser achieving "+-30mm" accuracy at range < 10 m. A mean of
                     0.0m and stddev of 0.01m will put 99.7% of samples within 0.03m of the true reading. -->
-               <mean>${laser_mean}</mean>
-               <stddev>${laser_stddev}</stddev>
+               <mean>${laser_noise_mean}</mean>
+               <stddev>${laser_noise_stddev}</stddev>
             </noise>
          </ray>

File: robot/description/urdf/constants.xacro (robot description, xacro)
@@ -26,9 +26,10 @@
     <xacro:property name="laser_horizontal_min_angle" value="-2.356"/>
     <xacro:property name="laser_horizontal_max_angle" value="2.356"/>
-    <xacro:property name="laser_range_min_angle" value="0.1"/>
-    <xacro:property name="laser_range_max_angle" value="5.6"/>
+    <xacro:property name="laser_range_min" value="0.1"/>
+    <xacro:property name="laser_range_max" value="5.6"/>
     <xacro:property name="laser_range_resolution" value="0.01"/>
-    <xacro:property name="laser_mean" value="0.0"/>
-    <xacro:property name="laser_stddev" value="0.1"/>
+    <xacro:property name="laser_noise_type" value="gaussian"/>
+    <xacro:property name="laser_noise_mean" value="0.0"/>
+    <xacro:property name="laser_noise_stddev" value="0.1"/>
     <xacro:property name="laser_topicName" value="scan"/>
     <xacro:property name="laser_frameName" value="base_laser"/>

Commit message: Added gazebo plugin, camera/optical links, and launch file for zed emulation with stereo_image_proc

File: robot/description/urdf/caffeine.gazebo.xacro (robot description, xacro)
@@ -7,5 +7,5 @@
     <gazebo>
         <plugin name="caffeine_drive_controller" filename="libgazebo_ros_diff_drive.so">
-            <robotNamespace>caffeine</robotNamespace>
+            <!-- <robotNamespace></robotNamespace> -->
             <updateRate>${diff_drive_update_rate}</updateRate>
             <leftJoint>left_wheel_joint</leftJoint>
@@ -31,6 +31,56 @@
     <gazebo>
         <plugin name="gazebo_ros_control" filename="libgazebo_ros_control.so">
-            <robotNamespace>caffeine</robotNamespace>
+            <!-- <robotNamespace></robotNamespace> -->
         </plugin>
     </gazebo>
+    <!-- TODO: double check these numbers -->
+    <!-- Gazebo multicamera plugin -->
+    <gazebo reference="camera_link">
+        <sensor type="multicamera" name="stereo_camera">
+            <update_rate>30.0</update_rate>
+            <camera name="left">
+            <horizontal_fov>1.571</horizontal_fov>
+            <image>
+                <width>1280</width>
+                <height>720</height>
+                <format>R8G8B8</format>
+            </image>
+            <clip>
+                <near>0.02</near>
+                <far>300</far>
+            </clip>
+            </camera>
+            <camera name="right">
+            <pose>0 ${-ZED_camera_length} 0 0 0 0</pose>
+            <horizontal_fov>1.571</horizontal_fov>
+            <image>
+                <width>1280</width>
+                <height>720</height>
+                <format>R8G8B8</format>
+            </image>
+            <clip>
+                <near>0.02</near>
+                <far>300</far>
+            </clip>
+            </camera>
+            <plugin name="stereo_camera_controller" filename="libgazebo_ros_multicamera.so">
+            <cameraName>zed/zed_node</cameraName>
+            <alwaysOn>true</alwaysOn>
+            <updateRate>0</updateRate>
+            <cameraName></cameraName>
+            <imageTopicName>image_raw</imageTopicName>
+            <cameraInfoTopicName>camera_info</cameraInfoTopicName>
+            <depthImageTopicName>depth/image_raw</depthImageTopicName>
+            <depthImageInfoTopicName>depth/camera_info</depthImageInfoTopicName>
+            <pointCloudTopicName>depth/points</pointCloudTopicName>
+            <frameName>zed_camera_link_optical</frameName>
+            <hackBaseline>${ZED_camera_length}</hackBaseline>
+            <distortionK1>0.0</distortionK1>
+            <distortionK2>0.0</distortionK2>
+            <distortionK3>0.0</distortionK3>
+            <distortionT1>0.0</distortionT1>
+            <distortionT2>0.0</distortionT2>
+            </plugin>
+        </sensor>
+    </gazebo>
 </robot>

File: robot/description/urdf/constants.xacro (robot description, xacro)
@@ -19,3 +19,14 @@
     <!-- Gazebo Motor -->
     <xacro:property name="diff_drive_update_rate" value="30.0"/>
+    <!-- ZED camera -->
+    <!-- NOTE: approx as a rectangular prism -->
+    <xacro:property name="ZED_camera_mass" value="0.1587573"/>
+    <xacro:property name="ZED_camera_length" value="0.175"/>
+    <xacro:property name="ZED_camera_width" value="0.03"/>
+    <xacro:property name="ZED_camera_height" value="0.033"/>
+    <!-- Stand -->
+    <xacro:property name="stand_length" value="0.412"/>
+    <xacro:property name="stand_width" value="0.254"/>
+    <xacro:property name="stand_height" value="1.324"/>
+    <xacro:property name="stand_mass" value="1.0"/>
 </robot>

File: robot/description/urdf/inertias.xacro (robot description, xacro)
@@ -32,3 +32,14 @@
         />
     </xacro:macro>
+    <!-- Camera -->
+    <xacro:macro name="box_inertia" params="mass length width height">
+        <inertia
+            ixx="${mass * (height*height + length*length)/12.0}"
+                        ixy="0.0"
+            ixz="0.0"
+                        iyy="${mass * (width*width + length*length)/12.0}"
+                        iyz="0.0"
+            izz="${mass * (width*width + height*height)/12.0}"
+        />
+    </xacro:macro>
 </robot>

File: robot/description/urdf/stand_link.urdf.xacro (robot description, xacro)
@@ -8,3 +8,53 @@
     <link name="stand_link">
     </link>
+    <!-- ZED Camera -->
+    <link name="zed_camera_link">
+        <visual>
+            <origin xyz="0 0 0" rpy="0 0 0"/>
+            <!-- TODO: should be using the mesh but couldn't get it to work -->
+            <geometry>
+            <box size="${ZED_camera_width} ${ZED_camera_length} ${ZED_camera_height}"/>
+            </geometry>
+        </visual>
+        <collision>
+            <origin xyz="0 0 0" rpy="0 0 0"/>
+            <geometry>
+                <box size="${ZED_camera_width} ${ZED_camera_length} ${ZED_camera_height}"/>
+            </geometry>
+        </collision>
+        <inertial>
+            <xacro:box_inertia mass="${ZED_camera_mass}" length="${ZED_camera_length}" width="${ZED_camera_width}" height="${ZED_camera_height}"/>
+            <mass value="${ZED_camera_mass}"/>
+        </inertial>
+    </link>
+    <joint name="zed_camera_joint" type="fixed">
+        <parent link="stand_link"/>
+        <child link="zed_camera_link"/>
+        <origin xyz="${stand_length/2} 0 ${stand_height + ZED_camera_height}" rpy="0 0 0"/>
+    </joint>
+    <!-- ZED camera lenses -->
+    <!-- NOTE: I'm only defining one and not visually showing any-->
+    <!-- I only need one for purposes of using the plugin -->
+    <!-- TODO: check if it's fine to call the left lense camera_link (rtabmap doesn't specify whether it wants the lense frame or the camera frame itself) -->
+    <link name="camera_link">
+        <!-- Inertial tag here to ensure that link does not phase through robot-->
+        <inertial>
+            <mass value="0.0001"/>
+            <inertia ixx="0.0001" ixy="0" ixz="0" iyy="0.0001" iyz="0" izz="0.00001"/>
+        </inertial>
+    </link>
+    <joint name="camera_link_joint" type="fixed">
+        <origin xyz="${ZED_camera_length/2.0} 0 0" rpy="0 0 0"/>
+        <parent link="zed_camera_link"/>
+        <child link="camera_link"/>
+    </joint>
+    <!-- Generate an optical frame http://www.ros.org/reps/rep-0103.html#suffix-frames so that ros and opencv can operate on the camera frame correctly -->
+    <link name="zed_camera_link_optical">
+    </link>
+    <joint name="zed_camera_link_optical_joint" type="fixed">
+        <!-- Transform b/w standard and optical frame -->
+        <origin xyz="0 0 0" rpy="${-pi/2} 0 ${-pi/2}"/>
+        <parent link="zed_camera_link"/>
+        <child link="zed_camera_link_optical"/>
+    </joint>
 </robot>

Commit message: Fixed constants.xacro parse error, namespaced scan topic and slightly moved the lidar

File: robot/description/urdf/caffeine.gazebo.xacro (robot description, xacro)
@@ -63,4 +63,5 @@
          </ray>
          <plugin name="gazebo_ros_hokuyo_controller" filename="libgazebo_ros_laser.so">
+            <robotNamespace>${robotNamespace}</robotNamespace>
             <topicName>${laser_topicName}</topicName>
             <frameName>${laser_frameName}</frameName>

File: robot/description/urdf/constants.xacro (robot description, xacro)
@@ -3,4 +3,8 @@
     <!-- Caffeine -->
     <xacro:property name="robotNamespace" value="caffeine"/>
+    <!-- Drivebase -->
+   <xacro:property name="base_length" value="1.268"/>
+   <xacro:property name="base_width" value="0.764"/>
+   <xacro:property name="base_height" value="0.01"/>
     <!-- Chassis -->
     <xacro:property name="chassis_to_base_link_dist" value="0.501747"/>
@@ -42,15 +46,15 @@
     <xacro:property name="laser_horizontal_samples" value="1080"/>
     <xacro:property name="laser_horizontal_resolution" value="1"/>
-    <xacro:property name="laser_field_of_view" value="240"/>
-    <xacro:property name="laser_horizontal_min_angle" value="$(-laser_field_of_view*pi/180)"/>
-    <xacro:property name="laser_horizontal_max_angle" value="$(laser_field_of_view*pi/180)"/>
+    <xacro:property name="laser_field_of_view" value="270"/>
+    <xacro:property name="laser_horizontal_min_angle" value="${-0.5*laser_field_of_view*pi/180}"/>
+    <xacro:property name="laser_horizontal_max_angle" value="${0.5*laser_field_of_view*pi/180}"/>
     <xacro:property name="laser_range_min" value="0.06"/>
     <xacro:property name="laser_range_max" value="4.095"/>
     <xacro:property name="laser_resolution_angle" value="0.36"/>
-    <xacro:property name="laser_range_resolution" value="$(laser_resolution_angle*pi/180)"/>
+    <xacro:property name="laser_range_resolution" value="${laser_resolution_angle*pi/180}"/>
     <xacro:property name="laser_noise_type" value="gaussian"/>
     <xacro:property name="laser_noise_mean" value="0.0"/>
     <xacro:property name="laser_noise_stddev" value="0.01/3"/>
-    <xacro:property name="laser_topicName" value="caffeine/scan"/>
+    <xacro:property name="laser_topicName" value="scan"/>
     <xacro:property name="laser_frameName" value="base_laser"/>
     <xacro:property name="laser_length" value="0.05"/>
@@ -58,5 +62,5 @@
     <xacro:property name="laser_height" value="0.07"/>
     <xacro:property name="laser_mass" value="0.16"/>
-    <xacro:property name="laser_x_dist" value="${0.634-laser_length}"/>
+    <xacro:property name="laser_x_dist" value="${base_length/2 - 2*laser_length}"/>
     <xacro:property name="laser_z_dist" value="${laser_height/2}"/>
 </robot>
