Commit message: Caff 3- LIDAR Plugin (#25)
* added Lidar Plug-in

* added Lidar Plug-in

* added Lidar plugin

* added Lidar plugin

* added Lidar plugin

* added Lidar plugin

* added Lidar plugin

* added Lidar plugin

* added Lidar plugin

* added Lidar plugin

* added Lidar plugin

* added Lidar plugin

* added Lidar plugin

* moved diff drive constants to constants file

* added constants from drive plugin

* changed 'hokuyo' name to 'laser' for consistency

* added extra line at the end

* added 'TODO' comment for parameters

* added robotNamespace constant

* added robotNamespace constant

* fixed syntax error

* placed topic under caffeine/scan

* fixed the positioning of laser

* removed robotnamespace under lidar plugin

* topic name under caffeine/scan

* fixed std dev acc to spec sheet/updated comments

* followed convention for comments

* fixed values acc to spec sheet/updated comments

* fixed code structure

* Fixed constants.xacro parse error, namespaced scan topic and slightly moved the lidar

Co-authored-by: Yviel Castillejos <yvielcastillejos@Yviels-MacBook-Pro.local>
Co-authored-by: Erick Mejia Uzeda <erickmu1@hotmail.com>

File: robot/description/urdf/caffeine.gazebo.xacro (robot description, xacro)
@@ -4,26 +4,25 @@
     <xacro:include filename="$(find description)/urdf/constants.xacro"/>
     <!-- differential drive control support -->
-    <!-- TODO: update parameters once they become known -->
     <gazebo>
         <plugin name="caffeine_drive_controller" filename="libgazebo_ros_diff_drive.so">
-            <robotNamespace>caffeine</robotNamespace>
+            <robotNamespace>${robotNamespace}</robotNamespace>
             <updateRate>${diff_drive_update_rate}</updateRate>
-            <leftJoint>left_wheel_joint</leftJoint>
-            <rightJoint>right_wheel_joint</rightJoint>
+            <leftJoint>${wheel_left_joint}</leftJoint>
+            <rightJoint>${wheel_right_joint}</rightJoint>
             <wheelSeparation>${wheels_separation}</wheelSeparation>
             <wheelDiameter>${wheel_diameter}</wheelDiameter>
-            <wheelAcceleration>1.0</wheelAcceleration>
-            <wheelTorque>20</wheelTorque>
-            <commandTopic>cmd_vel</commandTopic>
-            <odometryTopic>odom</odometryTopic>
-            <odometryFrame>odom</odometryFrame>
-            <robotBaseFrame>base_link</robotBaseFrame>
-            <odometrySource>encoder</odometrySource>
-            <publishWheelTF>false</publishWheelTF>
-            <publishOdomTF>true</publishOdomTF>
-            <publishTf>true</publishTf>
-            <publishWheelJointState>true</publishWheelJointState>
-            <legacyMode>false</legacyMode>
-            <rosDebugLevel>na</rosDebugLevel>
+            <wheelAcceleration>${wheel_acceleration}</wheelAcceleration>
+            <wheelTorque>${wheel_torque}</wheelTorque>
+            <commandTopic>${diff_drive_commandTopic}</commandTopic>
+            <odometryTopic>${diff_drive_odometryTopic}</odometryTopic>
+            <odometryFrame>${diff_drive_odometryFrame}</odometryFrame>
+            <robotBaseFrame>${diff_drive_robotBaseFrame}</robotBaseFrame>
+            <odometrySource>${diff_drive_odometrySource}</odometrySource>
+            <publishWheelTF>${diff_drive_publishWheelTF}</publishWheelTF>
+            <publishOdomTF>${diff_drive_publishOdomTF}</publishOdomTF>
+            <publishTf>${diff_drive_publishTf}</publishTf>
+            <publishWheelJointState>${diff_drive_publishWheelJointState}</publishWheelJointState>
+            <legacyMode>${diff_drive_legacymode}</legacyMode>
+            <rosDebugLevel>${diff_drive_rosDebugLevel}</rosDebugLevel>
         </plugin>
     </gazebo>
@@ -31,6 +30,42 @@
     <gazebo>
         <plugin name="gazebo_ros_control" filename="libgazebo_ros_control.so">
-            <robotNamespace>caffeine</robotNamespace>
+            <robotNamespace>${robotNamespace}</robotNamespace>
         </plugin>
     </gazebo>
+    <!-- LIDAR -->
+   <gazebo reference="base_laser">
+      <sensor type="ray" name="gpu_hokuyo_sensor">
+         <pose>0 0 0 0 0 0</pose>
+         <visualize>${laser_visualize}</visualize>
+        <update_rate>${laser_update_rate}</update_rate>
+         <ray>
+            <scan>
+               <horizontal>
+                  <samples>${laser_horizontal_samples}</samples>
+                  <resolution>${laser_horizontal_resolution}</resolution>
+                  <min_angle>${laser_horizontal_min_angle}</min_angle>
+                  <max_angle>${laser_horizontal_max_angle}</max_angle>
+               </horizontal>
+            </scan>
+            <range>
+               <min>${laser_range_min}</min>
+               <max>${laser_range_max}</max>
+               <resolution>${laser_range_resolution}</resolution>
+            </range>
+            <noise>
+               <type>${laser_noise_type}</type>
+               <!-- Noise based on gazebosim.org's tutorial on writing gazebo plugins w/ ROS. The comment they put will be reproduced:
+                    Noise parameters based on published spec for Hokuyo laser achieving "+-10mm" accuracy at range < 10 m. A mean of
+                    0.0m and stddev of (0.01/3), will put 99.8% of samples within 0.03m of the true reading. -->
+               <mean>${laser_noise_mean}</mean>
+               <stddev>${laser_noise_stddev}</stddev>
+            </noise>
+         </ray>
+         <plugin name="gazebo_ros_hokuyo_controller" filename="libgazebo_ros_laser.so">
+            <robotNamespace>${robotNamespace}</robotNamespace>
+            <topicName>${laser_topicName}</topicName>
+            <frameName>${laser_frameName}</frameName>
+         </plugin>
+      </sensor>
+   </gazebo>
 </robot>

File: robot/description/urdf/caffeine.urdf.xacro (robot description, xacro)
@@ -24,3 +24,10 @@
     <!-- wheels: front and back casters -->
     <xacro:include filename="$(find description)/urdf/casters.urdf.xacro"/>
+   <!-- base_laser: LIDAR at front of Caffeine -->
+   <xacro:include filename="$(find description)/urdf/base_laser.urdf.xacro"/>
+   <joint name="base_laser_joint" type="fixed">
+      <parent link="base_link"/>
+      <child link="base_laser"/>
+      <origin xyz="${laser_x_dist} 0 ${laser_z_dist}" rpy="0 0 0"/>
+   </joint>
 </robot>

File: robot/description/urdf/constants.xacro (robot description, xacro)
@@ -1,4 +1,10 @@
 <?xml version="1.0"?>
 <robot name="caffeine_constants" xmlns:xacro="http://ros.org/wiki/xacro">
+    <!-- Caffeine -->
+    <xacro:property name="robotNamespace" value="caffeine"/>
+    <!-- Drivebase -->
+   <xacro:property name="base_length" value="1.268"/>
+   <xacro:property name="base_width" value="0.764"/>
+   <xacro:property name="base_height" value="0.01"/>
     <!-- Chassis -->
     <xacro:property name="chassis_to_base_link_dist" value="0.501747"/>
@@ -13,9 +19,48 @@
     <xacro:property name="caster_link_to_wheel_dist_z" value="-0.04361749"/>
     <!-- Wheels -->
+    <!-- TODO: Update acceleration and torque parameters when known -->
     <xacro:property name="wheel_vertical_offset" value="-0.61759696"/>
+    <xacro:property name="wheel_left_joint" value="left_wheel_joint"/>
+    <xacro:property name="wheel_right_joint" value="right_wheel_joint"/>
     <xacro:property name="wheels_separation" value="0.875"/>
     <xacro:property name="wheel_diameter" value="0.25"/>
+    <xacro:property name="wheel_acceleration" value="1.0"/>
+    <xacro:property name="wheel_torque" value="20"/>
     <xacro:property name="wheel_mass" value="4.45"/>
     <!-- Gazebo Motor -->
     <xacro:property name="diff_drive_update_rate" value="30.0"/>
+    <xacro:property name="diff_drive_commandTopic" value="cmd_vel"/>
+    <xacro:property name="diff_drive_odometryTopic" value="odom"/>
+    <xacro:property name="diff_drive_odometryFrame" value="odom"/>
+    <xacro:property name="diff_drive_robotBaseFrame" value="base_link"/>
+    <xacro:property name="diff_drive_odometrySource" value="encoder"/>
+    <xacro:property name="diff_drive_publishWheelTF" value="false"/>
+    <xacro:property name="diff_drive_publishOdomTF" value="true"/>
+    <xacro:property name="diff_drive_publishTf" value="true"/>
+    <xacro:property name="diff_drive_publishWheelJointState" value="true"/>
+    <xacro:property name="diff_drive_legacymode" value="false"/>
+    <xacro:property name="diff_drive_rosDebugLevel" value="na"/>
+    <!-- Hokuyo 2D LIDAR sensor -->
+    <xacro:property name="laser_visualize" value="false"/>
+    <xacro:property name="laser_update_rate" value="10"/>
+    <xacro:property name="laser_horizontal_samples" value="1080"/>
+    <xacro:property name="laser_horizontal_resolution" value="1"/>
+    <xacro:property name="laser_field_of_view" value="270"/>
+    <xacro:property name="laser_horizontal_min_angle" value="${-0.5*laser_field_of_view*pi/180}"/>
+    <xacro:property name="laser_horizontal_max_angle" value="${0.5*laser_field_of_view*pi/180}"/>
+    <xacro:property name="laser_range_min" value="0.06"/>
+    <xacro:property name="laser_range_max" value="4.095"/>
+    <xacro:property name="laser_resolution_angle" value="0.36"/>
+    <xacro:property name="laser_range_resolution" value="${laser_resolution_angle*pi/180}"/>
+    <xacro:property name="laser_noise_type" value="gaussian"/>
+    <xacro:property name="laser_noise_mean" value="0.0"/>
+    <xacro:property name="laser_noise_stddev" value="0.01/3"/>
+    <xacro:property name="laser_topicName" value="scan"/>
+    <xacro:property name="laser_frameName" value="base_laser"/>
+    <xacro:property name="laser_length" value="0.05"/>
+    <xacro:property name="laser_width" value="0.05"/>
+    <xacro:property name="laser_height" value="0.07"/>
+    <xacro:property name="laser_mass" value="0.16"/>
+    <xacro:property name="laser_x_dist" value="${base_length/2 - 2*laser_length}"/>
+    <xacro:property name="laser_z_dist" value="${laser_height/2}"/>
 </robot>

File: robot/description/urdf/inertias.xacro (robot description, xacro)
@@ -32,3 +32,11 @@
         />
     </xacro:macro>
+    <!-- Lidar -->
+    <xacro:macro name="box_inertia" params="mass length width height">
+        <inertia
+            ixx="${mass * (height*height + length*length)/12.0}" ixy="0.0000" ixz="0.0000"
+            iyx = "0.0000" iyy="${mass * (width*width + length*length)/12.0}" iyz="0.0000"
+            izx="0.0000" izy="0.0000" izz="${mass * (width*width + height*height)/12.0}"
+        />
+    </xacro:macro>
 </robot>

Commit message: Added GPS link and gazebo plugin. Untested.

File: robot/description/urdf/caffeine.gazebo.xacro (robot description, xacro)
@@ -34,3 +34,21 @@
         </plugin>
     </gazebo>
+    <gazebo>
+      <plugin name="gps_controller" filename="libhector_gazebo_ros_gps.so">
+         <updateRate>5.0</updateRate>  <!-- 5 Hz -->
+         <bodyName>gps_link</bodyName>
+         <frameId>gps_link</frameId>
+         <topicName>gps/fix</topicName>
+         <velocityTopicName>gps/fix_velocity</velocityTopicName>
+         <!-- Set reference GPS coordinates to UofT -->
+         <referenceLatitude>43.6570</referenceLatitude>
+         <referenceLongitude>-79.3903</referenceLongitude>
+         <referenceAltitude>76</referenceAltitude>
+         <!-- Model GPS behaviour -->
+         <service>1</service> <!-- SERVICE_GPS = 1 -->
+         <drift>1.5 1.5 1.5</drift> <!-- m -->
+         <velocityDrift>0.05 0.05 0.05</velocityDrift> <!-- m/s-->
+         <!-- TODO: add Gaussian noise based off Garmin GPS -->
+      </plugin>
+   </gazebo>
 </robot>

File: robot/description/urdf/constants.xacro (robot description, xacro)
@@ -19,3 +19,8 @@
     <!-- Gazebo Motor -->
     <xacro:property name="diff_drive_update_rate" value="30.0"/>
+    <!-- Garmin GPS -->
+    <!-- NOTE: approx as a cylinder; garmin itself is similar to a hockey puck -->
+    <xacro:property name="gps_diam" value="0.061"/>
+    <xacro:property name="gps_length" value="0.0195"/>
+    <xacro:property name="gps_mass" value="0.165"/>
 </robot>

File: robot/description/urdf/inertias.xacro (robot description, xacro)
@@ -32,3 +32,14 @@
         />
     </xacro:macro>
+    <!-- Cynlinder inertia for GPS -->
+    <xacro:macro name="cylinder_inertia" params="mass length radius">
+        <inertia
+            ixx="${mass * (3*radius*radius + length*length)/12.0}"
+            ixy="0.0"
+            ixz="0.0"
+                        iyy="${mass * (3*radius*radius + length*length)/12.0}"
+            iyz="0.0"
+            izz="${0.5*mass*radius*radius}"
+        />
+    </xacro:macro>
 </robot>

File: robot/description/urdf/stand_link.urdf.xacro (robot description, xacro)
@@ -8,3 +8,28 @@
     <link name="stand_link">
     </link>
+    <!-- GPS -->
+    <link name="gps_link">
+        <inertial>
+            <mass value="${gps_mass}"/>
+            <xacro:cylinder_inertia mass="${gps_mass}" length="${gps_length}" radius="${gps_diam / 2.0}"/>
+        </inertial>
+        <visual>
+            <origin xyz="0 0 0" rpy="0 0 0"/>
+            <geometry>
+                <cylinder length="${gps_length}" radius="${gps_diam / 2.0}"/>
+            </geometry>
+        </visual>
+        <collision>
+            <origin xyz="0 0 0" rpy="0 0 0"/>
+            <geometry>
+                <cylinder length="${gps_length}" radius="${gps_diam / 2.0}"/>
+            </geometry>
+        </collision>
+    </link>
+    <!-- GPS: attach gps_link to base_link -->
+    <joint name="gps_joint" type="fixed">
+        <parent link="base_link"/>
+        <child link="gps_link"/>
+        <origin xyz="${-base_width / 2.0 - 0.1} 0 ${base_height / 2.0 + gps_length / 2.0}" rpy="0 0 0"/>
+    </joint>
 </robot>

Commit message: Fixed issues with LIDAR namespacing, changed default behavior to not using GUI and updated reference frame in rviz

File: robot/description/urdf/caffeine.gazebo.xacro (robot description, xacro)
@@ -65,5 +65,5 @@
             <robotNamespace>${robotNamespace}</robotNamespace>
             <topicName>${laser_topicName}</topicName>
-	    <frameName>${tf_prefix}/${laser_frameName}</frameName>
+	    <frameName>${laser_frameName}</frameName>
          </plugin>
       </sensor>

File: robot/description/urdf/constants.xacro (robot description, xacro)
@@ -43,5 +43,5 @@
     <xacro:property name="diff_drive_rosDebugLevel" value="na"/>
     <!-- Hokuyo 2D LIDAR sensor -->
-    <xacro:property name="laser_visualize" value="false"/>
+    <xacro:property name="laser_visualize" value="true"/>
     <xacro:property name="laser_update_rate" value="10"/>
     <xacro:property name="laser_horizontal_samples" value="1080"/>

Commit message: Fixing spacing and removing tf_prefix argument in caffeine_gazebo.launch

File: robot/description/urdf/caffeine.gazebo.xacro (robot description, xacro)
@@ -8,6 +8,6 @@
             <robotNamespace>${robotNamespace}</robotNamespace>
             <updateRate>${diff_drive_update_rate}</updateRate>
-	    <leftJoint>${tf_prefix}/${wheel_left_joint}</leftJoint>
-	    <rightJoint>${tf_prefix}/${wheel_right_joint}</rightJoint>
+	        <leftJoint>${tf_prefix}/${wheel_left_joint}</leftJoint>
+	        <rightJoint>${tf_prefix}/${wheel_right_joint}</rightJoint>
             <wheelSeparation>${wheels_separation}</wheelSeparation>
             <wheelDiameter>${wheel_diameter}</wheelDiameter>
@@ -38,5 +38,5 @@
          <pose>0 0 0 0 0 0</pose>
          <visualize>${laser_visualize}</visualize>
-        <update_rate>${laser_update_rate}</update_rate>
+         <update_rate>${laser_update_rate}</update_rate>
          <ray>
             <scan>
@@ -65,5 +65,5 @@
             <robotNamespace>${robotNamespace}</robotNamespace>
             <topicName>${laser_topicName}</topicName>
-	    <frameName>${laser_frameName}</frameName>
+            <frameName>${laser_frameName}</frameName>
          </plugin>
       </sensor>

File: robot/description/urdf/caffeine.urdf.xacro (robot description, xacro)
@@ -9,6 +9,6 @@
     <xacro:include filename="$(find description)/urdf/chassis_link.urdf.xacro"/>
     <joint name="${tf_prefix}/chassis_link_joint" type="fixed">
-	<parent link="${tf_prefix}/base_link"/>
-	<child link="${tf_prefix}/chassis_link"/>
+	    <parent link="${tf_prefix}/base_link"/>
+	    <child link="${tf_prefix}/chassis_link"/>
         <origin rpy="0 0 0" xyz="0 0 ${chassis_to_base_link_dist}"/>
     </joint>
@@ -16,6 +16,6 @@
     <xacro:include filename="$(find description)/urdf/stand_link.urdf.xacro"/>
     <joint name="${tf_prefix}/stand_link_joint" type="fixed">
-	<parent link="${tf_prefix}/chassis_link"/>
-	<child link="${tf_prefix}/stand_link"/>
+	    <parent link="${tf_prefix}/chassis_link"/>
+	    <child link="${tf_prefix}/stand_link"/>
         <origin rpy="0 0 0" xyz="0 0 ${chassis_to_stand_link_dist}"/>
     </joint>

File: robot/description/urdf/casters.urdf.xacro (robot description, xacro)
@@ -26,6 +26,6 @@
     <joint name="${tf_prefix}/front_caster_link_joint" type="fixed">
         <!-- <axis xyz="0 0 1"/> -->
-	<parent link="${tf_prefix}/chassis_link"/>
-	<child link="${tf_prefix}/front_caster_link"/>
+	    <parent link="${tf_prefix}/chassis_link"/>
+	    <child link="${tf_prefix}/front_caster_link"/>
         <origin rpy="0 0 0" xyz="${casters_separation / 2.0} 0 ${caster_vertical_offset}"/>
     </joint>
@@ -52,6 +52,6 @@
     <joint name="${tf_prefix}/back_caster_link_joint" type="fixed">
         <!-- <axis xyz="0 0 1"/> -->
-	<parent link="${tf_prefix}/chassis_link"/>
-	<child link="${tf_prefix}/back_caster_link"/>
+	    <parent link="${tf_prefix}/chassis_link"/>
+	    <child link="${tf_prefix}/back_caster_link"/>
         <origin rpy="0 0 0" xyz="-${casters_separation / 2.0} 0 ${caster_vertical_offset}"/>
     </joint>
@@ -76,6 +76,6 @@
     </link>
     <joint name="${tf_prefix}/front_caster_wheel_joint" type="continuous">
-	<parent link="${tf_prefix}/front_caster_link"/>
-	<child link="${tf_prefix}/front_caster_wheel"/>
+	    <parent link="${tf_prefix}/front_caster_link"/>
+	    <child link="${tf_prefix}/front_caster_wheel"/>
         <origin rpy="0 0 0" xyz="${caster_link_to_wheel_dist_x} 0 ${caster_link_to_wheel_dist_z}"/>
         <axis xyz="0 1 0"/>
@@ -101,6 +101,6 @@
     </link>
     <joint name="${tf_prefix}/back_caster_wheel_joint" type="continuous">
-	<parent link="${tf_prefix}/back_caster_link"/>
-	<child link="${tf_prefix}/back_caster_wheel"/>
+	    <parent link="${tf_prefix}/back_caster_link"/>
+	    <child link="${tf_prefix}/back_caster_wheel"/>
         <origin rpy="0 0 0" xyz="-${caster_link_to_wheel_dist_x} 0 ${caster_link_to_wheel_dist_z}"/>
         <axis xyz="0 1 0"/>

File: robot/description/urdf/side_wheels.urdf.xacro (robot description, xacro)
@@ -34,6 +34,6 @@
     </link>
     <joint name="${tf_prefix}/left_wheel_joint" type="continuous">
-	<parent link="${tf_prefix}/chassis_link"/>
-	<child link="${tf_prefix}/left_wheel_link"/>
+	    <parent link="${tf_prefix}/chassis_link"/>
+	    <child link="${tf_prefix}/left_wheel_link"/>
         <origin xyz= "0 ${wheels_separation / 2.0} ${wheel_vertical_offset}"/>
         <axis xyz="0 1 0"/>
@@ -60,6 +60,6 @@
     </link>
     <joint name="${tf_prefix}/right_wheel_joint" type="continuous">
-	<parent link="${tf_prefix}/chassis_link"/>
-	<child link="${tf_prefix}/right_wheel_link"/>
+	    <parent link="${tf_prefix}/chassis_link"/>
+    	<child link="${tf_prefix}/right_wheel_link"/>
         <origin xyz= "0 -${wheels_separation / 2.0} ${wheel_vertical_offset}"/>
         <axis xyz="0 1 0"/>
