Commit message: Fixing spaces once again

File: robot/description/urdf/caffeine.gazebo.xacro (robot description, xacro)
@@ -35,37 +35,37 @@
     <!-- LIDAR -->
     <gazebo reference="${tf_prefix}/base_laser">
-      <sensor type="ray" name="gpu_hokuyo_sensor">
-         <pose>0 0 0 0 0 0</pose>
-         <visualize>${laser_visualize}</visualize>
-         <update_rate>${laser_update_rate}</update_rate>
-         <ray>
-            <scan>
-               <horizontal>
-                  <samples>${laser_horizontal_samples}</samples>
-                  <resolution>${laser_horizontal_resolution}</resolution>
-                  <min_angle>${laser_horizontal_min_angle}</min_angle>
-                  <max_angle>${laser_horizontal_max_angle}</max_angle>
-               </horizontal>
-            </scan>
-            <range>
-               <min>${laser_range_min}</min>
-               <max>${laser_range_max}</max>
-               <resolution>${laser_range_resolution}</resolution>
-            </range>
-            <noise>
-               <type>${laser_noise_type}</type>
-               <!-- Noise based on gazebosim.org's tutorial on writing gazebo plugins w/ ROS. The comment they put will be reproduced:
-                    Noise parameters based on published spec for Hokuyo laser achieving "+-10mm" accuracy at range < 10 m. A mean of
-                    0.0m and stddev of (0.01/3), will put 99.8% of samples within 0.03m of the true reading. -->
-               <mean>${laser_noise_mean}</mean>
-               <stddev>${laser_noise_stddev}</stddev>
-            </noise>
-         </ray>
-         <plugin name="gazebo_ros_hokuyo_controller" filename="libgazebo_ros_laser.so">
-            <robotNamespace>${robotNamespace}</robotNamespace>
-            <topicName>${laser_topicName}</topicName>
-            <frameName>${laser_frameName}</frameName>
-         </plugin>
-      </sensor>
-   </gazebo>
+        <sensor type="ray" name="gpu_hokuyo_sensor">
+            <pose>0 0 0 0 0 0</pose>
+            <visualize>${laser_visualize}</visualize>
+            <update_rate>${laser_update_rate}</update_rate>
+            <ray>
+                <scan>
+                    <horizontal>
+                        <samples>${laser_horizontal_samples}</samples>
+                        <resolution>${laser_horizontal_resolution}</resolution>
+                        <min_angle>${laser_horizontal_min_angle}</min_angle>
+                        <max_angle>${laser_horizontal_max_angle}</max_angle>
+                    </horizontal>
+                </scan>
+                <range>
+                    <min>${laser_range_min}</min>
+                    <max>${laser_range_max}</max>
+                    <resolution>${laser_range_resolution}</resolution>
+                </range>
+                <noise>
+                    <type>${laser_noise_type}</type>
+                    <!-- Noise based on gazebosim.org's tutorial on writing gazebo plugins w/ ROS. The comment they put will be reproduced:
+                        Noise parameters based on published spec for Hokuyo laser achieving "+-10mm" accuracy at range < 10 m. A mean of
+                        0.0m and stddev of (0.01/3), will put 99.8% of samples within 0.03m of the true reading. -->
+                    <mean>${laser_noise_mean}</mean>
+                    <stddev>${laser_noise_stddev}</stddev>
+                </noise>
+            </ray>
+            <plugin name="gazebo_ros_hokuyo_controller" filename="libgazebo_ros_laser.so">
+                <robotNamespace>${robotNamespace}</robotNamespace>
+                <topicName>${laser_topicName}</topicName>
+                <frameName>${laser_frameName}</frameName>
+            </plugin>
+        </sensor>
+    </gazebo>
 </robot>

File: robot/description/urdf/caffeine.urdf.xacro (robot description, xacro)
@@ -9,6 +9,6 @@
     <xacro:include filename="$(find description)/urdf/chassis_link.urdf.xacro"/>
     <joint name="${tf_prefix}/chassis_link_joint" type="fixed">
-	    <parent link="${tf_prefix}/base_link"/>
-	    <child link="${tf_prefix}/chassis_link"/>
+        <parent link="${tf_prefix}/base_link"/>
+        <child link="${tf_prefix}/chassis_link"/>
         <origin rpy="0 0 0" xyz="0 0 ${chassis_to_base_link_dist}"/>
     </joint>
@@ -16,6 +16,6 @@
     <xacro:include filename="$(find description)/urdf/stand_link.urdf.xacro"/>
     <joint name="${tf_prefix}/stand_link_joint" type="fixed">
-	    <parent link="${tf_prefix}/chassis_link"/>
-	    <child link="${tf_prefix}/stand_link"/>
+        <parent link="${tf_prefix}/chassis_link"/>
+        <child link="${tf_prefix}/stand_link"/>
         <origin rpy="0 0 0" xyz="0 0 ${chassis_to_stand_link_dist}"/>
     </joint>
@@ -26,8 +26,8 @@
    <!-- base_laser: LIDAR at front of Caffeine -->
    <xacro:include filename="$(find description)/urdf/base_laser.urdf.xacro"/>
-   <joint name="${tf_prefix}/base_laser_joint" type="fixed">
-      <parent link="${tf_prefix}/base_link"/>
-      <child link="${tf_prefix}/base_laser"/>
-      <origin xyz="${laser_x_dist} 0 ${laser_z_dist}" rpy="0 0 0"/>
-   </joint>
+    <joint name="${tf_prefix}/base_laser_joint" type="fixed">
+        <parent link="${tf_prefix}/base_link"/>
+        <child link="${tf_prefix}/base_laser"/>
+        <origin xyz="${laser_x_dist} 0 ${laser_z_dist}" rpy="0 0 0"/>
+    </joint>
 </robot>

Commit message: Caff 26: Adding TF prefixes  (#30)
* Added tf_prefix to all elements of our URDF

* Added tf_prefix to all links

* Fixed issues with LIDAR namespacing, changed default behavior to not using GUI and updated reference frame in rviz

* Fixing spacing and removing tf_prefix argument in caffeine_gazebo.launch

* Fixing spaces once again

* Testing if spacing issue is resolved

* Resolving spacing issues

* Turning off LIDAR visualization in Gazebo

* Updated README to explain spawner fail error (benign) in caffeine_gazebo.launch

* Added friction to casters and wheels (values are guess-timated)

Co-authored-by: Erick Mejia Uzeda <erickmu1@hotmail.com>

File: robot/description/urdf/caffeine.gazebo.xacro (robot description, xacro)
@@ -8,6 +8,6 @@
             <robotNamespace>${robotNamespace}</robotNamespace>
             <updateRate>${diff_drive_update_rate}</updateRate>
-            <leftJoint>${wheel_left_joint}</leftJoint>
-            <rightJoint>${wheel_right_joint}</rightJoint>
+            <leftJoint>${tf_prefix}/${wheel_left_joint}</leftJoint>
+            <rightJoint>${tf_prefix}/${wheel_right_joint}</rightJoint>
             <wheelSeparation>${wheels_separation}</wheelSeparation>
             <wheelDiameter>${wheel_diameter}</wheelDiameter>
@@ -34,38 +34,38 @@
     </gazebo>
     <!-- LIDAR -->
-   <gazebo reference="base_laser">
-      <sensor type="ray" name="gpu_hokuyo_sensor">
-         <pose>0 0 0 0 0 0</pose>
-         <visualize>${laser_visualize}</visualize>
-        <update_rate>${laser_update_rate}</update_rate>
-         <ray>
-            <scan>
-               <horizontal>
-                  <samples>${laser_horizontal_samples}</samples>
-                  <resolution>${laser_horizontal_resolution}</resolution>
-                  <min_angle>${laser_horizontal_min_angle}</min_angle>
-                  <max_angle>${laser_horizontal_max_angle}</max_angle>
-               </horizontal>
-            </scan>
-            <range>
-               <min>${laser_range_min}</min>
-               <max>${laser_range_max}</max>
-               <resolution>${laser_range_resolution}</resolution>
-            </range>
-            <noise>
-               <type>${laser_noise_type}</type>
-               <!-- Noise based on gazebosim.org's tutorial on writing gazebo plugins w/ ROS. The comment they put will be reproduced:
-                    Noise parameters based on published spec for Hokuyo laser achieving "+-10mm" accuracy at range < 10 m. A mean of
-                    0.0m and stddev of (0.01/3), will put 99.8% of samples within 0.03m of the true reading. -->
-               <mean>${laser_noise_mean}</mean>
-               <stddev>${laser_noise_stddev}</stddev>
-            </noise>
-         </ray>
-         <plugin name="gazebo_ros_hokuyo_controller" filename="libgazebo_ros_laser.so">
-            <robotNamespace>${robotNamespace}</robotNamespace>
-            <topicName>${laser_topicName}</topicName>
-            <frameName>${laser_frameName}</frameName>
-         </plugin>
-      </sensor>
-   </gazebo>
+    <gazebo reference="${tf_prefix}/base_laser">
+        <sensor type="ray" name="gpu_hokuyo_sensor">
+            <pose>0 0 0 0 0 0</pose>
+            <visualize>${laser_visualize}</visualize>
+            <update_rate>${laser_update_rate}</update_rate>
+            <ray>
+                <scan>
+                    <horizontal>
+                        <samples>${laser_horizontal_samples}</samples>
+                        <resolution>${laser_horizontal_resolution}</resolution>
+                        <min_angle>${laser_horizontal_min_angle}</min_angle>
+                        <max_angle>${laser_horizontal_max_angle}</max_angle>
+                    </horizontal>
+                </scan>
+                <range>
+                    <min>${laser_range_min}</min>
+                    <max>${laser_range_max}</max>
+                    <resolution>${laser_range_resolution}</resolution>
+                </range>
+                <noise>
+                    <type>${laser_noise_type}</type>
+                    <!-- Noise based on gazebosim.org's tutorial on writing gazebo plugins w/ ROS. The comment they put will be reproduced:
+                        Noise parameters based on published spec for Hokuyo laser achieving "+-10mm" accuracy at range < 10 m. A mean of
+                        0.0m and stddev of (0.01/3), will put 99.8% of samples within 0.03m of the true reading. -->
+                    <mean>${laser_noise_mean}</mean>
+                    <stddev>${laser_noise_stddev}</stddev>
+                </noise>
+            </ray>
+            <plugin name="gazebo_ros_hokuyo_controller" filename="libgazebo_ros_laser.so">
+                <robotNamespace>${robotNamespace}</robotNamespace>
+                <topicName>${laser_topicName}</topicName>
+                <frameName>${laser_frameName}</frameName>
+            </plugin>
+        </sensor>
+    </gazebo>
 </robot>

File: robot/description/urdf/caffeine.urdf.xacro (robot description, xacro)
@@ -5,17 +5,17 @@
     <xacro:include filename="$(find description)/urdf/caffeine.gazebo.xacro"/>
     <!-- base_link: origin of the robot; located in the middle, on the top of the base plate -->
-    <link name="base_link"/>
+    <link name="${tf_prefix}/base_link"/>
     <!-- chassis_link: geometric center of the robot; used as the parent in which all other links connect to -->
     <xacro:include filename="$(find description)/urdf/chassis_link.urdf.xacro"/>
-    <joint name="chassis_link_joint" type="fixed">
-        <parent link="base_link"/>
-        <child link="chassis_link"/>
+    <joint name="${tf_prefix}/chassis_link_joint" type="fixed">
+        <parent link="${tf_prefix}/base_link"/>
+        <child link="${tf_prefix}/chassis_link"/>
         <origin rpy="0 0 0" xyz="0 0 ${chassis_to_base_link_dist}"/>
     </joint>
     <!-- stand_link: origin for anything on the stand; located in the middle, on the top of the stand plate -->
     <xacro:include filename="$(find description)/urdf/stand_link.urdf.xacro"/>
-    <joint name="stand_link_joint" type="fixed">
-        <parent link="chassis_link"/>
-        <child link="stand_link"/>
+    <joint name="${tf_prefix}/stand_link_joint" type="fixed">
+        <parent link="${tf_prefix}/chassis_link"/>
+        <child link="${tf_prefix}/stand_link"/>
         <origin rpy="0 0 0" xyz="0 0 ${chassis_to_stand_link_dist}"/>
     </joint>
@@ -26,8 +26,8 @@
    <!-- base_laser: LIDAR at front of Caffeine -->
    <xacro:include filename="$(find description)/urdf/base_laser.urdf.xacro"/>
-   <joint name="base_laser_joint" type="fixed">
-      <parent link="base_link"/>
-      <child link="base_laser"/>
-      <origin xyz="${laser_x_dist} 0 ${laser_z_dist}" rpy="0 0 0"/>
+   <joint name="${tf_prefix}/base_laser_joint" type="fixed">
+        <parent link="${tf_prefix}/base_link"/>
+        <child link="${tf_prefix}/base_laser"/>
+        <origin xyz="${laser_x_dist} 0 ${laser_z_dist}" rpy="0 0 0"/>
    </joint>
 </robot>

File: robot/description/urdf/casters.urdf.xacro (robot description, xacro)
@@ -5,5 +5,5 @@
     <xacro:include filename="$(find description)/urdf/inertias.xacro"/>
     <!-- Front caster definition -->
-    <link name="front_caster_link">
+    <link name="${tf_prefix}/front_caster_link">
         <visual>
             <origin rpy="0 0 0" xyz="0 0 0"/>
@@ -23,13 +23,18 @@
         </inertial>
     </link>
-    <!-- NOTE: using a fixed joint prevents Caffeine spawning tipped over -->
-    <joint name="front_caster_link_joint" type="fixed">
-        <!-- <axis xyz="0 0 1"/> -->
-        <parent link="chassis_link"/>
-        <child link="front_caster_link"/>
+    <joint name="${tf_prefix}/front_caster_link_joint" type="continuous">
+        <axis xyz="0 0 1"/>
+        <parent link="${tf_prefix}/chassis_link"/>
+        <child link="${tf_prefix}/front_caster_link"/>
         <origin rpy="0 0 0" xyz="${casters_separation / 2.0} 0 ${caster_vertical_offset}"/>
     </joint>
+    <gazebo reference="${tf_prefix}/front_caster_link">
+        <mu1 value="0.3"/>
+        <mu2 value="0.3"/>
+        <kp value="10000000.0" />
+        <kd value="1.0" />
+    </gazebo>
     <!-- Back caster definition -->
-    <link name="back_caster_link">
+    <link name="${tf_prefix}/back_caster_link">
         <visual>
             <origin rpy="0 0 0" xyz="0 0 0"/>
@@ -49,13 +54,18 @@
         </inertial>
     </link>
-    <!-- NOTE: using a fixed joint prevents Caffeine spawning tipped over -->
-    <joint name="back_caster_link_joint" type="fixed">
-        <!-- <axis xyz="0 0 1"/> -->
-        <parent link="chassis_link"/>
-        <child link="back_caster_link"/>
+    <joint name="${tf_prefix}/back_caster_link_joint" type="continuous">
+        <axis xyz="0 0 1"/>
+        <parent link="${tf_prefix}/chassis_link"/>
+        <child link="${tf_prefix}/back_caster_link"/>
         <origin rpy="0 0 0" xyz="-${casters_separation / 2.0} 0 ${caster_vertical_offset}"/>
     </joint>
+    <gazebo reference="${tf_prefix}/back_caster_link">
+        <mu1 value="0.3"/>
+        <mu2 value="0.3"/>
+        <kp value="10000000.0" />
+        <kd value="1.0" />
+    </gazebo>
     <!-- Front caster wheel definition -->
-    <link name="front_caster_wheel">
+    <link name="${tf_prefix}/front_caster_wheel">
         <visual>
             <origin rpy="0 0 0" xyz="0 0 0"/>
@@ -75,12 +85,18 @@
         </inertial>
     </link>
-    <joint name="front_caster_wheel_joint" type="continuous">
-        <parent link="front_caster_link"/>
-        <child link="front_caster_wheel"/>
+    <joint name="${tf_prefix}/front_caster_wheel_joint" type="continuous">
+        <parent link="${tf_prefix}/front_caster_link"/>
+        <child link="${tf_prefix}/front_caster_wheel"/>
         <origin rpy="0 0 0" xyz="${caster_link_to_wheel_dist_x} 0 ${caster_link_to_wheel_dist_z}"/>
         <axis xyz="0 1 0"/>
     </joint>
+    <gazebo reference="${tf_prefix}/front_caster_wheel">
+        <mu1 value="0.1"/>
+        <mu2 value="0.1"/>
+        <kp value="10000000.0" />
+        <kd value="1.0" />
+    </gazebo>
     <!-- Back caster wheel definition -->
-    <link name="back_caster_wheel">
+    <link name="${tf_prefix}/back_caster_wheel">
         <visual>
             <origin rpy="0 0 0" xyz="0 0 0"/>
@@ -100,9 +116,15 @@
         </inertial>
     </link>
-    <joint name="back_caster_wheel_joint" type="continuous">
-        <parent link="back_caster_link"/>
-        <child link="back_caster_wheel"/>
+    <joint name="${tf_prefix}/back_caster_wheel_joint" type="continuous">
+        <parent link="${tf_prefix}/back_caster_link"/>
+        <child link="${tf_prefix}/back_caster_wheel"/>
         <origin rpy="0 0 0" xyz="-${caster_link_to_wheel_dist_x} 0 ${caster_link_to_wheel_dist_z}"/>
         <axis xyz="0 1 0"/>
     </joint>
+    <gazebo reference="${tf_prefix}/back_caster_wheel">
+        <mu1 value="0.1"/>
+        <mu2 value="0.1"/>
+        <kp value="10000000.0" />
+        <kd value="1.0" />
+    </gazebo>
 </robot>

File: robot/description/urdf/chassis_link.urdf.xacro (robot description, xacro)
@@ -5,5 +5,5 @@
     <xacro:include filename="$(find description)/urdf/inertias.xacro"/>
     <!-- Chassis link definition; chassis link is associated with the centroid of the bounding box of the robot and the chassis_link.dae file-->
-    <link name="chassis_link">
+    <link name="${tf_prefix}/chassis_link">
         <visual>
             <origin rpy="0 0 0" xyz="0 0 0"/>

File: robot/description/urdf/side_wheels.urdf.xacro (robot description, xacro)
@@ -15,5 +15,5 @@
     </xacro:macro>
     <!-- left wheel -->
-    <link name="left_wheel_link">
+    <link name="${tf_prefix}/left_wheel_link">
         <visual>
             <origin rpy="0 0 0" xyz="0 0 0"/>
@@ -33,13 +33,19 @@
         </inertial>
     </link>
-    <joint name="left_wheel_joint" type="continuous">
-        <parent link="chassis_link"/>
-        <child link="left_wheel_link"/>
+    <joint name="${tf_prefix}/left_wheel_joint" type="continuous">
+        <parent link="${tf_prefix}/chassis_link"/>
+        <child link="${tf_prefix}/left_wheel_link"/>
         <origin xyz= "0 ${wheels_separation / 2.0} ${wheel_vertical_offset}"/>
         <axis xyz="0 1 0"/>
     </joint>
-    <xacro:Transmission joint="left_wheel_joint"/>
+    <gazebo reference="${tf_prefix}/left_wheel_link">
+        <mu1 value="1.0"/>
+        <mu2 value="1.0"/>
+        <kp value="10000000.0" />
+        <kd value="1.0" />
+    </gazebo>
+    <xacro:Transmission joint="${tf_prefix}/left_wheel_joint"/>
     <!-- right wheel -->
-    <link name="right_wheel_link">
+    <link name="${tf_prefix}/right_wheel_link">
         <visual>
             <origin rpy="0 0 0" xyz="0 0 0"/>
@@ -59,10 +65,16 @@
         </inertial>
     </link>
-    <joint name="right_wheel_joint" type="continuous">
-        <parent link="chassis_link"/>
-        <child link="right_wheel_link"/>
+    <joint name="${tf_prefix}/right_wheel_joint" type="continuous">
+        <parent link="${tf_prefix}/chassis_link"/>
+        <child link="${tf_prefix}/right_wheel_link"/>
         <origin xyz= "0 -${wheels_separation / 2.0} ${wheel_vertical_offset}"/>
         <axis xyz="0 1 0"/>
     </joint>
-    <xacro:Transmission joint="right_wheel_joint"/>
+    <gazebo reference="${tf_prefix}/right_wheel_link">
+        <mu1 value="1.0"/>
+        <mu2 value="1.0"/>
+        <kp value="10000000.0" />
+        <kd value="1.0" />
+    </gazebo>
+    <xacro:Transmission joint="${tf_prefix}/right_wheel_joint"/>
 </robot>

File: robot/description/urdf/stand_link.urdf.xacro (robot description, xacro)
@@ -6,5 +6,5 @@
     <!-- Stand link; this is a dummy link that is used to make camera placement and other sensors on the stand more convenient -->
     <!-- Stand link definition. Note: purposely left blank -->
-    <link name="stand_link">
+    <link name="${tf_prefix}/stand_link">
     </link>
 </robot>

Commit message: fixing merge conflicts in urdf files

File: robot/description/urdf/caffeine.gazebo.xacro (robot description, xacro)
@@ -34,5 +34,4 @@
     <gazebo>
         <plugin name="gazebo_ros_control" filename="libgazebo_ros_control.so">
-<<<<<<< HEAD
             <robotNamespace>${robotNamespace}</robotNamespace>
         </plugin>
@@ -73,8 +72,4 @@
             </plugin>
         </sensor>
-    </gazebo>
-=======
-            <!-- <robotNamespace></robotNamespace> -->
-        </plugin>
     </gazebo>
     <!-- TODO: double check these numbers -->
@@ -128,4 +123,3 @@
         </sensor>
     </gazebo>
->>>>>>> 9f8b0a61cddf46fc7b7b52e5512b828974b6028a
 </robot>

File: robot/description/urdf/caffeine.urdf.xacro (robot description, xacro)
@@ -5,9 +5,5 @@
     <xacro:include filename="$(find description)/urdf/caffeine.gazebo.xacro"/>
     <!-- base_link: origin of the robot; located in the middle, on the top of the base plate -->
-<<<<<<< HEAD
     <link name="${tf_prefix}/base_link"/>
-=======
-    <link name="base_link"/>
->>>>>>> 9f8b0a61cddf46fc7b7b52e5512b828974b6028a
     <!-- chassis_link: geometric center of the robot; used as the parent in which all other links connect to -->
     <xacro:include filename="$(find description)/urdf/chassis_link.urdf.xacro"/>
