Commit message: adding transform prefix to remaining links

File: robot/description/urdf/caffeine.gazebo.xacro (robot description, xacro)
@@ -6,9 +6,5 @@
     <gazebo>
         <plugin name="caffeine_drive_controller" filename="libgazebo_ros_diff_drive.so">
-<<<<<<< HEAD
             <robotNamespace>${robotNamespace}</robotNamespace>
-=======
-            <!-- <robotNamespace></robotNamespace> -->
->>>>>>> 9f8b0a61cddf46fc7b7b52e5512b828974b6028a
             <updateRate>${diff_drive_update_rate}</updateRate>
             <leftJoint>${tf_prefix}/${wheel_left_joint}</leftJoint>

File: robot/description/urdf/casters.urdf.xacro (robot description, xacro)
@@ -116,13 +116,7 @@
         </inertial>
     </link>
-<<<<<<< HEAD
-    <joint name="back_caster_wheel_joint" type="continuous">
-        <parent link="back_caster_link"/>
-        <child link="back_caster_wheel"/>
-=======
     <joint name="${tf_prefix}/back_caster_wheel_joint" type="continuous">
         <parent link="${tf_prefix}/back_caster_link"/>
         <child link="${tf_prefix}/back_caster_wheel"/>
->>>>>>> 3e3c6deaa9438f8a3a68e9a89c9fcb679f226f31
         <origin rpy="0 0 0" xyz="-${caster_link_to_wheel_dist_x} 0 ${caster_link_to_wheel_dist_z}"/>
         <axis xyz="0 1 0"/>

File: robot/description/urdf/constants.xacro (robot description, xacro)
@@ -31,5 +31,4 @@
     <!-- Gazebo Motor -->
     <xacro:property name="diff_drive_update_rate" value="30.0"/>
-<<<<<<< HEAD
     <xacro:property name="diff_drive_commandTopic" value="cmd_vel"/>
     <xacro:property name="diff_drive_odometryTopic" value="odom"/>
@@ -66,5 +65,4 @@
     <xacro:property name="laser_x_dist" value="${base_length/2 - 2*laser_length}"/>
     <xacro:property name="laser_z_dist" value="${laser_height/2}"/>
-=======
     <!-- ZED camera -->
     <!-- NOTE: approx as a rectangular prism -->
@@ -78,4 +76,3 @@
     <xacro:property name="stand_height" value="1.324"/>
     <xacro:property name="stand_mass" value="1.0"/>
->>>>>>> 9f8b0a61cddf46fc7b7b52e5512b828974b6028a
 </robot>

File: robot/description/urdf/inertias.xacro (robot description, xacro)
@@ -32,5 +32,4 @@
         />
     </xacro:macro>
-<<<<<<< HEAD
     <!-- Lidar -->
     <xacro:macro name="box_inertia" params="mass length width height">
@@ -41,5 +40,4 @@
         />
     </xacro:macro>
-=======
     <!-- Camera -->
     <xacro:macro name="box_inertia" params="mass length width height">
@@ -53,4 +51,3 @@
         />
     </xacro:macro>
->>>>>>> 9f8b0a61cddf46fc7b7b52e5512b828974b6028a
 </robot>

File: robot/description/urdf/stand_link.urdf.xacro (robot description, xacro)
@@ -6,11 +6,8 @@
     <!-- Stand link; this is a dummy link that is used to make camera placement and other sensors on the stand more convenient -->
     <!-- Stand link definition. Note: purposely left blank -->
-<<<<<<< HEAD
     <link name="${tf_prefix}/stand_link">
-=======
-    <link name="stand_link">
     </link>
     <!-- ZED Camera -->
-    <link name="zed_camera_link">
+    <link name="${tf_prefix}/zed_camera_link">
         <visual>
             <origin xyz="0 0 0" rpy="0 0 0"/>
@@ -31,8 +28,8 @@
         </inertial>
     </link>
-    <joint name="zed_camera_joint" type="fixed">
-        <parent link="stand_link"/>
-        <child link="zed_camera_link"/>
+    <joint name="${tf_prefix}/zed_camera_joint" type="fixed">
         <origin xyz="${stand_length/2} 0 ${stand_height + ZED_camera_height}" rpy="0 0 0"/>
+        <parent link="${tf_prefix}/stand_link"/>
+        <child link="${tf_prefix}/zed_camera_link"/>
     </joint>
     <!-- ZED camera lenses -->
@@ -40,5 +37,5 @@
     <!-- I only need one for purposes of using the plugin -->
     <!-- TODO: check if it's fine to call the left lense camera_link (rtabmap doesn't specify whether it wants the lense frame or the camera frame itself) -->
-    <link name="camera_link">
+    <link name="${tf_prefix}/camera_link">
         <!-- Inertial tag here to ensure that link does not phase through robot-->
         <inertial>
@@ -47,18 +44,17 @@
         </inertial>
     </link>
-    <joint name="camera_link_joint" type="fixed">
+    <joint name="${tf_prefix}/camera_link_joint" type="fixed">
         <origin xyz="${ZED_camera_length/2.0} 0 0" rpy="0 0 0"/>
-        <parent link="zed_camera_link"/>
-        <child link="camera_link"/>
+        <parent link="${tf_prefix}/zed_camera_link"/>
+        <child link="${tf_prefix}/camera_link"/>
     </joint>
     <!-- Generate an optical frame http://www.ros.org/reps/rep-0103.html#suffix-frames so that ros and opencv can operate on the camera frame correctly -->
-    <link name="zed_camera_link_optical">
->>>>>>> 9f8b0a61cddf46fc7b7b52e5512b828974b6028a
+    <link name="${tf_prefix}/zed_camera_link_optical">
     </link>
-    <joint name="zed_camera_link_optical_joint" type="fixed">
+    <joint name="${tf_prefix}/zed_camera_link_optical_joint" type="fixed">
         <!-- Transform b/w standard and optical frame -->
         <origin xyz="0 0 0" rpy="${-pi/2} 0 ${-pi/2}"/>
-        <parent link="zed_camera_link"/>
-        <child link="zed_camera_link_optical"/>
+        <parent link="${tf_prefix}/zed_camera_link"/>
+        <child link="${tf_prefix}/zed_camera_link_optical"/>
     </joint>
 </robot>

Commit message: editing transform prefixes

File: robot/description/urdf/caffeine.gazebo.xacro (robot description, xacro)
@@ -71,5 +71,5 @@
     <!-- TODO: double check these numbers -->
     <!-- Gazebo multicamera plugin -->
-    <gazebo reference="camera_link">
+    <gazebo reference="${tf_prefix}/camera_link">
         <sensor type="multicamera" name="stereo_camera">
             <update_rate>30.0</update_rate>

File: robot/description/urdf/stand_link.urdf.xacro (robot description, xacro)
@@ -29,5 +29,5 @@
     </link>
     <joint name="${tf_prefix}/zed_camera_joint" type="fixed">
-        <origin xyz="${stand_length/2} 0 ${stand_height + ZED_camera_height}" rpy="0 0 0"/>
+        <origin xyz="${stand_length/2} 0 ${stand_height + ZED_camera_height - 1.42}" rpy="0 0 0"/>
         <parent link="${tf_prefix}/stand_link"/>
         <child link="${tf_prefix}/zed_camera_link"/>

Commit message: Caff 4 - simulate GPS #33
Co-authored-by: Erick Mejia Uzeda <erickmu1@hotmail.com>

File: robot/description/urdf/caffeine.gazebo.xacro (robot description, xacro)
@@ -69,3 +69,23 @@
         </sensor>
     </gazebo>
+    <!-- GPS -->
+    <gazebo>
+        <plugin name="gps_controller" filename="libhector_gazebo_ros_gps.so">
+            <robotNamespace>${robotNamespace}</robotNamespace>
+            <updateRate>5.0</updateRate>  <!-- 5 Hz -->
+            <bodyName>${tf_prefix}/gps_link</bodyName>
+            <frameId>${tf_prefix}/gps_link</frameId>
+            <topicName>gps/fix</topicName>
+            <velocityTopicName>gps/fix_velocity</velocityTopicName>
+            <!-- Set reference GPS coordinates to UofT -->
+            <referenceLatitude>43.6570</referenceLatitude>
+            <referenceLongitude>-79.3903</referenceLongitude>
+            <referenceAltitude>76</referenceAltitude>
+            <!-- Model GPS behaviour -->
+            <service>1</service> <!-- SERVICE_GPS = 1 -->
+            <drift>1.5 1.5 1.5</drift> <!-- m -->
+            <velocityDrift>0.05 0.05 0.05</velocityDrift> <!-- m/s-->
+            <!-- TODO: add Gaussian noise based off Garmin GPS -->
+        </plugin>
+    </gazebo>
 </robot>

File: robot/description/urdf/constants.xacro (robot description, xacro)
@@ -65,3 +65,8 @@
     <xacro:property name="laser_x_dist" value="${base_length/2 - 2*laser_length}"/>
     <xacro:property name="laser_z_dist" value="${laser_height/2}"/>
+    <!-- Garmin GPS -->
+    <!-- NOTE: approx. as a cylinder, Garmin itself is similar to a hockey puck -->
+    <xacro:property name="gps_diam" value="0.061"/>
+    <xacro:property name="gps_length" value="0.0195"/>
+    <xacro:property name="gps_mass" value="0.165"/>
 </robot>

File: robot/description/urdf/inertias.xacro (robot description, xacro)
@@ -32,10 +32,18 @@
         />
     </xacro:macro>
-    <!-- Lidar -->
+    <!-- Box Inertia -->
     <xacro:macro name="box_inertia" params="mass length width height">
         <inertia
-            ixx="${mass * (height*height + length*length)/12.0}" ixy="0.0000" ixz="0.0000"
-            iyx = "0.0000" iyy="${mass * (width*width + length*length)/12.0}" iyz="0.0000"
-            izx="0.0000" izy="0.0000" izz="${mass * (width*width + height*height)/12.0}"
+            ixx="${mass * (height*height + length*length)/12.0}" ixy="0.0" ixz="0.0"
+            iyx = "0.0" iyy="${mass * (width*width + length*length)/12.0}" iyz="0.0"
+            izx="0.0" izy="0.0" izz="${mass * (width*width + height*height)/12.0}"
+        />
+    </xacro:macro>
+    <!-- Cynlinder Inertia -->
+    <xacro:macro name="cylinder_inertia" params="mass length radius">
+        <inertia
+            ixx="${mass * (3*radius*radius + length*length)/12.0}" ixy="0.0" ixz="0.0"
+            iyx="0.0" iyy="${mass * (3*radius*radius + length*length)/12.0}" iyz="0.0"
+            izx="0.0" izy="0.0" izz="${0.5*mass*radius*radius}"
         />
     </xacro:macro>

File: robot/description/urdf/stand_link.urdf.xacro (robot description, xacro)
@@ -8,3 +8,28 @@
     <link name="${tf_prefix}/stand_link">
     </link>
+    <!-- GPS -->
+    <link name="${tf_prefix}/gps_link">
+        <inertial>
+            <mass value="${gps_mass}"/>
+            <xacro:cylinder_inertia mass="${gps_mass}" length="${gps_length}" radius="${gps_diam / 2.0}"/>
+        </inertial>
+        <visual>
+            <origin xyz="0 0 0" rpy="0 0 0"/>
+            <geometry>
+                <cylinder length="${gps_length}" radius="${gps_diam / 2.0}"/>
+            </geometry>
+        </visual>
+        <collision>
+            <origin xyz="0 0 0" rpy="0 0 0"/>
+            <geometry>
+                <cylinder length="${gps_length}" radius="${gps_diam / 2.0}"/>
+            </geometry>
+        </collision>
+    </link>
+    <!-- GPS: attach gps_link to base_link -->
+    <joint name="${tf_prefix}/gps_joint" type="fixed">
+        <parent link="${tf_prefix}/stand_link"/>
+        <child link="${tf_prefix}/gps_link"/>
+        <origin xyz="0 0 0" rpy="0 0 0"/>
+    </joint>
 </robot>

Commit message: Added IMU link and plugin

File: robot/description/urdf/caffeine.gazebo.xacro (robot description, xacro)
@@ -89,3 +89,24 @@
         </plugin>
     </gazebo>
+    <!-- IMU -->
+    <gazebo reference="${tf_prefix}/imu_link">
+        <material>Gazebo/Black</material>
+        <gravity>true</gravity>
+        <sensor name="imu_sensor" type="imu">
+            <always_on>true</always_on>
+            <update_rate>128.0</update_rate>
+            <topic>__default_topic__</topic>
+            <plugin filename="libgazebo_ros_imu_sensor.so" name="imu_plugin">
+                <topicName>${robotNamespace}/imu/data</topicName>
+                <bodyName>${tf_prefix}/imu_link</bodyName>
+                <frameName>${tf_prefix}/imu_link</frameName>
+                <updateRateHZ>128.0</updateRateHZ>
+                <gaussianNoise>0.0</gaussianNoise>
+                <xyzOffset>0 0 0</xyzOffset>
+                <rpyOffset>0 0 0</rpyOffset>
+                <initialOrientationAsReference>false</initialOrientationAsReference>
+            </plugin>
+            <pose>0 0 0 0 0 0</pose>
+        </sensor>
+    </gazebo>
 </robot>

File: robot/description/urdf/caffeine.urdf.xacro (robot description, xacro)
@@ -11,5 +11,5 @@
         <parent link="${tf_prefix}/base_link"/>
         <child link="${tf_prefix}/chassis_link"/>
-        <origin rpy="0 0 0" xyz="0 0 ${chassis_to_base_link_dist}"/>
+        <origin xyz="0 0 ${chassis_to_base_link_dist}" rpy="0 0 0"/>
     </joint>
     <!-- stand_link: origin for anything on the stand; located in the middle, on the top of the stand plate -->
@@ -18,5 +18,5 @@
         <parent link="${tf_prefix}/chassis_link"/>
         <child link="${tf_prefix}/stand_link"/>
-        <origin rpy="0 0 0" xyz="0 0 ${chassis_to_stand_link_dist}"/>
+        <origin xyz="0 0 ${chassis_to_stand_link_dist}" rpy="0 0 0" />
     </joint>
     <!-- wheels: associated to wheels that can be moved by a motor -->

File: robot/description/urdf/constants.xacro (robot description, xacro)
@@ -10,5 +10,5 @@
     <!-- Chassis -->
     <xacro:property name="chassis_to_base_link_dist" value="0.501747"/>
-    <xacro:property name="chassis_to_stand_link_dist" value="0.713459"/>
+    <xacro:property name="chassis_to_stand_link_dist" value="0.698253"/>
     <xacro:property name="chassis_link_mass" value="33.9"/>
     <!-- Casters -->
@@ -70,3 +70,8 @@
     <xacro:property name="gps_length" value="0.0195"/>
     <xacro:property name="gps_mass" value="0.165"/>
+    <!-- Phidget IMU -->
+   <xacro:property name="phidget_length" value="0.04"/>
+   <xacro:property name="phidget_width" value="0.0375"/>
+   <xacro:property name="phidget_height" value="0.01"/>
+   <xacro:property name="phidget_mass" value="0.04"/>
 </robot>

File: robot/description/urdf/stand_link.urdf.xacro (robot description, xacro)
@@ -27,8 +27,33 @@
         </collision>
     </link>
-    <!-- GPS: attach gps_link to base_link -->
+    <!-- GPS: attach gps_link to stand_link -->
     <joint name="${tf_prefix}/gps_joint" type="fixed">
         <parent link="${tf_prefix}/stand_link"/>
         <child link="${tf_prefix}/gps_link"/>
+        <origin xyz="0 0 ${(gps_length + phidget_height) / 2.0}" rpy="0 0 0"/>
+    </joint>
+    <!-- IMU -->
+    <link name="${tf_prefix}/imu_link">
+        <inertial>
+            <mass value="${phidget_mass}"/>
+            <xacro:box_inertia mass="${phidget_mass}" length="${phidget_length}" width="${phidget_width}" height="${phidget_height}"/>
+        </inertial>
+        <visual>
+            <origin xyz="0 0 0" rpy="0 0 0"/>
+            <geometry>
+            <box size="${phidget_length} ${phidget_width} ${phidget_height}"/>
+            </geometry>
+        </visual>
+        <collision>
+            <origin xyz="0 0 0" rpy="0 0 0"/>
+            <geometry>
+            <box size="${phidget_length} ${phidget_width} ${phidget_height}"/>
+            </geometry>
+        </collision>
+    </link>
+    <!-- IMU: attach imu_link to stand_link -->
+    <joint name="${tf_prefix}/base_link_to_imu_link" type="fixed">
+        <parent link="${tf_prefix}/stand_link"/>
+        <child link="${tf_prefix}/imu_link"/>
         <origin xyz="0 0 0" rpy="0 0 0"/>
     </joint>

Commit message: visual odometry complete

File: robot/description/urdf/caffeine.gazebo.xacro (robot description, xacro)
@@ -120,20 +120,20 @@
             </camera>
             <plugin name="stereo_camera_controller" filename="libgazebo_ros_multicamera.so">
-            <cameraName>zed/zed_node</cameraName>
-            <alwaysOn>true</alwaysOn>
-            <updateRate>0</updateRate>
-            <cameraName></cameraName>
-            <imageTopicName>image_raw</imageTopicName>
-            <cameraInfoTopicName>camera_info</cameraInfoTopicName>
-            <depthImageTopicName>depth/image_raw</depthImageTopicName>
-            <depthImageInfoTopicName>depth/camera_info</depthImageInfoTopicName>
-            <pointCloudTopicName>depth/points</pointCloudTopicName>
-            <frameName>zed_camera_link_optical</frameName>
-            <hackBaseline>${ZED_camera_length}</hackBaseline>
-            <distortionK1>0.0</distortionK1>
-            <distortionK2>0.0</distortionK2>
-            <distortionK3>0.0</distortionK3>
-            <distortionT1>0.0</distortionT1>
-            <distortionT2>0.0</distortionT2>
+                <cameraName>zed/zed_node</cameraName>
+                <alwaysOn>true</alwaysOn>
+                <updateRate>0</updateRate>
+                <cameraName></cameraName>
+                <imageTopicName>image_raw</imageTopicName>
+                <cameraInfoTopicName>camera_info</cameraInfoTopicName>
+                <depthImageTopicName>depth/image_raw</depthImageTopicName>
+                <depthImageInfoTopicName>depth/camera_info</depthImageInfoTopicName>
+                <pointCloudTopicName>depth/points</pointCloudTopicName>
+                <frameName>${tf_prefix}/zed_camera_link_optical</frameName>
+                <hackBaseline>${ZED_camera_length}</hackBaseline>
+                <distortionK1>0.0</distortionK1>
+                <distortionK2>0.0</distortionK2>
+                <distortionK3>0.0</distortionK3>
+                <distortionT1>0.0</distortionT1>
+                <distortionT2>0.0</distortionT2>
             </plugin>
         </sensor>

File: robot/description/urdf/stand_link.urdf.xacro (robot description, xacro)
@@ -29,4 +29,5 @@
     </link>
     <joint name="${tf_prefix}/zed_camera_joint" type="fixed">
+        <!-- magic number to be fixed: 1.42 -->
         <origin xyz="${stand_length/2} 0 ${stand_height + ZED_camera_height - 1.42}" rpy="0 0 0"/>
         <parent link="${tf_prefix}/stand_link"/>
@@ -69,5 +70,5 @@
         </inertial>
     </link>
-    <joint name="${tf_prefix}/camera_link_joint" type="fixed">
+    <joint name="${tf_prefix}/zed_camera_link_joint" type="fixed">
         <origin xyz="${ZED_camera_length/2.0} 0 0" rpy="0 0 0"/>
         <parent link="${tf_prefix}/zed_camera_link"/>
@@ -75,6 +76,5 @@
     </joint>
     <!-- Generate an optical frame http://www.ros.org/reps/rep-0103.html#suffix-frames so that ros and opencv can operate on the camera frame correctly -->
-    <link name="${tf_prefix}/zed_camera_link_optical">
-    </link>
+    <link name="${tf_prefix}/zed_camera_link_optical"/>
     <joint name="${tf_prefix}/zed_camera_link_optical_joint" type="fixed">
         <!-- Transform b/w standard and optical frame -->

Commit message: Moved defined values for GPS and IMU into constants.xacro

File: robot/description/urdf/caffeine.gazebo.xacro (robot description, xacro)
@@ -73,17 +73,14 @@
         <plugin name="gps_controller" filename="libhector_gazebo_ros_gps.so">
             <robotNamespace>${robotNamespace}</robotNamespace>
-            <updateRate>5.0</updateRate>  <!-- 5 Hz -->
-            <bodyName>${tf_prefix}/gps_link</bodyName>
-            <frameId>${tf_prefix}/gps_link</frameId>
-            <topicName>gps/fix</topicName>
-            <velocityTopicName>gps/fix_velocity</velocityTopicName>
-            <!-- Set reference GPS coordinates to UofT -->
-            <referenceLatitude>43.6570</referenceLatitude>
-            <referenceLongitude>-79.3903</referenceLongitude>
-            <referenceAltitude>76</referenceAltitude>
-            <!-- Model GPS behaviour -->
-            <service>1</service> <!-- SERVICE_GPS = 1 -->
-            <drift>1.5 1.5 1.5</drift> <!-- m -->
-            <velocityDrift>0.05 0.05 0.05</velocityDrift> <!-- m/s-->
+            <updateRate>${gps_update_rate}</updateRate>
+            <bodyName>${tf_prefix}/${gps_frame}</bodyName>
+            <frameId>${tf_prefix}/${gps_frame}</frameId>
+            <topicName>${gps_topic}</topicName>
+            <velocityTopicName>${gps_vel_topic}</velocityTopicName>
+            <referenceLatitude>${ref_lat}</referenceLatitude>
+            <referenceLongitude>${ref_lon}</referenceLongitude>
+            <referenceAltitude>${ref_alt}</referenceAltitude>
+            <drift>${gps_drift}</drift> <!-- m -->
+            <velocityDrift>${gps_vel_drift}</velocityDrift> <!-- m/s-->
             <!-- TODO: add Gaussian noise based off Garmin GPS -->
         </plugin>
@@ -95,13 +92,13 @@
         <sensor name="imu_sensor" type="imu">
             <always_on>true</always_on>
-            <update_rate>128.0</update_rate>
+            <update_rate>${imu_update_rate}</update_rate>
             <topic>__default_topic__</topic>
-            <!-- TODO: set Drift based off Phidget IMU -->
+            <!-- TODO: add Drift based on Phidget IMU -->
             <plugin filename="libgazebo_ros_imu_sensor.so" name="imu_plugin">
-                <topicName>${robotNamespace}/imu/data</topicName>
-                <bodyName>${tf_prefix}/imu_link</bodyName>
-                <frameName>${tf_prefix}/imu_link</frameName>
-                <updateRateHZ>128.0</updateRateHZ>
-                <gaussianNoise>0.0</gaussianNoise>  <!-- TODO: set Gaussian noise based off Phidget IMU -->
+                <topicName>${robotNamespace}/${imu_topic}</topicName>
+                <bodyName>${tf_prefix}/${imu_frame}</bodyName>
+                <frameName>${tf_prefix}/${imu_frame}</frameName>
+                <updateRateHZ>${imu_update_rate}</updateRateHZ>
+                <gaussianNoise>0.0</gaussianNoise>  <!-- TODO: set Gaussian noise based on Phidget IMU -->
                 <xyzOffset>0 0 0</xyzOffset>
                 <rpyOffset>0 0 0</rpyOffset>

File: robot/description/urdf/constants.xacro (robot description, xacro)
@@ -70,4 +70,14 @@
     <xacro:property name="gps_length" value="0.0195"/>
     <xacro:property name="gps_mass" value="0.165"/>
+    <xacro:property name="gps_frame" value="gps_link"/>
+    <xacro:property name="gps_topic" value="gps/fix"/>
+    <xacro:property name="gps_vel_topic" value="gps/fix_velocity"/>
+    <xacro:property name="gps_update_rate" value="5.0"/>
+    <!-- NOTE: GPS coordinates for UofT St. George Campus -->
+    <xacro:property name="ref_lat" value="43.6570"/>
+    <xacro:property name="ref_lon" value="-79.3903"/>
+    <xacro:property name="ref_alt" value="76.0000"/>
+    <xacro:property name="gps_drift" value="1.5 1.5 1.5"/>
+    <xacro:property name="gps_vel_drift" value="0.05 0.05 0.05"/>
     <!-- Phidget IMU -->
    <xacro:property name="phidget_length" value="0.04"/>
@@ -75,3 +85,6 @@
    <xacro:property name="phidget_height" value="0.01"/>
    <xacro:property name="phidget_mass" value="0.04"/>
+   <xacro:property name="imu_frame" value="imu_link"/>
+   <xacro:property name="imu_topic" value="imu/data"/>
+   <xacro:property name="imu_update_rate" value="128.0"/>
 </robot>
