Commit message: Caff 2 - Simulate IMU (#35)
* Added IMU link and plugin

* Added TODO to simulate IMU noise and drift (not necessary atm)

* Moved defined values for GPS and IMU into constants.xacro

File: robot/description/urdf/caffeine.gazebo.xacro (robot description, xacro)
@@ -73,19 +73,38 @@
         <plugin name="gps_controller" filename="libhector_gazebo_ros_gps.so">
             <robotNamespace>${robotNamespace}</robotNamespace>
-            <updateRate>5.0</updateRate>  <!-- 5 Hz -->
-            <bodyName>${tf_prefix}/gps_link</bodyName>
-            <frameId>${tf_prefix}/gps_link</frameId>
-            <topicName>gps/fix</topicName>
-            <velocityTopicName>gps/fix_velocity</velocityTopicName>
-            <!-- Set reference GPS coordinates to UofT -->
-            <referenceLatitude>43.6570</referenceLatitude>
-            <referenceLongitude>-79.3903</referenceLongitude>
-            <referenceAltitude>76</referenceAltitude>
-            <!-- Model GPS behaviour -->
-            <service>1</service> <!-- SERVICE_GPS = 1 -->
-            <drift>1.5 1.5 1.5</drift> <!-- m -->
-            <velocityDrift>0.05 0.05 0.05</velocityDrift> <!-- m/s-->
+            <updateRate>${gps_update_rate}</updateRate>
+            <bodyName>${tf_prefix}/${gps_frame}</bodyName>
+            <frameId>${tf_prefix}/${gps_frame}</frameId>
+            <topicName>${gps_topic}</topicName>
+            <velocityTopicName>${gps_vel_topic}</velocityTopicName>
+            <referenceLatitude>${ref_lat}</referenceLatitude>
+            <referenceLongitude>${ref_lon}</referenceLongitude>
+            <referenceAltitude>${ref_alt}</referenceAltitude>
+            <drift>${gps_drift}</drift> <!-- m -->
+            <velocityDrift>${gps_vel_drift}</velocityDrift> <!-- m/s-->
             <!-- TODO: add Gaussian noise based off Garmin GPS -->
         </plugin>
     </gazebo>
+    <!-- IMU -->
+    <gazebo reference="${tf_prefix}/imu_link">
+        <material>Gazebo/Black</material>
+        <gravity>true</gravity>
+        <sensor name="imu_sensor" type="imu">
+            <always_on>true</always_on>
+            <update_rate>${imu_update_rate}</update_rate>
+            <topic>__default_topic__</topic>
+            <!-- TODO: add Drift based on Phidget IMU -->
+            <plugin filename="libgazebo_ros_imu_sensor.so" name="imu_plugin">
+                <topicName>${robotNamespace}/${imu_topic}</topicName>
+                <bodyName>${tf_prefix}/${imu_frame}</bodyName>
+                <frameName>${tf_prefix}/${imu_frame}</frameName>
+                <updateRateHZ>${imu_update_rate}</updateRateHZ>
+                <gaussianNoise>0.0</gaussianNoise>  <!-- TODO: set Gaussian noise based on Phidget IMU -->
+                <xyzOffset>0 0 0</xyzOffset>
+                <rpyOffset>0 0 0</rpyOffset>
+                <initialOrientationAsReference>false</initialOrientationAsReference>
+            </plugin>
+            <pose>0 0 0 0 0 0</pose>
+        </sensor>
+    </gazebo>
 </robot>

File: robot/description/urdf/constants.xacro (robot description, xacro)
@@ -10,5 +10,5 @@
     <!-- Chassis -->
     <xacro:property name="chassis_to_base_link_dist" value="0.501747"/>
-    <xacro:property name="chassis_to_stand_link_dist" value="0.713459"/>
+    <xacro:property name="chassis_to_stand_link_dist" value="0.698253"/>
     <xacro:property name="chassis_link_mass" value="33.9"/>
     <!-- Casters -->
@@ -70,3 +70,21 @@
     <xacro:property name="gps_length" value="0.0195"/>
     <xacro:property name="gps_mass" value="0.165"/>
+    <xacro:property name="gps_frame" value="gps_link"/>
+    <xacro:property name="gps_topic" value="gps/fix"/>
+    <xacro:property name="gps_vel_topic" value="gps/fix_velocity"/>
+    <xacro:property name="gps_update_rate" value="5.0"/>
+    <!-- NOTE: GPS coordinates for UofT St. George Campus -->
+    <xacro:property name="ref_lat" value="43.6570"/>
+    <xacro:property name="ref_lon" value="-79.3903"/>
+    <xacro:property name="ref_alt" value="76.0000"/>
+    <xacro:property name="gps_drift" value="1.5 1.5 1.5"/>
+    <xacro:property name="gps_vel_drift" value="0.05 0.05 0.05"/>
+    <!-- Phidget IMU -->
+   <xacro:property name="phidget_length" value="0.04"/>
+   <xacro:property name="phidget_width" value="0.0375"/>
+   <xacro:property name="phidget_height" value="0.01"/>
+   <xacro:property name="phidget_mass" value="0.04"/>
+   <xacro:property name="imu_frame" value="imu_link"/>
+   <xacro:property name="imu_topic" value="imu/data"/>
+   <xacro:property name="imu_update_rate" value="128.0"/>
 </robot>

Commit message: resolving pull req comments

File: robot/description/urdf/caffeine.gazebo.xacro (robot description, xacro)
@@ -89,15 +89,14 @@
         </plugin>
     </gazebo>
-    <!-- TODO: double check these numbers -->
     <!-- Gazebo multicamera plugin -->
     <gazebo reference="${tf_prefix}/camera_link">
         <sensor type="multicamera" name="stereo_camera">
-            <update_rate>30.0</update_rate>
+            <update_rate>${ZED_image_refresh}</update_rate>
             <camera name="left">
-            <horizontal_fov>1.571</horizontal_fov>
+            <horizontal_fov>${ZED_image_horizontal_fov} * (3.14/180)</horizontal_fov>
             <image>
-                <width>1280</width>
-                <height>720</height>
-                <format>R8G8B8</format>
+                <width>${ZED_image_width}</width>
+                <height>${ZED_image_height}</height>
+                <format>${ZED_image_format}</format>
             </image>
             <clip>
@@ -108,9 +107,9 @@
             <camera name="right">
             <pose>0 ${-ZED_camera_length} 0 0 0 0</pose>
-            <horizontal_fov>1.571</horizontal_fov>
+            <horizontal_fov>${ZED_image_horizontal_fov} * (3.14/180)</horizontal_fov>
             <image>
-                <width>1280</width>
-                <height>720</height>
-                <format>R8G8B8</format>
+                <width>${ZED_image_width}</width>
+                <height>${ZED_image_height}</height>
+                <format>${ZED_image_format}</format>
             </image>
             <clip>
@@ -131,4 +130,5 @@
                 <frameName>${tf_prefix}/zed_camera_link_optical</frameName>
                 <hackBaseline>${ZED_camera_length}</hackBaseline>
+                <!-- TODO: Get distortion parameters from real camera -->
                 <distortionK1>0.0</distortionK1>
                 <distortionK2>0.0</distortionK2>

File: robot/description/urdf/constants.xacro (robot description, xacro)
@@ -12,4 +12,9 @@
     <xacro:property name="chassis_to_stand_link_dist" value="0.713459"/>
     <xacro:property name="chassis_link_mass" value="33.9"/>
+    <!-- Stand -->
+    <xacro:property name="stand_length" value="0.412"/>
+    <xacro:property name="stand_width" value="0.254"/>
+    <xacro:property name="stand_height" value="1.324"/>
+    <xacro:property name="stand_mass" value="1.0"/>
     <!-- Casters -->
     <xacro:property name="caster_link_mass" value="0.5"/>
@@ -76,8 +81,9 @@
     <xacro:property name="ZED_camera_width" value="0.03"/>
     <xacro:property name="ZED_camera_height" value="0.033"/>
-    <!-- Stand -->
-    <xacro:property name="stand_length" value="0.412"/>
-    <xacro:property name="stand_width" value="0.254"/>
-    <xacro:property name="stand_height" value="1.324"/>
-    <xacro:property name="stand_mass" value="1.0"/>
+    <!-- ZED image height/width corresponds to image size for 60Hz refresh-->
+    <xacro:property name="ZED_image_refresh" value="60"/>
+    <xacro:property name="ZED_image_width" value="3840"/>
+    <xacro:property name="ZED_image_height" value="1080"/>
+    <xacro:property name="ZED_image_format" value="R8G8B8"/>
+    <xacro:property name="ZED_image_horizontal_fov" value="90"/>
 </robot>

File: robot/description/urdf/inertias.xacro (robot description, xacro)
@@ -48,14 +48,3 @@
         />
     </xacro:macro>
-    <!-- Camera -->
-    <xacro:macro name="box_inertia" params="mass length width height">
-        <inertia
-            ixx="${mass * (height*height + length*length)/12.0}"
-                        ixy="0.0"
-            ixz="0.0"
-                        iyy="${mass * (width*width + length*length)/12.0}"
-                        iyz="0.0"
-            izz="${mass * (width*width + height*height)/12.0}"
-        />
-    </xacro:macro>
 </robot>

File: robot/description/urdf/stand_link.urdf.xacro (robot description, xacro)
@@ -6,11 +6,9 @@
     <!-- Stand link; this is a dummy link that is used to make camera placement and other sensors on the stand more convenient -->
     <!-- Stand link definition. Note: purposely left blank -->
-    <link name="${tf_prefix}/stand_link">
-    </link>
+    <link name="${tf_prefix}/stand_link"/>
     <!-- ZED Camera -->
     <link name="${tf_prefix}/zed_camera_link">
         <visual>
             <origin xyz="0 0 0" rpy="0 0 0"/>
-            <!-- TODO: should be using the mesh but couldn't get it to work -->
             <geometry>
             <box size="${ZED_camera_width} ${ZED_camera_length} ${ZED_camera_height}"/>

Commit message: resolved pr comments except missing topics

File: robot/description/urdf/caffeine.gazebo.xacro (robot description, xacro)
@@ -94,5 +94,5 @@
             <update_rate>${ZED_image_refresh}</update_rate>
             <camera name="left">
-            <horizontal_fov>${ZED_image_horizontal_fov} * (3.14/180)</horizontal_fov>
+            <horizontal_fov>${ZED_image_hfov * (3.14/180)}</horizontal_fov>
             <image>
                 <width>${ZED_image_width}</width>
@@ -107,5 +107,5 @@
             <camera name="right">
             <pose>0 ${-ZED_camera_length} 0 0 0 0</pose>
-            <horizontal_fov>${ZED_image_horizontal_fov} * (3.14/180)</horizontal_fov>
+            <horizontal_fov>${ZED_image_hfov * (3.14/180)}</horizontal_fov>
             <image>
                 <width>${ZED_image_width}</width>

File: robot/description/urdf/constants.xacro (robot description, xacro)
@@ -86,4 +86,4 @@
     <xacro:property name="ZED_image_height" value="1080"/>
     <xacro:property name="ZED_image_format" value="R8G8B8"/>
-    <xacro:property name="ZED_image_horizontal_fov" value="90"/>
+    <xacro:property name="ZED_image_hfov" value="90"/>
 </robot>

File: robot/description/urdf/inertias.xacro (robot description, xacro)
@@ -36,5 +36,5 @@
         <inertia
             ixx="${mass * (height*height + length*length)/12.0}" ixy="0.0" ixz="0.0"
-            iyx = "0.0" iyy="${mass * (width*width + length*length)/12.0}" iyz="0.0"
+            iyx="0.0" iyy="${mass * (width*width + length*length)/12.0}" iyz="0.0"
             izx="0.0" izy="0.0" izz="${mass * (width*width + height*height)/12.0}"
         />

File: robot/description/urdf/stand_link.urdf.xacro (robot description, xacro)
@@ -27,6 +27,5 @@
     </link>
     <joint name="${tf_prefix}/zed_camera_joint" type="fixed">
-        <!-- magic number to be fixed: 1.42 -->
-        <origin xyz="${stand_length/2} 0 ${stand_height + ZED_camera_height - 1.42}" rpy="0 0 0"/>
+        <origin xyz="${stand_length/2 - ZED_camera_width} 0 0" rpy="0 0 0"/>
         <parent link="${tf_prefix}/stand_link"/>
         <child link="${tf_prefix}/zed_camera_link"/>

Commit message: made ZED constants

File: robot/description/urdf/caffeine.gazebo.xacro (robot description, xacro)
@@ -116,14 +116,14 @@
             </camera>
             <plugin name="stereo_camera_controller" filename="libgazebo_ros_multicamera.so">
-                <cameraName>zed/zed_node</cameraName>
-                <alwaysOn>true</alwaysOn>
-                <updateRate>0</updateRate>
+                <cameraName>${ZED_name}</cameraName>
+                <alwaysOn>${ZED_always_on}</alwaysOn>
+                <updateRate>${ZED_update_rate}</updateRate>
                 <cameraName></cameraName>
-                <imageTopicName>image_raw_color</imageTopicName>
-                <cameraInfoTopicName>camera_info</cameraInfoTopicName>
-                <depthImageTopicName>depth/image_raw</depthImageTopicName>
-                <depthImageInfoTopicName>depth/camera_info</depthImageInfoTopicName>
-                <pointCloudTopicName>depth/points</pointCloudTopicName>
-                <frameName>${tf_prefix}/zed_camera_link_optical</frameName>
+                <imageTopicName>${ZED_image_topicName}</imageTopicName>
+                <cameraInfoTopicName>${ZED_image_info_topicName}</cameraInfoTopicName>
+                <depthImageTopicName>${ZED_depth_topicName}</depthImageTopicName>
+                <depthImageInfoTopicName>${ZED_depth_info_topicName}</depthImageInfoTopicName>
+                <pointCloudTopicName>${ZED_depth_points_topicName}</pointCloudTopicName>
+                <frameName>${tf_prefix}/${ZED_frameName}</frameName>
                 <hackBaseline>${ZED_camera_length}</hackBaseline>
                 <!-- TODO: Get distortion parameters from real camera -->

File: robot/description/urdf/constants.xacro (robot description, xacro)
@@ -80,4 +80,13 @@
     <xacro:property name="ZED_image_format" value="R8G8B8"/>
     <xacro:property name="ZED_image_hfov" value="90"/>
+    <xacro:property name="ZED_name" value="zed/zed_node"/>
+    <xacro:property name="ZED_always_on" value="true"/>
+    <xacro:property name="ZED_update_rate" value="0"/>
+    <xacro:property name="ZED_image_topicName" value="image_raw_color"/>
+    <xacro:property name="ZED_image_info_topicName" value="camera_info"/>
+    <xacro:property name="ZED_depth_topicName" value="depth/image_raw"/>
+    <xacro:property name="ZED_depth_info_topicName" value="depth/camera_info"/>
+    <xacro:property name="ZED_depth_points_topicName" value="depth/points"/>
+    <xacro:property name="ZED_frameName" value="zed_camera_link_optical"/>
     <!-- Garmin GPS -->
     <!-- NOTE: approx. as a cylinder, Garmin itself is similar to a hockey puck -->
