Commit message: Caff 5 - Emulate ZED Camera (#37)
* saving progress on getting igvc world working on new code base

* Added gazebo plugin, camera/optical links, and launch file for zed emulation with stereo_image_proc

* completed walls for outer ring

* Complete inner loop of walls

* completed all walls and make required world copies

* merged master into caff-7 branch

* updated caffeine_gazebo.launch and added color to ramps

* added ramp color to all worlds

* updated worlds' package README

* removed ramp spawn and plain world in caffeine_gazebo.launch

* updated readme

* updated caffeine_gazebo.launch default world, and generated world with no ramp/walls

* actually commiting changes from caffeine_gazebo.launch

* removing random empty line

* fixing merge conflicts

* fix readme conflict in worlds readme

* fixing merge conflicts in urdf files

* adding transform prefix to remaining links

* saving progress

* editing transform prefixes

* visual odometry complete

* vis odom works

* reset gui to false

* returned spawn location to start

* resolving pull req comments

* resolved pr comments except missing topics

* fixing zed camera height

* saving progress

* remapped depth,cloud,disparity topics

* renamed zed topics

* removed unnecessary remaps

* made ZED constants

Co-authored-by: Trudie Cheung <trudie.cheung@gmail.com>
Co-authored-by: michruan <Michael Ruan>

File: robot/description/urdf/caffeine.gazebo.xacro (robot description, xacro)
@@ -86,4 +86,54 @@
         </plugin>
     </gazebo>
+    <!-- Gazebo multicamera plugin -->
+    <gazebo reference="${tf_prefix}/camera_link">
+        <sensor type="multicamera" name="stereo_camera">
+            <update_rate>${ZED_image_refresh}</update_rate>
+            <camera name="left">
+            <horizontal_fov>${ZED_image_hfov * (3.14/180)}</horizontal_fov>
+            <image>
+                <width>${ZED_image_width}</width>
+                <height>${ZED_image_height}</height>
+                <format>${ZED_image_format}</format>
+            </image>
+            <clip>
+                <near>0.02</near>
+                <far>300</far>
+            </clip>
+            </camera>
+            <camera name="right">
+            <pose>0 ${-ZED_camera_length} 0 0 0 0</pose>
+            <horizontal_fov>${ZED_image_hfov * (3.14/180)}</horizontal_fov>
+            <image>
+                <width>${ZED_image_width}</width>
+                <height>${ZED_image_height}</height>
+                <format>${ZED_image_format}</format>
+            </image>
+            <clip>
+                <near>0.02</near>
+                <far>300</far>
+            </clip>
+            </camera>
+            <plugin name="stereo_camera_controller" filename="libgazebo_ros_multicamera.so">
+                <cameraName>${ZED_name}</cameraName>
+                <alwaysOn>${ZED_always_on}</alwaysOn>
+                <updateRate>${ZED_update_rate}</updateRate>
+                <cameraName></cameraName>
+                <imageTopicName>${ZED_image_topicName}</imageTopicName>
+                <cameraInfoTopicName>${ZED_image_info_topicName}</cameraInfoTopicName>
+                <depthImageTopicName>${ZED_depth_topicName}</depthImageTopicName>
+                <depthImageInfoTopicName>${ZED_depth_info_topicName}</depthImageInfoTopicName>
+                <pointCloudTopicName>${ZED_depth_points_topicName}</pointCloudTopicName>
+                <frameName>${tf_prefix}/${ZED_frameName}</frameName>
+                <hackBaseline>${ZED_camera_length}</hackBaseline>
+                <!-- TODO: Get distortion parameters from real camera -->
+                <distortionK1>0.0</distortionK1>
+                <distortionK2>0.0</distortionK2>
+                <distortionK3>0.0</distortionK3>
+                <distortionT1>0.0</distortionT1>
+                <distortionT2>0.0</distortionT2>
+            </plugin>
+        </sensor>
+    </gazebo>
     <!-- IMU -->
     <gazebo reference="${tf_prefix}/imu_link">

File: robot/description/urdf/constants.xacro (robot description, xacro)
@@ -12,4 +12,9 @@
     <xacro:property name="chassis_to_stand_link_dist" value="0.698253"/>
     <xacro:property name="chassis_link_mass" value="33.9"/>
+    <!-- Stand -->
+    <xacro:property name="stand_length" value="0.412"/>
+    <xacro:property name="stand_width" value="0.254"/>
+    <xacro:property name="stand_height" value="1.324"/>
+    <xacro:property name="stand_mass" value="1.0"/>
     <!-- Casters -->
     <xacro:property name="caster_link_mass" value="1.2"/>
@@ -63,4 +68,25 @@
     <xacro:property name="laser_x_dist" value="${base_length/2 - 2*laser_length}"/>
     <xacro:property name="laser_z_dist" value="${laser_height/2}"/>
+    <!-- ZED camera -->
+    <!-- NOTE: approx as a rectangular prism -->
+    <xacro:property name="ZED_camera_mass" value="0.1587573"/>
+    <xacro:property name="ZED_camera_length" value="0.175"/>
+    <xacro:property name="ZED_camera_width" value="0.03"/>
+    <xacro:property name="ZED_camera_height" value="0.033"/>
+    <!-- ZED image height/width corresponds to image size for 60Hz refresh-->
+    <xacro:property name="ZED_image_refresh" value="60"/>
+    <xacro:property name="ZED_image_width" value="3840"/>
+    <xacro:property name="ZED_image_height" value="1080"/>
+    <xacro:property name="ZED_image_format" value="R8G8B8"/>
+    <xacro:property name="ZED_image_hfov" value="90"/>
+    <xacro:property name="ZED_name" value="zed/zed_node"/>
+    <xacro:property name="ZED_always_on" value="true"/>
+    <xacro:property name="ZED_update_rate" value="0"/>
+    <xacro:property name="ZED_image_topicName" value="image_raw_color"/>
+    <xacro:property name="ZED_image_info_topicName" value="camera_info"/>
+    <xacro:property name="ZED_depth_topicName" value="depth/image_raw"/>
+    <xacro:property name="ZED_depth_info_topicName" value="depth/camera_info"/>
+    <xacro:property name="ZED_depth_points_topicName" value="depth/points"/>
+    <xacro:property name="ZED_frameName" value="zed_camera_link_optical"/>
     <!-- Garmin GPS -->
     <!-- NOTE: approx. as a cylinder, Garmin itself is similar to a hockey puck -->

File: robot/description/urdf/inertias.xacro (robot description, xacro)
@@ -21,5 +21,5 @@
         <inertia
             ixx="${mass * (height*height + length*length)/12.0}" ixy="0.0" ixz="0.0"
-            iyx = "0.0" iyy="${mass * (width*width + length*length)/12.0}" iyz="0.0"
+            iyx="0.0" iyy="${mass * (width*width + length*length)/12.0}" iyz="0.0"
             izx="0.0" izy="0.0" izz="${mass * (width*width + height*height)/12.0}"
         />

File: robot/description/urdf/stand_link.urdf.xacro (robot description, xacro)
@@ -6,6 +6,29 @@
     <!-- Stand link; this is a dummy link that is used to make camera placement and other sensors on the stand more convenient -->
     <!-- Stand link definition. Note: purposely left blank -->
-    <link name="${tf_prefix}/stand_link">
+    <link name="${tf_prefix}/stand_link"/>
+    <!-- ZED Camera -->
+    <link name="${tf_prefix}/zed_camera_link">
+        <visual>
+            <origin xyz="0 0 0" rpy="0 0 0"/>
+            <geometry>
+            <box size="${ZED_camera_width} ${ZED_camera_length} ${ZED_camera_height}"/>
+            </geometry>
+        </visual>
+        <collision>
+            <origin xyz="0 0 0" rpy="0 0 0"/>
+            <geometry>
+                <box size="${ZED_camera_width} ${ZED_camera_length} ${ZED_camera_height}"/>
+            </geometry>
+        </collision>
+        <inertial>
+            <xacro:box_inertia mass="${ZED_camera_mass}" length="${ZED_camera_length}" width="${ZED_camera_width}" height="${ZED_camera_height}"/>
+            <mass value="${ZED_camera_mass}"/>
+        </inertial>
     </link>
+    <joint name="${tf_prefix}/zed_camera_joint" type="fixed">
+        <origin xyz="${stand_length/2 - ZED_camera_width} 0 ${ZED_camera_height / 2.0}" rpy="0 0 0"/>
+        <parent link="${tf_prefix}/stand_link"/>
+        <child link="${tf_prefix}/zed_camera_link"/>
+    </joint>
     <!-- GPS -->
     <link name="${tf_prefix}/gps_link">
@@ -58,3 +81,27 @@
         <origin xyz="0 0 0" rpy="0 0 0"/>
     </joint>
+    <!-- ZED camera lenses -->
+    <!-- NOTE: I'm only defining one and not visually showing any-->
+    <!-- I only need one for purposes of using the plugin -->
+    <!-- TODO: check if it's fine to call the left lense camera_link (rtabmap doesn't specify whether it wants the lense frame or the camera frame itself) -->
+    <link name="${tf_prefix}/camera_link">
+        <!-- Inertial tag here to ensure that link does not phase through robot-->
+        <inertial>
+            <mass value="0.0001"/>
+            <inertia ixx="0.0001" ixy="0" ixz="0" iyy="0.0001" iyz="0" izz="0.00001"/>
+        </inertial>
+    </link>
+    <joint name="${tf_prefix}/zed_camera_link_joint" type="fixed">
+        <origin xyz="${ZED_camera_length/2.0} 0 0" rpy="0 0 0"/>
+        <parent link="${tf_prefix}/zed_camera_link"/>
+        <child link="${tf_prefix}/camera_link"/>
+    </joint>
+    <!-- Generate an optical frame http://www.ros.org/reps/rep-0103.html#suffix-frames so that ros and opencv can operate on the camera frame correctly -->
+    <link name="${tf_prefix}/zed_camera_link_optical"/>
+    <joint name="${tf_prefix}/zed_camera_link_optical_joint" type="fixed">
+        <!-- Transform b/w standard and optical frame -->
+        <origin xyz="0 0 0" rpy="${-pi/2} 0 ${-pi/2}"/>
+        <parent link="${tf_prefix}/zed_camera_link"/>
+        <child link="${tf_prefix}/zed_camera_link_optical"/>
+    </joint>
 </robot>

Commit message: saving progress

File: robot/description/urdf/caffeine.gazebo.xacro (robot description, xacro)
@@ -91,5 +91,5 @@
             <update_rate>${ZED_image_refresh}</update_rate>
             <camera name="left">
-            <horizontal_fov>${ZED_image_hfov * (3.14/180)}</horizontal_fov>
+            <horizontal_fov>${ZED_image_hfov}</horizontal_fov>
             <image>
                 <width>${ZED_image_width}</width>
@@ -104,5 +104,5 @@
             <camera name="right">
             <pose>0 ${-ZED_camera_length} 0 0 0 0</pose>
-            <horizontal_fov>${ZED_image_hfov * (3.14/180)}</horizontal_fov>
+            <horizontal_fov>${ZED_image_hfov}</horizontal_fov>
             <image>
                 <width>${ZED_image_width}</width>
@@ -119,5 +119,4 @@
                 <alwaysOn>${ZED_always_on}</alwaysOn>
                 <updateRate>${ZED_update_rate}</updateRate>
-                <cameraName></cameraName>
                 <imageTopicName>${ZED_image_topicName}</imageTopicName>
                 <cameraInfoTopicName>${ZED_image_info_topicName}</cameraInfoTopicName>

File: robot/description/urdf/constants.xacro (robot description, xacro)
@@ -74,4 +74,5 @@
     <xacro:property name="ZED_camera_width" value="0.03"/>
     <xacro:property name="ZED_camera_height" value="0.033"/>
+    <xacro:property name="ZED_camera_pitch" value="${15 * pi/180}"/>
     <!-- ZED image height/width corresponds to image size for 60Hz refresh-->
     <xacro:property name="ZED_image_refresh" value="60"/>
@@ -79,5 +80,5 @@
     <xacro:property name="ZED_image_height" value="1080"/>
     <xacro:property name="ZED_image_format" value="R8G8B8"/>
-    <xacro:property name="ZED_image_hfov" value="90"/>
+    <xacro:property name="ZED_image_hfov" value="${90 * pi/180}"/>
     <xacro:property name="ZED_name" value="zed/zed_node"/>
     <xacro:property name="ZED_always_on" value="true"/>

File: robot/description/urdf/stand_link.urdf.xacro (robot description, xacro)
@@ -27,5 +27,5 @@
     </link>
     <joint name="${tf_prefix}/zed_camera_joint" type="fixed">
-        <origin xyz="${stand_length/2 - ZED_camera_width} 0 ${ZED_camera_height / 2.0}" rpy="0 0 0"/>
+        <origin xyz="${stand_length/2 - ZED_camera_width} 0 ${ZED_camera_height / 2.0}" rpy="0 ${ZED_camera_pitch} 0"/>
         <parent link="${tf_prefix}/stand_link"/>
         <child link="${tf_prefix}/zed_camera_link"/>
