Commit message: added Lidar plugin

File: robot/description/urdf/constants.xacro (robot description, xacro)
@@ -37,5 +37,5 @@
     <xacro:property name="hokuyo_height" value="0.07"/>
     <xacro:property name="hokuyo_mass" value="0.16"/>
-    <xacro:property name="laser_x_dist" value="0.3"/>
+    <xacro:property name="laser_x_dist" value="0.65"/>
     <xacro:property name="laser_z_dist" value="0.0"/>
 </robot>

Commit message: added constants from drive plugin

File: robot/description/urdf/constants.xacro (robot description, xacro)
@@ -14,9 +14,25 @@
     <!-- Wheels -->
     <xacro:property name="wheel_vertical_offset" value="-0.61759696"/>
+    <xacro:property name="wheel_left_joint" value="left_wheel_joint"/>
+    <xacro:property name="wheel_right_joint" value="right_wheel_joint"/>
     <xacro:property name="wheels_separation" value="0.875"/>
     <xacro:property name="wheel_diameter" value="0.25"/>
+    <xacro:property name="wheel_acceleration" value="1.0"/>
+    <xacro:property name="wheel_torque" value="20"/>
     <xacro:property name="wheel_mass" value="4.45"/>
     <!-- Gazebo Motor -->
+    <xacro:property name="diff_drive_robotNamespace" value="caffeine"/>
     <xacro:property name="diff_drive_update_rate" value="30.0"/>
+    <xacro:property name="diff_drive_commandTopic" value="cmd_vel"/>
+    <xacro:property name="diff_drive_odometryTopic" value="odom"/>
+    <xacro:property name="diff_drive_odometryFrame" value="odom"/>
+    <xacro:property name="diff_drive_robotBaseFrame" value="base_link"/>
+    <xacro:property name="diff_drive_odometrySource" value="encoder"/>
+    <xacro:property name="diff_drive_publishWheelTF" value="false"/>
+    <xacro:property name="diff_drive_publishOdomTF" value="true"/>
+    <xacro:property name="diff_drive_publishTf" value="true"/>
+    <xacro:property name="diff_drive_publishWheelJointState" value="true"/>
+    <xacro:property name="diff_drive_legacymode" value="false"/>
+    <xacro:property name="diff_drive_rosDebugLevel" value="na"/>
     <!-- Constants for hokuyo 2D LIDAR sensor -->
     <xacro:property name="laser_visualize" value="false"/>
@@ -34,8 +50,8 @@
     <xacro:property name="laser_topicName" value="scan"/>
     <xacro:property name="laser_frameName" value="base_laser"/>
-    <xacro:property name="hokuyo_length" value="0.05"/>
-    <xacro:property name="hokuyo_width" value="0.05"/>
-    <xacro:property name="hokuyo_height" value="0.07"/>
-    <xacro:property name="hokuyo_mass" value="0.16"/>
+    <xacro:property name="laser_length" value="0.05"/>
+    <xacro:property name="laser_width" value="0.05"/>
+    <xacro:property name="laser_height" value="0.07"/>
+    <xacro:property name="laser_mass" value="0.16"/>
     <xacro:property name="laser_x_dist" value="0.65"/>
     <xacro:property name="laser_z_dist" value="0.0"/>

Commit message: added robotNamespace constant

File: robot/description/urdf/constants.xacro (robot description, xacro)
@@ -1,4 +1,6 @@
 <?xml version="1.0"?>
 <robot name="caffeine_constants" xmlns:xacro="http://ros.org/wiki/xacro">
+    <!-- Caffeine -->
+    <xacro:property name="robotNamespace" value="caffeine"/>
     <!-- Chassis -->
     <xacro:property name="chassis_to_base_link_dist" value="0.501747"/>
@@ -24,5 +26,4 @@
     <!-- Gazebo Motor -->
     <!-- TODO: update parameters once they become known -->
-    <xacro:property name="diff_drive_robotNamespace" value="caffeine"/>
     <xacro:property name="diff_drive_update_rate" value="30.0"/>
     <xacro:property name="diff_drive_commandTopic" value="cmd_vel"/>

Commit message: fixed the positioning of laser

File: robot/description/urdf/constants.xacro (robot description, xacro)
@@ -57,5 +57,5 @@
     <xacro:property name="laser_height" value="0.07"/>
     <xacro:property name="laser_mass" value="0.16"/>
-    <xacro:property name="laser_x_dist" value="0.65"/>
-    <xacro:property name="laser_z_dist" value="0.0"/>
+    <xacro:property name="laser_x_dist" value="0.55"/>
+    <xacro:property name="laser_z_dist" value="${laser_height/2}"/>
 </robot>

Commit message: topic name under caffeine/scan

File: robot/description/urdf/constants.xacro (robot description, xacro)
@@ -51,5 +51,5 @@
     <xacro:property name="laser_noise_mean" value="0.0"/>
     <xacro:property name="laser_noise_stddev" value="0.1"/>
-    <xacro:property name="laser_topicName" value="scan"/>
+    <xacro:property name="laser_topicName" value="caffeine/scan"/>
     <xacro:property name="laser_frameName" value="base_laser"/>
     <xacro:property name="laser_length" value="0.05"/>

Commit message: fixed values acc to spec sheet/updated comments

File: robot/description/urdf/constants.xacro (robot description, xacro)
@@ -15,5 +15,5 @@
     <xacro:property name="caster_link_to_wheel_dist_z" value="-0.04361749"/>
     <!-- Wheels -->
-    <!-- TODO: update parameters once they become known -->
+    <!-- TODO: Update acceleration and torque parameters when known -->
     <xacro:property name="wheel_vertical_offset" value="-0.61759696"/>
     <xacro:property name="wheel_left_joint" value="left_wheel_joint"/>
@@ -25,5 +25,4 @@
     <xacro:property name="wheel_mass" value="4.45"/>
     <!-- Gazebo Motor -->
-    <!-- TODO: update parameters once they become known -->
     <xacro:property name="diff_drive_update_rate" value="30.0"/>
     <xacro:property name="diff_drive_commandTopic" value="cmd_vel"/>
@@ -38,17 +37,19 @@
     <xacro:property name="diff_drive_legacymode" value="false"/>
     <xacro:property name="diff_drive_rosDebugLevel" value="na"/>
-    <!-- Constants for hokuyo 2D LIDAR sensor -->
+    <!-- Hokuyo 2D LIDAR sensor -->
     <xacro:property name="laser_visualize" value="false"/>
-    <xacro:property name="laser_update_rate" value="30"/>
+    <xacro:property name="laser_update_rate" value="10"/>
     <xacro:property name="laser_horizontal_samples" value="1080"/>
     <xacro:property name="laser_horizontal_resolution" value="1"/>
-    <xacro:property name="laser_horizontal_min_angle" value="-2.356"/>
-    <xacro:property name="laser_horizontal_max_angle" value="2.356"/>
-    <xacro:property name="laser_range_min" value="0.1"/>
-    <xacro:property name="laser_range_max" value="5.6"/>
-    <xacro:property name="laser_range_resolution" value="0.01"/>
+    <xacro:property name="laser_field_of_view" value="240"/>
+    <xacro:property name="laser_horizontal_min_angle" value="$(-laser_field_of_view*pi/180)"/>
+    <xacro:property name="laser_horizontal_max_angle" value="$(laser_field_of_view*pi/180)"/>
+    <xacro:property name="laser_range_min" value="0.06"/>
+    <xacro:property name="laser_range_max" value="4.095"/>
+    <xacro:property name="laser_resolution_angle" value="0.36"/>
+    <xacro:property name="laser_range_resolution" value="$(laser_resolution_angle*pi/180)"/>
     <xacro:property name="laser_noise_type" value="gaussian"/>
     <xacro:property name="laser_noise_mean" value="0.0"/>
-    <xacro:property name="laser_noise_stddev" value="0.1"/>
+    <xacro:property name="laser_noise_stddev" value="0.01/3"/>
     <xacro:property name="laser_topicName" value="caffeine/scan"/>
     <xacro:property name="laser_frameName" value="base_laser"/>
@@ -57,5 +58,5 @@
     <xacro:property name="laser_height" value="0.07"/>
     <xacro:property name="laser_mass" value="0.16"/>
-    <xacro:property name="laser_x_dist" value="0.55"/>
+    <xacro:property name="laser_x_dist" value="${0.634-laser_length}"/>
     <xacro:property name="laser_z_dist" value="${laser_height/2}"/>
 </robot>

Commit message: Turning off LIDAR visualization in Gazebo

File: robot/description/urdf/constants.xacro (robot description, xacro)
@@ -43,5 +43,5 @@
     <xacro:property name="diff_drive_rosDebugLevel" value="na"/>
     <!-- Hokuyo 2D LIDAR sensor -->
-    <xacro:property name="laser_visualize" value="true"/>
+    <xacro:property name="laser_visualize" value="false"/>
     <xacro:property name="laser_update_rate" value="10"/>
     <xacro:property name="laser_horizontal_samples" value="1080"/>

Commit message: Updated caster ball radius to 0.0825

File: robot/description/urdf/constants.xacro (robot description, xacro)
@@ -16,5 +16,5 @@
     <xacro:property name="casters_separation" value="1.12"/>
     <xacro:property name="caster_vertical_offset" value="-0.59"/>
-    <xacro:property name="caster_link_radius" value="0.075"/>
+    <xacro:property name="caster_link_radius" value="0.0825"/>
     <!-- Wheels -->
     <!-- TODO: Update acceleration and torque parameters when known -->

Commit message: Removed GPS velocity drift and navsat uses zero altitude

File: robot/description/urdf/constants.xacro (robot description, xacro)
@@ -103,5 +103,5 @@
     <xacro:property name="ref_alt" value="76.0000"/>
     <xacro:property name="gps_drift" value="1.5 1.5 1.5"/>
-    <xacro:property name="gps_vel_drift" value="0.05 0.05 0.05"/>
+    <xacro:property name="gps_vel_drift" value="0.00 0.00 0.05"/>
     <!-- Phidget IMU -->
    <xacro:property name="phidget_length" value="0.04"/>

Commit message: Set all gps drift velocities to 0

File: robot/description/urdf/constants.xacro (robot description, xacro)
@@ -103,5 +103,5 @@
     <xacro:property name="ref_alt" value="76.0000"/>
     <xacro:property name="gps_drift" value="1.5 1.5 1.5"/>
-    <xacro:property name="gps_vel_drift" value="0.00 0.00 0.05"/>
+    <xacro:property name="gps_vel_drift" value="0.00 0.00 0.00"/>
     <!-- Phidget IMU -->
    <xacro:property name="phidget_length" value="0.04"/>

Commit message: Updated localization.yaml to include zed & modified odom frame to be published by robot localization instead of gazebo

File: robot/description/urdf/constants.xacro (robot description, xacro)
@@ -40,5 +40,5 @@
     <xacro:property name="diff_drive_odometrySource" value="encoder"/>
     <xacro:property name="diff_drive_publishWheelTF" value="false"/>
-    <xacro:property name="diff_drive_publishOdomTF" value="true"/>
+    <xacro:property name="diff_drive_publishOdomTF" value="false"/>
     <xacro:property name="diff_drive_publishTf" value="true"/>
     <xacro:property name="diff_drive_publishWheelJointState" value="true"/>

Commit message: Caff 9 - Add Navsat Transform Node (#42)
* Created odom package and added the navsat_transform_node. Currently GPS odom is subject to significant drift

* Removed GPS velocity drift and navsat uses zero altitude

* Set all gps drift velocities to 0

* Added odom.launch in caffeine_gazebo.launch

* Added ending newline to caffeine_navsat.yaml

* Removed comments from boilerplate code

File: robot/description/urdf/constants.xacro (robot description, xacro)
@@ -103,5 +103,5 @@
     <xacro:property name="ref_alt" value="76.0000"/>
     <xacro:property name="gps_drift" value="1.5 1.5 1.5"/>
-    <xacro:property name="gps_vel_drift" value="0.05 0.05 0.05"/>
+    <xacro:property name="gps_vel_drift" value="0.00 0.00 0.00"/>
     <!-- Phidget IMU -->
    <xacro:property name="phidget_length" value="0.04"/>

Commit message: Changed lidar update rate to 30 (temporarily) in constants.xacro and updated depth topic name in rtab.launch

File: robot/description/urdf/constants.xacro (robot description, xacro)
@@ -47,5 +47,5 @@
     <!-- Hokuyo 2D LIDAR sensor -->
     <xacro:property name="laser_visualize" value="false"/>
-    <xacro:property name="laser_update_rate" value="10"/>
+    <xacro:property name="laser_update_rate" value="30.0"/>
     <xacro:property name="laser_horizontal_samples" value="1080"/>
     <xacro:property name="laser_horizontal_resolution" value="1"/>

Commit message: Setting update LIDAR constant rate back to what it was

File: robot/description/urdf/constants.xacro (robot description, xacro)
@@ -47,5 +47,5 @@
     <!-- Hokuyo 2D LIDAR sensor -->
     <xacro:property name="laser_visualize" value="false"/>
-    <xacro:property name="laser_update_rate" value="30.0"/>
+    <xacro:property name="laser_update_rate" value="10"/>
     <xacro:property name="laser_horizontal_samples" value="1080"/>
     <xacro:property name="laser_horizontal_resolution" value="1"/>

Commit message: Updated camera pitch

File: robot/description/urdf/constants.xacro (robot description, xacro)
@@ -74,4 +74,5 @@
     <xacro:property name="ZED_camera_width" value="0.03"/>
     <xacro:property name="ZED_camera_height" value="0.033"/>
+    <xacro:property name="ZED_camera_pitch" value="${21.25 * pi/180}"/>
     <!-- ZED image height/width corresponds to image size for 60Hz refresh-->
     <xacro:property name="ZED_image_refresh" value="60"/>

Commit message: Updated pitch value and horizontal fov in constants and removed redunant camera name tag

File: robot/description/urdf/constants.xacro (robot description, xacro)
@@ -74,5 +74,5 @@
     <xacro:property name="ZED_camera_width" value="0.03"/>
     <xacro:property name="ZED_camera_height" value="0.033"/>
-    <xacro:property name="ZED_camera_pitch" value="${21.25 * pi/180}"/>
+    <xacro:property name="ZED_camera_pitch" value="${15 * pi/180}"/>
     <!-- ZED image height/width corresponds to image size for 60Hz refresh-->
     <xacro:property name="ZED_image_refresh" value="60"/>
@@ -80,5 +80,5 @@
     <xacro:property name="ZED_image_height" value="1080"/>
     <xacro:property name="ZED_image_format" value="R8G8B8"/>
-    <xacro:property name="ZED_image_hfov" value="90"/>
+    <xacro:property name="ZED_image_hfov" value="${90 * pi/180}"/>
     <xacro:property name="ZED_name" value="zed/zed_node"/>
     <xacro:property name="ZED_always_on" value="true"/>

Commit message: made black box

File: robot/description/urdf/constants.xacro (robot description, xacro)
@@ -21,7 +21,13 @@
     <xacro:property name="casters_separation" value="1.12"/>
     <xacro:property name="caster_vertical_offset" value="-0.619167561"/>
-    <xacro:property name="caster_wheel_mass" value="20.7"/> <!-- CHANGED -->
+    <xacro:property name="caster_wheel_mass" value="0.7"/>
     <xacro:property name="caster_link_to_wheel_dist_x" value="0.03621719"/>
     <xacro:property name="caster_link_to_wheel_dist_z" value="-0.04361749"/>
+    <!-- Battery -->
+    <xacro:property name="battery_width" value="0.05"/>
+    <xacro:property name="battery_length" value="0.1"/>
+    <xacro:property name="battery_height" value="0.05"/>
+    <xacro:property name="battery_mass" value="33"/>
+    <xacro:property name="battery_back_offset" value="0.17"/>
     <!-- Wheels -->
     <!-- TODO: Update acceleration and torque parameters when known -->

File: robot/description/urdf/stand_link.urdf.xacro (robot description, xacro)
@@ -7,4 +7,28 @@
     <!-- Stand link definition. Note: purposely left blank -->
     <link name="${tf_prefix}/stand_link"/>
+    <!-- Battery Link -->
+    <link name="${tf_prefix}/battery_link">
+        <visual>
+            <origin xyz="0 0 0" rpy="0 0 0"/>
+            <geometry>
+                <box size="${battery_width} ${battery_length} ${battery_height}"/>
+            </geometry>
+        </visual>
+        <collision>
+            <origin xyz="0 0 0" rpy="0 0 0"/>
+            <geometry>
+                <box size="${battery_width} ${battery_length} ${battery_height}"/>
+            </geometry>
+        </collision>
+        <inertial>
+            <xacro:box_inertia mass="${battery_mass}" length="${battery_length}" width="${battery_width}" height="${battery_height}"/>
+            <mass value="${battery_mass}"/>
+        </inertial>
+    </link>
+    <joint name="${tf_prefix}/battery_joint" type="fixed">
+        <origin xyz="${-1*(stand_length/2 + battery_width + battery_back_offset)} 0 ${wheel_diameter - (3*battery_height/2) - stand_height/2}" rpy="0 0 0"/>
+        <parent link="${tf_prefix}/chassis_link"/>
+        <child link="${tf_prefix}/battery_link"/>
+    </joint>
     <!-- ZED Camera -->
     <link name="${tf_prefix}/zed_camera_link">
@@ -12,5 +36,5 @@
             <origin xyz="0 0 0" rpy="0 0 0"/>
             <geometry>
-            <box size="${ZED_camera_width} ${ZED_camera_length} ${ZED_camera_height}"/>
+                <box size="${ZED_camera_width} ${ZED_camera_length} ${ZED_camera_height}"/>
             </geometry>
         </visual>

Commit message: played around with the values some more

File: robot/description/urdf/constants.xacro (robot description, xacro)
@@ -54,5 +54,5 @@
     <xacro:property name="diff_drive_rosDebugLevel" value="na"/>
     <!-- Hokuyo 2D LIDAR sensor -->
-    <xacro:property name="laser_visualize" value="false"/>
+    <xacro:property name="laser_visualize" value="true"/>
     <xacro:property name="laser_update_rate" value="10"/>
     <xacro:property name="laser_horizontal_samples" value="1080"/>

Commit message: comm

File: robot/description/urdf/constants.xacro (robot description, xacro)
@@ -18,5 +18,5 @@
     <xacro:property name="stand_mass" value="1.0"/>
     <!-- Casters -->
-    <xacro:property name="caster_link_mass" value="0.5"/>
+    <xacro:property name="caster_link_mass" value="1.2"/>
     <xacro:property name="casters_separation" value="1.12"/>
     <xacro:property name="caster_vertical_offset" value="-0.619167561"/>
