Commit message: Added casters and caster wheels

File: robot/description/urdf/casters.urdf.xacro (robot description, xacro)
@@ -1,6 +1,9 @@
 <?xml version="1.0"?>
 <robot name="caster_wheels" xmlns:xacro="http://ros.org/wiki/xacro">
-    <!-- TODO: populate this with caster wheels definitions and constants -->
-    <!-- For convenience, include the support definitions and constants for them here too -->
+    <!-- TODO: make sure the inertias associated with each caster and wheel is correct -->
+    <!-- Note: this file contains definitions for both the casters & the caster wheels -->
+    <!-- When included, only use front_caster_link and back_caster_link (joints for the wheels are defined in this file) -->
+    <!-- Constants related to casters -->
+    <!-- Note: mass can be used across both casters -->
     <xacro:property name="caster_link_mass" value="0.5"/>
     <xacro:macro name="front_caster_link_inertia">
@@ -18,4 +21,5 @@
         />
     </xacro:macro>
+    <!-- Front caster link definition -->
     <link name="front_caster_link">
         <visual>
@@ -36,4 +40,5 @@
         </inertial>
     </link>
+    <!-- Back caster link definition -->
     <link name="back_caster_link">
         <visual>
@@ -55,3 +60,75 @@
     </link>
     <!-- Wheel definitions and joints -->
+    <!-- Constants related to caster wheel definition -->
+    <xacro:property name="caster_wheel_mass" value="0.7"/>
+    <xacro:macro name="front_caster_wheel_inertia">
+        <inertia
+            ixx="0.29" ixy="0.00" ixz="-0.27"
+            iyx="0.00" iyy="0.54" iyz="0.00"
+            izx="-0.27" izy="0.00" izz="0.25"
+        />
+    </xacro:macro>
+    <xacro:macro name="back_caster_wheel_inertia">
+        <inertia
+            ixx="0.29" ixy="0.00" ixz="0.27"
+            iyx="0.00" iyy="0.54" iyz="0.00"
+            izx="0.27" izy="0.00" izz="0.25"
+        />
+    </xacro:macro>
+    <!-- Constants related to caster wheel joint definition -->
+    <xacro:property name="front_caster_link_to_front_caster_wheel_dist_x" value="0.03621719"/>
+    <xacro:property name="back_caster_link_to_back_caster_wheel_dist_x" value="-0.03621719"/>
+    <xacro:property name="caster_link_to_caster_wheel_dist_z" value="-0.04361749"/>
+    <!-- Front caster wheel definition -->
+    <link name="front_caster_wheel">
+        <visual>
+            <origin rpy="0 0 0" xyz="0 0 0"/>
+            <geometry>
+                <mesh filename="package://description/urdf/meshes/front_caster_wheel.dae"/>
+            </geometry>
+        </visual>
+        <collision>
+            <origin rpy="0 0 0" xyz="0 0 0"/>
+            <geometry>
+                <mesh filename="package://description/urdf/meshes/front_caster_wheel.dae"/>
+            </geometry>
+        </collision>
+        <inertial>
+            <mass value="${caster_wheel_mass}"/>
+            <xacro:front_caster_wheel_inertia/>
+        </inertial>
+    </link>
+    <!-- Front caster wheel joint -->
+    <joint name="front_caster_wheel_joint" type="continuous">
+        <axis xyz="0 1 0"/>
+        <parent link="front_caster_link"/>
+        <child link="front_caster_wheel"/>
+        <origin rpy="0 0 0" xyz="${front_caster_link_to_front_caster_wheel_dist_x} 0 ${caster_link_to_caster_wheel_dist_z}"/>
+    </joint>
+     <!-- Back caster wheel definition -->
+     <link name="back_caster_wheel">
+         <visual>
+             <origin rpy="0 0 0" xyz="0 0 0"/>
+             <geometry>
+                 <mesh filename="package://description/urdf/meshes/back_caster_wheel.dae"/>
+             </geometry>
+         </visual>
+         <collision>
+             <origin rpy="0 0 0" xyz="0 0 0"/>
+             <geometry>
+                 <mesh filename="package://description/urdf/meshes/back_caster_wheel.dae"/>
+             </geometry>
+         </collision>
+         <inertial>
+             <mass value="${caster_wheel_mass}"/>
+             <xacro:back_caster_wheel_inertia/>
+         </inertial>
+     </link>
+    <!-- Back caster wheel joint -->
+     <joint name="back_caster_wheel_joint" type="continuous">
+         <axis xyz="0 1 0"/>
+         <parent link="back_caster_link"/>
+         <child link="back_caster_wheel"/>
+         <origin rpy="0 0 0" xyz="${back_caster_link_to_back_caster_wheel_dist_x} 0 ${caster_link_to_caster_wheel_dist_z}"/>
+     </joint>
 </robot>

Commit message: Added inertias.xacro

File: robot/description/urdf/casters.urdf.xacro (robot description, xacro)
@@ -4,22 +4,8 @@
     <!-- Note: this file contains definitions for both the casters & the caster wheels -->
     <!-- When included, only use front_caster_link and back_caster_link (joints for the wheels are defined in this file) -->
-    <!-- Constants -->
+    <!-- Includes -->
     <xacro:include filename="$(find description)/urdf/constants.xacro"/>
-    <!-- Note: mass can be used across both casters -->
-    <xacro:macro name="front_caster_link_inertia">
-        <inertia
-            ixx="0.07" ixy="0.00" ixz="-0.06"
-            iyx="0.00" iyy="0.12" iyz="0.00"
-            izx="-0.06" izy="0.00" izz="0.06"
-        />
-    </xacro:macro>
-    <xacro:macro name="back_caster_link_inertia">
-        <inertia
-            ixx="0.07" ixy="0.00" ixz="0.06"
-            iyx="0.00" iyy="0.00" iyz="0.00"
-            izx="0.06" izy="0.00" izz="0.06"
-        />
-    </xacro:macro>
-    <!-- Front caster link definition -->
+    <xacro:include filename="$(find description)/urdf/inertias.xacro"/>
+    <!-- Front caster definition -->
     <link name="front_caster_link">
         <visual>
@@ -40,5 +26,4 @@
         </inertial>
     </link>
-    <!-- Front caster joint definition -->
     <joint name="front_caster_link_joint" type="continuous">
         <axis xyz="0 0 1"/>
@@ -47,5 +32,5 @@
         <origin rpy="0 0 0" xyz="${casters_separation / 2.0} 0 ${caster_vertical_offset}"/>
     </joint>
-    <!-- Back caster link definition -->
+    <!-- Back caster definition -->
     <link name="back_caster_link">
         <visual>
@@ -66,5 +51,4 @@
         </inertial>
     </link>
-    <!-- Back caster joint definition -->
     <joint name="back_caster_link_joint" type="continuous">
         <axis xyz="0 0 1"/>
@@ -73,19 +57,4 @@
         <origin rpy="0 0 0" xyz="-${casters_separation / 2.0} 0 ${caster_vertical_offset}"/>
     </joint>
-    <!-- Wheel definitions and joints -->
-    <xacro:macro name="front_caster_wheel_inertia">
-        <inertia
-            ixx="0.29" ixy="0.00" ixz="-0.27"
-            iyx="0.00" iyy="0.54" iyz="0.00"
-            izx="-0.27" izy="0.00" izz="0.25"
-        />
-    </xacro:macro>
-    <xacro:macro name="back_caster_wheel_inertia">
-        <inertia
-            ixx="0.29" ixy="0.00" ixz="0.27"
-            iyx="0.00" iyy="0.54" iyz="0.00"
-            izx="0.27" izy="0.00" izz="0.25"
-        />
-    </xacro:macro>
     <!-- Front caster wheel definition -->
     <link name="front_caster_wheel">
@@ -107,5 +76,4 @@
         </inertial>
     </link>
-    <!-- Front caster wheel joint -->
     <joint name="front_caster_wheel_joint" type="continuous">
         <axis xyz="0 1 0"/>
@@ -114,24 +82,23 @@
         <origin rpy="0 0 0" xyz="${caster_link_to_wheel_dist_x} 0 ${caster_link_to_wheel_dist_z}"/>
     </joint>
-     <!-- Back caster wheel definition -->
-     <link name="back_caster_wheel">
-         <visual>
-             <origin rpy="0 0 0" xyz="0 0 0"/>
-             <geometry>
-                 <mesh filename="package://description/urdf/meshes/back_caster_wheel.dae"/>
-             </geometry>
-         </visual>
-         <collision>
-             <origin rpy="0 0 0" xyz="0 0 0"/>
-             <geometry>
-                 <mesh filename="package://description/urdf/meshes/back_caster_wheel.dae"/>
-             </geometry>
-         </collision>
-         <inertial>
-             <mass value="${caster_wheel_mass}"/>
-             <xacro:back_caster_wheel_inertia/>
-         </inertial>
-     </link>
-    <!-- Back caster wheel joint -->
+    <!-- Back caster wheel definition -->
+    <link name="back_caster_wheel">
+        <visual>
+            <origin rpy="0 0 0" xyz="0 0 0"/>
+            <geometry>
+                <mesh filename="package://description/urdf/meshes/back_caster_wheel.dae"/>
+            </geometry>
+        </visual>
+        <collision>
+            <origin rpy="0 0 0" xyz="0 0 0"/>
+            <geometry>
+                <mesh filename="package://description/urdf/meshes/back_caster_wheel.dae"/>
+            </geometry>
+        </collision>
+        <inertial>
+            <mass value="${caster_wheel_mass}"/>
+            <xacro:back_caster_wheel_inertia/>
+        </inertial>
+    </link>
     <joint name="back_caster_wheel_joint" type="continuous">
         <axis xyz="0 1 0"/>

File: robot/description/urdf/chassis_link.urdf.xacro (robot description, xacro)
@@ -1,14 +1,7 @@
 <?xml version="1.0"?>
 <robot name="chassis" xmlns:xacro="http://ros.org/wiki/xacro">
-    <!-- Constants -->
+    <!-- Includes -->
     <xacro:include filename="$(find description)/urdf/constants.xacro"/>
-    <!-- Inertias -->
-    <xacro:macro name="chassis_link_inertia">
-        <inertia
-            ixx="10.77" ixy="0.00" ixz="0.00"
-            iyx="0.00" iyy="10.74" iyz="0.00"
-            izx="0.00" izy="0.00" izz="2.14"
-        />
-    </xacro:macro>
+    <xacro:include filename="$(find description)/urdf/inertias.xacro"/>
     <!-- Chassis link definition; chassis link is associated with the centroid of the bounding box of the robot and the chassis_link.dae file-->
     <link name="chassis_link">

File: robot/description/urdf/side_wheels.urdf.xacro (robot description, xacro)
@@ -1,21 +1,7 @@
 <?xml version="1.0"?>
 <robot name="side_wheels" xmlns:xacro="http://ros.org/wiki/xacro">
-    <!-- Constants -->
+    <!-- Includes -->
     <xacro:include filename="$(find description)/urdf/constants.xacro"/>
-    <!-- Inertias -->
-    <xacro:macro name="left_wheel_inertia">
-        <inertia
-            ixx="2.43" ixy="0.00" ixz="0.00"
-            iyx="0.00" iyy="1.60" iyz="1.15"
-            izx="0.00" izy="1.15" izz="0.87"
-            />
-    </xacro:macro>
-    <xacro:macro name="right_wheel_inertia">
-        <inertia
-            ixx="2.43" ixy="0.00" ixz="0.00"
-            iyx="0.00" iyy="1.60" iyz="-1.15"
-            izx="0.00" izy="-1.15" izz="0.87"
-            />
-    </xacro:macro>
+    <xacro:include filename="$(find description)/urdf/inertias.xacro"/>
     <!-- Motor Transmissions -->
     <xacro:macro name="Transmission" params="joint">

File: robot/description/urdf/stand_link.urdf.xacro (robot description, xacro)
@@ -1,6 +1,7 @@
 <?xml version="1.0"?>
 <robot name="stand_link" xmlns:xacro="http://ros.org/wiki/xacro">
-    <!-- Constants -->
+    <!-- Includes -->
     <xacro:include filename="$(find description)/urdf/constants.xacro"/>
+    <xacro:include filename="$(find description)/urdf/inertias.xacro"/>
     <!-- Stand link; this is a dummy link that is used to make camera placement and other sensors on the stand more convenient -->
     <!-- Stand link definition. Note: purposely left blank -->

Commit message: Updated inertia values

File: robot/description/urdf/casters.urdf.xacro (robot description, xacro)
@@ -23,5 +23,5 @@
         <inertial>
             <mass value="${caster_link_mass}"/>
-            <xacro:front_caster_link_inertia/>
+            <xacro:caster_link_inertia/>
         </inertial>
     </link>
@@ -48,5 +48,5 @@
         <inertial>
             <mass value="${caster_link_mass}"/>
-            <xacro:back_caster_link_inertia/>
+            <xacro:caster_link_inertia/>
         </inertial>
     </link>
@@ -73,5 +73,5 @@
         <inertial>
             <mass value="${caster_wheel_mass}"/>
-            <xacro:front_caster_wheel_inertia/>
+            <xacro:caster_wheel_inertia/>
         </inertial>
     </link>
@@ -98,5 +98,5 @@
         <inertial>
             <mass value="${caster_wheel_mass}"/>
-            <xacro:back_caster_wheel_inertia/>
+            <xacro:caster_wheel_inertia/>
         </inertial>
     </link>

File: robot/description/urdf/inertias.xacro (robot description, xacro)
@@ -4,52 +4,31 @@
     <xacro:macro name="chassis_link_inertia">
         <inertia
-            ixx="10.77" ixy="0.00" ixz="0.00"
-            iyx="0.00" iyy="10.74" iyz="0.00"
-            izx="0.00" izy="0.00" izz="2.14"
+            ixx="10.9364" ixy="0.0000" ixz="0.0000"
+            iyx="0.0000" iyy="10.9070" iyz="0.0000"
+            izx="0.0000" izy="0.0000" izz="2.3961"
         />
     </xacro:macro>
     <!-- Casters -->
-    <xacro:macro name="front_caster_link_inertia">
+    <xacro:macro name="caster_link_inertia">
         <inertia
-            ixx="0.07" ixy="0.00" ixz="-0.06"
-            iyx="0.00" iyy="0.12" iyz="0.00"
-            izx="-0.06" izy="0.00" izz="0.06"
+            ixx="0.0020" ixy="0.0000" ixz="0.0000"
+            iyx="0.0000" iyy="0.0020" iyz="0.0000"
+            izx="0.0000" izy="0.0000" izz="0.0008"
         />
     </xacro:macro>
-    <xacro:macro name="back_caster_link_inertia">
+    <xacro:macro name="caster_wheel_inertia">
         <inertia
-            ixx="0.07" ixy="0.00" ixz="0.06"
-            iyx="0.00" iyy="0.12" iyz="0.00"
-            izx="0.06" izy="0.00" izz="0.06"
-        />
-    </xacro:macro>
-    <xacro:macro name="front_caster_wheel_inertia">
-        <inertia
-            ixx="0.29" ixy="0.00" ixz="-0.27"
-            iyx="0.00" iyy="0.54" iyz="0.00"
-            izx="-0.27" izy="0.00" izz="0.25"
-        />
-    </xacro:macro>
-    <xacro:macro name="back_caster_wheel_inertia">
-        <inertia
-            ixx="0.29" ixy="0.00" ixz="0.27"
-            iyx="0.00" iyy="0.54" iyz="0.00"
-            izx="0.27" izy="0.00" izz="0.25"
+            ixx="0.0012" ixy="0.0000" ixz="0.0000"
+            iyx="0.0000" iyy="0.0022" iyz="0.0000"
+            izx="0.0000" izy="0.0000" izz="0.0012"
         />
     </xacro:macro>
     <!-- Wheels -->
-    <xacro:macro name="left_wheel_inertia">
+    <xacro:macro name="side_wheel_inertia">
         <inertia
-            ixx="2.43" ixy="0.00" ixz="0.00"
-            iyx="0.00" iyy="1.60" iyz="1.15"
-            izx="0.00" izy="1.15" izz="0.87"
-            />
-    </xacro:macro>
-    <xacro:macro name="right_wheel_inertia">
-        <inertia
-            ixx="2.43" ixy="0.00" ixz="0.00"
-            iyx="0.00" iyy="1.60" iyz="-1.15"
-            izx="0.00" izy="-1.15" izz="0.87"
-            />
+            ixx="0.0231" ixy="0.0000" ixz="0.0000"
+            iyx="0.0000" iyy="0.0374" iyz="0.0000"
+            izx="0.0000" izy="0.0000" izz="0.0231"
+        />
     </xacro:macro>
 </robot>

File: robot/description/urdf/side_wheels.urdf.xacro (robot description, xacro)
@@ -30,5 +30,5 @@
         <inertial>
             <mass value="${wheel_mass}"/>
-            <xacro:left_wheel_inertia/>
+            <xacro:side_wheel_inertia/>
         </inertial>
     </link>
@@ -56,5 +56,5 @@
         <inertial>
             <mass value="${wheel_mass}"/>
-            <xacro:right_wheel_inertia/>
+            <xacro:side_wheel_inertia/>
         </inertial>
     </link>

Commit message: Made support caster joint a fixed one

File: robot/description/urdf/casters.urdf.xacro (robot description, xacro)
@@ -26,6 +26,7 @@
         </inertial>
     </link>
-    <joint name="front_caster_link_joint" type="continuous">
-        <axis xyz="0 0 1"/>
+    <!-- NOTE: using a fixed joint prevents Caffeine spawning tipped over -->
+    <joint name="front_caster_link_joint" type="fixed">
+        <!-- <axis xyz="0 0 1"/> -->
         <parent link="chassis_link"/>
         <child link="front_caster_link"/>
@@ -51,6 +52,7 @@
         </inertial>
     </link>
-    <joint name="back_caster_link_joint" type="continuous">
-        <axis xyz="0 0 1"/>
+    <!-- NOTE: using a fixed joint prevents Caffeine spawning tipped over -->
+    <joint name="back_caster_link_joint" type="fixed">
+        <!-- <axis xyz="0 0 1"/> -->
         <parent link="chassis_link"/>
         <child link="back_caster_link"/>
@@ -77,8 +79,8 @@
     </link>
     <joint name="front_caster_wheel_joint" type="continuous">
-        <axis xyz="0 1 0"/>
         <parent link="front_caster_link"/>
         <child link="front_caster_wheel"/>
         <origin rpy="0 0 0" xyz="${caster_link_to_wheel_dist_x} 0 ${caster_link_to_wheel_dist_z}"/>
+        <axis xyz="0 1 0"/>
     </joint>
     <!-- Back caster wheel definition -->
@@ -102,8 +104,8 @@
     </link>
     <joint name="back_caster_wheel_joint" type="continuous">
-        <axis xyz="0 1 0"/>
         <parent link="back_caster_link"/>
         <child link="back_caster_wheel"/>
         <origin rpy="0 0 0" xyz="-${caster_link_to_wheel_dist_x} 0 ${caster_link_to_wheel_dist_z}"/>
+        <axis xyz="0 1 0"/>
     </joint>
 </robot>

Commit message: Removed unnecessary comments

File: robot/description/urdf/casters.urdf.xacro (robot description, xacro)
@@ -1,7 +1,4 @@
 <?xml version="1.0"?>
 <robot name="caster_wheels" xmlns:xacro="http://ros.org/wiki/xacro">
-    <!-- TODO: make sure the inertias associated with each caster and wheel is correct -->
-    <!-- Note: this file contains definitions for both the casters & the caster wheels -->
-    <!-- When included, only use front_caster_link and back_caster_link (joints for the wheels are defined in this file) -->
     <!-- Includes -->
     <xacro:include filename="$(find description)/urdf/constants.xacro"/>

File: robot/description/urdf/constants.xacro (robot description, xacro)
@@ -15,5 +15,5 @@
     <xacro:property name="wheel_vertical_offset" value="-0.61759696"/>
     <xacro:property name="wheels_separation" value="0.875"/>
-    <xacro:property name="wheel_diameter" value="0.25"/> <!-- TODO: update this value -->
+    <xacro:property name="wheel_diameter" value="0.25"/>
     <xacro:property name="wheel_mass" value="4.45"/>
     <!-- Gazebo Motor -->

Commit message: Added friction to casters and wheels (values are guess-timated)

File: robot/description/urdf/casters.urdf.xacro (robot description, xacro)
@@ -23,11 +23,16 @@
         </inertial>
     </link>
-    <!-- NOTE: using a fixed joint prevents Caffeine spawning tipped over -->
-    <joint name="${tf_prefix}/front_caster_link_joint" type="fixed">
-        <!-- <axis xyz="0 0 1"/> -->
+    <joint name="${tf_prefix}/front_caster_link_joint" type="continuous">
+        <axis xyz="0 0 1"/>
         <parent link="${tf_prefix}/chassis_link"/>
         <child link="${tf_prefix}/front_caster_link"/>
         <origin rpy="0 0 0" xyz="${casters_separation / 2.0} 0 ${caster_vertical_offset}"/>
     </joint>
+    <gazebo reference="${tf_prefix}/front_caster_link">
+        <mu1 value="0.3"/>
+        <mu2 value="0.3"/>
+        <kp value="10000000.0" />
+        <kd value="1.0" />
+    </gazebo>
     <!-- Back caster definition -->
     <link name="${tf_prefix}/back_caster_link">
@@ -49,11 +54,16 @@
         </inertial>
     </link>
-    <!-- NOTE: using a fixed joint prevents Caffeine spawning tipped over -->
-    <joint name="${tf_prefix}/back_caster_link_joint" type="fixed">
-        <!-- <axis xyz="0 0 1"/> -->
+    <joint name="${tf_prefix}/back_caster_link_joint" type="continuous">
+        <axis xyz="0 0 1"/>
         <parent link="${tf_prefix}/chassis_link"/>
         <child link="${tf_prefix}/back_caster_link"/>
         <origin rpy="0 0 0" xyz="-${casters_separation / 2.0} 0 ${caster_vertical_offset}"/>
     </joint>
+    <gazebo reference="${tf_prefix}/back_caster_link">
+        <mu1 value="0.3"/>
+        <mu2 value="0.3"/>
+        <kp value="10000000.0" />
+        <kd value="1.0" />
+    </gazebo>
     <!-- Front caster wheel definition -->
     <link name="${tf_prefix}/front_caster_wheel">
@@ -81,4 +91,10 @@
         <axis xyz="0 1 0"/>
     </joint>
+    <gazebo reference="${tf_prefix}/front_caster_wheel">
+        <mu1 value="0.1"/>
+        <mu2 value="0.1"/>
+        <kp value="10000000.0" />
+        <kd value="1.0" />
+    </gazebo>
     <!-- Back caster wheel definition -->
     <link name="${tf_prefix}/back_caster_wheel">
@@ -106,3 +122,9 @@
         <axis xyz="0 1 0"/>
     </joint>
+    <gazebo reference="${tf_prefix}/back_caster_wheel">
+        <mu1 value="0.1"/>
+        <mu2 value="0.1"/>
+        <kp value="10000000.0" />
+        <kd value="1.0" />
+    </gazebo>
 </robot>

File: robot/description/urdf/side_wheels.urdf.xacro (robot description, xacro)
@@ -39,4 +39,10 @@
         <axis xyz="0 1 0"/>
     </joint>
+    <gazebo reference="${tf_prefix}/left_wheel_link">
+        <mu1 value="1.0"/>
+        <mu2 value="1.0"/>
+        <kp value="10000000.0" />
+        <kd value="1.0" />
+    </gazebo>
     <xacro:Transmission joint="${tf_prefix}/left_wheel_joint"/>
     <!-- right wheel -->
@@ -65,4 +71,10 @@
         <axis xyz="0 1 0"/>
     </joint>
+    <gazebo reference="${tf_prefix}/right_wheel_link">
+        <mu1 value="1.0"/>
+        <mu2 value="1.0"/>
+        <kp value="10000000.0" />
+        <kd value="1.0" />
+    </gazebo>
     <xacro:Transmission joint="${tf_prefix}/right_wheel_joint"/>
 </robot>
