Commit message: Trying out ball casters

File: robot/description/urdf/casters.urdf.xacro (robot description, xacro)
@@ -9,5 +9,5 @@
             <origin rpy="0 0 0" xyz="0 0 0"/>
             <geometry>
-                <mesh filename="package://description/urdf/meshes/front_caster.dae"/>
+                <sphere radius="${caster_link_radius}"/>
             </geometry>
         </visual>
@@ -15,14 +15,13 @@
             <origin rpy="0 0 0" xyz="0 0 0"/>
             <geometry>
-                <mesh filename="package://description/urdf/meshes/front_caster.dae"/>
+                <sphere radius="${caster_link_radius}"/>
             </geometry>
         </collision>
         <inertial>
             <mass value="${caster_link_mass}"/>
-            <xacro:caster_link_inertia/>
+            <xacro:sphere_inertia mass="${caster_link_mass}" radius="${caster_link_radius}"/>
         </inertial>
     </link>
-    <joint name="${tf_prefix}/front_caster_link_joint" type="continuous">
-        <axis xyz="0 0 1"/>
+    <joint name="${tf_prefix}/front_caster_link_joint" type="fixed">
         <parent link="${tf_prefix}/chassis_link"/>
         <child link="${tf_prefix}/front_caster_link"/>
@@ -35,4 +34,23 @@
         <kd value="1.0" />
     </gazebo>
+    <gazebo>
+        <joint name='${tf_prefix}/front_caster_link_joint' type='ball'>
+           <parent>${tf_prefix}/chassis_link</parent>
+           <child>${tf_prefix}/front_caster_link</child>
+           <pose frame=''>0 0 0 0 0 0</pose>
+             <physics>
+                 <ode>
+                     <limit>
+                         <cfm>0</cfm>
+                         <erp>0.2</erp>
+                     </limit>
+                     <suspension>
+                         <cfm>0</cfm>
+                         <erp>0.2</erp>
+                     </suspension>
+                 </ode>
+             </physics>
+        </joint>
+    </gazebo>
     <!-- Back caster definition -->
     <link name="${tf_prefix}/back_caster_link">
@@ -40,5 +58,5 @@
             <origin rpy="0 0 0" xyz="0 0 0"/>
             <geometry>
-                <mesh filename="package://description/urdf/meshes/back_caster.dae"/>
+                <sphere radius="${caster_link_radius}"/>
             </geometry>
         </visual>
@@ -46,14 +64,13 @@
             <origin rpy="0 0 0" xyz="0 0 0"/>
             <geometry>
-                <mesh filename="package://description/urdf/meshes/back_caster.dae"/>
+                <sphere radius="${caster_link_radius}"/>
             </geometry>
         </collision>
         <inertial>
             <mass value="${caster_link_mass}"/>
-            <xacro:caster_link_inertia/>
+            <xacro:sphere_inertia mass="${caster_link_mass}" radius="${caster_link_radius}"/>
         </inertial>
     </link>
-    <joint name="${tf_prefix}/back_caster_link_joint" type="continuous">
-        <axis xyz="0 0 1"/>
+    <joint name="${tf_prefix}/back_caster_link_joint" type="fixed">
         <parent link="${tf_prefix}/chassis_link"/>
         <child link="${tf_prefix}/back_caster_link"/>
@@ -66,65 +83,22 @@
         <kd value="1.0" />
     </gazebo>
-    <!-- Front caster wheel definition -->
-    <link name="${tf_prefix}/front_caster_wheel">
-        <visual>
-            <origin rpy="0 0 0" xyz="0 0 0"/>
-            <geometry>
-                <mesh filename="package://description/urdf/meshes/front_caster_wheel.dae"/>
-            </geometry>
-        </visual>
-        <collision>
-            <origin rpy="0 0 0" xyz="0 0 0"/>
-            <geometry>
-                <mesh filename="package://description/urdf/meshes/front_caster_wheel.dae"/>
-            </geometry>
-        </collision>
-        <inertial>
-            <mass value="${caster_wheel_mass}"/>
-            <xacro:caster_wheel_inertia/>
-        </inertial>
-    </link>
-    <joint name="${tf_prefix}/front_caster_wheel_joint" type="continuous">
-        <parent link="${tf_prefix}/front_caster_link"/>
-        <child link="${tf_prefix}/front_caster_wheel"/>
-        <origin rpy="0 0 0" xyz="${caster_link_to_wheel_dist_x} 0 ${caster_link_to_wheel_dist_z}"/>
-        <axis xyz="0 1 0"/>
-    </joint>
-    <gazebo reference="${tf_prefix}/front_caster_wheel">
-        <mu1 value="0.1"/>
-        <mu2 value="0.1"/>
-        <kp value="10000000.0" />
-        <kd value="1.0" />
-    </gazebo>
-    <!-- Back caster wheel definition -->
-    <link name="${tf_prefix}/back_caster_wheel">
-        <visual>
-            <origin rpy="0 0 0" xyz="0 0 0"/>
-            <geometry>
-                <mesh filename="package://description/urdf/meshes/back_caster_wheel.dae"/>
-            </geometry>
-        </visual>
-        <collision>
-            <origin rpy="0 0 0" xyz="0 0 0"/>
-            <geometry>
-                <mesh filename="package://description/urdf/meshes/back_caster_wheel.dae"/>
-            </geometry>
-        </collision>
-        <inertial>
-            <mass value="${caster_wheel_mass}"/>
-            <xacro:caster_wheel_inertia/>
-        </inertial>
-    </link>
-    <joint name="${tf_prefix}/back_caster_wheel_joint" type="continuous">
-        <parent link="${tf_prefix}/back_caster_link"/>
-        <child link="${tf_prefix}/back_caster_wheel"/>
-        <origin rpy="0 0 0" xyz="-${caster_link_to_wheel_dist_x} 0 ${caster_link_to_wheel_dist_z}"/>
-        <axis xyz="0 1 0"/>
-    </joint>
-    <gazebo reference="${tf_prefix}/back_caster_wheel">
-        <mu1 value="0.1"/>
-        <mu2 value="0.1"/>
-        <kp value="10000000.0" />
-        <kd value="1.0" />
+    <gazebo>
+        <joint name='${tf_prefix}/back_caster_link_joint' type='ball'>
+            <parent>${tf_prefix}/chassis_link</parent>
+            <child>${tf_prefix}/back_caster_link</child>
+            <pose frame=''>0 0 0 0 0 0</pose>
+            <physics>
+                <ode>
+                    <limit>
+                        <cfm>0</cfm>
+                        <erp>0.2</erp>
+                    </limit>
+                    <suspension>
+                        <cfm>0</cfm>
+                        <erp>0.2</erp>
+                    </suspension>
+                </ode>
+            </physics>
+        </joint>
     </gazebo>
 </robot>

File: robot/description/urdf/constants.xacro (robot description, xacro)
@@ -13,10 +13,8 @@
     <xacro:property name="chassis_link_mass" value="33.9"/>
     <!-- Casters -->
-    <xacro:property name="caster_link_mass" value="0.5"/>
+    <xacro:property name="caster_link_mass" value="1.2"/>
     <xacro:property name="casters_separation" value="1.12"/>
     <xacro:property name="caster_vertical_offset" value="-0.619167561"/>
-    <xacro:property name="caster_wheel_mass" value="0.7"/>
-    <xacro:property name="caster_link_to_wheel_dist_x" value="0.03621719"/>
-    <xacro:property name="caster_link_to_wheel_dist_z" value="-0.04361749"/>
+    <xacro:property name="caster_link_radius" value="0.075"/>
     <!-- Wheels -->
     <!-- TODO: Update acceleration and torque parameters when known -->

File: robot/description/urdf/inertias.xacro (robot description, xacro)
@@ -7,19 +7,4 @@
             iyx="0.0000" iyy="10.9070" iyz="0.0000"
             izx="0.0000" izy="0.0000" izz="2.3961"
-        />
-    </xacro:macro>
-    <!-- Casters -->
-    <xacro:macro name="caster_link_inertia">
-        <inertia
-            ixx="0.0020" ixy="0.0000" ixz="0.0000"
-            iyx="0.0000" iyy="0.0020" iyz="0.0000"
-            izx="0.0000" izy="0.0000" izz="0.0008"
-        />
-    </xacro:macro>
-    <xacro:macro name="caster_wheel_inertia">
-        <inertia
-            ixx="0.0012" ixy="0.0000" ixz="0.0000"
-            iyx="0.0000" iyy="0.0022" iyz="0.0000"
-            izx="0.0000" izy="0.0000" izz="0.0012"
         />
     </xacro:macro>
@@ -48,3 +33,11 @@
         />
     </xacro:macro>
+     <!-- Sphere Inertia -->
+     <xacro:macro name="sphere_inertia" params="mass radius">
+         <inertia
+             ixx="${(2.0 * mass * radius * radius) / 5.0}" ixy="0.0" ixz="0.0"
+             iyx="0.0" iyy="${(2.0 * mass * radius * radius) / 5.0}" iyz="0.0"
+             izx="0.0" izy="0.0" izz="${(2.0 * mass * radius * radius) / 5.0}"
+         />
+     </xacro:macro>
 </robot>

Commit message: Can go over ramp currently but robot spawns non-level

File: robot/description/urdf/casters.urdf.xacro (robot description, xacro)
@@ -39,16 +39,4 @@
            <child>${tf_prefix}/front_caster_link</child>
            <pose frame=''>0 0 0 0 0 0</pose>
-             <physics>
-                 <ode>
-                     <limit>
-                         <cfm>0</cfm>
-                         <erp>0.2</erp>
-                     </limit>
-                     <suspension>
-                         <cfm>0</cfm>
-                         <erp>0.2</erp>
-                     </suspension>
-                 </ode>
-             </physics>
         </joint>
     </gazebo>
@@ -88,16 +76,4 @@
             <child>${tf_prefix}/back_caster_link</child>
             <pose frame=''>0 0 0 0 0 0</pose>
-            <physics>
-                <ode>
-                    <limit>
-                        <cfm>0</cfm>
-                        <erp>0.2</erp>
-                    </limit>
-                    <suspension>
-                        <cfm>0</cfm>
-                        <erp>0.2</erp>
-                    </suspension>
-                </ode>
-            </physics>
         </joint>
     </gazebo>

File: robot/description/urdf/constants.xacro (robot description, xacro)
@@ -15,5 +15,5 @@
     <xacro:property name="caster_link_mass" value="1.2"/>
     <xacro:property name="casters_separation" value="1.12"/>
-    <xacro:property name="caster_vertical_offset" value="-0.619167561"/>
+    <xacro:property name="caster_vertical_offset" value="-0.59"/>
     <xacro:property name="caster_link_radius" value="0.075"/>
     <!-- Wheels -->

Commit message: Removed ball joint and put all the original caster code in casters_original.urdf.xacro

File: robot/description/urdf/casters.urdf.xacro (robot description, xacro)
@@ -34,11 +34,4 @@
         <kd value="1.0" />
     </gazebo>
-    <gazebo>
-        <joint name='${tf_prefix}/front_caster_link_joint' type='ball'>
-           <parent>${tf_prefix}/chassis_link</parent>
-           <child>${tf_prefix}/front_caster_link</child>
-           <pose frame=''>0 0 0 0 0 0</pose>
-        </joint>
-    </gazebo>
     <!-- Back caster definition -->
     <link name="${tf_prefix}/back_caster_link">
@@ -71,10 +64,3 @@
         <kd value="1.0" />
     </gazebo>
-    <gazebo>
-        <joint name='${tf_prefix}/back_caster_link_joint' type='ball'>
-            <parent>${tf_prefix}/chassis_link</parent>
-            <child>${tf_prefix}/back_caster_link</child>
-            <pose frame=''>0 0 0 0 0 0</pose>
-        </joint>
-    </gazebo>
 </robot>

Commit message: Caff 28 - Navigate over ramps (#38)
* Created odom package, localization.yaml, odom.launch and modified caffeine_gazebo.launch to launch odometry. Currently does not work

* Trying out ball casters

* Can go over ramp currently but robot spawns non-level

* Removed odom packages that were accidentally added to this branch

* Restoring caffeine_gazebo launch file to initial state

* Updated caster ball radius to 0.0825

* Removed ball joint and put all the original caster code in casters_original.urdf.xacro

* set default world to ramp+walls

* reset gui to false

Co-authored-by: michruan <Michael Ruan>

File: robot/description/urdf/casters.urdf.xacro (robot description, xacro)
@@ -9,5 +9,5 @@
             <origin rpy="0 0 0" xyz="0 0 0"/>
             <geometry>
-                <mesh filename="package://description/urdf/meshes/front_caster.dae"/>
+                <sphere radius="${caster_link_radius}"/>
             </geometry>
         </visual>
@@ -15,14 +15,13 @@
             <origin rpy="0 0 0" xyz="0 0 0"/>
             <geometry>
-                <mesh filename="package://description/urdf/meshes/front_caster.dae"/>
+                <sphere radius="${caster_link_radius}"/>
             </geometry>
         </collision>
         <inertial>
             <mass value="${caster_link_mass}"/>
-            <xacro:caster_link_inertia/>
+            <xacro:sphere_inertia mass="${caster_link_mass}" radius="${caster_link_radius}"/>
         </inertial>
     </link>
-    <joint name="${tf_prefix}/front_caster_link_joint" type="continuous">
-        <axis xyz="0 0 1"/>
+    <joint name="${tf_prefix}/front_caster_link_joint" type="fixed">
         <parent link="${tf_prefix}/chassis_link"/>
         <child link="${tf_prefix}/front_caster_link"/>
@@ -40,5 +39,5 @@
             <origin rpy="0 0 0" xyz="0 0 0"/>
             <geometry>
-                <mesh filename="package://description/urdf/meshes/back_caster.dae"/>
+                <sphere radius="${caster_link_radius}"/>
             </geometry>
         </visual>
@@ -46,14 +45,13 @@
             <origin rpy="0 0 0" xyz="0 0 0"/>
             <geometry>
-                <mesh filename="package://description/urdf/meshes/back_caster.dae"/>
+                <sphere radius="${caster_link_radius}"/>
             </geometry>
         </collision>
         <inertial>
             <mass value="${caster_link_mass}"/>
-            <xacro:caster_link_inertia/>
+            <xacro:sphere_inertia mass="${caster_link_mass}" radius="${caster_link_radius}"/>
         </inertial>
     </link>
-    <joint name="${tf_prefix}/back_caster_link_joint" type="continuous">
-        <axis xyz="0 0 1"/>
+    <joint name="${tf_prefix}/back_caster_link_joint" type="fixed">
         <parent link="${tf_prefix}/chassis_link"/>
         <child link="${tf_prefix}/back_caster_link"/>
@@ -66,65 +64,3 @@
         <kd value="1.0" />
     </gazebo>
-    <!-- Front caster wheel definition -->
-    <link name="${tf_prefix}/front_caster_wheel">
-        <visual>
-            <origin rpy="0 0 0" xyz="0 0 0"/>
-            <geometry>
-                <mesh filename="package://description/urdf/meshes/front_caster_wheel.dae"/>
-            </geometry>
-        </visual>
-        <collision>
-            <origin rpy="0 0 0" xyz="0 0 0"/>
-            <geometry>
-                <mesh filename="package://description/urdf/meshes/front_caster_wheel.dae"/>
-            </geometry>
-        </collision>
-        <inertial>
-            <mass value="${caster_wheel_mass}"/>
-            <xacro:caster_wheel_inertia/>
-        </inertial>
-    </link>
-    <joint name="${tf_prefix}/front_caster_wheel_joint" type="continuous">
-        <parent link="${tf_prefix}/front_caster_link"/>
-        <child link="${tf_prefix}/front_caster_wheel"/>
-        <origin rpy="0 0 0" xyz="${caster_link_to_wheel_dist_x} 0 ${caster_link_to_wheel_dist_z}"/>
-        <axis xyz="0 1 0"/>
-    </joint>
-    <gazebo reference="${tf_prefix}/front_caster_wheel">
-        <mu1 value="0.1"/>
-        <mu2 value="0.1"/>
-        <kp value="10000000.0" />
-        <kd value="1.0" />
-    </gazebo>
-    <!-- Back caster wheel definition -->
-    <link name="${tf_prefix}/back_caster_wheel">
-        <visual>
-            <origin rpy="0 0 0" xyz="0 0 0"/>
-            <geometry>
-                <mesh filename="package://description/urdf/meshes/back_caster_wheel.dae"/>
-            </geometry>
-        </visual>
-        <collision>
-            <origin rpy="0 0 0" xyz="0 0 0"/>
-            <geometry>
-                <mesh filename="package://description/urdf/meshes/back_caster_wheel.dae"/>
-            </geometry>
-        </collision>
-        <inertial>
-            <mass value="${caster_wheel_mass}"/>
-            <xacro:caster_wheel_inertia/>
-        </inertial>
-    </link>
-    <joint name="${tf_prefix}/back_caster_wheel_joint" type="continuous">
-        <parent link="${tf_prefix}/back_caster_link"/>
-        <child link="${tf_prefix}/back_caster_wheel"/>
-        <origin rpy="0 0 0" xyz="-${caster_link_to_wheel_dist_x} 0 ${caster_link_to_wheel_dist_z}"/>
-        <axis xyz="0 1 0"/>
-    </joint>
-    <gazebo reference="${tf_prefix}/back_caster_wheel">
-        <mu1 value="0.1"/>
-        <mu2 value="0.1"/>
-        <kp value="10000000.0" />
-        <kd value="1.0" />
-    </gazebo>
 </robot>

File: robot/description/urdf/constants.xacro (robot description, xacro)
@@ -13,10 +13,8 @@
     <xacro:property name="chassis_link_mass" value="33.9"/>
     <!-- Casters -->
-    <xacro:property name="caster_link_mass" value="0.5"/>
+    <xacro:property name="caster_link_mass" value="1.2"/>
     <xacro:property name="casters_separation" value="1.12"/>
-    <xacro:property name="caster_vertical_offset" value="-0.619167561"/>
-    <xacro:property name="caster_wheel_mass" value="0.7"/>
-    <xacro:property name="caster_link_to_wheel_dist_x" value="0.03621719"/>
-    <xacro:property name="caster_link_to_wheel_dist_z" value="-0.04361749"/>
+    <xacro:property name="caster_vertical_offset" value="-0.59"/>
+    <xacro:property name="caster_link_radius" value="0.0825"/>
     <!-- Wheels -->
     <!-- TODO: Update acceleration and torque parameters when known -->
