Commit message: Making robot use CAD only instead of ball casters

File: robot/description/urdf/casters.urdf.xacro (robot description, xacro)
@@ -9,5 +9,5 @@
             <origin rpy="0 0 0" xyz="0 0 0"/>
             <geometry>
-                <sphere radius="${caster_link_radius}"/>
+                <mesh filename="package://description/urdf/meshes/front_caster.dae"/>
             </geometry>
         </visual>
@@ -15,13 +15,14 @@
             <origin rpy="0 0 0" xyz="0 0 0"/>
             <geometry>
-                <sphere radius="${caster_link_radius}"/>
+                <mesh filename="package://description/urdf/meshes/front_caster.dae"/>
             </geometry>
         </collision>
         <inertial>
             <mass value="${caster_link_mass}"/>
-            <xacro:sphere_inertia mass="${caster_link_mass}" radius="${caster_link_radius}"/>
+            <xacro:caster_link_inertia/>
         </inertial>
     </link>
-    <joint name="${tf_prefix}/front_caster_link_joint" type="fixed">
+    <joint name="${tf_prefix}/front_caster_link_joint" type="continuous">
+        <axis xyz="0 0 1"/>
         <parent link="${tf_prefix}/chassis_link"/>
         <child link="${tf_prefix}/front_caster_link"/>
@@ -39,5 +40,5 @@
             <origin rpy="0 0 0" xyz="0 0 0"/>
             <geometry>
-                <sphere radius="${caster_link_radius}"/>
+                <mesh filename="package://description/urdf/meshes/back_caster.dae"/>
             </geometry>
         </visual>
@@ -45,13 +46,14 @@
             <origin rpy="0 0 0" xyz="0 0 0"/>
             <geometry>
-                <sphere radius="${caster_link_radius}"/>
+                <mesh filename="package://description/urdf/meshes/back_caster.dae"/>
             </geometry>
         </collision>
         <inertial>
             <mass value="${caster_link_mass}"/>
-            <xacro:sphere_inertia mass="${caster_link_mass}" radius="${caster_link_radius}"/>
+            <xacro:caster_link_inertia/>
         </inertial>
     </link>
-    <joint name="${tf_prefix}/back_caster_link_joint" type="fixed">
+    <joint name="${tf_prefix}/back_caster_link_joint" type="continuous">
+        <axis xyz="0 0 1"/>
         <parent link="${tf_prefix}/chassis_link"/>
         <child link="${tf_prefix}/back_caster_link"/>
@@ -64,3 +66,65 @@
         <kd value="1.0" />
     </gazebo>
+    <!-- Front caster wheel definition -->
+    <link name="${tf_prefix}/front_caster_wheel">
+        <visual>
+            <origin rpy="0 0 0" xyz="0 0 0"/>
+            <geometry>
+                <mesh filename="package://description/urdf/meshes/front_caster_wheel.dae"/>
+            </geometry>
+        </visual>
+        <collision>
+            <origin rpy="0 0 0" xyz="0 0 0"/>
+            <geometry>
+                <mesh filename="package://description/urdf/meshes/front_caster_wheel.dae"/>
+            </geometry>
+        </collision>
+        <inertial>
+            <mass value="${caster_wheel_mass}"/>
+            <xacro:caster_wheel_inertia/>
+        </inertial>
+    </link>
+    <joint name="${tf_prefix}/front_caster_wheel_joint" type="continuous">
+        <parent link="${tf_prefix}/front_caster_link"/>
+        <child link="${tf_prefix}/front_caster_wheel"/>
+        <origin rpy="0 0 0" xyz="${caster_link_to_wheel_dist_x} 0 ${caster_link_to_wheel_dist_z}"/>
+        <axis xyz="0 1 0"/>
+    </joint>
+    <gazebo reference="${tf_prefix}/front_caster_wheel">
+        <mu1 value="0.1"/>
+        <mu2 value="0.1"/>
+        <kp value="10000000.0" />
+        <kd value="1.0" />
+    </gazebo>
+    <!-- Back caster wheel definition -->
+    <link name="${tf_prefix}/back_caster_wheel">
+        <visual>
+            <origin rpy="0 0 0" xyz="0 0 0"/>
+            <geometry>
+                <mesh filename="package://description/urdf/meshes/back_caster_wheel.dae"/>
+            </geometry>
+        </visual>
+        <collision>
+            <origin rpy="0 0 0" xyz="0 0 0"/>
+            <geometry>
+                <mesh filename="package://description/urdf/meshes/back_caster_wheel.dae"/>
+            </geometry>
+        </collision>
+        <inertial>
+            <mass value="${caster_wheel_mass}"/>
+            <xacro:caster_wheel_inertia/>
+        </inertial>
+    </link>
+    <joint name="${tf_prefix}/back_caster_wheel_joint" type="continuous">
+        <parent link="${tf_prefix}/back_caster_link"/>
+        <child link="${tf_prefix}/back_caster_wheel"/>
+        <origin rpy="0 0 0" xyz="-${caster_link_to_wheel_dist_x} 0 ${caster_link_to_wheel_dist_z}"/>
+        <axis xyz="0 1 0"/>
+    </joint>
+    <gazebo reference="${tf_prefix}/back_caster_wheel">
+        <mu1 value="0.1"/>
+        <mu2 value="0.1"/>
+        <kp value="10000000.0" />
+        <kd value="1.0" />
+    </gazebo>
 </robot>

File: robot/description/urdf/constants.xacro (robot description, xacro)
@@ -18,8 +18,10 @@
     <xacro:property name="stand_mass" value="1.0"/>
     <!-- Casters -->
-    <xacro:property name="caster_link_mass" value="1.2"/>
+    <xacro:property name="caster_link_mass" value="0.5"/>
     <xacro:property name="casters_separation" value="1.12"/>
-    <xacro:property name="caster_vertical_offset" value="-0.59"/>
-    <xacro:property name="caster_link_radius" value="0.0825"/>
+    <xacro:property name="caster_vertical_offset" value="-0.619167561"/>
+    <xacro:property name="caster_wheel_mass" value="0.7"/>
+    <xacro:property name="caster_link_to_wheel_dist_x" value="0.03621719"/>
+    <xacro:property name="caster_link_to_wheel_dist_z" value="-0.04361749"/>
     <!-- Wheels -->
     <!-- TODO: Update acceleration and torque parameters when known -->

File: robot/description/urdf/inertias.xacro (robot description, xacro)
@@ -41,3 +41,18 @@
          />
      </xacro:macro>
-</robot>
+     <!-- Casters and casters wheel inertias -->
+     <xacro:macro name="caster_link_inertia">
+        <inertia
+           ixx="0.0020" ixy="0.0000" ixz="0.0000"
+           iyx="0.0000" iyy="0.0020" iyz="0.0000"
+           izx="0.0000" izy="0.0000" izz="0.0008"
+        />
+    </xacro:macro>
+    <xacro:macro name="caster_wheel_inertia">
+        <inertia
+           ixx="0.0012" ixy="0.0000" ixz="0.0000"
+           iyx="0.0000" iyy="0.0022" iyz="0.0000"
+           izx="0.0000" izy="0.0000" izz="0.0012"
+        />
+    </xacro:macro>
+ </robot>

Commit message: commented front caster and increased back caster weight

File: robot/description/urdf/casters.urdf.xacro (robot description, xacro)
@@ -5,5 +5,5 @@
     <xacro:include filename="$(find description)/urdf/inertias.xacro"/>
     <!-- Front caster definition -->
-    <link name="${tf_prefix}/front_caster_link">
+    <!-- <link name="${tf_prefix}/front_caster_link">
         <visual>
             <origin rpy="0 0 0" xyz="0 0 0"/>
@@ -34,5 +34,5 @@
         <kp value="10000000.0" />
         <kd value="1.0" />
-    </gazebo>
+    </gazebo> -->
     <!-- Back caster definition -->
     <link name="${tf_prefix}/back_caster_link">
@@ -67,5 +67,5 @@
     </gazebo>
     <!-- Front caster wheel definition -->
-    <link name="${tf_prefix}/front_caster_wheel">
+    <!-- <link name="${tf_prefix}/front_caster_wheel">
         <visual>
             <origin rpy="0 0 0" xyz="0 0 0"/>
@@ -96,5 +96,5 @@
         <kp value="10000000.0" />
         <kd value="1.0" />
-    </gazebo>
+    </gazebo> -->
     <!-- Back caster wheel definition -->
     <link name="${tf_prefix}/back_caster_wheel">

File: robot/description/urdf/constants.xacro (robot description, xacro)
@@ -21,5 +21,5 @@
     <xacro:property name="casters_separation" value="1.12"/>
     <xacro:property name="caster_vertical_offset" value="-0.619167561"/>
-    <xacro:property name="caster_wheel_mass" value="0.7"/>
+    <xacro:property name="caster_wheel_mass" value="20.7"/> <!-- CHANGED -->
     <xacro:property name="caster_link_to_wheel_dist_x" value="0.03621719"/>
     <xacro:property name="caster_link_to_wheel_dist_z" value="-0.04361749"/>

Commit message: documented 3-wheel drive changes

File: robot/description/urdf/casters.urdf.xacro (robot description, xacro)
@@ -4,4 +4,14 @@
     <xacro:include filename="$(find description)/urdf/constants.xacro"/>
     <xacro:include filename="$(find description)/urdf/inertias.xacro"/>
+    <!--
+        ************************* HACK/FIX *************************
+        Previously, we had spheres in sim that would allow
+        our drive system to go over ramps, at the cost of a tilted
+        robot. A proposed hack/fix is to remove the front caster,
+        making Caffeine a 3-wheel drive robot, and adding a
+        counterweight at the back, representative of a battery, for
+        example.
+        *Leave Front Caster+Wheel Definitions Commented Out*
+    -->
     <!-- Front caster definition -->
     <!-- <link name="${tf_prefix}/front_caster_link">
@@ -32,4 +42,35 @@
         <mu1 value="0.3"/>
         <mu2 value="0.3"/>
+        <kp value="10000000.0" />
+        <kd value="1.0" />
+    </gazebo> -->
+    <!-- Front caster wheel definition -->
+    <!-- <link name="${tf_prefix}/front_caster_wheel">
+        <visual>
+            <origin rpy="0 0 0" xyz="0 0 0"/>
+            <geometry>
+                <mesh filename="package://description/urdf/meshes/front_caster_wheel.dae"/>
+            </geometry>
+        </visual>
+        <collision>
+            <origin rpy="0 0 0" xyz="0 0 0"/>
+            <geometry>
+                <mesh filename="package://description/urdf/meshes/front_caster_wheel.dae"/>
+            </geometry>
+        </collision>
+        <inertial>
+            <mass value="${caster_wheel_mass}"/>
+            <xacro:caster_wheel_inertia/>
+        </inertial>
+    </link>
+    <joint name="${tf_prefix}/front_caster_wheel_joint" type="continuous">
+        <parent link="${tf_prefix}/front_caster_link"/>
+        <child link="${tf_prefix}/front_caster_wheel"/>
+        <origin rpy="0 0 0" xyz="${caster_link_to_wheel_dist_x} 0 ${caster_link_to_wheel_dist_z}"/>
+        <axis xyz="0 1 0"/>
+    </joint>
+    <gazebo reference="${tf_prefix}/front_caster_wheel">
+        <mu1 value="0.1"/>
+        <mu2 value="0.1"/>
         <kp value="10000000.0" />
         <kd value="1.0" />
@@ -66,35 +107,4 @@
         <kd value="1.0" />
     </gazebo>
-    <!-- Front caster wheel definition -->
-    <!-- <link name="${tf_prefix}/front_caster_wheel">
-        <visual>
-            <origin rpy="0 0 0" xyz="0 0 0"/>
-            <geometry>
-                <mesh filename="package://description/urdf/meshes/front_caster_wheel.dae"/>
-            </geometry>
-        </visual>
-        <collision>
-            <origin rpy="0 0 0" xyz="0 0 0"/>
-            <geometry>
-                <mesh filename="package://description/urdf/meshes/front_caster_wheel.dae"/>
-            </geometry>
-        </collision>
-        <inertial>
-            <mass value="${caster_wheel_mass}"/>
-            <xacro:caster_wheel_inertia/>
-        </inertial>
-    </link>
-    <joint name="${tf_prefix}/front_caster_wheel_joint" type="continuous">
-        <parent link="${tf_prefix}/front_caster_link"/>
-        <child link="${tf_prefix}/front_caster_wheel"/>
-        <origin rpy="0 0 0" xyz="${caster_link_to_wheel_dist_x} 0 ${caster_link_to_wheel_dist_z}"/>
-        <axis xyz="0 1 0"/>
-    </joint>
-    <gazebo reference="${tf_prefix}/front_caster_wheel">
-        <mu1 value="0.1"/>
-        <mu2 value="0.1"/>
-        <kp value="10000000.0" />
-        <kd value="1.0" />
-    </gazebo> -->
     <!-- Back caster wheel definition -->
     <link name="${tf_prefix}/back_caster_wheel">

File: robot/description/urdf/constants.xacro (robot description, xacro)
@@ -28,4 +28,5 @@
     <xacro:property name="battery_length" value="0.1"/>
     <xacro:property name="battery_height" value="0.05"/>
+    <!-- HACK/FIX: Left very heavy to ensure for 3-wheel drive, caffeine doesn't tilt forward-->
     <xacro:property name="battery_mass" value="33"/>
     <xacro:property name="battery_back_offset" value="0.17"/>

Commit message: CAFF-39 - Implement Workaround to address robot tilt + inability to go over ramps: 3-Wheel Drive (#59)
* Making robot use CAD only instead of ball casters

* commented front caster and increased back caster weight

* made black box

* documented 3-wheel drive changes

* comm

Co-authored-by: kajananchinniah <kajananchinniah@gmail.com>
Co-authored-by: michruan <Michael Ruan>

File: robot/description/urdf/casters.urdf.xacro (robot description, xacro)
@@ -4,10 +4,20 @@
     <xacro:include filename="$(find description)/urdf/constants.xacro"/>
     <xacro:include filename="$(find description)/urdf/inertias.xacro"/>
+    <!--
+        ************************* HACK/FIX *************************
+        Previously, we had spheres in sim that would allow
+        our drive system to go over ramps, at the cost of a tilted
+        robot. A proposed hack/fix is to remove the front caster,
+        making Caffeine a 3-wheel drive robot, and adding a
+        counterweight at the back, representative of a battery, for
+        example.
+        *Leave Front Caster+Wheel Definitions Commented Out*
+    -->
     <!-- Front caster definition -->
-    <link name="${tf_prefix}/front_caster_link">
+    <!-- <link name="${tf_prefix}/front_caster_link">
         <visual>
             <origin rpy="0 0 0" xyz="0 0 0"/>
             <geometry>
-                <sphere radius="${caster_link_radius}"/>
+                <mesh filename="package://description/urdf/meshes/front_caster.dae"/>
             </geometry>
         </visual>
@@ -15,13 +25,14 @@
             <origin rpy="0 0 0" xyz="0 0 0"/>
             <geometry>
-                <sphere radius="${caster_link_radius}"/>
+                <mesh filename="package://description/urdf/meshes/front_caster.dae"/>
             </geometry>
         </collision>
         <inertial>
             <mass value="${caster_link_mass}"/>
-            <xacro:sphere_inertia mass="${caster_link_mass}" radius="${caster_link_radius}"/>
+            <xacro:caster_link_inertia/>
         </inertial>
     </link>
-    <joint name="${tf_prefix}/front_caster_link_joint" type="fixed">
+    <joint name="${tf_prefix}/front_caster_link_joint" type="continuous">
+        <axis xyz="0 0 1"/>
         <parent link="${tf_prefix}/chassis_link"/>
         <child link="${tf_prefix}/front_caster_link"/>
@@ -33,5 +44,36 @@
         <kp value="10000000.0" />
         <kd value="1.0" />
-    </gazebo>
+    </gazebo> -->
+    <!-- Front caster wheel definition -->
+    <!-- <link name="${tf_prefix}/front_caster_wheel">
+        <visual>
+            <origin rpy="0 0 0" xyz="0 0 0"/>
+            <geometry>
+                <mesh filename="package://description/urdf/meshes/front_caster_wheel.dae"/>
+            </geometry>
+        </visual>
+        <collision>
+            <origin rpy="0 0 0" xyz="0 0 0"/>
+            <geometry>
+                <mesh filename="package://description/urdf/meshes/front_caster_wheel.dae"/>
+            </geometry>
+        </collision>
+        <inertial>
+            <mass value="${caster_wheel_mass}"/>
+            <xacro:caster_wheel_inertia/>
+        </inertial>
+    </link>
+    <joint name="${tf_prefix}/front_caster_wheel_joint" type="continuous">
+        <parent link="${tf_prefix}/front_caster_link"/>
+        <child link="${tf_prefix}/front_caster_wheel"/>
+        <origin rpy="0 0 0" xyz="${caster_link_to_wheel_dist_x} 0 ${caster_link_to_wheel_dist_z}"/>
+        <axis xyz="0 1 0"/>
+    </joint>
+    <gazebo reference="${tf_prefix}/front_caster_wheel">
+        <mu1 value="0.1"/>
+        <mu2 value="0.1"/>
+        <kp value="10000000.0" />
+        <kd value="1.0" />
+    </gazebo> -->
     <!-- Back caster definition -->
     <link name="${tf_prefix}/back_caster_link">
@@ -39,5 +81,5 @@
             <origin rpy="0 0 0" xyz="0 0 0"/>
             <geometry>
-                <sphere radius="${caster_link_radius}"/>
+                <mesh filename="package://description/urdf/meshes/back_caster.dae"/>
             </geometry>
         </visual>
@@ -45,13 +87,14 @@
             <origin rpy="0 0 0" xyz="0 0 0"/>
             <geometry>
-                <sphere radius="${caster_link_radius}"/>
+                <mesh filename="package://description/urdf/meshes/back_caster.dae"/>
             </geometry>
         </collision>
         <inertial>
             <mass value="${caster_link_mass}"/>
-            <xacro:sphere_inertia mass="${caster_link_mass}" radius="${caster_link_radius}"/>
+            <xacro:caster_link_inertia/>
         </inertial>
     </link>
-    <joint name="${tf_prefix}/back_caster_link_joint" type="fixed">
+    <joint name="${tf_prefix}/back_caster_link_joint" type="continuous">
+        <axis xyz="0 0 1"/>
         <parent link="${tf_prefix}/chassis_link"/>
         <child link="${tf_prefix}/back_caster_link"/>
@@ -64,3 +107,34 @@
         <kd value="1.0" />
     </gazebo>
+    <!-- Back caster wheel definition -->
+    <link name="${tf_prefix}/back_caster_wheel">
+        <visual>
+            <origin rpy="0 0 0" xyz="0 0 0"/>
+            <geometry>
+                <mesh filename="package://description/urdf/meshes/back_caster_wheel.dae"/>
+            </geometry>
+        </visual>
+        <collision>
+            <origin rpy="0 0 0" xyz="0 0 0"/>
+            <geometry>
+                <mesh filename="package://description/urdf/meshes/back_caster_wheel.dae"/>
+            </geometry>
+        </collision>
+        <inertial>
+            <mass value="${caster_wheel_mass}"/>
+            <xacro:caster_wheel_inertia/>
+        </inertial>
+    </link>
+    <joint name="${tf_prefix}/back_caster_wheel_joint" type="continuous">
+        <parent link="${tf_prefix}/back_caster_link"/>
+        <child link="${tf_prefix}/back_caster_wheel"/>
+        <origin rpy="0 0 0" xyz="-${caster_link_to_wheel_dist_x} 0 ${caster_link_to_wheel_dist_z}"/>
+        <axis xyz="0 1 0"/>
+    </joint>
+    <gazebo reference="${tf_prefix}/back_caster_wheel">
+        <mu1 value="0.1"/>
+        <mu2 value="0.1"/>
+        <kp value="10000000.0" />
+        <kd value="1.0" />
+    </gazebo>
 </robot>

File: robot/description/urdf/constants.xacro (robot description, xacro)
@@ -20,6 +20,15 @@
     <xacro:property name="caster_link_mass" value="1.2"/>
     <xacro:property name="casters_separation" value="1.12"/>
-    <xacro:property name="caster_vertical_offset" value="-0.59"/>
-    <xacro:property name="caster_link_radius" value="0.0825"/>
+    <xacro:property name="caster_vertical_offset" value="-0.619167561"/>
+    <xacro:property name="caster_wheel_mass" value="0.7"/>
+    <xacro:property name="caster_link_to_wheel_dist_x" value="0.03621719"/>
+    <xacro:property name="caster_link_to_wheel_dist_z" value="-0.04361749"/>
+    <!-- Battery -->
+    <xacro:property name="battery_width" value="0.05"/>
+    <xacro:property name="battery_length" value="0.1"/>
+    <xacro:property name="battery_height" value="0.05"/>
+    <!-- HACK/FIX: Left very heavy to ensure for 3-wheel drive, caffeine doesn't tilt forward-->
+    <xacro:property name="battery_mass" value="33"/>
+    <xacro:property name="battery_back_offset" value="0.17"/>
     <!-- Wheels -->
     <!-- TODO: Update acceleration and torque parameters when known -->
