Commit message: Moved joint definition to inside their respective files

File: description/urdf/base_laser.urdf.xacro (robot description, xacro)
@@ -6,8 +6,8 @@
    <!-- LIDAR link -->
    <link name="${tf_prefix}/base_laser">
-        <inertial>
+      <inertial>
             <mass value="${laser_mass}"/>
             <xacro:box_inertia mass="${laser_mass}" length="${laser_length}" width="${laser_width}" height="${laser_height}"/>
-        </inertial>
+      </inertial>
       <visual>
          <origin xyz="0 0 0" rpy="0 0 0"/>
@@ -23,3 +23,8 @@
       </collision>
    </link>
+   <joint name="${tf_prefix}/base_laser_joint" type="fixed">
+      <parent link="${tf_prefix}/base_link"/>
+      <child link="${tf_prefix}/base_laser"/>
+      <origin xyz="${laser_x_dist} 0 ${laser_z_dist}" rpy="0 0 0"/>
+   </joint>
 </robot>

File: description/urdf/caffeine.urdf.xacro (robot description, xacro)
@@ -8,16 +8,6 @@
     <!-- chassis_link: geometric center of the robot; used as the parent in which all other links connect to -->
     <xacro:include filename="$(find description)/urdf/chassis_link.urdf.xacro"/>
-    <joint name="${tf_prefix}/chassis_link_joint" type="fixed">
-        <parent link="${tf_prefix}/base_link"/>
-        <child link="${tf_prefix}/chassis_link"/>
-        <origin xyz="0 0 ${chassis_to_base_link_dist}" rpy="0 0 0"/>
-    </joint>
     <!-- stand_link: origin for anything on the stand; located in the middle, on the top of the stand plate -->
     <xacro:include filename="$(find description)/urdf/stand_link.urdf.xacro"/>
-    <joint name="${tf_prefix}/stand_link_joint" type="fixed">
-        <parent link="${tf_prefix}/chassis_link"/>
-        <child link="${tf_prefix}/stand_link"/>
-        <origin xyz="0 0 ${chassis_to_stand_link_dist}" rpy="0 0 0" />
-    </joint>
     <!-- wheels: associated to wheels that can be moved by a motor -->
     <xacro:include filename="$(find description)/urdf/side_wheels.urdf.xacro"/>
@@ -26,8 +16,3 @@
    <!-- base_laser: LIDAR at front of Caffeine -->
    <xacro:include filename="$(find description)/urdf/base_laser.urdf.xacro"/>
-   <joint name="${tf_prefix}/base_laser_joint" type="fixed">
-        <parent link="${tf_prefix}/base_link"/>
-        <child link="${tf_prefix}/base_laser"/>
-        <origin xyz="${laser_x_dist} 0 ${laser_z_dist}" rpy="0 0 0"/>
-   </joint>
 </robot>

File: description/urdf/chassis_link.urdf.xacro (robot description, xacro)
@@ -23,4 +23,9 @@
         </inertial>
     </link>
+    <joint name="${tf_prefix}/chassis_link_joint" type="fixed">
+        <parent link="${tf_prefix}/base_link"/>
+        <child link="${tf_prefix}/chassis_link"/>
+        <origin xyz="0 0 ${chassis_to_base_link_dist}" rpy="0 0 0"/>
+    </joint>
     <!-- Battery Link -->
     <link name="${tf_prefix}/battery_link">

File: description/urdf/stand_link.urdf.xacro (robot description, xacro)
@@ -7,4 +7,9 @@
     <!-- Stand link definition. Note: purposely left blank -->
     <link name="${tf_prefix}/stand_link"/>
+    <joint name="${tf_prefix}/stand_link_joint" type="fixed">
+        <parent link="${tf_prefix}/chassis_link"/>
+        <child link="${tf_prefix}/stand_link"/>
+        <origin xyz="0 0 ${chassis_to_stand_link_dist}" rpy="0 0 0" />
+    </joint>
     <!-- ZED Camera -->
     <link name="${tf_prefix}/zed_camera_link">
