Commit message: remove caffeine namespace everywhere

File: description/urdf/caffeine.gazebo.xacro (robot description, xacro)
@@ -6,8 +6,7 @@
     <gazebo>
         <plugin name="caffeine_drive_controller" filename="libgazebo_ros_diff_drive.so">
-            <robotNamespace>${robotNamespace}</robotNamespace>
             <updateRate>${diff_drive_update_rate}</updateRate>
-            <leftJoint>${tf_prefix}/${wheel_left_joint}</leftJoint>
-            <rightJoint>${tf_prefix}/${wheel_right_joint}</rightJoint>
+            <leftJoint>${wheel_left_joint}</leftJoint>
+            <rightJoint>${wheel_right_joint}</rightJoint>
             <wheelSeparation>${wheels_separation}</wheelSeparation>
             <wheelDiameter>${wheel_diameter}</wheelDiameter>
@@ -29,10 +28,8 @@
     <!-- lets all the transmission tags be read -->
     <gazebo>
-        <plugin name="gazebo_ros_control" filename="libgazebo_ros_control.so">
-            <robotNamespace>${robotNamespace}</robotNamespace>
-        </plugin>
+        <plugin name="gazebo_ros_control" filename="libgazebo_ros_control.so"/>
     </gazebo>
     <!-- LIDAR -->
-    <gazebo reference="${tf_prefix}/base_laser">
+    <gazebo reference="base_laser">
         <sensor type="ray" name="gpu_hokuyo_sensor">
             <pose>0 0 0 0 0 0</pose>
@@ -63,5 +60,4 @@
             </ray>
             <plugin name="gazebo_ros_hokuyo_controller" filename="libgazebo_ros_laser.so">
-                <robotNamespace>${robotNamespace}</robotNamespace>
                 <topicName>${laser_topicName}</topicName>
                 <frameName>${laser_frameName}</frameName>
@@ -72,8 +68,7 @@
     <gazebo>
         <plugin name="gps_controller" filename="libhector_gazebo_ros_gps.so">
-            <robotNamespace>${robotNamespace}</robotNamespace>
             <updateRate>${gps_update_rate}</updateRate>
-            <bodyName>${tf_prefix}/${gps_frame}</bodyName>
-            <frameId>${tf_prefix}/${gps_frame}</frameId>
+            <bodyName>${gps_frame}</bodyName>
+            <frameId>${gps_frame}</frameId>
             <topicName>${gps_topic}</topicName>
             <velocityTopicName>${gps_vel_topic}</velocityTopicName>
@@ -87,5 +82,5 @@
     </gazebo>
     <!-- Gazebo multicamera plugin -->
-    <gazebo reference="${tf_prefix}/camera_link">
+    <gazebo reference="camera_link">
         <sensor type="multicamera" name="stereo_camera">
             <update_rate>${ZED_image_refresh}</update_rate>
@@ -124,5 +119,5 @@
                 <depthImageInfoTopicName>${ZED_depth_info_topicName}</depthImageInfoTopicName>
                 <pointCloudTopicName>${ZED_depth_points_topicName}</pointCloudTopicName>
-                <frameName>${tf_prefix}/${ZED_frameName}</frameName>
+                <frameName>${ZED_frameName}</frameName>
                 <hackBaseline>${ZED_camera_length}</hackBaseline>
                 <!-- TODO: Get distortion parameters from real camera -->
@@ -136,5 +131,5 @@
     </gazebo>
     <!-- IMU -->
-    <gazebo reference="${tf_prefix}/imu_link">
+    <gazebo reference="imu_link">
         <material>Gazebo/Black</material>
         <gravity>true</gravity>
@@ -145,7 +140,7 @@
             <!-- TODO: add Drift based on Phidget IMU -->
             <plugin filename="libgazebo_ros_imu_sensor.so" name="imu_plugin">
-                <topicName>${robotNamespace}/${imu_topic}</topicName>
-                <bodyName>${tf_prefix}/${imu_frame}</bodyName>
-                <frameName>${tf_prefix}/${imu_frame}</frameName>
+                <topicName>${imu_topic}</topicName>
+                <bodyName>${imu_frame}</bodyName>
+                <frameName>${imu_frame}</frameName>
                 <updateRateHZ>${imu_update_rate}</updateRateHZ>
                 <gaussianNoise>0.0</gaussianNoise>  <!-- TODO: set Gaussian noise based on Phidget IMU -->

File: description/urdf/caffeine.urdf.xacro (robot description, xacro)
@@ -5,5 +5,5 @@
     <xacro:include filename="$(find description)/urdf/caffeine.gazebo.xacro"/>
     <!-- base_link: origin of the robot; located in the middle, on the top of the base plate -->
-    <link name="${tf_prefix}/base_link"/>
+    <link name="base_link"/>
     <!-- chassis_link: geometric center of the robot; used as the parent in which all other links connect to -->
     <xacro:include filename="$(find description)/urdf/chassis_link.urdf.xacro"/>
@@ -15,5 +15,5 @@
     <xacro:include filename="$(find description)/urdf/casters.urdf.xacro"/>
     <!-- base_laser: LIDAR at front of Caffeine -->
-    <link name="${tf_prefix}/base_laser">
+    <link name="base_laser">
         <inertial>
             <mass value="${laser_mass}"/>
@@ -33,7 +33,7 @@
         </collision>
     </link>
-    <joint name="${tf_prefix}/base_laser_joint" type="fixed">
-        <parent link="${tf_prefix}/base_link"/>
-        <child link="${tf_prefix}/base_laser"/>
+    <joint name="base_laser_joint" type="fixed">
+        <parent link="base_link"/>
+        <child link="base_laser"/>
         <origin xyz="${laser_x_dist} 0 ${laser_z_dist}" rpy="0 0 0"/>
     </joint>

File: description/urdf/casters.urdf.xacro (robot description, xacro)
@@ -15,5 +15,5 @@
     -->
     <!-- Front caster definition -->
-    <!-- <link name="${tf_prefix}/front_caster_link">
+    <!-- <link name="front_caster_link">
         <visual>
             <origin rpy="0 0 0" xyz="0 0 0"/>
@@ -33,11 +33,11 @@
         </inertial>
     </link>
-    <joint name="${tf_prefix}/front_caster_link_joint" type="continuous">
+    <joint name="front_caster_link_joint" type="continuous">
         <axis xyz="0 0 1"/>
-        <parent link="${tf_prefix}/chassis_link"/>
-        <child link="${tf_prefix}/front_caster_link"/>
+        <parent link="chassis_link"/>
+        <child link="front_caster_link"/>
         <origin rpy="0 0 0" xyz="${casters_separation / 2.0} 0 ${caster_vertical_offset}"/>
     </joint>
-    <gazebo reference="${tf_prefix}/front_caster_link">
+    <gazebo reference="front_caster_link">
         <mu1 value="0.3"/>
         <mu2 value="0.3"/>
@@ -46,5 +46,5 @@
     </gazebo> -->
     <!-- Front caster wheel definition -->
-    <!-- <link name="${tf_prefix}/front_caster_wheel">
+    <!-- <link name="front_caster_wheel">
         <visual>
             <origin rpy="0 0 0" xyz="0 0 0"/>
@@ -64,11 +64,11 @@
         </inertial>
     </link>
-    <joint name="${tf_prefix}/front_caster_wheel_joint" type="continuous">
-        <parent link="${tf_prefix}/front_caster_link"/>
-        <child link="${tf_prefix}/front_caster_wheel"/>
+    <joint name="front_caster_wheel_joint" type="continuous">
+        <parent link="front_caster_link"/>
+        <child link="front_caster_wheel"/>
         <origin rpy="0 0 0" xyz="${caster_link_to_wheel_dist_x} 0 ${caster_link_to_wheel_dist_z}"/>
         <axis xyz="0 1 0"/>
     </joint>
-    <gazebo reference="${tf_prefix}/front_caster_wheel">
+    <gazebo reference="front_caster_wheel">
         <mu1 value="0.1"/>
         <mu2 value="0.1"/>
@@ -77,5 +77,5 @@
     </gazebo> -->
     <!-- Back caster definition -->
-    <link name="${tf_prefix}/back_caster_link">
+    <link name="back_caster_link">
         <visual>
             <origin rpy="0 0 0" xyz="0 0 0"/>
@@ -95,11 +95,11 @@
         </inertial>
     </link>
-    <joint name="${tf_prefix}/back_caster_link_joint" type="continuous">
+    <joint name="back_caster_link_joint" type="continuous">
         <axis xyz="0 0 1"/>
-        <parent link="${tf_prefix}/chassis_link"/>
-        <child link="${tf_prefix}/back_caster_link"/>
+        <parent link="chassis_link"/>
+        <child link="back_caster_link"/>
         <origin rpy="0 0 0" xyz="-${casters_separation / 2.0} 0 ${caster_vertical_offset}"/>
     </joint>
-    <gazebo reference="${tf_prefix}/back_caster_link">
+    <gazebo reference="back_caster_link">
         <mu1 value="0.3"/>
         <mu2 value="0.3"/>
@@ -108,5 +108,5 @@
     </gazebo>
     <!-- Back caster wheel definition -->
-    <link name="${tf_prefix}/back_caster_wheel">
+    <link name="back_caster_wheel">
         <visual>
             <origin rpy="0 0 0" xyz="0 0 0"/>
@@ -126,11 +126,11 @@
         </inertial>
     </link>
-    <joint name="${tf_prefix}/back_caster_wheel_joint" type="continuous">
-        <parent link="${tf_prefix}/back_caster_link"/>
-        <child link="${tf_prefix}/back_caster_wheel"/>
+    <joint name="back_caster_wheel_joint" type="continuous">
+        <parent link="back_caster_link"/>
+        <child link="back_caster_wheel"/>
         <origin rpy="0 0 0" xyz="-${caster_link_to_wheel_dist_x} 0 ${caster_link_to_wheel_dist_z}"/>
         <axis xyz="0 1 0"/>
     </joint>
-    <gazebo reference="${tf_prefix}/back_caster_wheel">
+    <gazebo reference="back_caster_wheel">
         <mu1 value="0.1"/>
         <mu2 value="0.1"/>

File: description/urdf/casters_original.urdf.xacro (robot description, xacro)
@@ -31,5 +31,5 @@
     <xacro:include filename="$(find description)/urdf/inertias.xacro"/>
     <!-- Front caster definition -->
-    <link name="${tf_prefix}/front_caster_link">
+    <link name="front_caster_link">
         <visual>
             <origin rpy="0 0 0" xyz="0 0 0"/>
@@ -49,11 +49,11 @@
         </inertial>
     </link>
-    <joint name="${tf_prefix}/front_caster_link_joint" type="continuous">
+    <joint name="front_caster_link_joint" type="continuous">
         <axis xyz="0 0 1"/>
-        <parent link="${tf_prefix}/chassis_link"/>
-        <child link="${tf_prefix}/front_caster_link"/>
+        <parent link="chassis_link"/>
+        <child link="front_caster_link"/>
         <origin rpy="0 0 0" xyz="${casters_separation / 2.0} 0 ${caster_vertical_offset}"/>
     </joint>
-    <gazebo reference="${tf_prefix}/front_caster_link">
+    <gazebo reference="front_caster_link">
         <mu1 value="0.3"/>
         <mu2 value="0.3"/>
@@ -62,5 +62,5 @@
     </gazebo>
     <!-- Back caster definition -->
-    <link name="${tf_prefix}/back_caster_link">
+    <link name="back_caster_link">
         <visual>
             <origin rpy="0 0 0" xyz="0 0 0"/>
@@ -80,11 +80,11 @@
         </inertial>
     </link>
-    <joint name="${tf_prefix}/back_caster_link_joint" type="continuous">
+    <joint name="back_caster_link_joint" type="continuous">
         <axis xyz="0 0 1"/>
-        <parent link="${tf_prefix}/chassis_link"/>
-        <child link="${tf_prefix}/back_caster_link"/>
+        <parent link="chassis_link"/>
+        <child link="back_caster_link"/>
         <origin rpy="0 0 0" xyz="-${casters_separation / 2.0} 0 ${caster_vertical_offset}"/>
     </joint>
-    <gazebo reference="${tf_prefix}/back_caster_link">
+    <gazebo reference="/back_caster_link">
         <mu1 value="0.3"/>
         <mu2 value="0.3"/>
@@ -93,5 +93,5 @@
     </gazebo>
     <!-- Front caster wheel definition -->
-    <link name="${tf_prefix}/front_caster_wheel">
+    <link name="front_caster_wheel">
         <visual>
             <origin rpy="0 0 0" xyz="0 0 0"/>
@@ -111,11 +111,11 @@
         </inertial>
     </link>
-    <joint name="${tf_prefix}/front_caster_wheel_joint" type="continuous">
-        <parent link="${tf_prefix}/front_caster_link"/>
-        <child link="${tf_prefix}/front_caster_wheel"/>
+    <joint name="front_caster_wheel_joint" type="continuous">
+        <parent link="front_caster_link"/>
+        <child link="front_caster_wheel"/>
         <origin rpy="0 0 0" xyz="${caster_link_to_wheel_dist_x} 0 ${caster_link_to_wheel_dist_z}"/>
         <axis xyz="0 1 0"/>
     </joint>
-    <gazebo reference="${tf_prefix}/front_caster_wheel">
+    <gazebo reference="front_caster_wheel">
         <mu1 value="0.1"/>
         <mu2 value="0.1"/>
@@ -124,5 +124,5 @@
     </gazebo>
     <!-- Back caster wheel definition -->
-    <link name="${tf_prefix}/back_caster_wheel">
+    <link name="back_caster_wheel">
         <visual>
             <origin rpy="0 0 0" xyz="0 0 0"/>
@@ -142,11 +142,11 @@
         </inertial>
     </link>
-    <joint name="${tf_prefix}/back_caster_wheel_joint" type="continuous">
-        <parent link="${tf_prefix}/back_caster_link"/>
-        <child link="${tf_prefix}/back_caster_wheel"/>
+    <joint name="back_caster_wheel_joint" type="continuous">
+        <parent link="back_caster_link"/>
+        <child link="back_caster_wheel"/>
         <origin rpy="0 0 0" xyz="-${caster_link_to_wheel_dist_x} 0 ${caster_link_to_wheel_dist_z}"/>
         <axis xyz="0 1 0"/>
     </joint>
-    <gazebo reference="${tf_prefix}/back_caster_wheel">
+    <gazebo reference="back_caster_wheel">
         <mu1 value="0.1"/>
         <mu2 value="0.1"/>

File: description/urdf/chassis_link.urdf.xacro (robot description, xacro)
@@ -5,5 +5,5 @@
     <xacro:include filename="$(find description)/urdf/inertias.xacro"/>
     <!-- Chassis link definition; chassis link is associated with the centroid of the bounding box of the robot and the chassis_link.dae file-->
-    <link name="${tf_prefix}/chassis_link">
+    <link name="chassis_link">
         <visual>
             <origin rpy="0 0 0" xyz="0 0 0"/>
@@ -23,11 +23,11 @@
         </inertial>
     </link>
-    <joint name="${tf_prefix}/chassis_link_joint" type="fixed">
-        <parent link="${tf_prefix}/base_link"/>
-        <child link="${tf_prefix}/chassis_link"/>
+    <joint name="chassis_link_joint" type="fixed">
+        <parent link="base_link"/>
+        <child link="chassis_link"/>
         <origin xyz="0 0 ${chassis_to_base_link_dist}" rpy="0 0 0"/>
     </joint>
     <!-- Battery Link -->
-    <link name="${tf_prefix}/battery_link">
+    <link name="battery_link">
         <visual>
             <origin xyz="0 0 0" rpy="0 0 0"/>
@@ -47,8 +47,8 @@
         </inertial>
     </link>
-    <joint name="${tf_prefix}/battery_joint" type="fixed">
+    <joint name="battery_joint" type="fixed">
         <origin xyz="${-1*(stand_length/2 + battery_width + battery_back_offset)} 0 ${wheel_diameter - (3*battery_height/2) - stand_height/2}" rpy="0 0 0"/>
-        <parent link="${tf_prefix}/chassis_link"/>
-        <child link="${tf_prefix}/battery_link"/>
+        <parent link="chassis_link"/>
+        <child link="battery_link"/>
     </joint>
 </robot>

File: description/urdf/constants.xacro (robot description, xacro)
@@ -1,11 +1,8 @@
 <?xml version="1.0"?>
 <robot name="caffeine_constants" xmlns:xacro="http://ros.org/wiki/xacro">
-    <!-- Caffeine -->
-    <xacro:property name="robotNamespace" value="caffeine"/>
-    <xacro:property name="tf_prefix" value="caffeine"/>
     <!-- Drivebase -->
-   <xacro:property name="base_length" value="1.268"/>
-   <xacro:property name="base_width" value="0.764"/>
-   <xacro:property name="base_height" value="0.01"/>
+    <xacro:property name="base_length" value="1.268"/>
+    <xacro:property name="base_width" value="0.764"/>
+    <xacro:property name="base_height" value="0.01"/>
     <!-- Chassis -->
     <xacro:property name="chassis_to_base_link_dist" value="0.501747"/>
@@ -115,10 +112,10 @@
     <xacro:property name="gps_vel_drift" value="0.00 0.00 0.00"/>
     <!-- Phidget IMU -->
-   <xacro:property name="phidget_length" value="0.04"/>
-   <xacro:property name="phidget_width" value="0.0375"/>
-   <xacro:property name="phidget_height" value="0.01"/>
-   <xacro:property name="phidget_mass" value="0.04"/>
-   <xacro:property name="imu_frame" value="imu_link"/>
-   <xacro:property name="imu_topic" value="imu/data"/>
-   <xacro:property name="imu_update_rate" value="128.0"/>
+    <xacro:property name="phidget_length" value="0.04"/>
+    <xacro:property name="phidget_width" value="0.0375"/>
+    <xacro:property name="phidget_height" value="0.01"/>
+    <xacro:property name="phidget_mass" value="0.04"/>
+    <xacro:property name="imu_frame" value="imu_link"/>
+    <xacro:property name="imu_topic" value="imu/data"/>
+    <xacro:property name="imu_update_rate" value="128.0"/>
 </robot>

File: description/urdf/side_wheels.urdf.xacro (robot description, xacro)
@@ -15,5 +15,5 @@
     </xacro:macro>
     <!-- left wheel -->
-    <link name="${tf_prefix}/left_wheel_link">
+    <link name="left_wheel_link">
         <visual>
             <origin rpy="0 0 0" xyz="0 0 0"/>
@@ -33,11 +33,11 @@
         </inertial>
     </link>
-    <joint name="${tf_prefix}/left_wheel_joint" type="continuous">
-        <parent link="${tf_prefix}/chassis_link"/>
-        <child link="${tf_prefix}/left_wheel_link"/>
+    <joint name="left_wheel_joint" type="continuous">
+        <parent link="chassis_link"/>
+        <child link="left_wheel_link"/>
         <origin xyz= "0 ${wheels_separation / 2.0} ${wheel_vertical_offset}"/>
         <axis xyz="0 1 0"/>
     </joint>
-    <gazebo reference="${tf_prefix}/left_wheel_link">
+    <gazebo reference="left_wheel_link">
         <mu1 value="1.0"/>
         <mu2 value="1.0"/>
@@ -45,7 +45,7 @@
         <kd value="1.0" />
     </gazebo>
-    <xacro:Transmission joint="${tf_prefix}/left_wheel_joint"/>
+    <xacro:Transmission joint="left_wheel_joint"/>
     <!-- right wheel -->
-    <link name="${tf_prefix}/right_wheel_link">
+    <link name="right_wheel_link">
         <visual>
             <origin rpy="0 0 0" xyz="0 0 0"/>
@@ -65,11 +65,11 @@
         </inertial>
     </link>
-    <joint name="${tf_prefix}/right_wheel_joint" type="continuous">
-        <parent link="${tf_prefix}/chassis_link"/>
-        <child link="${tf_prefix}/right_wheel_link"/>
+    <joint name="right_wheel_joint" type="continuous">
+        <parent link="chassis_link"/>
+        <child link="right_wheel_link"/>
         <origin xyz= "0 -${wheels_separation / 2.0} ${wheel_vertical_offset}"/>
         <axis xyz="0 1 0"/>
     </joint>
-    <gazebo reference="${tf_prefix}/right_wheel_link">
+    <gazebo reference="right_wheel_link">
         <mu1 value="1.0"/>
         <mu2 value="1.0"/>
@@ -77,4 +77,4 @@
         <kd value="1.0" />
     </gazebo>
-    <xacro:Transmission joint="${tf_prefix}/right_wheel_joint"/>
+    <xacro:Transmission joint="right_wheel_joint"/>
 </robot>

File: description/urdf/stand_link.urdf.xacro (robot description, xacro)
@@ -6,12 +6,12 @@
     <!-- Stand link; this is a dummy link that is used to make camera placement and other sensors on the stand more convenient -->
     <!-- Stand link definition. Note: purposely left blank -->
-    <link name="${tf_prefix}/stand_link"/>
-    <joint name="${tf_prefix}/stand_link_joint" type="fixed">
-        <parent link="${tf_prefix}/chassis_link"/>
-        <child link="${tf_prefix}/stand_link"/>
+    <link name="stand_link"/>
+    <joint name="stand_link_joint" type="fixed">
+        <parent link="chassis_link"/>
+        <child link="stand_link"/>
         <origin xyz="0 0 ${chassis_to_stand_link_dist}" rpy="0 0 0" />
     </joint>
     <!-- ZED Camera -->
-    <link name="${tf_prefix}/zed_camera_link">
+    <link name="zed_camera_link">
         <visual>
             <origin xyz="0 0 0" rpy="0 0 0"/>
@@ -31,11 +31,11 @@
         </inertial>
     </link>
-    <joint name="${tf_prefix}/zed_camera_joint" type="fixed">
+    <joint name="zed_camera_joint" type="fixed">
         <origin xyz="${stand_length/2 - ZED_camera_width} 0 ${ZED_camera_height / 2.0}" rpy="0 ${ZED_camera_pitch} 0"/>
-        <parent link="${tf_prefix}/stand_link"/>
-        <child link="${tf_prefix}/zed_camera_link"/>
+        <parent link="stand_link"/>
+        <child link="zed_camera_link"/>
     </joint>
     <!-- GPS -->
-    <link name="${tf_prefix}/gps_link">
+    <link name="gps_link">
         <inertial>
             <mass value="${gps_mass}"/>
@@ -56,11 +56,11 @@
     </link>
     <!-- GPS: attach gps_link to stand_link -->
-    <joint name="${tf_prefix}/gps_joint" type="fixed">
-        <parent link="${tf_prefix}/stand_link"/>
-        <child link="${tf_prefix}/gps_link"/>
+    <joint name="gps_joint" type="fixed">
+        <parent link="stand_link"/>
+        <child link="gps_link"/>
         <origin xyz="0 0 ${(gps_length + phidget_height) / 2.0}" rpy="0 0 0"/>
     </joint>
     <!-- IMU -->
-    <link name="${tf_prefix}/imu_link">
+    <link name="imu_link">
         <inertial>
             <mass value="${phidget_mass}"/>
@@ -81,7 +81,7 @@
     </link>
     <!-- IMU: attach imu_link to stand_link -->
-    <joint name="${tf_prefix}/base_link_to_imu_link" type="fixed">
-        <parent link="${tf_prefix}/stand_link"/>
-        <child link="${tf_prefix}/imu_link"/>
+    <joint name="base_link_to_imu_link" type="fixed">
+        <parent link="stand_link"/>
+        <child link="imu_link"/>
         <origin xyz="0 0 0" rpy="0 0 0"/>
     </joint>
@@ -89,5 +89,5 @@
     <!-- NOTE: I'm only defining one and not visually showing any-->
     <!-- I only need one for purposes of using the plugin -->
-    <link name="${tf_prefix}/camera_link">
+    <link name="camera_link">
         <!-- Inertial tag here to ensure that link does not phase through robot-->
         <inertial>
@@ -96,16 +96,16 @@
         </inertial>
     </link>
-    <joint name="${tf_prefix}/zed_camera_link_joint" type="fixed">
+    <joint name="zed_camera_link_joint" type="fixed">
         <origin xyz="${ZED_camera_length/2.0} 0 0" rpy="0 0 0"/>
-        <parent link="${tf_prefix}/zed_camera_link"/>
-        <child link="${tf_prefix}/camera_link"/>
+        <parent link="zed_camera_link"/>
+        <child link="camera_link"/>
     </joint>
     <!-- Generate an optical frame http://www.ros.org/reps/rep-0103.html#suffix-frames so that ros and opencv can operate on the camera frame correctly -->
-    <link name="${tf_prefix}/zed_camera_link_optical"/>
-    <joint name="${tf_prefix}/zed_camera_link_optical_joint" type="fixed">
+    <link name="zed_camera_link_optical"/>
+    <joint name="zed_camera_link_optical_joint" type="fixed">
         <!-- Transform b/w standard and optical frame -->
         <origin xyz="0 0 0" rpy="${-pi/2} 0 ${-pi/2}"/>
-        <parent link="${tf_prefix}/zed_camera_link"/>
-        <child link="${tf_prefix}/zed_camera_link_optical"/>
+        <parent link="zed_camera_link"/>
+        <child link="zed_camera_link_optical"/>
     </joint>
 </robot>
