Commit message: ffffff changed model

File: description/urdf/casters.urdf.xacro (robot description, xacro)
@@ -15,5 +15,5 @@
     -->
     <!-- Front caster definition -->
-    <!-- <link name="front_caster_link">
+    <link name="front_caster_link">
         <visual>
             <origin rpy="0 0 0" xyz="0 0 0"/>
@@ -44,7 +44,7 @@
         <kp value="10000000.0" />
         <kd value="1.0" />
-    </gazebo> -->
+    </gazebo>
     <!-- Front caster wheel definition -->
-    <!-- <link name="front_caster_wheel">
+    <link name="front_caster_wheel">
         <visual>
             <origin rpy="0 0 0" xyz="0 0 0"/>
@@ -75,7 +75,7 @@
         <kp value="10000000.0" />
         <kd value="1.0" />
-    </gazebo> -->
+    </gazebo>
     <!-- Back caster definition -->
-    <link name="back_caster_link">
+    <!-- <link name="back_caster_link">
         <visual>
             <origin rpy="0 0 0" xyz="0 0 0"/>
@@ -106,7 +106,7 @@
         <kp value="10000000.0" />
         <kd value="1.0" />
-    </gazebo>
+    </gazebo> -->
     <!-- Back caster wheel definition -->
-    <link name="back_caster_wheel">
+    <!-- <link name="back_caster_wheel">
         <visual>
             <origin rpy="0 0 0" xyz="0 0 0"/>
@@ -137,4 +137,4 @@
         <kp value="10000000.0" />
         <kd value="1.0" />
-    </gazebo>
+    </gazebo> -->
 </robot>

File: description/urdf/chassis_link.urdf.xacro (robot description, xacro)
@@ -48,5 +48,5 @@
     </link>
     <joint name="battery_joint" type="fixed">
-        <origin xyz="${-1*(stand_length/2 + battery_width + battery_back_offset)} 0 ${wheel_diameter - (3*battery_height/2) - stand_height/2}" rpy="0 0 0"/>
+        <origin xyz="${(stand_length/2 + battery_width + battery_back_offset)} 0 ${wheel_diameter - (3*battery_height/2) - stand_height/2}" rpy="0 0 0"/>
         <parent link="chassis_link"/>
         <child link="battery_link"/>

File: description/urdf/constants.xacro (robot description, xacro)
@@ -11,6 +11,6 @@
     <!-- Stand -->
     <xacro:property name="stand_length" value="0.412"/>
-    <xacro:property name="stand_width" value="0.254"/>
-    <xacro:property name="stand_height" value="1.324"/>
+    <xacro:property name="stand_width" value="0.33"/>
+    <xacro:property name="stand_height" value="1.335"/>
     <xacro:property name="stand_mass" value="1.0"/>
     <!-- Casters -->
@@ -79,5 +79,5 @@
     <xacro:property name="ZED_camera_length" value="0.175"/>
     <xacro:property name="ZED_camera_width" value="0.03"/>
-    <xacro:property name="ZED_camera_height" value="0.033"/>
+    <xacro:property name="ZED_camera_height" value="0.06"/>
     <xacro:property name="ZED_camera_pitch" value="${50 * pi/180}"/>
     <!-- ZED image height/width corresponds to image size for 60Hz refresh-->
@@ -119,3 +119,6 @@
     <xacro:property name="imu_topic" value="imu/data"/>
     <xacro:property name="imu_update_rate" value="128.0"/>
+    <xacro:property name="imu_x_dist" value="0.28"/>
+    <xacro:property name="imu_y_dist" value="0.295"/>
+    <xacro:property name="imu_z_dist" value="0.34"/>
 </robot>

File: description/urdf/stand_link.urdf.xacro (robot description, xacro)
@@ -34,5 +34,5 @@
         <parent link="stand_link"/>
         <child link="gps_link"/>
-        <origin xyz="0 0 ${(gps_length + phidget_height) / 2.0}" rpy="0 0 0"/>
+        <origin xyz="0 0 0" rpy="0 0 0"/>
     </joint>
     <!-- IMU -->
@@ -56,9 +56,9 @@
     </link>
     <joint name="base_link_to_imu_link" type="fixed">
-        <parent link="stand_link"/>
+        <parent link="base_link"/>
         <child link="imu_link"/>
-        <origin xyz="0 0 0" rpy="0 0 0"/>
+        <origin xyz="${imu_x_dist} ${imu_y_dist} ${imu_z_dist}" rpy="0 0 0"/>
     </joint>
-<!-- </robot> -->
+    <!-- </robot> -->
     <!-- ZED Camera -->
     <!-- NOTE: this frame is for convenience, multicamera will use the subsequent left camera frames -->
@@ -84,5 +84,5 @@
         <parent link="stand_link"/>
         <child link="zed_base_link"/>
-        <origin xyz="${stand_length / 2.0 - ZED_camera_width} 0 ${ZED_camera_height / 2.0}" rpy="0 ${ZED_camera_pitch} 0"/>
+        <origin xyz="${0.05 + (stand_width / 2.0) - ZED_camera_width} 0 ${ZED_camera_height / 2.0}" rpy="0 ${ZED_camera_pitch} 0"/>
     </joint>
     <!-- Generate Left Camera frame -->
@@ -96,6 +96,6 @@
     </joint> -->
     <!-- Generate an optical frame http://www.ros.org/reps/rep-0103.html#suffix-frames so that ros and opencv can operate on the camera frame correctly -->
-    <!-- <link name="left_camera_link_optical"/>
-    <joint name="left_camera_link_optical_joint" type="fixed">
+    <!-- <link name="left_camera_link_optical"/> -->
+    <!-- <joint name="left_camera_link_optical_joint" type="fixed">
         <parent link="left_camera_link"/>
         <child link="left_camera_link_optical"/>
