Commit message: All changes for today. Various updates

File: description/urdf/casters_original.urdf.xacro (robot description, xacro)
@@ -62,5 +62,5 @@
     </gazebo>
     <!-- Back caster definition -->
-    <link name="back_caster_link">
+    <!-- <link name="back_caster_link">
         <visual>
             <origin rpy="0 0 0" xyz="0 0 0"/>
@@ -91,5 +91,5 @@
         <kp value="10000000.0" />
         <kd value="1.0" />
-    </gazebo>
+    </gazebo> -->
     <!-- Front caster wheel definition -->
     <link name="front_caster_wheel">
@@ -124,5 +124,5 @@
     </gazebo>
     <!-- Back caster wheel definition -->
-    <link name="back_caster_wheel">
+    <!-- <link name="back_caster_wheel">
         <visual>
             <origin rpy="0 0 0" xyz="0 0 0"/>
@@ -153,4 +153,4 @@
         <kp value="10000000.0" />
         <kd value="1.0" />
-    </gazebo>
+    </gazebo> -->
 </robot>
