Commit message: fixing odom

File: description/urdf/plugins.gazebo.xacro (robot description, xacro)
@@ -77,5 +77,7 @@
             <referenceAltitude>${ref_alt}</referenceAltitude>
             <drift>${gps_drift}</drift> <!-- m -->
+            <gaussianNoise>0.1 0.1 0.1</gaussianNoise>
             <velocityDrift>${gps_vel_drift}</velocityDrift> <!-- m/s-->
+            <velocityGaussianNoise>0.1 0.1 0.1</velocityGaussianNoise>
             <!-- TODO: add Gaussian noise based off Garmin GPS -->
         </plugin>
@@ -144,9 +146,51 @@
                 <frameName>${imu_frame}</frameName>
                 <updateRateHZ>${imu_update_rate}</updateRateHZ>
-                <gaussianNoise>0.0</gaussianNoise>  <!-- TODO: set Gaussian noise based on Phidget IMU -->
+                <gaussianNoise>0.1</gaussianNoise>  <!-- TODO: set Gaussian noise based on Phidget IMU -->
                 <xyzOffset>0 0 0</xyzOffset>
                 <rpyOffset>0 0 0</rpyOffset>
                 <initialOrientationAsReference>false</initialOrientationAsReference>
             </plugin>
+            <imu>
+                <angular_velocity>
+                    <x>
+                        <noise type="gaussian">
+                            <mean>0.0</mean>
+                            <stddev>2e-4</stddev>
+                        </noise>
+                    </x>
+                    <y>
+                        <noise type="gaussian">
+                            <mean>0.0</mean>
+                            <stddev>2e-4</stddev>
+                        </noise>
+                    </y>
+                    <z>
+                        <noise type="gaussian">
+                            <mean>0.0</mean>
+                            <stddev>2e-4</stddev>
+                        </noise>
+                    </z>
+                </angular_velocity>
+                <linear_acceleration>
+                    <x>
+                        <noise type="gaussian">
+                            <mean>0.0</mean>
+                            <stddev>1.7e-2</stddev>
+                        </noise>
+                    </x>
+                    <y>
+                        <noise type="gaussian">
+                            <mean>0.0</mean>
+                            <stddev>1.7e-2</stddev>
+                        </noise>
+                    </y>
+                    <y>
+                        <noise type="gaussian">
+                            <mean>0.0</mean>
+                            <stddev>1.7e-2</stddev>
+                        </noise>
+                    </y>
+                </linear_acceleration>
+            </imu>
             <pose>0 0 0 0 0 0</pose>
         </sensor>

File: description/urdf/stand_link.urdf.xacro (robot description, xacro)
@@ -63,5 +63,5 @@
     <!-- ZED Camera -->
     <!-- NOTE: this frame is for convenience, multicamera will use the subsequent left camera frames -->
-    <link name="zed_base_link">
+    <link name="zed_camera_link">
         <visual>
             <origin xyz="0 0 0" rpy="0 0 0"/>
@@ -83,5 +83,5 @@
     <joint name="zed_camera_joint" type="fixed">
         <parent link="stand_link"/>
-        <child link="zed_base_link"/>
+        <child link="zed_camera_link"/>
         <origin xyz="${0.05 + (stand_width / 2.0) - ZED_camera_width} 0 ${ZED_camera_height / 2.0}" rpy="0 ${ZED_camera_pitch} 0"/>
     </joint>
@@ -89,16 +89,16 @@
     <!-- NOTE: specify frame of left camera (lens) because right one is specified relative to it by the multicamera plugin -->
     <!-- NOTE: we are assuming the lens are located at the edges of the camera (hence the use of 'camera_length' and not a 'stereo_offset') -->
-    <!-- <link name="left_camera_link"/> -->
-    <!-- <joint name="left_camera_link_joint" type="fixed">
-        <parent link="zed_base_link"/>
+    <link name="left_camera_link"/>
+    <joint name="left_camera_link_joint" type="fixed">
+        <parent link="zed_camera_link"/>
         <child link="left_camera_link"/>
         <origin xyz="0 ${ZED_camera_length / 2.0} 0" rpy="0 0 0"/>
-    </joint> -->
+    </joint>
     <!-- Generate an optical frame http://www.ros.org/reps/rep-0103.html#suffix-frames so that ros and opencv can operate on the camera frame correctly -->
-    <!-- <link name="left_camera_link_optical"/> -->
-    <!-- <joint name="left_camera_link_optical_joint" type="fixed">
+    <link name="left_camera_link_optical"/>
+    <joint name="left_camera_link_optical_joint" type="fixed">
         <parent link="left_camera_link"/>
         <child link="left_camera_link_optical"/>
         <origin xyz="0 0 0" rpy="${-pi/2} 0 ${-pi/2}"/>
-    </joint> -->
+    </joint>
 </robot>
