Commit message: Big messy commit for hardware integration.
Added motor odometry.
Added motor feedback loop.
Integrated teleop override of nav_stack.
Fixed rosserial issues.
Added testing launch scripts.
Fixed build error with VL.

File: description/urdf/stand_link.urdf.xacro (robot description, xacro)
@@ -60,7 +60,8 @@
         <origin xyz="0 0 0" rpy="0 0 0"/>
     </joint>
+<!-- </robot> -->
     <!-- ZED Camera -->
     <!-- NOTE: this frame is for convenience, multicamera will use the subsequent left camera frames -->
-    <link name="zed_camera_link">
+    <link name="zed_base_link">
         <visual>
             <origin xyz="0 0 0" rpy="0 0 0"/>
@@ -82,5 +83,5 @@
     <joint name="zed_camera_joint" type="fixed">
         <parent link="stand_link"/>
-        <child link="zed_camera_link"/>
+        <child link="zed_base_link"/>
         <origin xyz="${stand_length / 2.0 - ZED_camera_width} 0 ${ZED_camera_height / 2.0}" rpy="0 ${ZED_camera_pitch} 0"/>
     </joint>
@@ -88,16 +89,16 @@
     <!-- NOTE: specify frame of left camera (lens) because right one is specified relative to it by the multicamera plugin -->
     <!-- NOTE: we are assuming the lens are located at the edges of the camera (hence the use of 'camera_length' and not a 'stereo_offset') -->
-    <link name="left_camera_link"/>
-    <joint name="left_camera_link_joint" type="fixed">
-        <parent link="zed_camera_link"/>
+    <!-- <link name="left_camera_link"/> -->
+    <!-- <joint name="left_camera_link_joint" type="fixed">
+        <parent link="zed_base_link"/>
         <child link="left_camera_link"/>
         <origin xyz="0 ${ZED_camera_length / 2.0} 0" rpy="0 0 0"/>
-    </joint>
+    </joint> -->
     <!-- Generate an optical frame http://www.ros.org/reps/rep-0103.html#suffix-frames so that ros and opencv can operate on the camera frame correctly -->
-    <link name="left_camera_link_optical"/>
+    <!-- <link name="left_camera_link_optical"/>
     <joint name="left_camera_link_optical_joint" type="fixed">
         <parent link="left_camera_link"/>
         <child link="left_camera_link_optical"/>
         <origin xyz="0 0 0" rpy="${-pi/2} 0 ${-pi/2}"/>
-    </joint>
+    </joint> -->
 </robot>

Commit message: cv topic changes frame set for ros

File: description/urdf/stand_link.urdf.xacro (robot description, xacro)
@@ -60,8 +60,8 @@
         <origin xyz="0 0 0" rpy="0 0 0"/>
     </joint>
-<!-- </robot> -->
+    <!-- </robot> -->
     <!-- ZED Camera -->
     <!-- NOTE: this frame is for convenience, multicamera will use the subsequent left camera frames -->
-    <link name="zed_base_link">
+    <link name="zed_camera_link">
         <visual>
             <origin xyz="0 0 0" rpy="0 0 0"/>
@@ -83,5 +83,5 @@
     <joint name="zed_camera_joint" type="fixed">
         <parent link="stand_link"/>
-        <child link="zed_base_link"/>
+        <child link="zed_camera_link"/>
         <origin xyz="${stand_length / 2.0 - ZED_camera_width} 0 ${ZED_camera_height / 2.0}" rpy="0 ${ZED_camera_pitch} 0"/>
     </joint>
@@ -89,16 +89,16 @@
     <!-- NOTE: specify frame of left camera (lens) because right one is specified relative to it by the multicamera plugin -->
     <!-- NOTE: we are assuming the lens are located at the edges of the camera (hence the use of 'camera_length' and not a 'stereo_offset') -->
-    <!-- <link name="left_camera_link"/> -->
-    <!-- <joint name="left_camera_link_joint" type="fixed">
-        <parent link="zed_base_link"/>
+    <link name="left_camera_link"/>
+    <joint name="left_camera_link_joint" type="fixed">
+        <parent link="zed_camera_link"/>
         <child link="left_camera_link"/>
         <origin xyz="0 ${ZED_camera_length / 2.0} 0" rpy="0 0 0"/>
-    </joint> -->
+    </joint>
     <!-- Generate an optical frame http://www.ros.org/reps/rep-0103.html#suffix-frames so that ros and opencv can operate on the camera frame correctly -->
-    <!-- <link name="left_camera_link_optical"/>
+    <link name="left_camera_link_optical"/>
     <joint name="left_camera_link_optical_joint" type="fixed">
         <parent link="left_camera_link"/>
         <child link="left_camera_link_optical"/>
         <origin xyz="0 0 0" rpy="${-pi/2} 0 ${-pi/2}"/>
-    </joint> -->
+    </joint>
 </robot>

Commit message: merge ready for IGVC branch

File: description/urdf/stand_link.urdf.xacro (robot description, xacro)
@@ -63,5 +63,5 @@
     <!-- ZED Camera -->
     <!-- NOTE: this frame is for convenience, multicamera will use the subsequent left camera frames -->
-    <link name="zed_camera_link">
+    <link name="zed_base_link">
         <visual>
             <origin xyz="0 0 0" rpy="0 0 0"/>
@@ -83,5 +83,5 @@
     <joint name="zed_camera_joint" type="fixed">
         <parent link="stand_link"/>
-        <child link="zed_camera_link"/>
+        <child link="zed_base_link"/>
         <origin xyz="${0.05 + (stand_width / 2.0) - ZED_camera_width} 0 ${ZED_camera_height / 2.0}" rpy="0 ${ZED_camera_pitch} 0"/>
     </joint>
@@ -89,16 +89,16 @@
     <!-- NOTE: specify frame of left camera (lens) because right one is specified relative to it by the multicamera plugin -->
     <!-- NOTE: we are assuming the lens are located at the edges of the camera (hence the use of 'camera_length' and not a 'stereo_offset') -->
-    <link name="left_camera_link"/>
-    <joint name="left_camera_link_joint" type="fixed">
-        <parent link="zed_camera_link"/>
+    <!-- <link name="left_camera_link"/> -->
+    <!-- <joint name="left_camera_link_joint" type="fixed">
+        <parent link="zed_base_link"/>
         <child link="left_camera_link"/>
         <origin xyz="0 ${ZED_camera_length / 2.0} 0" rpy="0 0 0"/>
-    </joint>
+    </joint> -->
     <!-- Generate an optical frame http://www.ros.org/reps/rep-0103.html#suffix-frames so that ros and opencv can operate on the camera frame correctly -->
-    <link name="left_camera_link_optical"/>
-    <joint name="left_camera_link_optical_joint" type="fixed">
+    <!-- <link name="left_camera_link_optical"/> -->
+    <!-- <joint name="left_camera_link_optical_joint" type="fixed">
         <parent link="left_camera_link"/>
         <child link="left_camera_link_optical"/>
         <origin xyz="0 0 0" rpy="${-pi/2} 0 ${-pi/2}"/>
-    </joint>
+    </joint> -->
 </robot>

Commit message: revert unneeded things

File: description/urdf/stand_link.urdf.xacro (robot description, xacro)
@@ -63,5 +63,5 @@
     <!-- ZED Camera -->
     <!-- NOTE: this frame is for convenience, multicamera will use the subsequent left camera frames -->
-    <link name="zed_camera_link">
+    <link name="zed_base_link">
         <visual>
             <origin xyz="0 0 0" rpy="0 0 0"/>
@@ -83,5 +83,5 @@
     <joint name="zed_camera_joint" type="fixed">
         <parent link="stand_link"/>
-        <child link="zed_camera_link"/>
+        <child link="zed_base_link"/>
         <origin xyz="${0.05 + (stand_width / 2.0) - ZED_camera_width} 0 ${ZED_camera_height / 2.0}" rpy="0 ${ZED_camera_pitch} 0"/>
     </joint>
@@ -89,16 +89,16 @@
     <!-- NOTE: specify frame of left camera (lens) because right one is specified relative to it by the multicamera plugin -->
     <!-- NOTE: we are assuming the lens are located at the edges of the camera (hence the use of 'camera_length' and not a 'stereo_offset') -->
-    <link name="left_camera_link"/>
+    <!-- <link name="left_camera_link"/>
     <joint name="left_camera_link_joint" type="fixed">
-        <parent link="zed_camera_link"/>
+        <parent link="zed_base_link"/>
         <child link="left_camera_link"/>
         <origin xyz="0 ${ZED_camera_length / 2.0} 0" rpy="0 0 0"/>
-    </joint>
+    </joint> -->
     <!-- Generate an optical frame http://www.ros.org/reps/rep-0103.html#suffix-frames so that ros and opencv can operate on the camera frame correctly -->
-    <link name="left_camera_link_optical"/>
+    <!-- <link name="left_camera_link_optical"/>
     <joint name="left_camera_link_optical_joint" type="fixed">
         <parent link="left_camera_link"/>
         <child link="left_camera_link_optical"/>
         <origin xyz="0 0 0" rpy="${-pi/2} 0 ${-pi/2}"/>
-    </joint>
+    </joint> -->
 </robot>

Commit message: Vl cv integration (#122)
* Not working code based on simple layer tutorials

* Able to write obstacles to local costmap

* I broke simple_layers.cpp

* it works

* remove useless variables

* python to C++

* int to double

* separated function

* offset to 4,4

* fixed random function & reduced spacing btw points

* temp

* pull caff-57

* local to global

* 10sec delay before next set of points

* published dummy topic, not yet subscribed by virtual layer

* testing subscriber in virtual layer

* michael temp com

* temp comm

* remove nonfunctional subscriber from virtual layer

* fixed layer

* michael save

* Initial commit for CV wrapper.
    Loads in random test image from disk. Runs image preprocessing, loads in cv .onnx model, and runs a profile on inference speeds.
    Next commit will aim to integrate with ros nodes, subscribe to camera to load image and publish to a nav friendly format.

* Updatedd code - still not working

* Got inference working.

Left to do:
- Interface on both ends with ROS. Subscribe to ZED node to get images and publish results

* basic ros node skeleton & cleaning up inference code

* Able to get images from rviz

* deleted old model wrapper file

* removed local filepath from launch file

* added basic instructions to install onnxruntime, need to expand later

* minor cleanup in post process function

* cleaned up constructor code a bit

* made node handle private to allow params be accessible

* fixed gitignore end of line

* removed cv gitignore

* deleted unnecessary comments in package.xml

* fixed formatting in lane_detection_inference_node's constructor

* Added instructions to readme

* Update README.md

* Added zed wrapper

* Removed zed wrapper code - to add as submodule

* Added zed wrapper as submodule

* Overloaded cpp cv pipeline for python varient. Runs using communication to python3 inference using redis. Removes dependancy for onnxruntime built from scratch on arm.

Launch using roslaunch lane_detection lane_detection_server.launch

* added some cv code; currently not working

* added helper scripts in scripts folder

* Added 3D projection. Publishing to rostopic /cv/lane_detection. Does not include tf transforms yet, untested with rviz

* kj wants me to show caff-80 so pause here

* fixing vl

* Added default z mapping

* Added relative imports for script

* VL issue was offset and global var

* merge master

* cleanup

* return cv/lanes

* Finished lane detection. Refactored cv pipeline to allow for easy addition of pothole detection

* updated Readme

* Added new line (for Michael)

* Removed unused code

* Added comment for future todo

* Changed camera projection code to use zed parameters. Added checks full null data read - occurs when FPS drops below FPS set by ros.

* Removed unused files

* temp save

* Added checks for NoneType thoruhg redis. Added publishing of raw model output to topic cv/model/output

* I think it works, but cv/ros did diff frame definitions

* figured out cv transform I think, but cv revieweing their work

* left camera optical frame not just offset of zed frame so prev trans def wrong

* Updating and clean-up of functions

* Minor correction

* Preliminary (non-working) pothole detection pipeline

* Scaling camera intrinsics to accommodate resized images

* Got valid outputs + thresholding

* Reformatted, working.

* Correcting some inputs of the lane fit functions

* added unexplained x2 and +190/+80 xy offsets

* Added scaling of intrinsics. Fixed previous commit bugs

* fixed left/camera_info topic name again

* Added working pothole detection code!

* Fixed projection errors.

* testing ivy's changes

* remove cv_points clearing. Will need to combine similar points

* giant pink blobs

* kj's comments

* Caff 88b (#116)

* ffffff changed model

* change imu z dist

* saving progress, probably broken

* ffffff temp pause

* ffffff temp pausev2

* need to tune but it works

* update threshold

* imu local making issues, and idk why so coment out

* the freaking global costmap moves with me, so need to do save dict instead of set and deduct xy

* saving work

* builds but useless

* rotation is wrong...

* minor cleanup

* fff

* cleaner

* newer update

* global costmap is map frame translated to robot center...

* had to reset costmap. It works now with small probabilities

* merge ready for IGVC branch

* created local/global vl layers separately

* fixing odom

* revert unneeded things

Co-authored-by: kajananchinniah <kajananchinniah@gmail.com>
Co-authored-by: Jimin Kwon <kishyaut@gmail.com>
Co-authored-by: Spencer Teetaert <erickmu1@hotmail.com>
Co-authored-by: Spencer Teetaert <spencerteetaert@gmail.com>
Co-authored-by: Spencer Teetaert <45899408+spencerteetaert@users.noreply.github.com>
Co-authored-by: Jason-Y000 <57577805+Jason-Y000@users.noreply.github.com>

File: description/urdf/stand_link.urdf.xacro (robot description, xacro)
@@ -89,6 +89,6 @@
     <!-- NOTE: specify frame of left camera (lens) because right one is specified relative to it by the multicamera plugin -->
     <!-- NOTE: we are assuming the lens are located at the edges of the camera (hence the use of 'camera_length' and not a 'stereo_offset') -->
-    <!-- <link name="left_camera_link"/> -->
-    <!-- <joint name="left_camera_link_joint" type="fixed">
+    <!-- <link name="left_camera_link"/>
+    <joint name="left_camera_link_joint" type="fixed">
         <parent link="zed_base_link"/>
         <child link="left_camera_link"/>
@@ -96,6 +96,6 @@
     </joint> -->
     <!-- Generate an optical frame http://www.ros.org/reps/rep-0103.html#suffix-frames so that ros and opencv can operate on the camera frame correctly -->
-    <!-- <link name="left_camera_link_optical"/> -->
-    <!-- <joint name="left_camera_link_optical_joint" type="fixed">
+    <!-- <link name="left_camera_link_optical"/>
+    <joint name="left_camera_link_optical_joint" type="fixed">
         <parent link="left_camera_link"/>
         <child link="left_camera_link_optical"/>

Commit message: lane detection works with sim

File: description/urdf/stand_link.urdf.xacro (robot description, xacro)
@@ -89,16 +89,16 @@
     <!-- NOTE: specify frame of left camera (lens) because right one is specified relative to it by the multicamera plugin -->
     <!-- NOTE: we are assuming the lens are located at the edges of the camera (hence the use of 'camera_length' and not a 'stereo_offset') -->
-    <!-- <link name="left_camera_link"/> -->
-    <!-- <joint name="left_camera_link_joint" type="fixed">
+    <link name="left_camera_link"/>
+    <joint name="left_camera_link_joint" type="fixed">
         <parent link="zed_base_link"/>
         <child link="left_camera_link"/>
         <origin xyz="0 ${ZED_camera_length / 2.0} 0" rpy="0 0 0"/>
-    </joint> -->
+    </joint>
     <!-- Generate an optical frame http://www.ros.org/reps/rep-0103.html#suffix-frames so that ros and opencv can operate on the camera frame correctly -->
-    <!-- <link name="left_camera_link_optical"/> -->
-    <!-- <joint name="left_camera_link_optical_joint" type="fixed">
+    <link name="left_camera_link_optical"/>
+    <joint name="left_camera_link_optical_joint" type="fixed">
         <parent link="left_camera_link"/>
         <child link="left_camera_link_optical"/>
         <origin xyz="0 0 0" rpy="${-pi/2} 0 ${-pi/2}"/>
-    </joint> -->
+    </joint>
 </robot>
