Commit message: battery changes

File: description/urdf/chassis_link.urdf.xacro (robot description, xacro)
@@ -23,3 +23,27 @@
         </inertial>
     </link>
+    <!-- Battery Link -->
+    <link name="${tf_prefix}/battery_link">
+        <visual>
+            <origin xyz="0 0 0" rpy="0 0 0"/>
+            <geometry>
+                <box size="${battery_width} ${battery_length} ${battery_height}"/>
+            </geometry>
+        </visual>
+        <collision>
+            <origin xyz="0 0 0" rpy="0 0 0"/>
+            <geometry>
+                <box size="${battery_width} ${battery_length} ${battery_height}"/>
+            </geometry>
+        </collision>
+        <inertial>
+            <xacro:box_inertia mass="${battery_mass}" length="${battery_length}" width="${battery_width}" height="${battery_height}"/>
+            <mass value="${battery_mass}"/>
+        </inertial>
+    </link>
+    <joint name="${tf_prefix}/battery_joint" type="fixed">
+        <origin xyz="${-1*(stand_length/2 + battery_width + battery_back_offset)} 0 ${wheel_diameter - (3*battery_height/2) - stand_height/2}" rpy="0 0 0"/>
+        <parent link="${tf_prefix}/chassis_link"/>
+        <child link="${tf_prefix}/battery_link"/>
+    </joint>
 </robot>

File: description/urdf/stand_link.urdf.xacro (robot description, xacro)
@@ -7,28 +7,4 @@
     <!-- Stand link definition. Note: purposely left blank -->
     <link name="${tf_prefix}/stand_link"/>
-    <!-- Battery Link -->
-    <link name="${tf_prefix}/battery_link">
-        <visual>
-            <origin xyz="0 0 0" rpy="0 0 0"/>
-            <geometry>
-                <box size="${battery_width} ${battery_length} ${battery_height}"/>
-            </geometry>
-        </visual>
-        <collision>
-            <origin xyz="0 0 0" rpy="0 0 0"/>
-            <geometry>
-                <box size="${battery_width} ${battery_length} ${battery_height}"/>
-            </geometry>
-        </collision>
-        <inertial>
-            <xacro:box_inertia mass="${battery_mass}" length="${battery_length}" width="${battery_width}" height="${battery_height}"/>
-            <mass value="${battery_mass}"/>
-        </inertial>
-    </link>
-    <joint name="${tf_prefix}/battery_joint" type="fixed">
-        <origin xyz="${-1*(stand_length/2 + battery_width + battery_back_offset)} 0 ${wheel_diameter - (3*battery_height/2) - stand_height/2}" rpy="0 0 0"/>
-        <parent link="${tf_prefix}/chassis_link"/>
-        <child link="${tf_prefix}/battery_link"/>
-    </joint>
     <!-- ZED Camera -->
     <link name="${tf_prefix}/zed_camera_link">

Commit message: Changed chassis model and WIP of changing model of lanes

File: description/urdf/chassis_link.urdf.xacro (robot description, xacro)
@@ -9,5 +9,5 @@
             <origin rpy="0 0 0" xyz="0 0 0"/>
             <geometry>
-                <mesh filename="package://description/urdf/meshes/chassis_link.dae"/>
+                <mesh filename="package://description/urdf/meshes/chassis_link_new.dae"/>
             </geometry>
         </visual>
@@ -15,5 +15,5 @@
             <origin rpy="0 0 0" xyz="0 0 0"/>
             <geometry>
-                <mesh filename="package://description/urdf/meshes/chassis_link.dae"/>
+                <mesh filename="package://description/urdf/meshes/chassis_link_new.dae"/>
             </geometry>
         </collision>

File: description/urdf/constants.xacro (robot description, xacro)
@@ -6,7 +6,7 @@
     <xacro:property name="base_height" value="0.01"/>
     <!-- Chassis -->
-    <xacro:property name="chassis_to_base_link_dist" value="0.74424"/>
-    <xacro:property name="chassis_to_stand_link_dist" value="1.0357"/>
-    <xacro:property name="chassis_link_mass" value="32.46"/>
+    <xacro:property name="chassis_to_base_link_dist" value="0.501747"/>
+    <xacro:property name="chassis_to_stand_link_dist" value="0.428526"/>
+    <xacro:property name="chassis_link_mass" value="36.95"/>
     <!-- Stand -->
     <xacro:property name="stand_length" value="0.412"/>

File: description/urdf/inertias.xacro (robot description, xacro)
@@ -4,7 +4,7 @@
     <xacro:macro name="chassis_link_inertia">
         <inertia
-            ixx="21.200" ixy="0.000" ixz="0.0000"
-            iyx="0.0000" iyy="21.230" iyz="0.0000"
-            izx="0.0000" izy="0.0000" izz="2.2600"
+            ixx="13.1600" ixy="0.0000" ixz="0.0000"
+            iyx="0.0000" iyy="11.7000" iyz="0.0000"
+            izx="0.0000" izy="0.0000" izz="2.6800"
         />
     </xacro:macro>
@@ -25,5 +25,5 @@
         />
     </xacro:macro>
-    <!-- Cynlinder Inertia -->
+    <!-- Cylinder Inertia -->
     <xacro:macro name="cylinder_inertia" params="mass length radius">
         <inertia
