Commit message: move base_laser to caffeine urdf

File: description/urdf/caffeine.urdf.xacro (robot description, xacro)
@@ -15,4 +15,26 @@
     <xacro:include filename="$(find description)/urdf/casters.urdf.xacro"/>
     <!-- base_laser: LIDAR at front of Caffeine -->
-    <xacro:include filename="$(find description)/urdf/base_laser.urdf.xacro"/>
+    <link name="${tf_prefix}/base_laser">
+        <inertial>
+            <mass value="${laser_mass}"/>
+            <xacro:box_inertia mass="${laser_mass}" length="${laser_length}" width="${laser_width}" height="${laser_height}"/>
+        </inertial>
+        <visual>
+            <origin xyz="0 0 0" rpy="0 0 0"/>
+            <geometry>
+            <mesh filename="package://description/urdf/meshes/hokuyo.dae"/>
+            </geometry>
+        </visual>
+        <collision>
+            <origin xyz="0 0 0" rpy="0 0 0"/>
+            <geometry>
+            <mesh filename="package://description//urdf/meshes/hokuyo.dae"/>
+            </geometry>
+        </collision>
+    </link>
+    <joint name="${tf_prefix}/base_laser_joint" type="fixed">
+        <parent link="${tf_prefix}/base_link"/>
+        <child link="${tf_prefix}/base_laser"/>
+        <origin xyz="${laser_x_dist} 0 ${laser_z_dist}" rpy="0 0 0"/>
+    </joint>
 </robot>

Commit message: Corrected how links where created for the Gazebo stereo camera plugin. Renamed caffeine.gazebo to plugins.gazebo and made some minor edits

File: description/urdf/caffeine.urdf.xacro (robot description, xacro)
@@ -3,5 +3,5 @@
     <!-- Includes -->
     <xacro:include filename="$(find description)/urdf/constants.xacro"/>
-    <xacro:include filename="$(find description)/urdf/caffeine.gazebo.xacro"/>
+    <xacro:include filename="$(find description)/urdf/plugins.gazebo.xacro"/>
     <!-- base_link: origin of the robot; located in the middle, on the top of the base plate -->
     <link name="base_link"/>

File: description/urdf/constants.xacro (robot description, xacro)
@@ -95,5 +95,5 @@
     <xacro:property name="ZED_depth_info_topicName" value="depth/camera_info"/>
     <xacro:property name="ZED_depth_points_topicName" value="depth/points"/>
-    <xacro:property name="ZED_frameName" value="zed_camera_link_optical"/>
+    <xacro:property name="ZED_frameName" value="left_camera_link_optical"/>
     <!-- Garmin GPS -->
     <!-- NOTE: approx. as a cylinder, Garmin itself is similar to a hockey puck -->

File: description/urdf/plugins.gazebo.xacro (robot description, xacro)
@@ -1,4 +1,4 @@
 <?xml version="1.0"?>
-<robot name="caffeine_sim" xmlns:xacro="http://ros.org/wiki/xacro">
+<robot name="plugins" xmlns:xacro="http://ros.org/wiki/xacro">
     <!-- Constants -->
     <xacro:include filename="$(find description)/urdf/constants.xacro"/>
@@ -82,5 +82,5 @@
     </gazebo>
     <!-- Gazebo multicamera plugin -->
-    <gazebo reference="camera_link">
+    <gazebo reference="left_camera_link">
         <sensor type="multicamera" name="stereo_camera">
             <update_rate>${ZED_image_refresh}</update_rate>
@@ -98,5 +98,5 @@
             </camera>
             <camera name="right">
-            <pose>0 ${-ZED_camera_length} 0 0 0 0</pose>
+            <pose>0 -${ZED_camera_length} 0 0 0 0</pose>
             <horizontal_fov>${ZED_image_hfov}</horizontal_fov>
             <image>

File: description/urdf/stand_link.urdf.xacro (robot description, xacro)
@@ -11,28 +11,4 @@
         <child link="stand_link"/>
         <origin xyz="0 0 ${chassis_to_stand_link_dist}" rpy="0 0 0" />
-    </joint>
-    <!-- ZED Camera -->
-    <link name="zed_camera_link">
-        <visual>
-            <origin xyz="0 0 0" rpy="0 0 0"/>
-            <geometry>
-                <box size="${ZED_camera_width} ${ZED_camera_length} ${ZED_camera_height}"/>
-            </geometry>
-        </visual>
-        <collision>
-            <origin xyz="0 0 0" rpy="0 0 0"/>
-            <geometry>
-                <box size="${ZED_camera_width} ${ZED_camera_length} ${ZED_camera_height}"/>
-            </geometry>
-        </collision>
-        <inertial>
-            <xacro:box_inertia mass="${ZED_camera_mass}" length="${ZED_camera_length}" width="${ZED_camera_width}" height="${ZED_camera_height}"/>
-            <mass value="${ZED_camera_mass}"/>
-        </inertial>
-    </link>
-    <joint name="zed_camera_joint" type="fixed">
-        <origin xyz="${stand_length/2 - ZED_camera_width} 0 ${ZED_camera_height / 2.0}" rpy="0 ${ZED_camera_pitch} 0"/>
-        <parent link="stand_link"/>
-        <child link="zed_camera_link"/>
     </joint>
     <!-- GPS -->
@@ -55,5 +31,4 @@
         </collision>
     </link>
-    <!-- GPS: attach gps_link to stand_link -->
     <joint name="gps_joint" type="fixed">
         <parent link="stand_link"/>
@@ -80,5 +55,4 @@
         </collision>
     </link>
-    <!-- IMU: attach imu_link to stand_link -->
     <joint name="base_link_to_imu_link" type="fixed">
         <parent link="stand_link"/>
@@ -86,26 +60,44 @@
         <origin xyz="0 0 0" rpy="0 0 0"/>
     </joint>
-    <!-- ZED camera lenses -->
-    <!-- NOTE: I'm only defining one and not visually showing any-->
-    <!-- I only need one for purposes of using the plugin -->
-    <link name="camera_link">
-        <!-- Inertial tag here to ensure that link does not phase through robot-->
+    <!-- ZED Camera -->
+    <!-- NOTE: this frame is for convenience, multicamera will use the subsequent left camera frames -->
+    <link name="zed_camera_link">
+        <visual>
+            <origin xyz="0 0 0" rpy="0 0 0"/>
+            <geometry>
+                <box size="${ZED_camera_width} ${ZED_camera_length} ${ZED_camera_height}"/>
+            </geometry>
+        </visual>
+        <collision>
+            <origin xyz="0 0 0" rpy="0 0 0"/>
+            <geometry>
+                <box size="${ZED_camera_width} ${ZED_camera_length} ${ZED_camera_height}"/>
+            </geometry>
+        </collision>
         <inertial>
-            <mass value="0.0001"/>
-            <inertia ixx="0.0001" ixy="0" ixz="0" iyy="0.0001" iyz="0" izz="0.00001"/>
+            <xacro:box_inertia mass="${ZED_camera_mass}" length="${ZED_camera_length}" width="${ZED_camera_width}" height="${ZED_camera_height}"/>
+            <mass value="${ZED_camera_mass}"/>
         </inertial>
     </link>
-    <joint name="zed_camera_link_joint" type="fixed">
-        <origin xyz="${ZED_camera_length/2.0} 0 0" rpy="0 0 0"/>
+    <joint name="zed_camera_joint" type="fixed">
+        <parent link="stand_link"/>
+        <child link="zed_camera_link"/>
+        <origin xyz="${stand_length / 2.0 - ZED_camera_width} 0 ${ZED_camera_height / 2.0}" rpy="0 ${ZED_camera_pitch} 0"/>
+    </joint>
+    <!-- Generate Left Camera frame -->
+    <!-- NOTE: specify frame of left camera (lens) because right one is specified relative to it by the multicamera plugin -->
+    <!-- NOTE: we are assuming the lens are located at the edges of the camera (hence the use of 'camera_length' and not a 'stereo_offset') -->
+    <link name="left_camera_link"/>
+    <joint name="left_camera_link_joint" type="fixed">
         <parent link="zed_camera_link"/>
-        <child link="camera_link"/>
+        <child link="left_camera_link"/>
+        <origin xyz="0 ${ZED_camera_length / 2.0} 0" rpy="0 0 0"/>
     </joint>
     <!-- Generate an optical frame http://www.ros.org/reps/rep-0103.html#suffix-frames so that ros and opencv can operate on the camera frame correctly -->
-    <link name="zed_camera_link_optical"/>
-    <joint name="zed_camera_link_optical_joint" type="fixed">
-        <!-- Transform b/w standard and optical frame -->
+    <link name="left_camera_link_optical"/>
+    <joint name="left_camera_link_optical_joint" type="fixed">
+        <parent link="left_camera_link"/>
+        <child link="left_camera_link_optical"/>
         <origin xyz="0 0 0" rpy="${-pi/2} 0 ${-pi/2}"/>
-        <parent link="zed_camera_link"/>
-        <child link="zed_camera_link_optical"/>
     </joint>
 </robot>

Commit message: CAFF-54 - Repo Cleanup (#60)
* folder changes

* battery changes

* Moved joint definition to inside their respective files

* deal with to do

* indenc local_costmap_params.yaml

* add comment

* spacing

* move base_laser to caffeine urdf

* remove caffeine namespace everywhere

* IGVC worlds installation instructions on README + install_models.sh can be ran from any directory

* Split caffeine_gazebo into simulate and spawn. caffeine_rviz now just view. twist_mux renamed key_vel to man_vel

* Corrected how links where created for the Gazebo stereo camera plugin. Renamed caffeine.gazebo to plugins.gazebo and made some minor edits

* Removed keyboard teleop from move_base and instead left a todo (since will use rqt_steer for manual control)

* Missing new line for move_base

* remove useless comment

* re-add keyboard teleop twist mux topic

Co-authored-by: kajananchinniah <kajananchinniah@gmail.com>
Co-authored-by: Erick Mejia Uzeda <erickmu1@hotmail.com>

File: description/urdf/caffeine.urdf.xacro (robot description, xacro)
@@ -3,31 +3,38 @@
     <!-- Includes -->
     <xacro:include filename="$(find description)/urdf/constants.xacro"/>
-    <xacro:include filename="$(find description)/urdf/caffeine.gazebo.xacro"/>
+    <xacro:include filename="$(find description)/urdf/plugins.gazebo.xacro"/>
     <!-- base_link: origin of the robot; located in the middle, on the top of the base plate -->
-    <link name="${tf_prefix}/base_link"/>
+    <link name="base_link"/>
     <!-- chassis_link: geometric center of the robot; used as the parent in which all other links connect to -->
     <xacro:include filename="$(find description)/urdf/chassis_link.urdf.xacro"/>
-    <joint name="${tf_prefix}/chassis_link_joint" type="fixed">
-        <parent link="${tf_prefix}/base_link"/>
-        <child link="${tf_prefix}/chassis_link"/>
-        <origin xyz="0 0 ${chassis_to_base_link_dist}" rpy="0 0 0"/>
-    </joint>
     <!-- stand_link: origin for anything on the stand; located in the middle, on the top of the stand plate -->
     <xacro:include filename="$(find description)/urdf/stand_link.urdf.xacro"/>
-    <joint name="${tf_prefix}/stand_link_joint" type="fixed">
-        <parent link="${tf_prefix}/chassis_link"/>
-        <child link="${tf_prefix}/stand_link"/>
-        <origin xyz="0 0 ${chassis_to_stand_link_dist}" rpy="0 0 0" />
-    </joint>
     <!-- wheels: associated to wheels that can be moved by a motor -->
     <xacro:include filename="$(find description)/urdf/side_wheels.urdf.xacro"/>
     <!-- wheels: front and back casters -->
     <xacro:include filename="$(find description)/urdf/casters.urdf.xacro"/>
-   <!-- base_laser: LIDAR at front of Caffeine -->
-   <xacro:include filename="$(find description)/urdf/base_laser.urdf.xacro"/>
-   <joint name="${tf_prefix}/base_laser_joint" type="fixed">
-        <parent link="${tf_prefix}/base_link"/>
-        <child link="${tf_prefix}/base_laser"/>
+    <!-- base_laser: LIDAR at front of Caffeine -->
+    <link name="base_laser">
+        <inertial>
+            <mass value="${laser_mass}"/>
+            <xacro:box_inertia mass="${laser_mass}" length="${laser_length}" width="${laser_width}" height="${laser_height}"/>
+        </inertial>
+        <visual>
+            <origin xyz="0 0 0" rpy="0 0 0"/>
+            <geometry>
+            <mesh filename="package://description/urdf/meshes/hokuyo.dae"/>
+            </geometry>
+        </visual>
+        <collision>
+            <origin xyz="0 0 0" rpy="0 0 0"/>
+            <geometry>
+            <mesh filename="package://description//urdf/meshes/hokuyo.dae"/>
+            </geometry>
+        </collision>
+    </link>
+    <joint name="base_laser_joint" type="fixed">
+        <parent link="base_link"/>
+        <child link="base_laser"/>
         <origin xyz="${laser_x_dist} 0 ${laser_z_dist}" rpy="0 0 0"/>
-   </joint>
+    </joint>
 </robot>

File: description/urdf/constants.xacro (robot description, xacro)
@@ -1,11 +1,8 @@
 <?xml version="1.0"?>
 <robot name="caffeine_constants" xmlns:xacro="http://ros.org/wiki/xacro">
-    <!-- Caffeine -->
-    <xacro:property name="robotNamespace" value="caffeine"/>
-    <xacro:property name="tf_prefix" value="caffeine"/>
     <!-- Drivebase -->
-   <xacro:property name="base_length" value="1.268"/>
-   <xacro:property name="base_width" value="0.764"/>
-   <xacro:property name="base_height" value="0.01"/>
+    <xacro:property name="base_length" value="1.268"/>
+    <xacro:property name="base_width" value="0.764"/>
+    <xacro:property name="base_height" value="0.01"/>
     <!-- Chassis -->
     <xacro:property name="chassis_to_base_link_dist" value="0.501747"/>
@@ -98,5 +95,5 @@
     <xacro:property name="ZED_depth_info_topicName" value="depth/camera_info"/>
     <xacro:property name="ZED_depth_points_topicName" value="depth/points"/>
-    <xacro:property name="ZED_frameName" value="zed_camera_link_optical"/>
+    <xacro:property name="ZED_frameName" value="left_camera_link_optical"/>
     <!-- Garmin GPS -->
     <!-- NOTE: approx. as a cylinder, Garmin itself is similar to a hockey puck -->
@@ -115,10 +112,10 @@
     <xacro:property name="gps_vel_drift" value="0.00 0.00 0.00"/>
     <!-- Phidget IMU -->
-   <xacro:property name="phidget_length" value="0.04"/>
-   <xacro:property name="phidget_width" value="0.0375"/>
-   <xacro:property name="phidget_height" value="0.01"/>
-   <xacro:property name="phidget_mass" value="0.04"/>
-   <xacro:property name="imu_frame" value="imu_link"/>
-   <xacro:property name="imu_topic" value="imu/data"/>
-   <xacro:property name="imu_update_rate" value="128.0"/>
+    <xacro:property name="phidget_length" value="0.04"/>
+    <xacro:property name="phidget_width" value="0.0375"/>
+    <xacro:property name="phidget_height" value="0.01"/>
+    <xacro:property name="phidget_mass" value="0.04"/>
+    <xacro:property name="imu_frame" value="imu_link"/>
+    <xacro:property name="imu_topic" value="imu/data"/>
+    <xacro:property name="imu_update_rate" value="128.0"/>
 </robot>

File: description/urdf/plugins.gazebo.xacro (robot description, xacro)
@@ -1,4 +1,4 @@
 <?xml version="1.0"?>
-<robot name="caffeine_sim" xmlns:xacro="http://ros.org/wiki/xacro">
+<robot name="plugins" xmlns:xacro="http://ros.org/wiki/xacro">
     <!-- Constants -->
     <xacro:include filename="$(find description)/urdf/constants.xacro"/>
@@ -6,8 +6,7 @@
     <gazebo>
         <plugin name="caffeine_drive_controller" filename="libgazebo_ros_diff_drive.so">
-            <robotNamespace>${robotNamespace}</robotNamespace>
             <updateRate>${diff_drive_update_rate}</updateRate>
-            <leftJoint>${tf_prefix}/${wheel_left_joint}</leftJoint>
-            <rightJoint>${tf_prefix}/${wheel_right_joint}</rightJoint>
+            <leftJoint>${wheel_left_joint}</leftJoint>
+            <rightJoint>${wheel_right_joint}</rightJoint>
             <wheelSeparation>${wheels_separation}</wheelSeparation>
             <wheelDiameter>${wheel_diameter}</wheelDiameter>
@@ -29,10 +28,8 @@
     <!-- lets all the transmission tags be read -->
     <gazebo>
-        <plugin name="gazebo_ros_control" filename="libgazebo_ros_control.so">
-            <robotNamespace>${robotNamespace}</robotNamespace>
-        </plugin>
+        <plugin name="gazebo_ros_control" filename="libgazebo_ros_control.so"/>
     </gazebo>
     <!-- LIDAR -->
-    <gazebo reference="${tf_prefix}/base_laser">
+    <gazebo reference="base_laser">
         <sensor type="ray" name="gpu_hokuyo_sensor">
             <pose>0 0 0 0 0 0</pose>
@@ -63,5 +60,4 @@
             </ray>
             <plugin name="gazebo_ros_hokuyo_controller" filename="libgazebo_ros_laser.so">
-                <robotNamespace>${robotNamespace}</robotNamespace>
                 <topicName>${laser_topicName}</topicName>
                 <frameName>${laser_frameName}</frameName>
@@ -72,8 +68,7 @@
     <gazebo>
         <plugin name="gps_controller" filename="libhector_gazebo_ros_gps.so">
-            <robotNamespace>${robotNamespace}</robotNamespace>
             <updateRate>${gps_update_rate}</updateRate>
-            <bodyName>${tf_prefix}/${gps_frame}</bodyName>
-            <frameId>${tf_prefix}/${gps_frame}</frameId>
+            <bodyName>${gps_frame}</bodyName>
+            <frameId>${gps_frame}</frameId>
             <topicName>${gps_topic}</topicName>
             <velocityTopicName>${gps_vel_topic}</velocityTopicName>
@@ -87,5 +82,5 @@
     </gazebo>
     <!-- Gazebo multicamera plugin -->
-    <gazebo reference="${tf_prefix}/camera_link">
+    <gazebo reference="left_camera_link">
         <sensor type="multicamera" name="stereo_camera">
             <update_rate>${ZED_image_refresh}</update_rate>
@@ -103,5 +98,5 @@
             </camera>
             <camera name="right">
-            <pose>0 ${-ZED_camera_length} 0 0 0 0</pose>
+            <pose>0 -${ZED_camera_length} 0 0 0 0</pose>
             <horizontal_fov>${ZED_image_hfov}</horizontal_fov>
             <image>
@@ -124,5 +119,5 @@
                 <depthImageInfoTopicName>${ZED_depth_info_topicName}</depthImageInfoTopicName>
                 <pointCloudTopicName>${ZED_depth_points_topicName}</pointCloudTopicName>
-                <frameName>${tf_prefix}/${ZED_frameName}</frameName>
+                <frameName>${ZED_frameName}</frameName>
                 <hackBaseline>${ZED_camera_length}</hackBaseline>
                 <!-- TODO: Get distortion parameters from real camera -->
@@ -136,5 +131,5 @@
     </gazebo>
     <!-- IMU -->
-    <gazebo reference="${tf_prefix}/imu_link">
+    <gazebo reference="imu_link">
         <material>Gazebo/Black</material>
         <gravity>true</gravity>
@@ -145,7 +140,7 @@
             <!-- TODO: add Drift based on Phidget IMU -->
             <plugin filename="libgazebo_ros_imu_sensor.so" name="imu_plugin">
-                <topicName>${robotNamespace}/${imu_topic}</topicName>
-                <bodyName>${tf_prefix}/${imu_frame}</bodyName>
-                <frameName>${tf_prefix}/${imu_frame}</frameName>
+                <topicName>${imu_topic}</topicName>
+                <bodyName>${imu_frame}</bodyName>
+                <frameName>${imu_frame}</frameName>
                 <updateRateHZ>${imu_update_rate}</updateRateHZ>
                 <gaussianNoise>0.0</gaussianNoise>  <!-- TODO: set Gaussian noise based on Phidget IMU -->

File: description/urdf/side_wheels.urdf.xacro (robot description, xacro)
@@ -15,5 +15,5 @@
     </xacro:macro>
     <!-- left wheel -->
-    <link name="${tf_prefix}/left_wheel_link">
+    <link name="left_wheel_link">
         <visual>
             <origin rpy="0 0 0" xyz="0 0 0"/>
@@ -33,11 +33,11 @@
         </inertial>
     </link>
-    <joint name="${tf_prefix}/left_wheel_joint" type="continuous">
-        <parent link="${tf_prefix}/chassis_link"/>
-        <child link="${tf_prefix}/left_wheel_link"/>
+    <joint name="left_wheel_joint" type="continuous">
+        <parent link="chassis_link"/>
+        <child link="left_wheel_link"/>
         <origin xyz= "0 ${wheels_separation / 2.0} ${wheel_vertical_offset}"/>
         <axis xyz="0 1 0"/>
     </joint>
-    <gazebo reference="${tf_prefix}/left_wheel_link">
+    <gazebo reference="left_wheel_link">
         <mu1 value="1.0"/>
         <mu2 value="1.0"/>
@@ -45,7 +45,7 @@
         <kd value="1.0" />
     </gazebo>
-    <xacro:Transmission joint="${tf_prefix}/left_wheel_joint"/>
+    <xacro:Transmission joint="left_wheel_joint"/>
     <!-- right wheel -->
-    <link name="${tf_prefix}/right_wheel_link">
+    <link name="right_wheel_link">
         <visual>
             <origin rpy="0 0 0" xyz="0 0 0"/>
@@ -65,11 +65,11 @@
         </inertial>
     </link>
-    <joint name="${tf_prefix}/right_wheel_joint" type="continuous">
-        <parent link="${tf_prefix}/chassis_link"/>
-        <child link="${tf_prefix}/right_wheel_link"/>
+    <joint name="right_wheel_joint" type="continuous">
+        <parent link="chassis_link"/>
+        <child link="right_wheel_link"/>
         <origin xyz= "0 -${wheels_separation / 2.0} ${wheel_vertical_offset}"/>
         <axis xyz="0 1 0"/>
     </joint>
-    <gazebo reference="${tf_prefix}/right_wheel_link">
+    <gazebo reference="right_wheel_link">
         <mu1 value="1.0"/>
         <mu2 value="1.0"/>
@@ -77,4 +77,4 @@
         <kd value="1.0" />
     </gazebo>
-    <xacro:Transmission joint="${tf_prefix}/right_wheel_joint"/>
+    <xacro:Transmission joint="right_wheel_joint"/>
 </robot>

Commit message: guessed sensor positions

File: description/urdf/caffeine.urdf.xacro (robot description, xacro)
@@ -34,7 +34,7 @@
     </link>
     <joint name="base_laser_joint" type="fixed">
-        <parent link="base_link"/>
+        <parent link="chassis_link"/>
         <child link="base_laser"/>
-        <origin xyz="${laser_x_dist} 0 ${laser_z_dist}" rpy="0 0 0"/>
+        <origin xyz="${laser_x_dist} 0 ${wheel_diameter - (2.75 * laser_height / 3)  - stand_height / 2}" rpy="0 0 0"/>
     </joint>
 </robot>

File: description/urdf/stand_link.urdf.xacro (robot description, xacro)
@@ -58,5 +58,5 @@
         <parent link="stand_link"/>
         <child link="imu_link"/>
-        <origin xyz="0 0 0" rpy="0 0 0"/>
+        <origin xyz="-0.19 -0.28 ${-1.55 + phidget_height}" rpy="0 0 0"/>
     </joint>
     <!-- ZED Camera -->
