Commit message: Added second lidar

File: description/urdf/caffeine.urdf.xacro (robot description, xacro)
@@ -38,3 +38,27 @@
         <origin xyz="${laser_x_dist} 0 ${laser_z_dist}" rpy="0 0 0"/>
     </joint>
+    <!--another lidar for testing-->
+    <link name="another_laser">
+        <inertial>
+            <mass value="${laser_mass}"/>
+            <xacro:box_inertia mass="${laser_mass}" length="${laser_length}" width="${laser_width}" height="${laser_height}"/>
+        </inertial>
+        <visual>
+            <origin xyz="0 0 0" rpy="0 0 0"/>
+            <geometry>
+            <mesh filename="package://description/urdf/meshes/hokuyo.dae"/>
+            </geometry>
+        </visual>
+        <collision>
+            <origin xyz="0 0 0" rpy="0 0 0"/>
+            <geometry>
+            <mesh filename="package://description//urdf/meshes/hokuyo.dae"/>
+            </geometry>
+        </collision>
+    </link>
+    <joint name="another_laser_joint" type="fixed">
+        <parent link="base_link"/>
+        <child link="another_laser"/>
+        <origin xyz="${laser_x_dist} 0 ${laser_z_dist+distance_to_second_lidar}" rpy="0 0 0"/>
+    </joint>
 </robot>

File: description/urdf/constants.xacro (robot description, xacro)
@@ -68,4 +68,6 @@
     <xacro:property name="laser_topicName" value="scan"/>
     <xacro:property name="laser_frameName" value="base_laser"/>
+    <xacro:property name="another_laser_topicName" value="scan_upper"/>
+    <xacro:property name="another_laser_frameName" value="another_laser"/>
     <xacro:property name="laser_length" value="0.05"/>
     <xacro:property name="laser_width" value="0.05"/>
@@ -74,4 +76,5 @@
     <xacro:property name="laser_x_dist" value="${base_length/2 - 2*laser_length}"/>
     <xacro:property name="laser_z_dist" value="${laser_height/2}"/>
+    <xacro:property name="distance_to_second_lidar" value="0.2"/>
     <!-- ZED camera -->
     <!-- NOTE: approx as a rectangular prism -->

File: description/urdf/plugins.gazebo.xacro (robot description, xacro)
@@ -62,4 +62,39 @@
                 <topicName>${laser_topicName}</topicName>
                 <frameName>${laser_frameName}</frameName>
+            </plugin>
+        </sensor>
+    </gazebo>
+    <!-- Another LIDAR for testing-->
+    <gazebo reference="another_laser">
+        <sensor type="ray" name="gpu_hokuyo_sensor">
+            <pose>0 0 0 0 0 0</pose>
+            <visualize>${laser_visualize}</visualize>
+            <update_rate>${laser_update_rate}</update_rate>
+            <ray>
+                <scan>
+                    <horizontal>
+                        <samples>${laser_horizontal_samples}</samples>
+                        <resolution>${laser_horizontal_resolution}</resolution>
+                        <min_angle>${laser_horizontal_min_angle}</min_angle>
+                        <max_angle>${laser_horizontal_max_angle}</max_angle>
+                    </horizontal>
+                </scan>
+                <range>
+                    <min>${laser_range_min}</min>
+                    <max>${laser_range_max}</max>
+                    <resolution>${laser_range_resolution}</resolution>
+                </range>
+                <noise>
+                    <type>${laser_noise_type}</type>
+                    <!-- Noise based on gazebosim.org's tutorial on writing gazebo plugins w/ ROS. The comment they put will be reproduced:
+                        Noise parameters based on published spec for Hokuyo laser achieving "+-10mm" accuracy at range < 10 m. A mean of
+                        0.0m and stddev of (0.01/3), will put 99.8% of samples within 0.03m of the true reading. -->
+                    <mean>${laser_noise_mean}</mean>
+                    <stddev>${laser_noise_stddev}</stddev>
+                </noise>
+            </ray>
+            <plugin name="gazebo_ros_hokuyo_controller" filename="libgazebo_ros_laser.so">
+                <topicName>${another_laser_topicName}</topicName>
+                <frameName>${another_laser_frameName}</frameName>
             </plugin>
         </sensor>

Commit message: Adding back second lidar.

File: description/urdf/caffeine.urdf.xacro (robot description, xacro)
@@ -38,3 +38,27 @@
         <origin xyz="${laser_x_dist} 0 ${wheel_diameter - (2.75 * laser_height / 3)  - stand_height / 2}" rpy="0 0 0"/>
     </joint>
+    <!--another lidar for testing-->
+    <link name="upper_laser">
+        <inertial>
+            <mass value="${laser_mass}"/>
+            <xacro:box_inertia mass="${laser_mass}" length="${laser_length}" width="${laser_width}" height="${laser_height}"/>
+        </inertial>
+        <visual>
+            <origin xyz="0 0 0" rpy="0 0 0"/>
+            <geometry>
+            <mesh filename="package://description/urdf/meshes/hokuyo.dae"/>
+            </geometry>
+        </visual>
+        <collision>
+            <origin xyz="0 0 0" rpy="0 0 0"/>
+            <geometry>
+            <mesh filename="package://description//urdf/meshes/hokuyo.dae"/>
+            </geometry>
+        </collision>
+    </link>
+    <joint name="upper_laser_joint" type="fixed">
+        <parent link="base_link"/>
+        <child link="upper_laser"/>
+        <origin xyz="${laser_x_dist} 0 ${laser_z_dist+distance_to_second_lidar}" rpy="0 0 0"/>
+    </joint>
 </robot>

File: description/urdf/constants.xacro (robot description, xacro)
@@ -68,4 +68,6 @@
     <xacro:property name="laser_topicName" value="scan"/>
     <xacro:property name="laser_frameName" value="base_laser"/>
+    <xacro:property name="upper_laser_topicName" value="scan_upper"/>
+    <xacro:property name="upper_laser_frameName" value="upper_laser"/>
     <xacro:property name="laser_length" value="0.05"/>
     <xacro:property name="laser_width" value="0.05"/>
@@ -119,3 +121,7 @@
     <xacro:property name="imu_topic" value="imu/data"/>
     <xacro:property name="imu_update_rate" value="128.0"/>
+    <xacro:property name="imu_x_dist" value="0.28"/>
+    <xacro:property name="imu_y_dist" value="0.295"/>
+    <xacro:property name="imu_z_dist" value="0.0"/>
+    <!--<xacro:property name="imu_z_dist" value="0.195"/>-->
 </robot>

File: description/urdf/plugins.gazebo.xacro (robot description, xacro)
@@ -62,4 +62,39 @@
                 <topicName>${laser_topicName}</topicName>
                 <frameName>${laser_frameName}</frameName>
+            </plugin>
+        </sensor>
+    </gazebo>
+    <!-- Another LIDAR for testing-->
+    <gazebo reference="upper_laser">
+        <sensor type="ray" name="gpu_hokuyo_sensor">
+            <pose>0 0 0 0 0 0</pose>
+            <visualize>${laser_visualize}</visualize>
+            <update_rate>${laser_update_rate}</update_rate>
+            <ray>
+                <scan>
+                    <horizontal>
+                        <samples>${laser_horizontal_samples}</samples>
+                        <resolution>${laser_horizontal_resolution}</resolution>
+                        <min_angle>${laser_horizontal_min_angle}</min_angle>
+                        <max_angle>${laser_horizontal_max_angle}</max_angle>
+                    </horizontal>
+                </scan>
+                <range>
+                    <min>${laser_range_min}</min>
+                    <max>${laser_range_max}</max>
+                    <resolution>${laser_range_resolution}</resolution>
+                </range>
+                <noise>
+                    <type>${laser_noise_type}</type>
+                    <!-- Noise based on gazebosim.org's tutorial on writing gazebo plugins w/ ROS. The comment they put will be reproduced:
+                        Noise parameters based on published spec for Hokuyo laser achieving "+-10mm" accuracy at range < 10 m. A mean of
+                        0.0m and stddev of (0.01/3), will put 99.8% of samples within 0.03m of the true reading. -->
+                    <mean>${laser_noise_mean}</mean>
+                    <stddev>${laser_noise_stddev}</stddev>
+                </noise>
+            </ray>
+            <plugin name="gazebo_ros_hokuyo_controller" filename="libgazebo_ros_laser.so">
+                <topicName>${upper_laser_topicName}</topicName>
+                <frameName>${upper_laser_frameName}</frameName>
             </plugin>
         </sensor>

Commit message: Removed conflicting changes from much older code

File: description/urdf/caffeine.urdf.xacro (robot description, xacro)
@@ -34,7 +34,7 @@
     </link>
     <joint name="base_laser_joint" type="fixed">
-        <parent link="chassis_link"/>
+        <parent link="base_link"/>
         <child link="base_laser"/>
-        <origin xyz="${laser_x_dist} 0 ${wheel_diameter - (2.75 * laser_height / 3)  - stand_height / 2}" rpy="0 0 0"/>
+        <origin xyz="${laser_x_dist} 0 ${laser_z_dist}" rpy="0 0 0"/>
     </joint>
     <!--another lidar for testing-->

File: description/urdf/casters.urdf.xacro (robot description, xacro)
@@ -12,8 +12,8 @@
         counterweight at the back, representative of a battery, for
         example.
-        *Leave Front Caster+Wheel Definitions Commented Out*
+        *Leave BACK Caster+Wheel Definitions Commented Out*
     -->
-    <!-- Front caster definition -->
-    <!-- <link name="front_caster_link">
+       <!-- Front caster definition -->
+    <link name="front_caster_link">
         <visual>
             <origin rpy="0 0 0" xyz="0 0 0"/>
@@ -44,7 +44,7 @@
         <kp value="10000000.0" />
         <kd value="1.0" />
-    </gazebo> -->
+    </gazebo>
     <!-- Front caster wheel definition -->
-    <!-- <link name="front_caster_wheel">
+    <link name="front_caster_wheel">
         <visual>
             <origin rpy="0 0 0" xyz="0 0 0"/>
@@ -75,7 +75,7 @@
         <kp value="10000000.0" />
         <kd value="1.0" />
-    </gazebo> -->
+    </gazebo>
     <!-- Back caster definition -->
-    <link name="back_caster_link">
+    <!-- <link name="back_caster_link">
         <visual>
             <origin rpy="0 0 0" xyz="0 0 0"/>
@@ -106,7 +106,7 @@
         <kp value="10000000.0" />
         <kd value="1.0" />
-    </gazebo>
+    </gazebo> -->
     <!-- Back caster wheel definition -->
-    <link name="back_caster_wheel">
+    <!-- <link name="back_caster_wheel">
         <visual>
             <origin rpy="0 0 0" xyz="0 0 0"/>
@@ -137,4 +137,4 @@
         <kp value="10000000.0" />
         <kd value="1.0" />
-    </gazebo>
+    </gazebo> -->
 </robot>

File: description/urdf/chassis_link.urdf.xacro (robot description, xacro)
@@ -48,5 +48,5 @@
     </link>
     <joint name="battery_joint" type="fixed">
-        <origin xyz="${-1*(stand_length/2 + battery_width + battery_back_offset)} 0 ${wheel_diameter - (3*battery_height/2) - stand_height/2}" rpy="0 0 0"/>
+        <origin xyz="${(stand_length/2 + battery_width + battery_back_offset)} 0 ${wheel_diameter - (3*battery_height/2) - stand_height/2}" rpy="0 0 0"/>
         <parent link="chassis_link"/>
         <child link="battery_link"/>

File: description/urdf/constants.xacro (robot description, xacro)
@@ -11,6 +11,6 @@
     <!-- Stand -->
     <xacro:property name="stand_length" value="0.412"/>
-    <xacro:property name="stand_width" value="0.254"/>
-    <xacro:property name="stand_height" value="1.324"/>
+    <xacro:property name="stand_width" value="0.33"/>
+    <xacro:property name="stand_height" value="1.335"/>
     <xacro:property name="stand_mass" value="1.0"/>
     <!-- Casters -->

File: description/urdf/stand_link.urdf.xacro (robot description, xacro)
@@ -56,7 +56,7 @@
     </link>
     <joint name="base_link_to_imu_link" type="fixed">
-        <parent link="stand_link"/>
+        <parent link="base_link"/>
         <child link="imu_link"/>
-        <origin xyz="-0.19 -0.28 ${-1.55 + phidget_height}" rpy="0 0 0"/>
+        <origin xyz="${imu_x_dist} ${imu_y_dist} ${imu_z_dist}" rpy="0 0 0"/>
     </joint>
     <!-- ZED Camera -->

Commit message: 'another' naming switched to 'upper' for new lidar

File: description/urdf/caffeine.urdf.xacro (robot description, xacro)
@@ -39,5 +39,5 @@
     </joint>
     <!--another lidar for testing-->
-    <link name="another_laser">
+    <link name="upper_laser">
         <inertial>
             <mass value="${laser_mass}"/>
@@ -57,7 +57,7 @@
         </collision>
     </link>
-    <joint name="another_laser_joint" type="fixed">
+    <joint name="upper_laser_joint" type="fixed">
         <parent link="base_link"/>
-        <child link="another_laser"/>
+        <child link="upper_laser"/>
         <origin xyz="${laser_x_dist} 0 ${laser_z_dist+distance_to_second_lidar}" rpy="0 0 0"/>
     </joint>

File: description/urdf/constants.xacro (robot description, xacro)
@@ -68,6 +68,6 @@
     <xacro:property name="laser_topicName" value="scan"/>
     <xacro:property name="laser_frameName" value="base_laser"/>
-    <xacro:property name="another_laser_topicName" value="scan_upper"/>
-    <xacro:property name="another_laser_frameName" value="another_laser"/>
+    <xacro:property name="upper_laser_topicName" value="scan_upper"/>
+    <xacro:property name="upper_laser_frameName" value="upper_laser"/>
     <xacro:property name="laser_length" value="0.05"/>
     <xacro:property name="laser_width" value="0.05"/>

File: description/urdf/plugins.gazebo.xacro (robot description, xacro)
@@ -66,5 +66,5 @@
     </gazebo>
     <!-- Another LIDAR for testing-->
-    <gazebo reference="another_laser">
+    <gazebo reference="upper_laser">
         <sensor type="ray" name="gpu_hokuyo_sensor">
             <pose>0 0 0 0 0 0</pose>
@@ -95,6 +95,6 @@
             </ray>
             <plugin name="gazebo_ros_hokuyo_controller" filename="libgazebo_ros_laser.so">
-                <topicName>${another_laser_topicName}</topicName>
-                <frameName>${another_laser_frameName}</frameName>
+                <topicName>${upper_laser_topicName}</topicName>
+                <frameName>${upper_laser_frameName}</frameName>
             </plugin>
         </sensor>
