Commit message: Removed second lidar and changed distance between wheels to 1 m in urdf and in cmd_vel_to_motor.cpp

File: description/urdf/caffeine.urdf.xacro (robot description, xacro)
@@ -38,27 +38,3 @@
         <origin xyz="${laser_x_dist} 0 ${laser_z_dist}" rpy="0 0 0"/>
     </joint>
-    <!--another lidar for testing-->
-    <link name="upper_laser">
-        <inertial>
-            <mass value="${laser_mass}"/>
-            <xacro:box_inertia mass="${laser_mass}" length="${laser_length}" width="${laser_width}" height="${laser_height}"/>
-        </inertial>
-        <visual>
-            <origin xyz="0 0 0" rpy="0 0 0"/>
-            <geometry>
-            <mesh filename="package://description/urdf/meshes/hokuyo.dae"/>
-            </geometry>
-        </visual>
-        <collision>
-            <origin xyz="0 0 0" rpy="0 0 0"/>
-            <geometry>
-            <mesh filename="package://description//urdf/meshes/hokuyo.dae"/>
-            </geometry>
-        </collision>
-    </link>
-    <joint name="upper_laser_joint" type="fixed">
-        <parent link="base_link"/>
-        <child link="upper_laser"/>
-        <origin xyz="${laser_x_dist} 0 ${laser_z_dist+distance_to_second_lidar}" rpy="0 0 0"/>
-    </joint>
 </robot>

File: description/urdf/casters.urdf.xacro (robot description, xacro)
@@ -50,5 +50,6 @@
             <origin rpy="0 0 0" xyz="0 0 0"/>
             <geometry>
-                <mesh filename="package://description/urdf/meshes/front_caster_wheel.dae"/>
+                <mesh filename="package://description/urdf/meshes/front_caster_wheel_new.dae"/>
+                <!--<mesh filename="package://description/urdf/meshes/front_caster_wheel.dae"/>-->
             </geometry>
         </visual>
@@ -56,5 +57,6 @@
             <origin rpy="0 0 0" xyz="0 0 0"/>
             <geometry>
-                <mesh filename="package://description/urdf/meshes/front_caster_wheel.dae"/>
+                <mesh filename="package://description/urdf/meshes/front_caster_wheel_new.dae"/>
+                <!--<mesh filename="package://description/urdf/meshes/front_caster_wheel.dae"/>-->
             </geometry>
         </collision>

File: description/urdf/constants.xacro (robot description, xacro)
@@ -33,5 +33,6 @@
     <xacro:property name="wheel_left_joint" value="left_wheel_joint"/>
     <xacro:property name="wheel_right_joint" value="right_wheel_joint"/>
-    <xacro:property name="wheels_separation" value="0.875"/>
+    <!--<xacro:property name="wheels_separation" value="0.875"/>-->
+    <xacro:property name="wheels_separation" value="1.0"/>
     <xacro:property name="wheel_diameter" value="0.25"/>
     <xacro:property name="wheel_acceleration" value="1.0"/>
@@ -68,6 +69,4 @@
     <xacro:property name="laser_topicName" value="scan"/>
     <xacro:property name="laser_frameName" value="base_laser"/>
-    <xacro:property name="upper_laser_topicName" value="scan_upper"/>
-    <xacro:property name="upper_laser_frameName" value="upper_laser"/>
     <xacro:property name="laser_length" value="0.05"/>
     <xacro:property name="laser_width" value="0.05"/>
@@ -76,5 +75,4 @@
     <xacro:property name="laser_x_dist" value="${base_length/2 - 2*laser_length}"/>
     <xacro:property name="laser_z_dist" value="${laser_height/2}"/>
-    <xacro:property name="distance_to_second_lidar" value="0.2"/>
     <!-- ZED camera -->
     <!-- NOTE: approx as a rectangular prism -->

File: description/urdf/plugins.gazebo.xacro (robot description, xacro)
@@ -62,39 +62,4 @@
                 <topicName>${laser_topicName}</topicName>
                 <frameName>${laser_frameName}</frameName>
-            </plugin>
-        </sensor>
-    </gazebo>
-    <!-- Another LIDAR for testing-->
-    <gazebo reference="upper_laser">
-        <sensor type="ray" name="gpu_hokuyo_sensor">
-            <pose>0 0 0 0 0 0</pose>
-            <visualize>${laser_visualize}</visualize>
-            <update_rate>${laser_update_rate}</update_rate>
-            <ray>
-                <scan>
-                    <horizontal>
-                        <samples>${laser_horizontal_samples}</samples>
-                        <resolution>${laser_horizontal_resolution}</resolution>
-                        <min_angle>${laser_horizontal_min_angle}</min_angle>
-                        <max_angle>${laser_horizontal_max_angle}</max_angle>
-                    </horizontal>
-                </scan>
-                <range>
-                    <min>${laser_range_min}</min>
-                    <max>${laser_range_max}</max>
-                    <resolution>${laser_range_resolution}</resolution>
-                </range>
-                <noise>
-                    <type>${laser_noise_type}</type>
-                    <!-- Noise based on gazebosim.org's tutorial on writing gazebo plugins w/ ROS. The comment they put will be reproduced:
-                        Noise parameters based on published spec for Hokuyo laser achieving "+-10mm" accuracy at range < 10 m. A mean of
-                        0.0m and stddev of (0.01/3), will put 99.8% of samples within 0.03m of the true reading. -->
-                    <mean>${laser_noise_mean}</mean>
-                    <stddev>${laser_noise_stddev}</stddev>
-                </noise>
-            </ray>
-            <plugin name="gazebo_ros_hokuyo_controller" filename="libgazebo_ros_laser.so">
-                <topicName>${upper_laser_topicName}</topicName>
-                <frameName>${upper_laser_frameName}</frameName>
             </plugin>
         </sensor>

File: description/urdf/side_wheels.urdf.xacro (robot description, xacro)
@@ -19,5 +19,6 @@
             <origin rpy="0 0 0" xyz="0 0 0"/>
             <geometry>
-                <mesh filename="package://description/urdf/meshes/left_wheel.dae"/>
+                <mesh filename="package://description/urdf/meshes/left_wheel_new.dae"/>
+                <!--<mesh filename="package://description/urdf/meshes/left_wheel.dae"/>-->
             </geometry>
         </visual>
@@ -25,5 +26,6 @@
             <origin rpy="0 0 0" xyz="0 0 0"/>
             <geometry>
-                <mesh filename="package://description/urdf/meshes/left_wheel.dae"/>
+                <mesh filename="package://description/urdf/meshes/left_wheel_new.dae"/>
+                <!--<mesh filename="package://description/urdf/meshes/left_wheel.dae"/>-->
             </geometry>
         </collision>
@@ -51,5 +53,6 @@
             <origin rpy="0 0 0" xyz="0 0 0"/>
             <geometry>
-                <mesh filename="package://description/urdf/meshes/right_wheel.dae"/>
+                <mesh filename="package://description/urdf/meshes/right_wheel_new.dae"/>
+                <!--mesh filename="package://description/urdf/meshes/right_wheel.dae"/>-->
             </geometry>
         </visual>
@@ -57,5 +60,6 @@
             <origin rpy="0 0 0" xyz="0 0 0"/>
             <geometry>
-                <mesh filename="package://description/urdf/meshes/right_wheel.dae"/>
+                <mesh filename="package://description/urdf/meshes/right_wheel_new.dae"/>
+                <!--<mesh filename="package://description/urdf/meshes/right_wheel.dae"/>-->
             </geometry>
         </collision>

File: description/urdf/stand_link.urdf.xacro (robot description, xacro)
@@ -35,28 +35,4 @@
         <child link="gps_link"/>
         <origin xyz="0 0 ${(gps_length + phidget_height) / 2.0}" rpy="0 0 0"/>
-    </joint>
-    <!-- IMU -->
-    <link name="imu_link">
-        <inertial>
-            <mass value="${phidget_mass}"/>
-            <xacro:box_inertia mass="${phidget_mass}" length="${phidget_length}" width="${phidget_width}" height="${phidget_height}"/>
-        </inertial>
-        <visual>
-            <origin xyz="0 0 0" rpy="0 0 0"/>
-            <geometry>
-            <box size="${phidget_length} ${phidget_width} ${phidget_height}"/>
-            </geometry>
-        </visual>
-        <collision>
-            <origin xyz="0 0 0" rpy="0 0 0"/>
-            <geometry>
-            <box size="${phidget_length} ${phidget_width} ${phidget_height}"/>
-            </geometry>
-        </collision>
-    </link>
-    <joint name="base_link_to_imu_link" type="fixed">
-        <parent link="base_link"/>
-        <child link="imu_link"/>
-        <origin xyz="${imu_x_dist} ${imu_y_dist} ${imu_z_dist}" rpy="0 0 0"/>
     </joint>
     <!-- ZED Camera -->
@@ -101,3 +77,27 @@
         <origin xyz="0 0 0" rpy="${-pi/2} 0 ${-pi/2}"/>
     </joint>
+    <!-- IMU (IS CONNECTED TO BASE LINK) -->
+    <link name="imu_link">
+        <inertial>
+            <mass value="${phidget_mass}"/>
+            <xacro:box_inertia mass="${phidget_mass}" length="${phidget_length}" width="${phidget_width}" height="${phidget_height}"/>
+        </inertial>
+        <visual>
+            <origin xyz="0 0 0" rpy="0 0 0"/>
+            <geometry>
+            <box size="${phidget_length} ${phidget_width} ${phidget_height}"/>
+            </geometry>
+        </visual>
+        <collision>
+            <origin xyz="0 0 0" rpy="0 0 0"/>
+            <geometry>
+            <box size="${phidget_length} ${phidget_width} ${phidget_height}"/>
+            </geometry>
+        </collision>
+    </link>
+    <joint name="base_link_to_imu_link" type="fixed">
+        <parent link="base_link"/>
+        <child link="imu_link"/>
+        <origin xyz="${imu_x_dist} ${imu_y_dist} ${imu_z_dist}" rpy="0 0 0"/>
+    </joint>
 </robot>

Commit message: Moved imu to caffeine-urdf.xacro

File: description/urdf/caffeine.urdf.xacro (robot description, xacro)
@@ -38,3 +38,27 @@
         <origin xyz="${laser_x_dist} 0 ${laser_z_dist}" rpy="0 0 0"/>
     </joint>
+    <!-- IMU (IS CONNECTED TO BASE LINK) -->
+    <link name="imu_link">
+        <inertial>
+            <mass value="${phidget_mass}"/>
+            <xacro:box_inertia mass="${phidget_mass}" length="${phidget_length}" width="${phidget_width}" height="${phidget_height}"/>
+        </inertial>
+        <visual>
+            <origin xyz="0 0 0" rpy="0 0 0"/>
+            <geometry>
+            <box size="${phidget_length} ${phidget_width} ${phidget_height}"/>
+            </geometry>
+        </visual>
+        <collision>
+            <origin xyz="0 0 0" rpy="0 0 0"/>
+            <geometry>
+            <box size="${phidget_length} ${phidget_width} ${phidget_height}"/>
+            </geometry>
+        </collision>
+    </link>
+    <joint name="base_link_to_imu_link" type="fixed">
+        <parent link="base_link"/>
+        <child link="imu_link"/>
+        <origin xyz="${imu_x_dist} ${imu_y_dist} ${imu_z_dist}" rpy="0 0 0"/>
+    </joint>
 </robot>

File: description/urdf/stand_link.urdf.xacro (robot description, xacro)
@@ -77,27 +77,3 @@
         <origin xyz="0 0 0" rpy="${-pi/2} 0 ${-pi/2}"/>
     </joint>
-    <!-- IMU (IS CONNECTED TO BASE LINK) -->
-    <link name="imu_link">
-        <inertial>
-            <mass value="${phidget_mass}"/>
-            <xacro:box_inertia mass="${phidget_mass}" length="${phidget_length}" width="${phidget_width}" height="${phidget_height}"/>
-        </inertial>
-        <visual>
-            <origin xyz="0 0 0" rpy="0 0 0"/>
-            <geometry>
-            <box size="${phidget_length} ${phidget_width} ${phidget_height}"/>
-            </geometry>
-        </visual>
-        <collision>
-            <origin xyz="0 0 0" rpy="0 0 0"/>
-            <geometry>
-            <box size="${phidget_length} ${phidget_width} ${phidget_height}"/>
-            </geometry>
-        </collision>
-    </link>
-    <joint name="base_link_to_imu_link" type="fixed">
-        <parent link="base_link"/>
-        <child link="imu_link"/>
-        <origin xyz="${imu_x_dist} ${imu_y_dist} ${imu_z_dist}" rpy="0 0 0"/>
-    </joint>
 </robot>

Commit message: CAFF-88: Update Caffeine Model and Pavement World Maps (#138)
* updated stand position but seeing weird bugs

* guessed sensor positions

* Changed chassis model and WIP of changing model of lanes

* Adding back second lidar.

* Fixing missing distance_to_second_lidar

* Removed conflicting changes from much older code

* Fixed scene lighting so lanes appear as white.

* Updated all scenes.

* Removed second lidar and changed distance between wheels to 1 m in urdf and in cmd_vel_to_motor.cpp

* Moved imu to caffeine-urdf.xacro

* Making motor files consistent with master.

* Revert unneeded texture changes.

* Fixed camera positioning.

* Simulate.launch world is set to pavement full

---------

Co-authored-by: kajananchinniah <kajananchinniah@gmail.com>
Co-authored-by: Vicky <vhy.huang@mail.utoronto.ca>

File: description/urdf/caffeine.urdf.xacro (robot description, xacro)
@@ -38,3 +38,27 @@
         <origin xyz="${laser_x_dist} 0 ${laser_z_dist}" rpy="0 0 0"/>
     </joint>
+    <!-- IMU (IS CONNECTED TO BASE LINK) -->
+    <link name="imu_link">
+        <inertial>
+            <mass value="${phidget_mass}"/>
+            <xacro:box_inertia mass="${phidget_mass}" length="${phidget_length}" width="${phidget_width}" height="${phidget_height}"/>
+        </inertial>
+        <visual>
+            <origin xyz="0 0 0" rpy="0 0 0"/>
+            <geometry>
+            <box size="${phidget_length} ${phidget_width} ${phidget_height}"/>
+            </geometry>
+        </visual>
+        <collision>
+            <origin xyz="0 0 0" rpy="0 0 0"/>
+            <geometry>
+            <box size="${phidget_length} ${phidget_width} ${phidget_height}"/>
+            </geometry>
+        </collision>
+    </link>
+    <joint name="base_link_to_imu_link" type="fixed">
+        <parent link="base_link"/>
+        <child link="imu_link"/>
+        <origin xyz="${imu_x_dist} ${imu_y_dist} ${imu_z_dist}" rpy="0 0 0"/>
+    </joint>
 </robot>

File: description/urdf/casters.urdf.xacro (robot description, xacro)
@@ -12,5 +12,5 @@
         counterweight at the back, representative of a battery, for
         example.
-        *Leave Front Caster+Wheel Definitions Commented Out*
+        *Leave BACK Caster+Wheel Definitions Commented Out*
     -->
     <!-- Front caster definition -->
@@ -50,5 +50,6 @@
             <origin rpy="0 0 0" xyz="0 0 0"/>
             <geometry>
-                <mesh filename="package://description/urdf/meshes/front_caster_wheel.dae"/>
+                <mesh filename="package://description/urdf/meshes/front_caster_wheel_new.dae"/>
+                <!--<mesh filename="package://description/urdf/meshes/front_caster_wheel.dae"/>-->
             </geometry>
         </visual>
@@ -56,5 +57,6 @@
             <origin rpy="0 0 0" xyz="0 0 0"/>
             <geometry>
-                <mesh filename="package://description/urdf/meshes/front_caster_wheel.dae"/>
+                <mesh filename="package://description/urdf/meshes/front_caster_wheel_new.dae"/>
+                <!--<mesh filename="package://description/urdf/meshes/front_caster_wheel.dae"/>-->
             </geometry>
         </collision>

File: description/urdf/chassis_link.urdf.xacro (robot description, xacro)
@@ -9,5 +9,5 @@
             <origin rpy="0 0 0" xyz="0 0 0"/>
             <geometry>
-                <mesh filename="package://description/urdf/meshes/chassis_link.dae"/>
+                <mesh filename="package://description/urdf/meshes/chassis_link_new.dae"/>
             </geometry>
         </visual>
@@ -15,5 +15,5 @@
             <origin rpy="0 0 0" xyz="0 0 0"/>
             <geometry>
-                <mesh filename="package://description/urdf/meshes/chassis_link.dae"/>
+                <mesh filename="package://description/urdf/meshes/chassis_link_new.dae"/>
             </geometry>
         </collision>

File: description/urdf/constants.xacro (robot description, xacro)
@@ -7,9 +7,9 @@
     <!-- Chassis -->
     <xacro:property name="chassis_to_base_link_dist" value="0.501747"/>
-    <xacro:property name="chassis_to_stand_link_dist" value="0.698253"/>
-    <xacro:property name="chassis_link_mass" value="33.9"/>
+    <xacro:property name="chassis_to_stand_link_dist" value="0.428526"/>
+    <xacro:property name="chassis_link_mass" value="36.95"/>
     <!-- Stand -->
     <xacro:property name="stand_length" value="0.412"/>
-    <xacro:property name="stand_width" value="0.33"/>
+    <xacro:property name="stand_width" value="0.255"/>
     <xacro:property name="stand_height" value="1.335"/>
     <xacro:property name="stand_mass" value="1.0"/>
@@ -33,5 +33,6 @@
     <xacro:property name="wheel_left_joint" value="left_wheel_joint"/>
     <xacro:property name="wheel_right_joint" value="right_wheel_joint"/>
-    <xacro:property name="wheels_separation" value="0.875"/>
+    <!--<xacro:property name="wheels_separation" value="0.875"/>-->
+    <xacro:property name="wheels_separation" value="1.0"/>
     <xacro:property name="wheel_diameter" value="0.25"/>
     <xacro:property name="wheel_acceleration" value="1.0"/>
@@ -96,4 +97,7 @@
     <xacro:property name="ZED_depth_points_topicName" value="depth/points"/>
     <xacro:property name="ZED_frameName" value="left_camera_link_optical"/>
+    <!--ZED CAMERA JOINT PARAMETERS-->
+    <xacro:property name="ZED_camera_to_top_plate_x" value="${(stand_width / 2.0)-0.01}"/>
+    <xacro:property name="ZED_camera_to_top_plate_z" value="0.065"/>
     <!-- Garmin GPS -->
     <!-- NOTE: approx. as a cylinder, Garmin itself is similar to a hockey puck -->
@@ -121,4 +125,5 @@
     <xacro:property name="imu_x_dist" value="0.28"/>
     <xacro:property name="imu_y_dist" value="0.295"/>
-    <xacro:property name="imu_z_dist" value="0.195"/>
+    <xacro:property name="imu_z_dist" value="0.0"/>
+    <!--<xacro:property name="imu_z_dist" value="0.195"/>-->
 </robot>

File: description/urdf/inertias.xacro (robot description, xacro)
@@ -4,7 +4,7 @@
     <xacro:macro name="chassis_link_inertia">
         <inertia
-            ixx="10.9364" ixy="0.0000" ixz="0.0000"
-            iyx="0.0000" iyy="10.9070" iyz="0.0000"
-            izx="0.0000" izy="0.0000" izz="2.3961"
+            ixx="13.1600" ixy="0.0000" ixz="0.0000"
+            iyx="0.0000" iyy="11.7000" iyz="0.0000"
+            izx="0.0000" izy="0.0000" izz="2.6800"
         />
     </xacro:macro>
@@ -25,5 +25,5 @@
         />
     </xacro:macro>
-    <!-- Cynlinder Inertia -->
+    <!-- Cylinder Inertia -->
     <xacro:macro name="cylinder_inertia" params="mass length radius">
         <inertia

File: description/urdf/stand_link.urdf.xacro (robot description, xacro)
@@ -34,29 +34,5 @@
         <parent link="stand_link"/>
         <child link="gps_link"/>
-        <origin xyz="0 0 0" rpy="0 0 0"/>
-    </joint>
-    <!-- IMU -->
-    <link name="imu_link">
-        <inertial>
-            <mass value="${phidget_mass}"/>
-            <xacro:box_inertia mass="${phidget_mass}" length="${phidget_length}" width="${phidget_width}" height="${phidget_height}"/>
-        </inertial>
-        <visual>
-            <origin xyz="0 0 0" rpy="0 0 0"/>
-            <geometry>
-            <box size="${phidget_length} ${phidget_width} ${phidget_height}"/>
-            </geometry>
-        </visual>
-        <collision>
-            <origin xyz="0 0 0" rpy="0 0 0"/>
-            <geometry>
-            <box size="${phidget_length} ${phidget_width} ${phidget_height}"/>
-            </geometry>
-        </collision>
-    </link>
-    <joint name="base_link_to_imu_link" type="fixed">
-        <parent link="base_link"/>
-        <child link="imu_link"/>
-        <origin xyz="${imu_x_dist} ${imu_y_dist} ${imu_z_dist}" rpy="0 0 0"/>
+        <origin xyz="0 0 ${(gps_length + phidget_height) / 2.0}" rpy="0 0 0"/>
     </joint>
     <!-- </robot> -->
@@ -84,5 +60,5 @@
         <parent link="stand_link"/>
         <child link="zed_base_link"/>
-        <origin xyz="${0.05 + (stand_width / 2.0) - ZED_camera_width} 0 ${ZED_camera_height / 2.0}" rpy="0 ${ZED_camera_pitch} 0"/>
+        <origin xyz="${ZED_camera_to_top_plate_x} 0 ${ZED_camera_to_top_plate_z}" rpy="0 ${ZED_camera_pitch} 0"/>
     </joint>
     <!-- Generate Left Camera frame -->

Commit message: Adjusted files for merge v1

File: description/urdf/caffeine.urdf.xacro (robot description, xacro)
@@ -62,5 +62,5 @@
         <origin xyz="${imu_x_dist} ${imu_y_dist} ${imu_z_dist}" rpy="0 0 0"/>
     </joint>
-    <!--another lidar for testing-->
+    <!-- Second upper lidar -->
     <link name="upper_laser">
         <inertial>

File: description/urdf/constants.xacro (robot description, xacro)
@@ -92,5 +92,5 @@
     <xacro:property name="upper_laser_topicName" value="scan_upper"/>
     <xacro:property name="upper_laser_frameName" value="upper_laser"/>
-    <xacro:property name="distance_to_second_lidar" value="0.2"/>
+    <xacro:property name="distance_to_second_lidar" value="0.14"/>
     <!-- ZED camera -->
     <!-- NOTE: approx as a rectangular prism -->
