Commit message: Caff 132 - ramp detection + upper lidar mock (#151)
* Added second lidar

* 'another' naming switched to 'upper' for new lidar

* new node for ramp filter w parameters

* node functioning

* lidar sensor names have to be unique :(

* testing of ramp filter setup

* Added separately named parameters for upper laser.

* corrected constants referencing for upper lidar

* parameterized upper lidar, array and start, end indexing variable

* corrected world file

* ramp detect params

* spawn at course start

* Adjusted files for merge v1

* Prepare for merge v2 - start toggle

* Finished sim/IGVC toggle in launch file and scheduler.py

* Made toggling cleaner

---------

Co-authored-by: Vicky <vhy.huang@mail.utoronto.ca>
Co-authored-by: utra-art <art@utra.ca>
Co-authored-by: Ivy Tan <ivtn0912@gmail.com>

File: description/urdf/caffeine.urdf.xacro (robot description, xacro)
@@ -62,3 +62,27 @@
         <origin xyz="${imu_x_dist} ${imu_y_dist} ${imu_z_dist}" rpy="0 0 0"/>
     </joint>
+    <!-- Second upper lidar -->
+    <link name="upper_laser">
+        <inertial>
+            <mass value="${laser_mass}"/>
+            <xacro:box_inertia mass="${laser_mass}" length="${laser_length}" width="${laser_width}" height="${laser_height}"/>
+        </inertial>
+        <visual>
+            <origin xyz="0 0 0" rpy="0 0 0"/>
+            <geometry>
+            <mesh filename="package://description/urdf/meshes/hokuyo.dae"/>
+            </geometry>
+        </visual>
+        <collision>
+            <origin xyz="0 0 0" rpy="0 0 0"/>
+            <geometry>
+            <mesh filename="package://description//urdf/meshes/hokuyo.dae"/>
+            </geometry>
+        </collision>
+    </link>
+    <joint name="upper_laser_joint" type="fixed">
+        <parent link="base_link"/>
+        <child link="upper_laser"/>
+        <origin xyz="${laser_x_dist} 0 ${laser_z_dist+distance_to_second_lidar}" rpy="0 0 0"/>
+    </joint>
 </robot>

File: description/urdf/constants.xacro (robot description, xacro)
@@ -75,4 +75,22 @@
     <xacro:property name="laser_x_dist" value="${base_length/2 - 2*laser_length}"/>
     <xacro:property name="laser_z_dist" value="${laser_height/2}"/>
+    <!--RPlidar A1-->
+    <xacro:property name="upper_laser_visualize" value="false"/>
+    <xacro:property name="upper_laser_update_rate" value="10"/>
+    <xacro:property name="upper_laser_horizontal_samples" value="1080"/>
+    <xacro:property name="upper_laser_horizontal_resolution" value="1"/>
+    <xacro:property name="upper_laser_field_of_view" value="270"/>
+    <xacro:property name="upper_laser_horizontal_min_angle" value="${-0.5*upper_laser_field_of_view*pi/180}"/>
+    <xacro:property name="upper_laser_horizontal_max_angle" value="${0.5*upper_laser_field_of_view*pi/180}"/>
+    <xacro:property name="upper_laser_range_min" value="0.06"/>
+    <xacro:property name="upper_laser_range_max" value="4.095"/>
+    <xacro:property name="upper_laser_resolution_angle" value="0.36"/>
+    <xacro:property name="upper_laser_range_resolution" value="${upper_laser_resolution_angle*pi/180}"/>
+    <xacro:property name="upper_laser_noise_type" value="gaussian"/>
+    <xacro:property name="upper_laser_noise_mean" value="0.0"/>
+    <xacro:property name="upper_laser_noise_stddev" value="0.01/3"/>
+    <xacro:property name="upper_laser_topicName" value="scan_upper"/>
+    <xacro:property name="upper_laser_frameName" value="upper_laser"/>
+    <xacro:property name="distance_to_second_lidar" value="0.14"/>
     <!-- ZED camera -->
     <!-- NOTE: approx as a rectangular prism -->

File: description/urdf/plugins.gazebo.xacro (robot description, xacro)
@@ -32,5 +32,6 @@
     <!-- LIDAR -->
     <gazebo reference="base_laser">
-        <sensor type="ray" name="gpu_hokuyo_sensor">
+        <!-- make sure your sensor NAMES are unique :'( -->
+        <sensor type="ray" name="hokuyo_sensor_1">
             <pose>0 0 0 0 0 0</pose>
             <visualize>${laser_visualize}</visualize>
@@ -62,4 +63,40 @@
                 <topicName>${laser_topicName}</topicName>
                 <frameName>${laser_frameName}</frameName>
+            </plugin>
+        </sensor>
+    </gazebo>
+    <!-- Another LIDAR for testing-->
+    <gazebo reference="upper_laser">
+        <!-- make sure your sensor NAMES are unique :'( -->
+        <sensor type="ray" name="hokuyo_sensor_2">
+            <pose>0 0 0 0 0 0</pose>
+            <visualize>${upper_laser_visualize}</visualize>
+            <update_rate>${upper_laser_update_rate}</update_rate>
+            <ray>
+                <scan>
+                    <horizontal>
+                        <samples>${upper_laser_horizontal_samples}</samples>
+                        <resolution>${upper_laser_horizontal_resolution}</resolution>
+                        <min_angle>${upper_laser_horizontal_min_angle}</min_angle>
+                        <max_angle>${upper_laser_horizontal_max_angle}</max_angle>
+                    </horizontal>
+                </scan>
+                <range>
+                    <min>${upper_laser_range_min}</min>
+                    <max>${upper_laser_range_max}</max>
+                    <resolution>${upper_laser_range_resolution}</resolution>
+                </range>
+                <noise>
+                    <type>${upper_laser_noise_type}</type>
+                    <!-- Noise based on gazebosim.org's tutorial on writing gazebo plugins w/ ROS. The comment they put will be reproduced:
+                        Noise parameters based on published spec for Hokuyo laser achieving "+-10mm" accuracy at range < 10 m. A mean of
+                        0.0m and stddev of (0.01/3), will put 99.8% of samples within 0.03m of the true reading. -->
+                    <mean>${upper_laser_noise_mean}</mean>
+                    <stddev>${upper_laser_noise_stddev}</stddev>
+                </noise>
+            </ray>
+            <plugin name="gazebo_ros_hokuyo_controller" filename="libgazebo_ros_laser.so">
+                <topicName>${upper_laser_topicName}</topicName>
+                <frameName>${upper_laser_frameName}</frameName>
             </plugin>
         </sensor>
