Commit message: Temporarily set GPS drifts to 0 for a perfect GPS

File: description/urdf/constants.xacro (robot description, xacro)
@@ -109,5 +109,5 @@
     <xacro:property name="ref_lon" value="-79.3903"/>
     <xacro:property name="ref_alt" value="76.0000"/>
-    <xacro:property name="gps_drift" value="1.5 1.5 1.5"/>
+    <xacro:property name="gps_drift" value="0.00 0.00 0.00"/>
     <xacro:property name="gps_vel_drift" value="0.00 0.00 0.00"/>
     <!-- Phidget IMU -->

Commit message: Quick updates to test_gps to get it working

File: description/urdf/constants.xacro (robot description, xacro)
@@ -109,5 +109,5 @@
     <xacro:property name="ref_lon" value="-79.3903"/>
     <xacro:property name="ref_alt" value="76.0000"/>
-    <xacro:property name="gps_drift" value="0.00 0.00 0.00"/>
+    <xacro:property name="gps_drift" value="1.5 1.5 1.5"/>
     <xacro:property name="gps_vel_drift" value="0.00 0.00 0.00"/>
     <!-- Phidget IMU -->

Commit message: lowered camera angle to avoid detecting ground as obstacle

File: description/urdf/constants.xacro (robot description, xacro)
@@ -80,5 +80,5 @@
     <xacro:property name="ZED_camera_width" value="0.03"/>
     <xacro:property name="ZED_camera_height" value="0.033"/>
-    <xacro:property name="ZED_camera_pitch" value="${15 * pi/180}"/>
+    <xacro:property name="ZED_camera_pitch" value="${25 * pi/180}"/>
     <!-- ZED image height/width corresponds to image size for 60Hz refresh-->
     <xacro:property name="ZED_image_refresh" value="60"/>

Commit message: Linked rtabmap to global cost map, fixed wheel jittering

File: description/urdf/constants.xacro (robot description, xacro)
@@ -65,5 +65,5 @@
     <xacro:property name="laser_noise_type" value="gaussian"/>
     <xacro:property name="laser_noise_mean" value="0.0"/>
-    <xacro:property name="laser_noise_stddev" value="0.01/3"/>
+    <xacro:property name="laser_noise_stddev" value="0.0"/>
     <xacro:property name="laser_topicName" value="scan"/>
     <xacro:property name="laser_frameName" value="base_laser"/>
@@ -109,5 +109,5 @@
     <xacro:property name="ref_lon" value="-79.3903"/>
     <xacro:property name="ref_alt" value="76.0000"/>
-    <xacro:property name="gps_drift" value="1.5 1.5 1.5"/>
+    <xacro:property name="gps_drift" value="0 0 0"/>
     <xacro:property name="gps_vel_drift" value="0.00 0.00 0.00"/>
     <!-- Phidget IMU -->

Commit message: navigation to first waypoint

File: description/urdf/constants.xacro (robot description, xacro)
@@ -80,5 +80,5 @@
     <xacro:property name="ZED_camera_width" value="0.03"/>
     <xacro:property name="ZED_camera_height" value="0.033"/>
-    <xacro:property name="ZED_camera_pitch" value="${25 * pi/180}"/>
+    <xacro:property name="ZED_camera_pitch" value="${19.66 * pi/180}"/> <!-- 19.66 degrees ensures the camera's field of view overlaps with the end of the lidar readings-->
     <!-- ZED image height/width corresponds to image size for 60Hz refresh-->
     <xacro:property name="ZED_image_refresh" value="60"/>

Commit message: merge changes

File: description/urdf/constants.xacro (robot description, xacro)
@@ -59,5 +59,5 @@
     <xacro:property name="laser_horizontal_min_angle" value="${-0.5*laser_field_of_view*pi/180}"/>
     <xacro:property name="laser_horizontal_max_angle" value="${0.5*laser_field_of_view*pi/180}"/>
-    <xacro:property name="laser_range_min" value="0.06"/>
+    <xacro:property name="laser_range_min" value="0.1"/>
     <xacro:property name="laser_range_max" value="4.095"/>
     <xacro:property name="laser_resolution_angle" value="0.36"/>
@@ -65,5 +65,5 @@
     <xacro:property name="laser_noise_type" value="gaussian"/>
     <xacro:property name="laser_noise_mean" value="0.0"/>
-    <xacro:property name="laser_noise_stddev" value="0.0"/>
+    <xacro:property name="laser_noise_stddev" value="0.01/3"/>
     <xacro:property name="laser_topicName" value="scan"/>
     <xacro:property name="laser_frameName" value="base_laser"/>
@@ -109,5 +109,5 @@
     <xacro:property name="ref_lon" value="-79.3903"/>
     <xacro:property name="ref_alt" value="76.0000"/>
-    <xacro:property name="gps_drift" value="0 0 0"/>
+    <xacro:property name="gps_drift" value="1.5 1.5 1.5"/>
     <xacro:property name="gps_vel_drift" value="0.00 0.00 0.00"/>
     <!-- Phidget IMU -->

Commit message: cleaning for PR

File: description/urdf/constants.xacro (robot description, xacro)
@@ -59,5 +59,5 @@
     <xacro:property name="laser_horizontal_min_angle" value="${-0.5*laser_field_of_view*pi/180}"/>
     <xacro:property name="laser_horizontal_max_angle" value="${0.5*laser_field_of_view*pi/180}"/>
-    <xacro:property name="laser_range_min" value="0.1"/>
+    <xacro:property name="laser_range_min" value="0.06"/>
     <xacro:property name="laser_range_max" value="4.095"/>
     <xacro:property name="laser_resolution_angle" value="0.36"/>

Commit message: revert camera tilt back to 15

File: description/urdf/constants.xacro (robot description, xacro)
@@ -80,5 +80,5 @@
     <xacro:property name="ZED_camera_width" value="0.03"/>
     <xacro:property name="ZED_camera_height" value="0.033"/>
-    <xacro:property name="ZED_camera_pitch" value="${19.66 * pi/180}"/> <!-- 19.66 degrees ensures the camera's field of view overlaps with the end of the lidar readings-->
+    <xacro:property name="ZED_camera_pitch" value="${15 * pi/180}"/> <!-- 19.66 degrees ensures the camera's field of view overlaps with the end of the lidar readings-->
     <!-- ZED image height/width corresponds to image size for 60Hz refresh-->
     <xacro:property name="ZED_image_refresh" value="60"/>

Commit message: Caff 80 (#92)
* added support for x-y coordinate waypoints

* lowered camera angle to avoid detecting ground as obstacle

* added global carrot planner

* navigation to first waypoint

* michael tests

* adjust pilones and local costmap issue due to lidar min/max obs height

* tuning planner vels and inflation radius

* basic functionality present. Path planning sucks tho

* need to tune planner

* cleaning for PR

* more cleanup

* create 2 files for waypoints

* newline

* revert camera tilt back to 15

Co-authored-by: Anthony Lem <anthonyjlem@gmail.com>

File: description/urdf/constants.xacro (robot description, xacro)
@@ -80,5 +80,5 @@
     <xacro:property name="ZED_camera_width" value="0.03"/>
     <xacro:property name="ZED_camera_height" value="0.033"/>
-    <xacro:property name="ZED_camera_pitch" value="${15 * pi/180}"/>
+    <xacro:property name="ZED_camera_pitch" value="${15 * pi/180}"/> <!-- 19.66 degrees ensures the camera's field of view overlaps with the end of the lidar readings-->
     <!-- ZED image height/width corresponds to image size for 60Hz refresh-->
     <xacro:property name="ZED_image_refresh" value="60"/>

Commit message: added unexplained x2 and +190/+80 xy offsets

File: description/urdf/constants.xacro (robot description, xacro)
@@ -80,9 +80,9 @@
     <xacro:property name="ZED_camera_width" value="0.03"/>
     <xacro:property name="ZED_camera_height" value="0.033"/>
-    <xacro:property name="ZED_camera_pitch" value="${15 * pi/180}"/> <!-- 19.66 degrees ensures the camera's field of view overlaps with the end of the lidar readings-->
+    <xacro:property name="ZED_camera_pitch" value="${50 * pi/180}"/> <!-- 19.66 degrees ensures the camera's field of view overlaps with the end of the lidar readings-->
     <!-- ZED image height/width corresponds to image size for 60Hz refresh-->
     <xacro:property name="ZED_image_refresh" value="60"/>
-    <xacro:property name="ZED_image_width" value="3840"/>
-    <xacro:property name="ZED_image_height" value="1080"/>
+    <xacro:property name="ZED_image_width" value="640"/>
+    <xacro:property name="ZED_image_height" value="360"/>
     <xacro:property name="ZED_image_format" value="R8G8B8"/>
     <xacro:property name="ZED_image_hfov" value="${90 * pi/180}"/>

Commit message: testing ivy's changes

File: description/urdf/constants.xacro (robot description, xacro)
@@ -109,5 +109,5 @@
     <xacro:property name="ref_lon" value="-79.3903"/>
     <xacro:property name="ref_alt" value="76.0000"/>
-    <xacro:property name="gps_drift" value="1.5 1.5 1.5"/>
+    <xacro:property name="gps_drift" value="0 0 0"/>
     <xacro:property name="gps_vel_drift" value="0.00 0.00 0.00"/>
     <!-- Phidget IMU -->

Commit message: kj's comments

File: description/urdf/constants.xacro (robot description, xacro)
@@ -80,5 +80,5 @@
     <xacro:property name="ZED_camera_width" value="0.03"/>
     <xacro:property name="ZED_camera_height" value="0.033"/>
-    <xacro:property name="ZED_camera_pitch" value="${50 * pi/180}"/> <!-- 19.66 degrees ensures the camera's field of view overlaps with the end of the lidar readings-->
+    <xacro:property name="ZED_camera_pitch" value="${50 * pi/180}"/>
     <!-- ZED image height/width corresponds to image size for 60Hz refresh-->
     <xacro:property name="ZED_image_refresh" value="60"/>
@@ -109,5 +109,5 @@
     <xacro:property name="ref_lon" value="-79.3903"/>
     <xacro:property name="ref_alt" value="76.0000"/>
-    <xacro:property name="gps_drift" value="0 0 0"/>
+    <xacro:property name="gps_drift" value="1.5 1.5 1.5"/>
     <xacro:property name="gps_vel_drift" value="0.00 0.00 0.00"/>
     <!-- Phidget IMU -->

Commit message: Vl cv integration (#108)
* Not working code based on simple layer tutorials

* Able to write obstacles to local costmap

* I broke simple_layers.cpp

* it works

* remove useless variables

* python to C++

* int to double

* separated function

* offset to 4,4

* fixed random function & reduced spacing btw points

* temp

* pull caff-57

* local to global

* 10sec delay before next set of points

* published dummy topic, not yet subscribed by virtual layer

* testing subscriber in virtual layer

* michael temp com

* temp comm

* remove nonfunctional subscriber from virtual layer

* fixed layer

* michael save

* Initial commit for CV wrapper.
    Loads in random test image from disk. Runs image preprocessing, loads in cv .onnx model, and runs a profile on inference speeds.
    Next commit will aim to integrate with ros nodes, subscribe to camera to load image and publish to a nav friendly format.

* Updatedd code - still not working

* Got inference working.

Left to do:
- Interface on both ends with ROS. Subscribe to ZED node to get images and publish results

* basic ros node skeleton & cleaning up inference code

* Able to get images from rviz

* deleted old model wrapper file

* removed local filepath from launch file

* added basic instructions to install onnxruntime, need to expand later

* minor cleanup in post process function

* cleaned up constructor code a bit

* made node handle private to allow params be accessible

* fixed gitignore end of line

* removed cv gitignore

* deleted unnecessary comments in package.xml

* fixed formatting in lane_detection_inference_node's constructor

* Added instructions to readme

* Update README.md

* Added zed wrapper

* Removed zed wrapper code - to add as submodule

* Added zed wrapper as submodule

* Overloaded cpp cv pipeline for python varient. Runs using communication to python3 inference using redis. Removes dependancy for onnxruntime built from scratch on arm.

Launch using roslaunch lane_detection lane_detection_server.launch

* added some cv code; currently not working

* added helper scripts in scripts folder

* Added 3D projection. Publishing to rostopic /cv/lane_detection. Does not include tf transforms yet, untested with rviz

* kj wants me to show caff-80 so pause here

* fixing vl

* Added default z mapping

* Added relative imports for script

* VL issue was offset and global var

* merge master

* cleanup

* return cv/lanes

* Finished lane detection. Refactored cv pipeline to allow for easy addition of pothole detection

* updated Readme

* Added new line (for Michael)

* Removed unused code

* Added comment for future todo

* Changed camera projection code to use zed parameters. Added checks full null data read - occurs when FPS drops below FPS set by ros.

* Removed unused files

* temp save

* Added checks for NoneType thoruhg redis. Added publishing of raw model output to topic cv/model/output

* I think it works, but cv/ros did diff frame definitions

* figured out cv transform I think, but cv revieweing their work

* left camera optical frame not just offset of zed frame so prev trans def wrong

* Updating and clean-up of functions

* Minor correction

* Preliminary (non-working) pothole detection pipeline

* Scaling camera intrinsics to accommodate resized images

* Got valid outputs + thresholding

* Reformatted, working.

* Correcting some inputs of the lane fit functions

* added unexplained x2 and +190/+80 xy offsets

* Added scaling of intrinsics. Fixed previous commit bugs

* fixed left/camera_info topic name again

* Added working pothole detection code!

* Fixed projection errors.

* testing ivy's changes

* remove cv_points clearing. Will need to combine similar points

* giant pink blobs

* kj's comments

Co-authored-by: kajananchinniah <kajananchinniah@gmail.com>
Co-authored-by: Jimin Kwon <kishyaut@gmail.com>
Co-authored-by: Spencer Teetaert <erickmu1@hotmail.com>
Co-authored-by: Spencer Teetaert <spencerteetaert@gmail.com>
Co-authored-by: Spencer Teetaert <45899408+spencerteetaert@users.noreply.github.com>
Co-authored-by: Jason-Y000 <57577805+Jason-Y000@users.noreply.github.com>

File: description/urdf/constants.xacro (robot description, xacro)
@@ -80,9 +80,9 @@
     <xacro:property name="ZED_camera_width" value="0.03"/>
     <xacro:property name="ZED_camera_height" value="0.033"/>
-    <xacro:property name="ZED_camera_pitch" value="${15 * pi/180}"/> <!-- 19.66 degrees ensures the camera's field of view overlaps with the end of the lidar readings-->
+    <xacro:property name="ZED_camera_pitch" value="${50 * pi/180}"/>
     <!-- ZED image height/width corresponds to image size for 60Hz refresh-->
     <xacro:property name="ZED_image_refresh" value="60"/>
-    <xacro:property name="ZED_image_width" value="3840"/>
-    <xacro:property name="ZED_image_height" value="1080"/>
+    <xacro:property name="ZED_image_width" value="640"/>
+    <xacro:property name="ZED_image_height" value="360"/>
     <xacro:property name="ZED_image_format" value="R8G8B8"/>
     <xacro:property name="ZED_image_hfov" value="${90 * pi/180}"/>

Commit message: updated stand position but seeing weird bugs

File: description/urdf/constants.xacro (robot description, xacro)
@@ -6,7 +6,7 @@
     <xacro:property name="base_height" value="0.01"/>
     <!-- Chassis -->
-    <xacro:property name="chassis_to_base_link_dist" value="0.501747"/>
-    <xacro:property name="chassis_to_stand_link_dist" value="0.698253"/>
-    <xacro:property name="chassis_link_mass" value="33.9"/>
+    <xacro:property name="chassis_to_base_link_dist" value="0.74424"/>
+    <xacro:property name="chassis_to_stand_link_dist" value="1.0357"/>
+    <xacro:property name="chassis_link_mass" value="32.46"/>
     <!-- Stand -->
     <xacro:property name="stand_length" value="0.412"/>

File: description/urdf/inertias.xacro (robot description, xacro)
@@ -4,7 +4,7 @@
     <xacro:macro name="chassis_link_inertia">
         <inertia
-            ixx="10.9364" ixy="0.0000" ixz="0.0000"
-            iyx="0.0000" iyy="10.9070" iyz="0.0000"
-            izx="0.0000" izy="0.0000" izz="2.3961"
+            ixx="21.200" ixy="0.000" ixz="0.0000"
+            iyx="0.0000" iyy="21.230" iyz="0.0000"
+            izx="0.0000" izy="0.0000" izz="2.2600"
         />
     </xacro:macro>

Commit message: change imu z dist

File: description/urdf/constants.xacro (robot description, xacro)
@@ -121,4 +121,4 @@
     <xacro:property name="imu_x_dist" value="0.28"/>
     <xacro:property name="imu_y_dist" value="0.295"/>
-    <xacro:property name="imu_z_dist" value="0.34"/>
+    <xacro:property name="imu_z_dist" value="0.195"/>
 </robot>

Commit message: Fixing missing distance_to_second_lidar

File: description/urdf/constants.xacro (robot description, xacro)
@@ -76,4 +76,5 @@
     <xacro:property name="laser_x_dist" value="${base_length/2 - 2*laser_length}"/>
     <xacro:property name="laser_z_dist" value="${laser_height/2}"/>
+    <xacro:property name="distance_to_second_lidar" value="0.2"/>
     <!-- ZED camera -->
     <!-- NOTE: approx as a rectangular prism -->

Commit message: node functioning

File: description/urdf/constants.xacro (robot description, xacro)
@@ -76,7 +76,7 @@
     <xacro:property name="laser_x_dist" value="${base_length/2 - 2*laser_length}"/>
     <xacro:property name="laser_z_dist" value="${laser_height/2}"/>
-    <xacro:property name="distance_to_second_lidar" value="0.2"/>
+    <xacro:property name="distance_to_second_lidar" value="0.6"/>
     <!-- ZED camera -->
-    <!-- NOTE: approx as a rectangular prism -->
+    <!-- NOTE: approx as a rectangulSar prism -->
     <xacro:property name="ZED_camera_mass" value="0.1587573"/>
     <xacro:property name="ZED_camera_length" value="0.175"/>

Commit message: lidar sensor names have to be unique :(

File: description/urdf/constants.xacro (robot description, xacro)
@@ -76,5 +76,5 @@
     <xacro:property name="laser_x_dist" value="${base_length/2 - 2*laser_length}"/>
     <xacro:property name="laser_z_dist" value="${laser_height/2}"/>
-    <xacro:property name="distance_to_second_lidar" value="0.6"/>
+    <xacro:property name="distance_to_second_lidar" value="0.2"/>
     <!-- ZED camera -->
     <!-- NOTE: approx as a rectangulSar prism -->

File: description/urdf/plugins.gazebo.xacro (robot description, xacro)
@@ -32,5 +32,6 @@
     <!-- LIDAR -->
     <gazebo reference="base_laser">
-        <sensor type="ray" name="gpu_hokuyo_sensor">
+        <!-- make sure your sensor NAMES are unique :'( -->
+        <sensor type="ray" name="hokuyo_sensor_1">
             <pose>0 0 0 0 0 0</pose>
             <visualize>${laser_visualize}</visualize>
@@ -67,5 +68,6 @@
     <!-- Another LIDAR for testing-->
     <gazebo reference="upper_laser">
-        <sensor type="ray" name="gpu_hokuyo_sensor">
+        <!-- make sure your sensor NAMES are unique :'( -->
+        <sensor type="ray" name="hokuyo_sensor_2">
             <pose>0 0 0 0 0 0</pose>
             <visualize>${laser_visualize}</visualize>

Commit message: Fixed camera positioning.

File: description/urdf/constants.xacro (robot description, xacro)
@@ -11,5 +11,5 @@
     <!-- Stand -->
     <xacro:property name="stand_length" value="0.412"/>
-    <xacro:property name="stand_width" value="0.33"/>
+    <xacro:property name="stand_width" value="0.255"/>
     <xacro:property name="stand_height" value="1.335"/>
     <xacro:property name="stand_mass" value="1.0"/>
@@ -97,4 +97,7 @@
     <xacro:property name="ZED_depth_points_topicName" value="depth/points"/>
     <xacro:property name="ZED_frameName" value="left_camera_link_optical"/>
+    <!--ZED CAMERA JOINT PARAMETERS-->
+    <xacro:property name="ZED_camera_to_top_plate_x" value="${(stand_width / 2.0)-0.01}"/>
+    <xacro:property name="ZED_camera_to_top_plate_z" value="0.065"/>
     <!-- Garmin GPS -->
     <!-- NOTE: approx. as a cylinder, Garmin itself is similar to a hockey puck -->

File: description/urdf/stand_link.urdf.xacro (robot description, xacro)
@@ -60,5 +60,5 @@
         <parent link="stand_link"/>
         <child link="zed_base_link"/>
-        <origin xyz="${0.05 + (stand_width / 2.0) - ZED_camera_width} 0 ${ZED_camera_height / 2.0}" rpy="0 ${ZED_camera_pitch} 0"/>
+        <origin xyz="${ZED_camera_to_top_plate_x} 0 ${ZED_camera_to_top_plate_z}" rpy="0 ${ZED_camera_pitch} 0"/>
     </joint>
     <!-- Generate Left Camera frame -->

Commit message: Updated wheel separation.

File: description/urdf/constants.xacro (robot description, xacro)
@@ -34,5 +34,5 @@
     <xacro:property name="wheel_right_joint" value="right_wheel_joint"/>
     <!--<xacro:property name="wheels_separation" value="0.875"/>-->
-    <xacro:property name="wheels_separation" value="1.0"/>
+    <xacro:property name="wheels_separation" value="0.926"/>
     <xacro:property name="wheel_diameter" value="0.25"/>
     <xacro:property name="wheel_acceleration" value="1.0"/>

Commit message: Changed camera angle

File: description/urdf/constants.xacro (robot description, xacro)
@@ -81,5 +81,6 @@
     <xacro:property name="ZED_camera_width" value="0.03"/>
     <xacro:property name="ZED_camera_height" value="0.06"/>
-    <xacro:property name="ZED_camera_pitch" value="${50 * pi/180}"/>
+    <xacro:property name="ZED_camera_pitch" value="${34 * pi/180}"/>
+    <!--<xacro:property name="ZED_camera_pitch" value="${50 * pi/180}"/>-->
     <!-- ZED image height/width corresponds to image size for 60Hz refresh-->
     <xacro:property name="ZED_image_refresh" value="60"/>
