Commit message: CAFF-140: Merge Visual Odometry into Sensor Fusion and Add Ground Truth Plugin (#146)
* Using proper wheel separation.

* Added zed odom to odom_local

* Fuse VO with differential turned on

* Fix rtabmap on Vicky's machine

* Added ground truth plugin.

* Put in ground truth plugin.

* Create node to add contant offsets to ground truth

* Need to fix the ground_truth_script still

* Changed camera angle

* Fixed ground truth transform

* Implemented ground truth script.

* Move ground truth tf node to simulate.launch

* Deleted duplicated commented out code

* Removed old code.

---------

Co-authored-by: Vicky <vhy.huang@mail.utoronto.ca>

File: description/urdf/constants.xacro (robot description, xacro)
@@ -34,5 +34,5 @@
     <xacro:property name="wheel_right_joint" value="right_wheel_joint"/>
     <!--<xacro:property name="wheels_separation" value="0.875"/>-->
-    <xacro:property name="wheels_separation" value="1.0"/>
+    <xacro:property name="wheels_separation" value="0.926"/>
     <xacro:property name="wheel_diameter" value="0.25"/>
     <xacro:property name="wheel_acceleration" value="1.0"/>
@@ -81,5 +81,6 @@
     <xacro:property name="ZED_camera_width" value="0.03"/>
     <xacro:property name="ZED_camera_height" value="0.06"/>
-    <xacro:property name="ZED_camera_pitch" value="${50 * pi/180}"/>
+    <xacro:property name="ZED_camera_pitch" value="${34 * pi/180}"/>
+    <!--<xacro:property name="ZED_camera_pitch" value="${50 * pi/180}"/>-->
     <!-- ZED image height/width corresponds to image size for 60Hz refresh-->
     <xacro:property name="ZED_image_refresh" value="60"/>

File: description/urdf/plugins.gazebo.xacro (robot description, xacro)
@@ -152,3 +152,16 @@
         </sensor>
     </gazebo>
+    <!-- Ground Truth Plugin-->
+    <gazebo>
+        <plugin name="p3d_base_controller" filename="libgazebo_ros_p3d.so">
+        <alwaysOn>true</alwaysOn>
+        <updateRate>50.0</updateRate>
+        <bodyName>base_link</bodyName>
+        <topicName>ground_truth/state</topicName>
+        <gaussianNoise>0.01</gaussianNoise>
+        <frameName>world</frameName>
+        <xyzOffsets>0 0 0</xyzOffsets>
+        <rpyOffsets>0 0 0</rpyOffsets>
+        </plugin>
+    </gazebo>
 </robot>

Commit message: Added separately named parameters for upper laser.

File: description/urdf/constants.xacro (robot description, xacro)
@@ -68,6 +68,4 @@
     <xacro:property name="laser_topicName" value="scan"/>
     <xacro:property name="laser_frameName" value="base_laser"/>
-    <xacro:property name="upper_laser_topicName" value="scan_upper"/>
-    <xacro:property name="upper_laser_frameName" value="upper_laser"/>
     <xacro:property name="laser_length" value="0.05"/>
     <xacro:property name="laser_width" value="0.05"/>
@@ -76,7 +74,24 @@
     <xacro:property name="laser_x_dist" value="${base_length/2 - 2*laser_length}"/>
     <xacro:property name="laser_z_dist" value="${laser_height/2}"/>
+    <!--RPlidar A1-->
+    <xacro:property name="upper_laser_visualize" value="false"/>
+    <xacro:property name="upper_laser_update_rate" value="10"/>
+    <xacro:property name="upper_laser_horizontal_samples" value="1080"/>
+    <xacro:property name="upper_laser_horizontal_resolution" value="1"/>
+    <xacro:property name="upper_laser_field_of_view" value="270"/>
+    <xacro:property name="upper_laser_horizontal_min_angle" value="${-0.5*laser_field_of_view*pi/180}"/>
+    <xacro:property name="upper_laser_horizontal_max_angle" value="${0.5*laser_field_of_view*pi/180}"/>
+    <xacro:property name="upper_laser_range_min" value="0.06"/>
+    <xacro:property name="upper_laser_range_max" value="4.095"/>
+    <xacro:property name="upper_laser_resolution_angle" value="0.36"/>
+    <xacro:property name="upper_laser_range_resolution" value="${laser_resolution_angle*pi/180}"/>
+    <xacro:property name="upper_laser_noise_type" value="gaussian"/>
+    <xacro:property name="upper_laser_noise_mean" value="0.0"/>
+    <xacro:property name="upper_laser_noise_stddev" value="0.01/3"/>
+    <xacro:property name="upper_laser_topicName" value="scan_upper"/>
+    <xacro:property name="upper_laser_frameName" value="upper_laser"/>
     <xacro:property name="distance_to_second_lidar" value="0.2"/>
     <!-- ZED camera -->
-    <!-- NOTE: approx as a rectangulSar prism -->
+    <!-- NOTE: approx as a rectangular prism -->
     <xacro:property name="ZED_camera_mass" value="0.1587573"/>
     <xacro:property name="ZED_camera_length" value="0.175"/>

File: description/urdf/plugins.gazebo.xacro (robot description, xacro)
@@ -71,27 +71,27 @@
         <sensor type="ray" name="hokuyo_sensor_2">
             <pose>0 0 0 0 0 0</pose>
-            <visualize>${laser_visualize}</visualize>
-            <update_rate>${laser_update_rate}</update_rate>
+            <visualize>${upper_laser_visualize}</visualize>
+            <update_rate>${upper_laser_update_rate}</update_rate>
             <ray>
                 <scan>
                     <horizontal>
-                        <samples>${laser_horizontal_samples}</samples>
-                        <resolution>${laser_horizontal_resolution}</resolution>
-                        <min_angle>${laser_horizontal_min_angle}</min_angle>
-                        <max_angle>${laser_horizontal_max_angle}</max_angle>
+                        <samples>${upper_laser_horizontal_samples}</samples>
+                        <resolution>${upper_laser_horizontal_resolution}</resolution>
+                        <min_angle>${upper_laser_horizontal_min_angle}</min_angle>
+                        <max_angle>${upper_laser_horizontal_max_angle}</max_angle>
                     </horizontal>
                 </scan>
                 <range>
-                    <min>${laser_range_min}</min>
-                    <max>${laser_range_max}</max>
-                    <resolution>${laser_range_resolution}</resolution>
+                    <min>${upper_laser_range_min}</min>
+                    <max>${upper_laser_range_max}</max>
+                    <resolution>${upper_laser_range_resolution}</resolution>
                 </range>
                 <noise>
-                    <type>${laser_noise_type}</type>
+                    <type>${upper_laser_noise_type}</type>
                     <!-- Noise based on gazebosim.org's tutorial on writing gazebo plugins w/ ROS. The comment they put will be reproduced:
                         Noise parameters based on published spec for Hokuyo laser achieving "+-10mm" accuracy at range < 10 m. A mean of
                         0.0m and stddev of (0.01/3), will put 99.8% of samples within 0.03m of the true reading. -->
-                    <mean>${laser_noise_mean}</mean>
-                    <stddev>${laser_noise_stddev}</stddev>
+                    <mean>${upper_laser_noise_mean}</mean>
+                    <stddev>${upper_laser_noise_stddev}</stddev>
                 </noise>
             </ray>

Commit message: corrected constants referencing for upper lidar

File: description/urdf/constants.xacro (robot description, xacro)
@@ -80,10 +80,10 @@
     <xacro:property name="upper_laser_horizontal_resolution" value="1"/>
     <xacro:property name="upper_laser_field_of_view" value="270"/>
-    <xacro:property name="upper_laser_horizontal_min_angle" value="${-0.5*laser_field_of_view*pi/180}"/>
-    <xacro:property name="upper_laser_horizontal_max_angle" value="${0.5*laser_field_of_view*pi/180}"/>
+    <xacro:property name="upper_laser_horizontal_min_angle" value="${-0.5*upper_laser_field_of_view*pi/180}"/>
+    <xacro:property name="upper_laser_horizontal_max_angle" value="${0.5*upper_laser_field_of_view*pi/180}"/>
     <xacro:property name="upper_laser_range_min" value="0.06"/>
     <xacro:property name="upper_laser_range_max" value="4.095"/>
     <xacro:property name="upper_laser_resolution_angle" value="0.36"/>
-    <xacro:property name="upper_laser_range_resolution" value="${laser_resolution_angle*pi/180}"/>
+    <xacro:property name="upper_laser_range_resolution" value="${upper_laser_resolution_angle*pi/180}"/>
     <xacro:property name="upper_laser_noise_type" value="gaussian"/>
     <xacro:property name="upper_laser_noise_mean" value="0.0"/>

Commit message: Trying to rmove barrels from thresholded image

File: description/urdf/constants.xacro (robot description, xacro)
@@ -81,5 +81,5 @@
     <xacro:property name="ZED_camera_width" value="0.03"/>
     <xacro:property name="ZED_camera_height" value="0.06"/>
-    <xacro:property name="ZED_camera_pitch" value="${34 * pi/180}"/>
+    <xacro:property name="ZED_camera_pitch" value="${45 * pi/180}"/>
     <!--<xacro:property name="ZED_camera_pitch" value="${50 * pi/180}"/>-->
     <!-- ZED image height/width corresponds to image size for 60Hz refresh-->

Commit message: Michael Specific: Save 0 noise gps test

File: description/urdf/constants.xacro (robot description, xacro)
@@ -132,5 +132,5 @@
     <xacro:property name="ref_lon" value="-79.3903"/>
     <xacro:property name="ref_alt" value="76.0000"/>
-    <xacro:property name="gps_drift" value="1.5 1.5 1.5"/>
+    <xacro:property name="gps_drift" value="0 0 0"/>
     <xacro:property name="gps_vel_drift" value="0.00 0.00 0.00"/>
     <!-- Phidget IMU -->

Commit message: Update wheel separation

File: description/urdf/constants.xacro (robot description, xacro)
@@ -34,5 +34,5 @@
     <xacro:property name="wheel_right_joint" value="right_wheel_joint"/>
     <!--<xacro:property name="wheels_separation" value="0.875"/>-->
-    <xacro:property name="wheels_separation" value="0.926"/>
+    <xacro:property name="wheels_separation" value="0.916"/>
     <xacro:property name="wheel_diameter" value="0.25"/>
     <xacro:property name="wheel_acceleration" value="1.0"/>

Commit message: Added lane to lidar conversion in c++. Connected with cartographer by simulating two laser scans.

File: description/urdf/constants.xacro (robot description, xacro)
@@ -99,5 +99,5 @@
     <xacro:property name="ZED_camera_width" value="0.03"/>
     <xacro:property name="ZED_camera_height" value="0.06"/>
-    <xacro:property name="ZED_camera_pitch" value="${34 * pi/180}"/>
+    <xacro:property name="ZED_camera_pitch" value="${0 * pi/180}"/>
     <!--<xacro:property name="ZED_camera_pitch" value="${50 * pi/180}"/>-->
     <!-- ZED image height/width corresponds to image size for 60Hz refresh-->

Commit message: merge previous change in IGVC-2023 and master

File: description/urdf/constants.xacro (robot description, xacro)
@@ -99,5 +99,5 @@
     <xacro:property name="ZED_camera_width" value="0.03"/>
     <xacro:property name="ZED_camera_height" value="0.06"/>
-    <xacro:property name="ZED_camera_pitch" value="${34 * pi/180}"/>
+    <xacro:property name="ZED_camera_pitch" value="${32 * pi/180}"/>
     <!--<xacro:property name="ZED_camera_pitch" value="${50 * pi/180}"/>-->
     <!-- ZED image height/width corresponds to image size for 60Hz refresh-->
@@ -107,5 +107,5 @@
     <xacro:property name="ZED_image_format" value="R8G8B8"/>
     <xacro:property name="ZED_image_hfov" value="${90 * pi/180}"/>
-    <xacro:property name="ZED_name" value="zed/zed_node"/>
+    <xacro:property name="ZED_name" value="zed_node"/>
     <xacro:property name="ZED_always_on" value="true"/>
     <xacro:property name="ZED_update_rate" value="0"/>
